Commit message: fix orientation

File: auv_description/auv_common_descriptions/urdf/sensors/sonar.urdf.xacro (robot description, xacro)
@@ -4,5 +4,5 @@
     <link name="${name}_link">
       <visual>
-        <origin xyz="0 0 0" rpy="0 ${-math.pi/2} 0" />
+        <origin xyz="0 0 0" rpy="0 0 0" />
         <geometry>
           <mesh

File: auv_description/taluy_description/urdf/auv_base.urdf.xacro (robot description, xacro)
@@ -90,14 +90,14 @@
     <xacro:sonar name="base_link/sonar_front" parent="base_link"
       position="0.38 0.09 0.09"
-      orientation="0 ${math.pi/2} 0" />
+      orientation="0 0 0" />
     <xacro:sonar name="base_link/sonar_back" parent="base_link"
       position="-0.42 -0.09 0.09"
-      orientation="0 ${math.pi/2} ${math.pi}" />
+      orientation="0 0 ${math.pi}" />
     <xacro:sonar name="base_link/sonar_left" parent="base_link"
       position="0.02 -0.21 -0.14"
-      orientation="0 ${math.pi/2} ${-math.pi/2}" />
+      orientation="0 0 ${-math.pi/2}" />
     <xacro:sonar name="base_link/sonar_right" parent="base_link"
       position="0.02 0.21 -0.14"
-      orientation="0 ${math.pi/2} ${math.pi/2}" />
+      orientation="0 0 ${math.pi/2}" />
     <!-- <link name="base_footprint">
       <inertial>
