Commit message: use the uuv_simulator plugin for imu
- Replace the libgazebo_ros imu plugin with libuuv_gazebo_ros imu plugin. This is how it was in the legacy repo, so I thought this should be better.
- Changed the joint type of the IMU link from `fixed` to `revolute` (with movement limits) to resolve an issue where libuuv_gazebo_ros plugins couldn't detect fixed links in Gazebo.
- Noted that Gazebo doesn't recognize links with fixed joints as standalone links, which seems to cause this issue.

File: auv_description/auv_common_descriptions/urdf/sensors/xsens_mti_g710.urdf.xacro (robot description, xacro)
@@ -24,9 +24,10 @@
       </inertial>
     </link>
-    <joint name="${name}_joint" type="fixed">
+    <joint name="${name}_joint" type="revolute">
       <parent link="${parent}" />
       <child link="${name}_link" />
       <origin xyz="${position}" rpy="${orientation}" />
       <axis rpy="0 0 0" xyz="0 0 1" />
+      <limit upper="0" lower="0" effort="0" velocity="0" />
     </joint>
   </xacro:macro>

File: auv_sim/auv_sim_description/urdf/gazebo_plugins.urdf.xacro (robot description, xacro)
@@ -44,23 +44,24 @@
   <!-- imu plugin -->
   <xacro:macro name="xsens_mti_g710_sim" params="name">
-    <gazebo reference="${name}_link">
-      <gravity>true</gravity>
-      <sensor name="${name}_sensor" type="imu">
-        <always_on>true</always_on>
-        <update_rate>100</update_rate>
-        <visualize>true</visualize>
-        <topic>__default_topic__</topic>
-        <plugin filename="libgazebo_ros_imu_sensor.so" name="imu_plugin">
-          <topicName>sensors/imu/data</topicName>
-          <bodyName>${name}_link</bodyName>
-          <updateRateHZ>10.0</updateRateHZ>
-          <gaussianNoise>0.0</gaussianNoise>
-          <xyzOffset>0 0 0</xyzOffset>
-          <rpyOffset>0 0 0</rpyOffset>
-          <frameName>${name}_link</frameName>
-          <initialOrientationAsReference>false</initialOrientationAsReference>
-        </plugin>
-        <pose>0 0 0 0 0 0</pose>
-      </sensor>
+    <gazebo>
+      <plugin filename="libuuv_gazebo_ros_imu_plugin.so"
+        name="${name}_imu_plugin">
+        <robot_namespace>taluy</robot_namespace>
+        <link_name>${name}_link</link_name>
+        <sensor_topic>sensors/imu/data</sensor_topic>
+        <gyroscope_noise_density>0.0002514074</gyroscope_noise_density>
+        <gyroscope_random_walk>0.000038785</gyroscope_random_walk>
+        <gyroscope_bias_correlation_time>1000.0</gyroscope_bias_correlation_time>
+        <gyroscope_turn_on_bias_sigma>0.0087</gyroscope_turn_on_bias_sigma>
+        <accelerometer_noise_density>0.00104347826</accelerometer_noise_density>
+        <accelerometer_random_walk>0.006</accelerometer_random_walk>
+        <accelerometer_bias_correlation_time>300.0</accelerometer_bias_correlation_time>
+        <accelerometer_turn_on_bias_sigma>0.1960</accelerometer_turn_on_bias_sigma>
+        <orientation_noise>0.05</orientation_noise>
+        <update_rate>80</update_rate>
+        <enable_gazebo_messages>false</enable_gazebo_messages>
+        <enable_local_ned_frame>false</enable_local_ned_frame>
+        <static_reference_frame>world</static_reference_frame>
+      </plugin>
     </gazebo>
   </xacro:macro>

Commit message: use the uuv_simulator plugin for imu
- Replace the libgazebo_ros imu plugin with libuuv_gazebo_ros imu plugin. This is how it was in the legacy repo, so I thought this should be better.
- Changed the joint type of the IMU link from `fixed` to `revolute` (with movement limits) to resolve an issue where libuuv_gazebo_ros plugins couldn't detect fixed links in Gazebo.
- Noted that Gazebo doesn't recognize links with fixed joints as standalone links, which seems to cause this issue.

File: auv_description/auv_common_descriptions/urdf/sensors/xsens_mti_g710.urdf.xacro (robot description, xacro)
@@ -20,9 +20,10 @@
       </inertial>
     </link>
-    <joint name="${name}_joint" type="fixed">
-      <parent link="${parent}"/>
-      <child link="${name}_link"/>
-      <origin xyz="${position}" rpy="${orientation}"/>
-      <axis rpy="0 0 0" xyz="0 0 1"/>
+    <joint name="${name}_joint" type="revolute">
+      <parent link="${parent}" />
+      <child link="${name}_link" />
+      <origin xyz="${position}" rpy="${orientation}" />
+      <axis rpy="0 0 0" xyz="0 0 1" />
+      <limit upper="0" lower="0" effort="0" velocity="0" />
     </joint>
   </xacro:macro>

Commit message: revert IMU joint type from `revolute` to `fixed`
- add rotation to fix imu plugin values

File: auv_description/auv_common_descriptions/urdf/sensors/xsens_mti_g710.urdf.xacro (robot description, xacro)
@@ -24,10 +24,9 @@
       </inertial>
     </link>
-    <joint name="${name}_joint" type="revolute">
+    <joint name="${name}_joint" type="fixed">
       <parent link="${parent}" />
       <child link="${name}_link" />
       <origin xyz="${position}" rpy="${orientation}" />
       <axis rpy="0 0 0" xyz="0 0 1" />
-      <limit upper="0" lower="0" effort="0" velocity="0" />
     </joint>
   </xacro:macro>

File: auv_sim/auv_sim_description/auv_common_sim_descriptions/urdf/sensors/xsens_mti_g710.urdf.xacro (robot description, xacro)
@@ -2,9 +2,29 @@
 <robot name="xsens_mti_g710" xmlns:xacro="http://www.ros.org/wiki/xacro">
   <xacro:macro name="xsens_mti_g710_sim" params="name namespace static_reference_frame">
+    <link name="${name}_sim_link">
+      <inertial>
+        <mass value="0.001" />
+        <origin xyz="0 0 0" rpy="0 0 0" />
+        <inertia ixx="0.0000001" ixy="0" ixz="0" iyy="0.0000001" iyz="0" izz="0.0000001" />
+      </inertial>
+      <collision>
+        <geometry>
+          <cylinder length="${0.000001}" radius="${0.000001}" />
+        </geometry>
+        <origin xyz="0 0 0" rpy="0 ${0.5*pi} 0" />
+      </collision>
+    </link>
+    <joint name="${name}_sim_joint" type="revolute">
+      <parent link="${name}_link" />
+      <child link="${name}_sim_link" />
+      <origin xyz="0 0 0" rpy="${math.pi} ${math.pi} 0" />
+      <axis rpy="0 0 0" xyz="0 0 1" />
+      <limit lower="0.0" upper="0.0" effort="0.0" velocity="0.0" />
+    </joint>
     <gazebo>
       <plugin filename="libuuv_gazebo_ros_imu_plugin.so"
         name="${name}_imu_plugin">
         <robot_namespace>${namespace}</robot_namespace>
-        <link_name>${name}_link</link_name>
+        <link_name>${name}_sim_link</link_name>
         <sensor_topic>sensors/imu/data</sensor_topic>
         <gyroscope_noise_density>0.0002514074</gyroscope_noise_density>
