Commit message: namespace solved  issue

File: auv_description/auv_common_descriptions/urdf/sensors/realsense_d435.urdf.xacro (robot description, xacro)
@@ -11,5 +11,5 @@
         <joint name="${namespace}/camera_depth_optical_joint" type="fixed">
             <parent link="${name}"/>
-            <child link="${namespace}/camera_depth_optical_frame"/>
+            <child link="${namespace}/_camera_depth_optical_frame"/>
             <origin xyz="0 0 0" rpy="${-pi/2} 0 ${-pi/2}"/>
         </joint>

File: auv_description/taluy_description/urdf/auv_base.urdf.xacro (robot description, xacro)
@@ -58,5 +58,5 @@
     <xacro:sonar name="${namespace}/base_link/sonar_right" parent="${namespace}/base_link" position="0.02 -0.21 -0.14" orientation="0 0 ${-math.pi/2}"/>
     <xacro:sonar name="${namespace}/base_link/sonar_left" parent="${namespace}/base_link" position="0.02 0.21 -0.14" orientation="0 0 ${math.pi/2}"/>
-    <xacro:realsense_d435 name="${namespace}/camera" parent="${namespace}/_base_link" position="0.35 0 0" orientation="0 0 0"/>
+    <xacro:realsense_d435 name="${namespace}/camera" parent="${namespace}/base_link" position="0.35 0 0" orientation="0 0 0"/>
     <!-- <link name="base_footprint">
       <inertial>

Commit message: a

File: auv_description/auv_common_descriptions/urdf/sensors/realsense_d435.urdf.xacro (robot description, xacro)
@@ -8,5 +8,5 @@
             <origin xyz="${position}" rpy="${orientation}"/>
         </joint>
-        <link name="${namespace}/camera_depth_optical_frame"/>
+        <link name="${namespace}/_camera_depth_optical_frame"/>
         <joint name="${namespace}/camera_depth_optical_joint" type="fixed">
             <parent link="${name}"/>

Commit message: fix typo

File: auv_description/auv_common_descriptions/urdf/sensors/realsense_d435.urdf.xacro (robot description, xacro)
@@ -9,5 +9,5 @@
         </joint>
         <link name="${namespace}/_camera_depth_optical_frame"/>
-        <joint name="${namespace}/camera_depth_optical_joint" type="fixed">
+        <joint name="${namespace}/_camera_depth_optical_joint" type="fixed">
             <parent link="${name}"/>
             <child link="${namespace}/_camera_depth_optical_frame"/>

Commit message: new typo

File: auv_description/auv_common_descriptions/urdf/sensors/realsense_d435.urdf.xacro (robot description, xacro)
@@ -8,8 +8,8 @@
             <origin xyz="${position}" rpy="${orientation}"/>
         </joint>
-        <link name="${namespace}/_camera_depth_optical_frame"/>
+        <link name="${namespace}/_depth_optical_frame"/>
         <joint name="${namespace}/_camera_depth_optical_joint" type="fixed">
             <parent link="${name}"/>
-            <child link="${namespace}/_camera_depth_optical_frame"/>
+            <child link="${namespace}/_depth_optical_frame"/>
             <origin xyz="0 0 0" rpy="${-pi/2} 0 ${-pi/2}"/>
         </joint>

Commit message: fix camera frame 24 june

File: auv_description/auv_common_descriptions/urdf/sensors/realsense_d435.urdf.xacro (robot description, xacro)
@@ -8,8 +8,8 @@
             <origin xyz="${position}" rpy="${orientation}"/>
         </joint>
-        <link name="${namespace}/_depth_optical_frame"/>
-        <joint name="${namespace}/_camera_depth_optical_joint" type="fixed">
+        <link name="${name}_depth_optical_frame"/>
+        <joint name="${name}_depth_optical_joint" type="fixed">
             <parent link="${name}"/>
-            <child link="${namespace}/_depth_optical_frame"/>
+            <child link="${name}_depth_optical_frame"/>
             <origin xyz="0 0 0" rpy="${-pi/2} 0 ${-pi/2}"/>
         </joint>

File: auv_description/taluy_description/urdf/auv_base.urdf.xacro (robot description, xacro)
@@ -58,5 +58,5 @@
     <xacro:sonar name="${namespace}/base_link/sonar_right" parent="${namespace}/base_link" position="0.02 -0.21 -0.14" orientation="0 0 ${-math.pi/2}"/>
     <xacro:sonar name="${namespace}/base_link/sonar_left" parent="${namespace}/base_link" position="0.02 0.21 -0.14" orientation="0 0 ${math.pi/2}"/>
-    <xacro:realsense_d435 name="${namespace}/camera" parent="${namespace}/base_link" position="-0.35 0 0" orientation="0 0 0"/>
+    <xacro:realsense_d435 name="${namespace}/camera" parent="${namespace}/base_link" position="-0.35 0 0" orientation="0 0 ${math.pi}"/>
     <!-- <link name="base_footprint">
       <inertial>

Commit message: pre-commit

File: auv_description/auv_common_descriptions/urdf/sensors/realsense_d435.urdf.xacro (robot description, xacro)
@@ -1,17 +1,17 @@
 <?xml version="1.0"?>
 <robot xmlns:xacro="http://www.ros.org/wiki/xacro">
-    <xacro:macro name="realsense_d435" params="name parent position orientation">
-        <link name="${name}"/>
-        <joint name="${name}_joint" type="fixed">
-            <parent link="${parent}"/>
-            <child link="${name}"/>
-            <origin xyz="${position}" rpy="${orientation}"/>
-        </joint>
-        <link name="${name}_depth_optical_frame"/>
-        <joint name="${name}_depth_optical_joint" type="fixed">
-            <parent link="${name}"/>
-            <child link="${name}_depth_optical_frame"/>
-            <origin xyz="0 0 0" rpy="${-pi/2} 0 ${-pi/2}"/>
-        </joint>
-    </xacro:macro>
+  <xacro:macro name="realsense_d435" params="name parent position orientation">
+    <link name="${name}"/>
+    <joint name="${name}_joint" type="fixed">
+      <parent link="${parent}"/>
+      <child link="${name}"/>
+      <origin xyz="${position}" rpy="${orientation}"/>
+    </joint>
+    <link name="${name}_depth_optical_frame"/>
+    <joint name="${name}_depth_optical_joint" type="fixed">
+      <parent link="${name}"/>
+      <child link="${name}_depth_optical_frame"/>
+      <origin xyz="0 0 0" rpy="${-pi/2} 0 ${-pi/2}"/>
+    </joint>
+  </xacro:macro>
 </robot>

Commit message: Add RealSense D435 camera integration

File: auv_description/auv_common_descriptions/urdf/sensors/realsense_d435.urdf.xacro (robot description, xacro)
@@ -14,4 +14,10 @@
       <origin xyz="0 0 0" rpy="${-pi/2} 0 ${-pi/2}"/>
     </joint>
+    <link name="${name}_color_optical_frame"/>
+    <joint name="${name}_color_optical_joint" type="fixed">
+      <parent link="${name}"/>
+      <child link="${name}_color_optical_frame"/>
+      <origin xyz="0 0 0" rpy="${-pi/2} 0 ${-pi/2}"/>
+    </joint>
   </xacro:macro>
 </robot>

File: auv_sim/auv_sim_description/taluy_sim_description/urdf/sensors.urdf.xacro (robot description, xacro)
@@ -14,67 +14,5 @@
   <xacro:xsens_mti_g710_sim name="${namespace}/base_link/imu" namespace="${namespace}" static_reference_frame="${inertial_reference_frame}" update_rate="$(arg imu_update_rate)"/>
   <xacro:wayfinder_dvl_sim name="${namespace}/base_link/dvl" namespace="${namespace}" static_reference_frame="${inertial_reference_frame}" update_rate="$(arg dvl_update_rate)"/>
-  <!-- Include RealSense D435 camera -->
-  <xacro:include filename="$(find realsense2_description)/urdf/_d435.urdf.xacro"/>
-  <!-- Add RealSense camera to the front of the AUV -->
-  <xacro:sensor_d435 parent="$(arg namespace)/base_link" use_nominal_extrinsics="true" add_plug="true" use_mesh="true">
-    <origin xyz="-0.35 0 0" rpy="0 0 ${math.pi}"/>
-  </xacro:sensor_d435>
-  <!-- RealSense RGB Camera Gazebo plugin -->
-  <gazebo reference="camera_link">
-    <sensor type="camera" name="camera">
-      <update_rate>30.0</update_rate>
-      <camera name="camera">
-        <horizontal_fov>1.211</horizontal_fov>
-        <image>
-          <width>1280</width>
-          <height>720</height>
-          <format>RGB8</format>
-        </image>
-        <clip>
-          <near>0.1</near>
-          <far>100</far>
-        </clip>
-      </camera>
-      <plugin name="camera_controller" filename="libgazebo_ros_camera.so">
-        <alwaysOn>true</alwaysOn>
-        <updateRate>30.0</updateRate>
-        <cameraName>camera</cameraName>
-        <imageTopicName>rgb/image_raw</imageTopicName>
-        <cameraInfoTopicName>rgb/camera_info</cameraInfoTopicName>
-        <frameName>camera_color_optical_frame</frameName>
-        <hackBaseline>0.07</hackBaseline>
-      </plugin>
-    </sensor>
-  </gazebo>
-  <!-- RealSense Depth Camera Gazebo plugin -->
-  <gazebo reference="camera_depth_frame">
-    <sensor type="depth" name="depth_camera">
-      <update_rate>30.0</update_rate>
-      <camera name="depth_camera">
-        <horizontal_fov>1.487</horizontal_fov>
-        <image>
-          <width>1280</width>
-          <height>720</height>
-          <format>B8G8R8</format>
-        </image>
-        <clip>
-          <near>0.1</near>
-          <far>10</far>
-        </clip>
-      </camera>
-      <plugin name="depth_camera_controller" filename="libgazebo_ros_openni_kinect.so">
-        <alwaysOn>true</alwaysOn>
-        <updateRate>30.0</updateRate>
-        <cameraName>camera</cameraName>
-        <imageTopicName>depth/image_raw</imageTopicName>
-        <cameraInfoTopicName>depth/camera_info</cameraInfoTopicName>
-        <depthImageTopicName>depth/image_raw</depthImageTopicName>
-        <depthImageCameraInfoTopicName>depth/camera_info</depthImageCameraInfoTopicName>
-        <pointCloudTopicName>depth/points</pointCloudTopicName>
-        <frameName>taluy/camera_depth_optical_frame</frameName>
-        <pointCloudCutoff>0.1</pointCloudCutoff>
-        <pointCloudCutoffMax>10.0</pointCloudCutoffMax>
-      </plugin>
-    </sensor>
-  </gazebo>
+  <xacro:include filename="$(find taluy_sim_description)/urdf/realsense_sim.urdf.xacro"/>
+  <xacro:realsense_sim name="${namespace}/camera"/>
 </robot>

Commit message: fix

File: auv_description/auv_common_descriptions/urdf/sensors/realsense_d435.urdf.xacro (robot description, xacro)
@@ -8,14 +8,14 @@
       <origin xyz="${position}" rpy="${orientation}"/>
     </joint>
-    <link name="${name}_depth_optical_frame"/>
+    <link name="${name}_depth_optical_link"/>
     <joint name="${name}_depth_optical_joint" type="fixed">
       <parent link="${name}"/>
-      <child link="${name}_depth_optical_frame"/>
+      <child link="${name}_depth_optical_link"/>
       <origin xyz="0 0 0" rpy="${-pi/2} 0 ${-pi/2}"/>
     </joint>
-    <link name="${name}_color_optical_frame"/>
+    <link name="${name}_color_optical_link"/>
     <joint name="${name}_color_optical_joint" type="fixed">
       <parent link="${name}"/>
-      <child link="${name}_color_optical_frame"/>
+      <child link="${name}_color_optical_link"/>
       <origin xyz="0 0 0" rpy="${-pi/2} 0 ${-pi/2}"/>
     </joint>

File: auv_description/taluy_description/urdf/auv_base.urdf.xacro (robot description, xacro)
@@ -59,5 +59,5 @@
     <xacro:sonar name="${namespace}/base_link/sonar_left" parent="${namespace}/base_link" position="0.02 0.21 -0.14" orientation="0 0 ${math.pi/2}"/>
     <xacro:ball_dropper name="${namespace}/base_link/ball_dropper" parent="${namespace}/base_link" position="0.1004 0.0745 -0.1953" orientation="0 0 0"/>
-    <xacro:realsense_d435 name="${namespace}/camera" parent="${namespace}/base_link" position="-0.35 0 0" orientation="0 0 ${math.pi}"/>
+    <xacro:realsense_d435 name="${namespace}/base_link/back_camera" parent="${namespace}/base_link" position="-0.35 0 0" orientation="0 0 ${math.pi}"/>
     <!-- <link name="base_footprint">
       <inertial>

File: auv_sim/auv_sim_description/auv_common_sim_descriptions/urdf/sensors.urdf.xacro (robot description, xacro)
@@ -6,3 +6,4 @@
   <xacro:include filename="$(find auv_common_sim_descriptions)/urdf/sensors/sonar.urdf.xacro"/>
   <xacro:include filename="$(find auv_common_sim_descriptions)/urdf/sensors/wayfinder_dvl.urdf.xacro"/>
+  <xacro:include filename="$(find auv_common_sim_descriptions)/urdf/sensors/realsense_d435.urdf.xacro"/>
 </robot>

File: auv_sim/auv_sim_description/taluy_sim_description/urdf/sensors.urdf.xacro (robot description, xacro)
@@ -14,5 +14,4 @@
   <xacro:xsens_mti_g710_sim name="${namespace}/base_link/imu" namespace="${namespace}" static_reference_frame="${inertial_reference_frame}" update_rate="$(arg imu_update_rate)"/>
   <xacro:wayfinder_dvl_sim name="${namespace}/base_link/dvl" namespace="${namespace}" static_reference_frame="${inertial_reference_frame}" update_rate="$(arg dvl_update_rate)"/>
-  <xacro:include filename="$(find taluy_sim_description)/urdf/realsense_sim.urdf.xacro"/>
-  <xacro:realsense_sim name="${namespace}/camera"/>
+  <xacro:realsense_d435_sim name="${namespace}/base_link/back_camera" topic_name="cameras/cam_back"/>
 </robot>
