Commit message: create bar30 gazebo plugin
- use libuuv_gazebo_ros_subsea_pressure_plugin
- Changed the joint type of the bar30 link from `fixed` to `revolute` (with movement limits) to resolve an issue where libuuv_gazebo_ros plugins couldn't detect fixed links in Gazebo.
- Noted that Gazebo doesn't recognize links with fixed joints as standalone links, which seems to cause this issue.

File: auv_description/auv_common_descriptions/urdf/sensors/bar30.urdf.xacro (robot description, xacro)
@@ -25,9 +25,10 @@
     </link>
     <link name="${name}_link" />
-    <joint name="${name}_joint" type="fixed">
+    <joint name="${name}_joint" type="revolute">
       <parent link="${parent}" />
       <child link="${name}_chasis_link" />
       <origin xyz="${position}" rpy="${orientation}" />
       <axis rpy="0 0 0" xyz="0 0 1" />
+      <limit upper="0" lower="0" effort="0" velocity="0" />
     </joint>
     <joint name="${name}_sensor_joint" type="fixed">

File: auv_sim/auv_sim_description/urdf/gazebo_plugins.urdf.xacro (robot description, xacro)
@@ -91,3 +91,22 @@
     </gazebo>
   </xacro:macro>
+  <!-- bar30 plugin -->
+  <xacro:macro name="bar30_sim" params="name">
+    <gazebo>
+      <plugin filename="libuuv_gazebo_ros_subsea_pressure_plugin.so"
+        name="${name}_pressure_plugin">
+        <robot_namespace>taluy</robot_namespace>
+        <link_name>${name}_chasis_link</link_name>
+        <sensor_topic>sensors/pressure/data</sensor_topic>
+        <update_rate>50.0</update_rate>
+        <saturation>5000</saturation>
+        <noise_sigma>0.4</noise_sigma>
+        <noise_amplitude>0.13</noise_amplitude>
+        <estimate_depth_on>false</estimate_depth_on>
+        <standard_pressure>101.325</standard_pressure>
+        <kPa_per_meter>9.80638</kPa_per_meter>
+        <enable_gazebo_messages>false</enable_gazebo_messages>
+      </plugin>
+    </gazebo>
+  </xacro:macro>
 </robot>

File: auv_sim/auv_sim_description/urdf/taluy_sim.urdf.xacro (robot description, xacro)
@@ -16,4 +16,5 @@
   <xacro:t200_thruster_sim name="thruster_6" thruster_id="6" />
   <xacro:t200_thruster_sim name="thruster_7" thruster_id="7" />
+  <xacro:bar30_sim name="base_link/external_pressure_sensor" />
   <!--  -->
 </robot>

Commit message: create bar30 gazebo plugin
- use libuuv_gazebo_ros_subsea_pressure_plugin
- Changed the joint type of the bar30 link from `fixed` to `revolute` (with movement limits) to resolve an issue where libuuv_gazebo_ros plugins couldn't detect fixed links in Gazebo.
- Noted that Gazebo doesn't recognize links with fixed joints as standalone links, which seems to cause this issue.

File: auv_description/auv_common_descriptions/urdf/sensors/bar30.urdf.xacro (robot description, xacro)
@@ -20,10 +20,11 @@
       </inertial>
     </link>
-    <link name="${name}_link"/>
-    <joint name="${name}_joint" type="fixed">
-      <parent link="${parent}"/>
-      <child link="${name}_chasis_link"/>
-      <origin xyz="${position}" rpy="${orientation}"/>
-      <axis rpy="0 0 0" xyz="0 0 1"/>
+    <link name="${name}_link" />
+    <joint name="${name}_joint" type="revolute">
+      <parent link="${parent}" />
+      <child link="${name}_chasis_link" />
+      <origin xyz="${position}" rpy="${orientation}" />
+      <axis rpy="0 0 0" xyz="0 0 1" />
+      <limit upper="0" lower="0" effort="0" velocity="0" />
     </joint>
     <joint name="${name}_sensor_joint" type="fixed">

Commit message: revert Bar30 joint type from `revolute` to `fixed`

File: auv_description/auv_common_descriptions/urdf/sensors/bar30.urdf.xacro (robot description, xacro)
@@ -25,10 +25,9 @@
     </link>
     <link name="${name}_link" />
-    <joint name="${name}_joint" type="revolute">
+    <joint name="${name}_joint" type="fixed">
       <parent link="${parent}" />
       <child link="${name}_chasis_link" />
       <origin xyz="${position}" rpy="${orientation}" />
       <axis rpy="0 0 0" xyz="0 0 1" />
-      <limit upper="0" lower="0" effort="0" velocity="0" />
     </joint>
     <joint name="${name}_sensor_joint" type="fixed">

File: auv_sim/auv_sim_description/auv_common_sim_descriptions/urdf/sensors/bar30.urdf.xacro (robot description, xacro)
@@ -2,9 +2,29 @@
 <robot name="bar30" xmlns:xacro="http://www.ros.org/wiki/xacro">
   <xacro:macro name="bar30_sim" params="name">
+    <link name="${name}_sim_link">
+      <inertial>
+        <mass value="0.001" />
+        <origin xyz="0 0 0" rpy="0 0 0" />
+        <inertia ixx="0.0000001" ixy="0" ixz="0" iyy="0.0000001" iyz="0" izz="0.0000001" />
+      </inertial>
+      <collision>
+        <geometry>
+          <cylinder length="${0.000001}" radius="${0.000001}" />
+        </geometry>
+        <origin xyz="0 0 0" rpy="0 ${0.5*pi} 0" />
+      </collision>
+    </link>
+    <joint name="${name}_sim_joint" type="revolute">
+      <parent link="${name}_chasis_link" />
+      <child link="${name}_sim_link" />
+      <origin xyz="0 0 0" rpy="0 0 0" />
+      <axis rpy="0 0 0" xyz="0 0 1" />
+      <limit lower="0.0" upper="0.0" effort="0.0" velocity="0.0" />
+    </joint>
     <gazebo>
       <plugin filename="libuuv_gazebo_ros_subsea_pressure_plugin.so"
         name="${name}_pressure_plugin">
         <robot_namespace>taluy</robot_namespace>
-        <link_name>${name}_chasis_link</link_name>
+        <link_name>${name}_sim_link</link_name>
         <sensor_topic>sim/pressure</sensor_topic>
         <update_rate>50.0</update_rate>

Commit message: fix IMU, Sonar and Bar30 in simulation (#96)
* revert IMU joint type from `revolute` to `fixed`

- add rotation to fix imu plugin values

* fix sonar plugin topic name

- removed namespace at the start of the topic name since it was causing issues
- also change update rate and range according to sensor specifications

* revert Bar30 joint type from `revolute` to `fixed`

* add imu offset to simulation

* fix drift ros param

* rename topics

- renamed it in the code and remapped it to same place.
- this is just to make it more understandable

---------

Co-authored-by: Ozan Hakan Tunca <t.ozanhakan@gmail.com>

File: auv_description/auv_common_descriptions/urdf/sensors/bar30.urdf.xacro (robot description, xacro)
@@ -21,10 +21,9 @@
     </link>
     <link name="${name}_link" />
-    <joint name="${name}_joint" type="revolute">
+    <joint name="${name}_joint" type="fixed">
       <parent link="${parent}" />
       <child link="${name}_chasis_link" />
       <origin xyz="${position}" rpy="${orientation}" />
       <axis rpy="0 0 0" xyz="0 0 1" />
-      <limit upper="0" lower="0" effort="0" velocity="0" />
     </joint>
     <joint name="${name}_sensor_joint" type="fixed">

File: auv_description/auv_common_descriptions/urdf/sensors/xsens_mti_g710.urdf.xacro (robot description, xacro)
@@ -20,10 +20,9 @@
       </inertial>
     </link>
-    <joint name="${name}_joint" type="revolute">
+    <joint name="${name}_joint" type="fixed">
       <parent link="${parent}" />
       <child link="${name}_link" />
       <origin xyz="${position}" rpy="${orientation}" />
       <axis rpy="0 0 0" xyz="0 0 1" />
-      <limit upper="0" lower="0" effort="0" velocity="0" />
     </joint>
   </xacro:macro>

File: auv_sim/auv_sim_description/auv_common_sim_descriptions/urdf/sensors/xsens_mti_g710.urdf.xacro (robot description, xacro)
@@ -2,10 +2,30 @@
 <robot name="xsens_mti_g710" xmlns:xacro="http://www.ros.org/wiki/xacro">
   <xacro:macro name="xsens_mti_g710_sim" params="name namespace static_reference_frame">
+    <link name="${name}_sim_link">
+      <inertial>
+        <mass value="0.001" />
+        <origin xyz="0 0 0" rpy="0 0 0" />
+        <inertia ixx="0.0000001" ixy="0" ixz="0" iyy="0.0000001" iyz="0" izz="0.0000001" />
+      </inertial>
+      <collision>
+        <geometry>
+          <cylinder length="${0.000001}" radius="${0.000001}" />
+        </geometry>
+        <origin xyz="0 0 0" rpy="0 ${0.5*pi} 0" />
+      </collision>
+    </link>
+    <joint name="${name}_sim_joint" type="revolute">
+      <parent link="${name}_link" />
+      <child link="${name}_sim_link" />
+      <origin xyz="0 0 0" rpy="${math.pi} ${math.pi} 0" />
+      <axis rpy="0 0 0" xyz="0 0 1" />
+      <limit lower="0.0" upper="0.0" effort="0.0" velocity="0.0" />
+    </joint>
     <gazebo>
       <plugin filename="libuuv_gazebo_ros_imu_plugin.so"
         name="${name}_imu_plugin">
         <robot_namespace>${namespace}</robot_namespace>
-        <link_name>${name}_link</link_name>
-        <sensor_topic>sensors/imu/data</sensor_topic>
+        <link_name>${name}_sim_link</link_name>
+        <sensor_topic>sim/imu</sensor_topic>
         <gyroscope_noise_density>0.0002514074</gyroscope_noise_density>
         <gyroscope_random_walk>0.000038785</gyroscope_random_walk>

Commit message: Update bar30 sensor position and adjust camera orientations in auv_base

File: auv_description/auv_common_descriptions/urdf/sensors/bar30.urdf.xacro (robot description, xacro)
@@ -31,5 +31,5 @@
       <parent link="${name}_chasis_link"/>
       <child link="${name}_link"/>
-      <origin xyz="0 0 0.0075" rpy="0 0 0"/>
+      <origin xyz="0 0 0.0092" rpy="0 0 0"/>
     </joint>
   </xacro:macro>

File: auv_description/taluy_description/urdf/auv_base.urdf.xacro (robot description, xacro)
@@ -50,13 +50,14 @@
     <xacro:h2c_hydrophone name="${namespace}/base_link/hydrophone_3" parent="${namespace}/base_link" position="-0.315 -0.1675 0.1715" orientation="0 0 0"/>
     <xacro:ping360 name="${namespace}/base_link/ping360" parent="${namespace}/base_link" position="0.2 0 0.134" orientation="0 0 0"/>
-    <xacro:bar30 name="${namespace}/base_link/external_pressure_sensor" parent="${namespace}/base_link" position="0 0 0.07" orientation="0 0 0"/>
-    <xacro:logitech_c920_camera name="${namespace}/base_link/front_camera" parent="${namespace}/base_link" position="0.35 0 0" orientation="0 0 0"/>
+    <xacro:bar30 name="${namespace}/base_link/external_pressure_sensor" parent="${namespace}/base_link" position="0 0 0.079" orientation="0 0 0"/>
+    <xacro:logitech_c920_camera name="${namespace}/base_link/front_camera" parent="${namespace}/base_link" position="0.35 0 0" orientation="0 0.1234 0"/>
     <xacro:logitech_c920_camera name="${namespace}/base_link/bottom_camera" parent="${namespace}/base_link" position="0 0 -0.07" orientation="0 ${math.pi/2} ${-math.pi/2}"/>
-    <xacro:torpedo_upper name="${namespace}/base_link/torpedo_upper" parent="${namespace}/base_link" position="0.3916 -0.11 -0.056" orientation="0 0 0"/>
-    <xacro:torpedo_bottom name="${namespace}/base_link/torpedo_bottom" parent="${namespace}/base_link" position="0.3916 -0.11 -0.091" orientation="0 0 0"/>
+    <xacro:torpedo_upper name="${namespace}/base_link/torpedo_upper" parent="${namespace}/base_link" position="0.4057 -0.1038 -0.049" orientation="0 0 0"/>
+    <xacro:torpedo_bottom name="${namespace}/base_link/torpedo_bottom" parent="${namespace}/base_link" position="0.4057 -0.1038 -0.084" orientation="0 0 0"/>
     <xacro:sonar name="${namespace}/base_link/sonar_front" parent="${namespace}/base_link" position="0.38 0.09 0.09" orientation="0 0 0"/>
     <xacro:sonar name="${namespace}/base_link/sonar_back" parent="${namespace}/base_link" position="-0.42 -0.09 0.09" orientation="0 0 ${math.pi}"/>
     <xacro:sonar name="${namespace}/base_link/sonar_right" parent="${namespace}/base_link" position="0.02 -0.21 -0.14" orientation="0 0 ${-math.pi/2}"/>
     <xacro:sonar name="${namespace}/base_link/sonar_left" parent="${namespace}/base_link" position="0.02 0.21 -0.14" orientation="0 0 ${math.pi/2}"/>
+    <!-- 0.0931 -->
     <xacro:ball_dropper name="${namespace}/base_link/ball_dropper" parent="${namespace}/base_link" position="0.1004 0.0745 -0.1953" orientation="0 0 0"/>
     <xacro:realsense_d435 name="${namespace}/camera" parent="${namespace}/base_link" position="-0.35 0 0" orientation="0 0 ${math.pi}"/>
