Commit message: create dvl plugin and bridge

File: auv_description/auv_common_descriptions/urdf/sensors/wayfinder_dvl.urdf.xacro (robot description, xacro)
@@ -19,4 +19,8 @@
         </geometry>
       </collision>
+      <inertial>
+        <mass value="0.0001" />
+        <inertia ixx="0.000001" ixy="0.0" ixz="0.0" iyy="0.000001" iyz="0.0" izz="0.000001" />
+      </inertial>
     </link>
     <link name="${name}_cog">
@@ -31,9 +35,10 @@
     <link name="${name}_sensor_surface_link" />
     <link name="${name}_link" />
-    <joint name="${name}_chasis_joint" type="fixed">
+    <joint name="${name}_chasis_joint" type="revolute">
       <parent link="${parent}" />
       <child link="${name}_mount_link" />
       <origin xyz="${position}" rpy="${orientation}" />
       <axis rpy="0 0 0" xyz="0 0 1" />
+      <limit upper="0" lower="0" effort="0" velocity="0" />
     </joint>
     <joint name="${name}_sensor_surface_joint" type="fixed">

File: auv_sim/auv_sim_description/auv_common_sim_descriptions/urdf/sensors.urdf.xacro (robot description, xacro)
@@ -9,3 +9,5 @@
   <xacro:include
     filename="$(find auv_common_sim_descriptions)/urdf/sensors/sonar.urdf.xacro" />
+  <xacro:include
+    filename="$(find auv_common_sim_descriptions)/urdf/sensors/wayfinder_dvl.urdf.xacro" />
 </robot>

File: auv_sim/auv_sim_description/taluy_sim_description/urdf/sensors.urdf.xacro (robot description, xacro)
@@ -13,3 +13,5 @@
   <xacro:xsens_mti_g710_sim name="${namespace}/base_link/imu" namespace="${namespace}"
     static_reference_frame="${inertial_reference_frame}" />
+  <xacro:wayfinder_dvl_sim name="${namespace}/base_link/dvl" namespace="${namespace}"
+    static_reference_frame="${inertial_reference_frame}" />
 </robot>

File: auv_sim/auv_sim_description/taluy_sim_description/urdf/taluy_sim.urdf.xacro (robot description, xacro)
@@ -30,5 +30,5 @@
     namespace="$(arg namespace)"
     parent_link="$(arg namespace)/base_link"
-    topic="odometry"
+    topic="odometry_gt"
     update_rate="$(arg control_rate)"
     noise_sigma="0.0"

Commit message: remove dvl plugin
- velocity and altitude values we get from uuv_simulator plugin is not consistent with the ground truth

File: auv_description/auv_common_descriptions/urdf/sensors/wayfinder_dvl.urdf.xacro (robot description, xacro)
@@ -19,8 +19,4 @@
         </geometry>
       </collision>
-      <inertial>
-        <mass value="0.0001" />
-        <inertia ixx="0.000001" ixy="0.0" ixz="0.0" iyy="0.000001" iyz="0.0" izz="0.000001" />
-      </inertial>
     </link>
     <link name="${name}_cog">
@@ -35,10 +31,9 @@
     <link name="${name}_sensor_surface_link" />
     <link name="${name}_link" />
-    <joint name="${name}_chasis_joint" type="revolute">
+    <joint name="${name}_chasis_joint" type="fixed">
       <parent link="${parent}" />
       <child link="${name}_mount_link" />
       <origin xyz="${position}" rpy="${orientation}" />
       <axis rpy="0 0 0" xyz="0 0 1" />
-      <limit upper="0" lower="0" effort="0" velocity="0" />
     </joint>
     <joint name="${name}_sensor_surface_joint" type="fixed">

File: auv_sim/auv_sim_description/auv_common_sim_descriptions/urdf/sensors.urdf.xacro (robot description, xacro)
@@ -9,5 +9,3 @@
   <xacro:include
     filename="$(find auv_common_sim_descriptions)/urdf/sensors/sonar.urdf.xacro" />
-  <xacro:include
-    filename="$(find auv_common_sim_descriptions)/urdf/sensors/wayfinder_dvl.urdf.xacro" />
 </robot>

File: auv_sim/auv_sim_description/taluy_sim_description/urdf/sensors.urdf.xacro (robot description, xacro)
@@ -13,5 +13,3 @@
   <xacro:xsens_mti_g710_sim name="${namespace}/base_link/imu" namespace="${namespace}"
     static_reference_frame="${inertial_reference_frame}" />
-  <xacro:wayfinder_dvl_sim name="${namespace}/base_link/dvl" namespace="${namespace}"
-    static_reference_frame="${inertial_reference_frame}" />
 </robot>

Commit message: format

File: auv_description/auv_common_descriptions/urdf/sensors/wayfinder_dvl.urdf.xacro (robot description, xacro)
@@ -2,6 +2,5 @@
 <robot xmlns:xacro="http://ros.org/wiki/xacro" name="wayfinder_dvl">
   <xacro:macro name="wayfinder_dvl" params="name parent position:='0 0 0' orientation:='0 0 0'">
-    <link name="${name}_mount_link">
-    </link>
+    <link name="${name}_mount_link"/>
     <link name="${name}_cog">
       <inertial>

Commit message: vehicle changes

File: auv_description/auv_common_descriptions/urdf/sensors/wayfinder_dvl.urdf.xacro (robot description, xacro)
@@ -2,5 +2,5 @@
 <robot xmlns:xacro="http://ros.org/wiki/xacro" name="wayfinder_dvl">
   <xacro:macro name="wayfinder_dvl" params="name parent position:='0 0 0' orientation:='0 0 0' use_models:='false'">
-    <xacro:property name="sensor_orientation" value="${math.pi/3 if 'taluy_mini' in name else -3*math.pi/4}"/>
+    <xacro:property name="sensor_orientation" value="${1.244419 if 'taluy_mini' in name else -3*math.pi/4}"/>
     <link name="${name}_mount_link">
       <xacro:if value="${use_models}">
