Commit message: remove gazebo ref from xacro

File: auv_description/auv_common_descriptions/urdf/sensors/wayfinder_dvl.urdf.xacro (robot description, xacro)
@@ -56,10 +56,4 @@
       <origin xyz="0 0 0" rpy="0 0 ${sensor_orientation}"/>
     </joint>
-    <!-- <gazebo reference="${name}_propeller_link">
-      <material>Gazebo/Orange</material>
-    </gazebo>
-    <gazebo reference="${name}_link">
-      <material>Gazebo/Orange</material>
-    </gazebo> -->
   </xacro:macro>
 </robot>
