Commit message: update

File: auv_sim/auv_sim_description/urdf/dynamics.urdf.xacro (robot description, xacro)
@@ -23,5 +23,5 @@
   <xacro:macro name="auv_hydro_model" params="namespace">
     <link name="${namespace}/base_link">
-      <neutrally_buoyant>0</neutrally_buoyant>
+      <neutrally_buoyant>1</neutrally_buoyant>
       <volume>${volume}</volume>
       <box>
@@ -42,8 +42,8 @@
         </added_mass>
         <linear_damping>
-          -30 -31 -89 0 0 -1.87
+          -30 -31 -89 -1.87 -1.87 -1.87
         </linear_damping>
         <quadratic_damping>
-          -77 -155 -136 0 0 -7.98
+          -77 -155 -136 -7.98 -7.98 -7.98
         </quadratic_damping>
       </hydrodynamic_model>

File: auv_sim/auv_sim_description/urdf/gazebo_plugins.urdf.xacro (robot description, xacro)
@@ -43,9 +43,9 @@
   </xacro:macro>
   <!-- imu plugin -->
-  <xacro:macro name="xsens_mti_g710_sim" params="name">
+  <xacro:macro name="xsens_mti_g710_sim" params="name namespace static_reference_frame">
     <gazebo>
       <plugin filename="libuuv_gazebo_ros_imu_plugin.so"
         name="${name}_imu_plugin">
-        <robot_namespace>taluy</robot_namespace>
+        <robot_namespace>${namespace}</robot_namespace>
         <link_name>${name}_link</link_name>
         <sensor_topic>sensors/imu/data</sensor_topic>
@@ -62,5 +62,5 @@
         <enable_gazebo_messages>false</enable_gazebo_messages>
         <enable_local_ned_frame>false</enable_local_ned_frame>
-        <static_reference_frame>world</static_reference_frame>
+        <static_reference_frame>${static_reference_frame}</static_reference_frame>
       </plugin>
     </gazebo>
@@ -73,7 +73,8 @@
         <jointName>${name}_propeller_joint</jointName>
         <thrusterID>${thruster_id}</thrusterID>
+        <gain>1</gain>
         <dynamics>
           <type>FirstOrder</type>
-          <timeConstant>0.05</timeConstant>
+          <timeConstant>0.04</timeConstant>
         </dynamics>
         <conversion>
@@ -82,17 +83,33 @@
           </type>
           <inputValues>
-            0 1009 1100 1110 1120 1130 1140 1150 1160 1170 1180 1190 1200 1210 1220 1230 1240 1250
-            1260 1270 1280 1290 1300 1310 1320 1330 1340 1350 1360 1370 1380 1390 1400 1410 1420
-            1430 1440 1450 1460 1470 1480 1490 1500 1510 1520 1530 1540 1550 1560 1570 1580 1590
-            1600 1610 1620 1630 1640 1650 1660 1670 1680 1690 1700 1710 1720 1730 1740 1750 1760
-            1770 1780 1790 1800 1810 1820 1830 1840 1850 1860 1870 1880 1890 1900 1901 1902
+            0 1099 1100 1104 1108 1112 1116 1120 1124 1128 1132 1136 1140 1144 1148 1152 1156 1160
+            1164 1168 1172 1176 1180 1184 1188 1192 1196 1200 1204 1208 1212 1216 1220 1224 1228
+            1232 1236 1240 1244 1248 1252 1256 1260 1264 1268 1272 1276 1280 1284 1288 1292 1296
+            1300 1304 1308 1312 1316 1320 1324 1328 1332 1336 1340 1344 1348 1352 1356 1360 1364
+            1368 1372 1376 1380 1384 1388 1392 1396 1400 1404 1408 1412 1416 1420 1424 1428 1432
+            1436 1440 1444 1448 1452 1456 1460 1464 1468 1472 1476 1480 1484 1488 1492 1496 1500
+            1504 1508 1512 1516 1520 1524 1528 1532 1536 1540 1544 1548 1552 1556 1560 1564 1568
+            1572 1576 1580 1584 1588 1592 1596 1600 1604 1608 1612 1616 1620 1624 1628 1632 1636
+            1640 1644 1648 1652 1656 1660 1664 1668 1672 1676 1680 1684 1688 1692 1696 1700 1704
+            1708 1712 1716 1720 1724 1728 1732 1736 1740 1744 1748 1752 1756 1760 1764 1768 1772
+            1776 1780 1784 1788 1792 1796 1800 1804 1808 1812 1816 1820 1824 1828 1832 1836 1840
+            1844 1848 1852 1856 1860 1864 1868 1872 1876 1880 1884 1888 1892 1896 1900 1902
           </inputValues>
           <outputValues>
-            0 0 -17.34 -16.09 -15.47 -14.98 -14.13 -13.73 -12.97 -12.35 -11.86 -11.41 -10.83 -10.21
-            -9.72 -9.09 -8.38 -7.76 -7.40 -6.91 -6.55 -6.11 -5.71 -5.22 -4.64 -4.19 -3.92 -3.61
-            -3.21 -2.67 -2.27 -1.96 -1.65 -1.38 -1.03 -0.71 -0.49 -0.31 -0.13 -0.09 0.00 0.00 0.00
-            0.00 0.00 0.09 0.36 0.62 1.03 1.43 1.92 2.50 3.03 3.61 4.23 4.73 5.35 6.02 6.73 7.22
-            7.89 8.65 9.45 10.39 11.10 11.63 12.30 12.79 13.60 14.62 15.47 16.23 16.94 17.87 19.21
-            20.06 20.59 21.40 22.20 22.78 23.71 24.38 24.69 0 0
+            0 0 -28.48 -28.61 -28.38 -27.76 -27.32 -27.09 -26.69 -26.20 -25.49 -25.45 -25.14 -24.47
+            -23.93 -23.85 -23.40 -22.96 -22.60 -22.11 -21.84 -21.40 -21.00 -20.55 -20.29 -19.71
+            -19.44 -19.08 -18.46 -18.11 -17.70 -17.44 -16.99 -16.33 -16.19 -15.79 -15.30 -15.04
+            -14.63 -14.41 -14.10 -13.70 -13.43 -13.08 -12.68 -12.54 -11.96 -11.70 -11.30 -10.94
+            -10.63 -10.23 -10.01 -9.74 -9.43 -9.12 -8.85 -8.54 -8.18 -7.78 -7.56 -7.25 -7.07 -6.80
+            -6.45 -6.27 -5.91 -5.60 -5.33 -5.07 -4.85 -4.62 -4.31 -4.09 -3.82 -3.60 -3.33 -3.11
+            -2.89 -2.62 -2.40 -2.22 -2.00 -1.73 -1.60 -1.42 -1.20 -1.06 -0.88 -0.71 -0.57 -0.44
+            -0.35 0.00 0.00 0.00 0.00 0.00 0.00 0.00 0.00 0.00 0.00 0.00 0.00 0.00 0.00 0.00 0.00
+            0.00 0.00 0.00 0.40 0.53 0.71 0.93 1.11 1.29 1.51 1.73 1.95 2.18 2.49 2.71 3.02 3.24
+            3.60 3.87 4.18 4.49 4.80 5.07 5.38 5.78 6.14 6.40 6.71 6.98 7.43 7.74 8.14 8.41 8.76
+            9.12 9.47 9.83 10.18 10.63 11.16 11.39 11.74 12.10 12.54 12.85 13.26 13.74 14.06 14.55
+            14.99 15.35 16.01 16.41 16.77 17.35 17.84 18.11 18.68 18.86 19.26 19.93 20.46 20.91
+            21.35 21.93 22.29 22.87 23.53 24.16 24.60 25.14 25.67 26.03 26.60 27.23 27.89 28.16
+            28.74 29.50 29.85 30.25 30.97 31.63 31.99 32.52 33.15 33.37 33.81 34.35 35.01 35.68
+            36.35 36.22 36.43 0
           </outputValues>
         </conversion>
@@ -114,5 +131,5 @@
         <robot_namespace>taluy</robot_namespace>
         <link_name>${name}_chasis_link</link_name>
-        <sensor_topic>sensors/pressure/data</sensor_topic>
+        <sensor_topic>sim/pressure</sensor_topic>
         <update_rate>50.0</update_rate>
         <saturation>5000</saturation>

File: auv_sim/auv_sim_description/urdf/sensors.urdf.xacro (robot description, xacro)
@@ -11,4 +11,4 @@
   <xacro:logitech_c920_camera_sim name="${namespace}/base_link/bottom_camera"
     topic_name="cameras/cam_bottom" />
-  <xacro:xsens_mti_g710_sim name="${namespace}/base_link/imu" />
+  <xacro:xsens_mti_g710_sim name="${namespace}/base_link/imu" namespace="${namespace}" static_reference_frame="${inertial_reference_frame}" />
 </robot>

File: auv_sim/auv_sim_description/urdf/taluy_sim.urdf.xacro (robot description, xacro)
@@ -3,4 +3,5 @@
   <xacro:arg name="debug" default="0" />
   <xacro:arg name="namespace" default="taluy" />
+  <xacro:arg name="control_rate" default="20" />
   <xacro:arg name="inertial_reference_frame" default="world" />
   <xacro:include filename="$(find auv_sim_description)/urdf/base.urdf.xacro" />
@@ -20,4 +21,20 @@
   <!-- joint state publisher -->
   <xacro:include filename="$(find uuv_gazebo_ros_plugins)/urdf/misc.xacro" />
-  <xacro:default_joint_state_publisher namespace="$(arg namespace)" update_rate="50" />
+  <xacro:include filename="$(find uuv_sensor_ros_plugins)/urdf/pose_3d_snippets.xacro" />
+  <xacro:default_joint_state_publisher namespace="$(arg namespace)" update_rate="$(arg control_rate)" />
+  <!-- TODO: rename odometry back to pose_gt, to not use -->
+  <!-- ground truth odometry -->
+  <!-- and also the odom -->
+  <xacro:pose_3d_macro
+    namespace="$(arg namespace)"
+    parent_link="$(arg namespace)/base_link"
+    topic="odometry"
+    update_rate="$(arg control_rate)"
+    noise_sigma="0.0"
+    noise_amplitude="0.0"
+    suffix="default"
+    reference_frame="odom"
+    publish_ned_odom="false">
+    <origin xyz="0 0 0" rpy="0 0 0" />
+  </xacro:pose_3d_macro>
 </robot>
