Commit message: use dvl frame for dvl_altimeter
- rename altimeter to dvl_altimeter to make it easier to understand altimeter is used to mock the dvl in simulation

File: auv_sim/auv_sim_description/auv_common_sim_descriptions/urdf/sensors.urdf.xacro (robot description, xacro)
@@ -10,4 +10,4 @@
     filename="$(find auv_common_sim_descriptions)/urdf/sensors/sonar.urdf.xacro" />
   <xacro:include
-    filename="$(find auv_common_sim_descriptions)/urdf/sensors/altimeter.urdf.xacro" />
+    filename="$(find auv_common_sim_descriptions)/urdf/sensors/dvl_altimeter.urdf.xacro" />
 </robot>

File: auv_sim/auv_sim_description/auv_common_sim_descriptions/urdf/sensors/dvl_altimeter.urdf.xacro (robot description, xacro)
@@ -1,8 +1,8 @@
 <?xml version="1.0"?>
-<robot name="altimeter" xmlns:xacro="http://ros.org/wiki/xacro">
-  <xacro:macro name="altimeter_sim" params="name parent position:='0 0 0' orientation:='0 0 0'">
+<robot name="dvl_altimeter" xmlns:xacro="http://ros.org/wiki/xacro">
+  <xacro:macro name="dvl_altimeter_sim" params="name parent orientation:='0 0 0'">
     <link name="${name}_link" />
     <joint name="${name}_joint" type="fixed">
-      <origin xyz="${position}" rpy="${orientation}" />
+      <origin xyz="0 0 0" rpy="${orientation}" />
       <parent link="${parent}" />
       <child link="${name}_link" />
@@ -11,5 +11,5 @@
       <sensor type="ray" name="${name}">
         <pose>0 0 0 0 0 0</pose>
-        <visualize>false</visualize>
+        <visualize>true</visualize>
         <update_rate>20</update_rate>
         <ray>
@@ -17,5 +17,5 @@
             <horizontal>
               <samples>1</samples>
-              <resolution>0.15</resolution>
+              <resolution>0.01</resolution>
               <min_angle>-0.5*0.523599</min_angle>
               <max_angle>${0.5*0.523599}</max_angle>
@@ -23,5 +23,5 @@
             <vertical>
               <samples>1</samples>
-              <resolution>0.15</resolution>
+              <resolution>0.01</resolution>
               <min_angle>-${0.5*0.523599}</min_angle>
               <max_angle>${0.5*0.523599}</max_angle>
@@ -29,7 +29,7 @@
           </scan>
           <range>
-            <min>0.15</min>
+            <min>0.01</min>
             <max>100.0</max>
-            <resolution>0.15</resolution>
+            <resolution>0.01</resolution>
           </range>
           <noise>
@@ -40,5 +40,5 @@
         </ray>
         <plugin filename="libgazebo_ros_range.so" name="${name}_range_plugin">
-          <topicName>sim/altimeter</topicName>
+          <topicName>sim/dvl_altimeter</topicName>
           <frameName>${name}_link</frameName>
           <gaussianNoise>0.005</gaussianNoise>

File: auv_sim/auv_sim_description/taluy_sim_description/urdf/sensors.urdf.xacro (robot description, xacro)
@@ -13,5 +13,5 @@
   <xacro:xsens_mti_g710_sim name="${namespace}/base_link/imu" namespace="${namespace}"
     static_reference_frame="${inertial_reference_frame}" />
-  <xacro:altimeter_sim name="${namespace}/base_link/altimeter" parent="${namespace}/base_link"
-    position="0.2 0 -0.11" orientation="0 0 0" />
+  <xacro:dvl_altimeter_sim name="${namespace}/base_link/dvl_altimeter"
+    parent="${namespace}/base_link/dvl_link" orientation="0 ${math.pi/2} 0" />
 </robot>
