Commit message: create another link for sim dvl

File: auv_sim/auv_sim_description/auv_common_sim_descriptions/urdf/sensors/wayfinder_dvl.urdf.xacro (robot description, xacro)
@@ -66,5 +66,26 @@
     </gazebo>
   </xacro:macro>
-  <xacro:macro name="wayfinder_dvl_sim" params="name namespace static_reference_frame update_rate">
+  <xacro:macro name="wayfinder_dvl_sim"
+    params="name namespace static_reference_frame update_rate position orientation">
+    <link name="${name}_sim_link">
+      <inertial>
+        <mass value="0.001" />
+        <origin xyz="0 0 0" rpy="0 0 0" />
+        <inertia ixx="0.0000001" ixy="0" ixz="0" iyy="0.0000001" iyz="0" izz="0.0000001" />
+      </inertial>
+      <collision>
+        <geometry>
+          <cylinder length="${0.000001}" radius="${0.000001}" />
+        </geometry>
+        <origin xyz="0 0 0" rpy="0 ${0.5*pi} 0" />
+      </collision>
+    </link>
+    <joint name="${name}_sim_joint" type="revolute">
+      <parent link="${name}_mount_link" />
+      <child link="${name}_sim_link" />
+      <origin xyz="${position}" rpy="${orientation}" />
+      <axis rpy="0 0 0" xyz="0 0 1" />
+      <limit lower="0.0" upper="0.0" effort="0.0" velocity="0.0" />
+    </joint>
     <xacro:dvl_single_sonar
       namespace="${namespace}"
@@ -94,5 +115,5 @@
       <plugin filename="libuuv_gazebo_ros_dvl_plugin.so" name="libuuv_gazebo_dvl_plugin">
         <robot_namespace>${namespace}</robot_namespace>
-        <link_name>${name}_mount_link</link_name>
+        <link_name>${name}_sim_link</link_name>
         <sensor_topic>sim/dvl</sensor_topic>
         <update_rate>${update_rate}</update_rate>

File: auv_sim/auv_sim_description/taluy_sim_description/urdf/sensors.urdf.xacro (robot description, xacro)
@@ -14,4 +14,5 @@
     static_reference_frame="${inertial_reference_frame}" />
   <xacro:wayfinder_dvl_sim name="${namespace}/base_link/dvl" namespace="${namespace}"
-    static_reference_frame="${inertial_reference_frame}" update_rate="10" />
+    static_reference_frame="${inertial_reference_frame}" position="0.2 0 -0.11"
+    orientation="0 0 0" update_rate="10" />
 </robot>

Commit message: remove position and orientation params

File: auv_sim/auv_sim_description/auv_common_sim_descriptions/urdf/sensors/wayfinder_dvl.urdf.xacro (robot description, xacro)
@@ -84,5 +84,5 @@
       <parent link="${name}_mount_link" />
       <child link="${name}_sim_link" />
-      <origin xyz="${position}" rpy="${orientation}" />
+      <origin xyz="0 0 0" rpy="0 0 0" />
       <axis rpy="0 0 0" xyz="0 0 1" />
       <limit lower="0.0" upper="0.0" effort="0.0" velocity="0.0" />

File: auv_sim/auv_sim_description/taluy_sim_description/urdf/sensors.urdf.xacro (robot description, xacro)
@@ -14,5 +14,4 @@
     static_reference_frame="${inertial_reference_frame}" />
   <xacro:wayfinder_dvl_sim name="${namespace}/base_link/dvl" namespace="${namespace}"
-    static_reference_frame="${inertial_reference_frame}" position="0.2 0 -0.11"
-    orientation="0 0 0" update_rate="10" />
+    static_reference_frame="${inertial_reference_frame}" update_rate="10" />
 </robot>
