Commit message: fix sonar plugin topic name
- removed namespace at the start of the topic name since it was causing issues
- also change update rate and range according to sensor specifications

File: auv_sim/auv_sim_description/auv_common_sim_descriptions/urdf/sensors/sonar.urdf.xacro (robot description, xacro)
@@ -1,10 +1,10 @@
 <?xml version="1.0"?>
 <robot name="sonar" xmlns:xacro="http://ros.org/wiki/xacro">
-  <xacro:macro name="sonar_sim" params="name">
+  <xacro:macro name="sonar_sim" params="name topic">
     <gazebo reference="${name}_link">
       <sensor type="ray" name="${name}">
         <pose>0 0 0 0 0 0</pose>
         <visualize>false</visualize>
-        <update_rate>10</update_rate>
+        <update_rate>20</update_rate>
         <ray>
           <scan>
@@ -23,7 +23,7 @@
           </scan>
           <range>
-            <min>0.5</min>
-            <max>30.0</max>
-            <resolution>0.15</resolution>
+            <min>0.3</min>
+            <max>100.0</max>
+            <resolution>0.1</resolution>
           </range>
           <noise>
@@ -34,9 +34,9 @@
         </ray>
         <plugin filename="libgazebo_ros_range.so" name="${name}_range_plugin">
-          <topicName>${name}/data</topicName>
+          <topicName>${topic}/data</topicName>
           <frameName>${name}_link</frameName>
           <gaussianNoise>0.005</gaussianNoise>
           <alwaysOn>true</alwaysOn>
-          <updateRate>10</updateRate>
+          <updateRate>20</updateRate>
           <visualize>true</visualize>
           <radiation>infrared</radiation>

File: auv_sim/auv_sim_description/taluy_sim_description/urdf/sensors.urdf.xacro (robot description, xacro)
@@ -3,8 +3,8 @@
   <xacro:include filename="$(find auv_common_sim_descriptions)/urdf/sensors.urdf.xacro" />
   <xacro:bar30_sim name="${namespace}/base_link/external_pressure_sensor" />
-  <xacro:sonar_sim name="${namespace}/base_link/sonar_front" />
-  <xacro:sonar_sim name="${namespace}/base_link/sonar_back" />
-  <xacro:sonar_sim name="${namespace}/base_link/sonar_right" />
-  <xacro:sonar_sim name="${namespace}/base_link/sonar_left" />
+  <xacro:sonar_sim name="${namespace}/base_link/sonar_front" topic="sensors/sonar_front" />
+  <xacro:sonar_sim name="${namespace}/base_link/sonar_back" topic="sensors/sonar_back" />
+  <xacro:sonar_sim name="${namespace}/base_link/sonar_right" topic="sensors/sonar_right" />
+  <xacro:sonar_sim name="${namespace}/base_link/sonar_left" topic="sensors/sonar_left" />
   <xacro:logitech_c920_camera_sim name="${namespace}/base_link/front_camera"
     topic_name="cameras/cam_front" />
