Commit message: add update rate across files

File: auv_sim/auv_sim_description/auv_common_sim_descriptions/urdf/sensors/bar30.urdf.xacro (robot description, xacro)
@@ -1,5 +1,5 @@
 <?xml version="1.0"?>
 <robot xmlns:xacro="http://www.ros.org/wiki/xacro" name="bar30">
-  <xacro:macro name="bar30_sim" params="name">
+  <xacro:macro name="bar30_sim" params="name update_rate">
     <link name="${name}_sim_link">
       <inertial>
@@ -27,5 +27,5 @@
         <link_name>${name}_sim_link</link_name>
         <sensor_topic>sim/pressure</sensor_topic>
-        <update_rate>50.0</update_rate>
+        <update_rate>${update_rate}</update_rate>
         <saturation>5000</saturation>
         <noise_sigma>0.4</noise_sigma>

File: auv_sim/auv_sim_description/auv_common_sim_descriptions/urdf/sensors/xsens_mti_g710.urdf.xacro (robot description, xacro)
@@ -1,5 +1,5 @@
 <?xml version="1.0"?>
 <robot xmlns:xacro="http://www.ros.org/wiki/xacro" name="xsens_mti_g710">
-  <xacro:macro name="xsens_mti_g710_sim" params="name namespace static_reference_frame">
+  <xacro:macro name="xsens_mti_g710_sim" params="name namespace static_reference_frame update_rate">
     <link name="${name}_sim_link">
       <inertial>
@@ -36,5 +36,5 @@
         <accelerometer_turn_on_bias_sigma>0.1960</accelerometer_turn_on_bias_sigma>
         <orientation_noise>0.05</orientation_noise>
-        <update_rate>80</update_rate>
+        <update_rate>${update_rate}</update_rate>
         <enable_gazebo_messages>false</enable_gazebo_messages>
         <enable_local_ned_frame>false</enable_local_ned_frame>

File: auv_sim/auv_sim_description/taluy_sim_description/urdf/sensors.urdf.xacro (robot description, xacro)
@@ -1,6 +1,8 @@
 <?xml version="1.0"?>
 <robot xmlns:xacro="http://www.ros.org/wiki/xacro">
+  <xacro:arg name="imu_update_rate" default="20"/>
+  <xacro:arg name="dvl_update_rate" default="20"/>
+  <xacro:arg name="pressure_update_rate" default="20"/>
   <xacro:include filename="$(find auv_common_sim_descriptions)/urdf/sensors.urdf.xacro"/>
-  <xacro:bar30_sim name="${namespace}/base_link/external_pressure_sensor"/>
   <xacro:sonar_sim name="${namespace}/base_link/sonar_front" topic="sensors/sonar_front"/>
   <xacro:sonar_sim name="${namespace}/base_link/sonar_back" topic="sensors/sonar_back"/>
@@ -9,5 +11,6 @@
   <xacro:logitech_c920_camera_sim name="${namespace}/base_link/front_camera" topic_name="cameras/cam_front"/>
   <xacro:logitech_c920_camera_sim name="${namespace}/base_link/bottom_camera" topic_name="cameras/cam_bottom"/>
-  <xacro:xsens_mti_g710_sim name="${namespace}/base_link/imu" namespace="${namespace}" static_reference_frame="${inertial_reference_frame}"/>
-  <xacro:wayfinder_dvl_sim name="${namespace}/base_link/dvl" namespace="${namespace}" static_reference_frame="${inertial_reference_frame}" update_rate="10"/>
+  <xacro:bar30_sim name="${namespace}/base_link/external_pressure_sensor" update_rate="$(arg pressure_update_rate)"/>
+  <xacro:xsens_mti_g710_sim name="${namespace}/base_link/imu" namespace="${namespace}" static_reference_frame="${inertial_reference_frame}" update_rate="$(arg imu_update_rate)"/>
+  <xacro:wayfinder_dvl_sim name="${namespace}/base_link/dvl" namespace="${namespace}" static_reference_frame="${inertial_reference_frame}" update_rate="$(arg dvl_update_rate)"/>
 </robot>
