Commit message: changed the simulation bottom camera to use real values, removed a trajectory frame, removed unused state, fixes

File: auv_sim/auv_sim_description/auv_common_sim_descriptions/urdf/sensors/logitech_c920_camera.urdf.xacro (robot description, xacro)
@@ -1,13 +1,16 @@
 <?xml version="1.0"?>
 <robot xmlns:xacro="http://ros.org/wiki/xacro" name="logitech_c920_camera">
-  <xacro:macro name="logitech_c920_camera_sim" params="name topic_name">
+  <xacro:macro name="logitech_c920_camera_sim" params="name topic_name
+    image_width:=640 image_height:=480 hfov:=1.229
+    distortion_k1:=0.0 distortion_k2:=0.0 distortion_k3:=0.0
+    distortion_t1:=0.0 distortion_t2:=0.0">
     <gazebo reference="${name}_link">
       <sensor type="camera" name="${name}_sensor">
         <update_rate>30.0</update_rate>
         <camera name="head">
-          <horizontal_fov>1.229</horizontal_fov>
+          <horizontal_fov>${hfov}</horizontal_fov>
           <image>
-            <width>640</width>
-            <height>480</height>
+            <width>${image_width}</width>
+            <height>${image_height}</height>
             <format>B8G8R8</format>
           </image>
@@ -24,4 +27,12 @@
             <stddev>0.007</stddev>
           </noise>
+          <distortion>
+            <k1>${distortion_k1}</k1>
+            <k2>${distortion_k2}</k2>
+            <k3>${distortion_k3}</k3>
+            <p1>${distortion_t1}</p1>
+            <p2>${distortion_t2}</p2>
+            <center>0.5 0.5</center>
+          </distortion>
         </camera>
         <plugin name="camera_controller" filename="libgazebo_ros_camera.so">
@@ -32,9 +43,9 @@
           <frameName>${name}_link</frameName>
           <hackBaseline>0.07</hackBaseline>
-          <distortionK1>0.0</distortionK1>
-          <distortionK2>0.0</distortionK2>
-          <distortionK3>0.0</distortionK3>
-          <distortionT1>0.0</distortionT1>
-          <distortionT2>0.0</distortionT2>
+          <distortionK1>${distortion_k1}</distortionK1>
+          <distortionK2>${distortion_k2}</distortionK2>
+          <distortionK3>${distortion_k3}</distortionK3>
+          <distortionT1>${distortion_t1}</distortionT1>
+          <distortionT2>${distortion_t2}</distortionT2>
         </plugin>
       </sensor>

File: auv_sim/auv_sim_description/taluy_sim_description/urdf/sensors.urdf.xacro (robot description, xacro)
@@ -10,5 +10,8 @@
   <xacro:sonar_sim name="${namespace}/base_link/sonar_left" topic="sensors/sonar_left"/>
   <xacro:logitech_c920_camera_sim name="${namespace}/base_link/front_camera" topic_name="cameras/cam_front"/>
-  <xacro:logitech_c920_camera_sim name="${namespace}/base_link/bottom_camera" topic_name="cameras/cam_bottom"/>
+  <xacro:logitech_c920_camera_sim name="${namespace}/base_link/bottom_camera" topic_name="cameras/cam_bottom"
+    image_width="1920" image_height="1080" hfov="1.2724"
+    distortion_k1="-0.330122" distortion_k2="0.135823" distortion_k3="0.0"
+    distortion_t1="0.001839" distortion_t2="0.000819"/>
   <xacro:logitech_c920_camera_sim name="${namespace}/base_link/torpedo_camera" topic_name="cameras/cam_torpedo"/>
   <xacro:bar30_sim name="${namespace}/base_link/external_pressure_sensor" update_rate="$(arg pressure_update_rate)"/>

Commit message: changed the simulation bottom camera to use real values, removed a trajectory frame, removed unused state, fixes

File: auv_sim/auv_sim_description/auv_common_sim_descriptions/urdf/sensors/logitech_c920_camera.urdf.xacro (robot description, xacro)
@@ -1,13 +1,16 @@
 <?xml version="1.0"?>
 <robot xmlns:xacro="http://ros.org/wiki/xacro" name="logitech_c920_camera">
-  <xacro:macro name="logitech_c920_camera_sim" params="name topic_name">
+  <xacro:macro name="logitech_c920_camera_sim" params="name topic_name
+    image_width:=640 image_height:=480 hfov:=1.229
+    distortion_k1:=0.0 distortion_k2:=0.0 distortion_k3:=0.0
+    distortion_t1:=0.0 distortion_t2:=0.0">
     <gazebo reference="${name}_link">
       <sensor type="camera" name="${name}_sensor">
         <update_rate>30.0</update_rate>
         <camera name="head">
-          <horizontal_fov>1.229</horizontal_fov>
+          <horizontal_fov>${hfov}</horizontal_fov>
           <image>
-            <width>640</width>
-            <height>480</height>
+            <width>${image_width}</width>
+            <height>${image_height}</height>
             <format>B8G8R8</format>
           </image>
@@ -24,4 +27,12 @@
             <stddev>0.007</stddev>
           </noise>
+          <distortion>
+            <k1>${distortion_k1}</k1>
+            <k2>${distortion_k2}</k2>
+            <k3>${distortion_k3}</k3>
+            <p1>${distortion_t1}</p1>
+            <p2>${distortion_t2}</p2>
+            <center>0.5 0.5</center>
+          </distortion>
         </camera>
         <plugin name="camera_controller" filename="libgazebo_ros_camera.so">
@@ -32,9 +43,9 @@
           <frameName>${name}_optical_link</frameName>
           <hackBaseline>0.07</hackBaseline>
-          <distortionK1>0.0</distortionK1>
-          <distortionK2>0.0</distortionK2>
-          <distortionK3>0.0</distortionK3>
-          <distortionT1>0.0</distortionT1>
-          <distortionT2>0.0</distortionT2>
+          <distortionK1>${distortion_k1}</distortionK1>
+          <distortionK2>${distortion_k2}</distortionK2>
+          <distortionK3>${distortion_k3}</distortionK3>
+          <distortionT1>${distortion_t1}</distortionT1>
+          <distortionT2>${distortion_t2}</distortionT2>
         </plugin>
       </sensor>

File: auv_sim/auv_sim_description/taluy_sim_description/urdf/sensors.urdf.xacro (robot description, xacro)
@@ -10,5 +10,8 @@
   <xacro:sonar_sim name="${namespace}/base_link/sonar_left" topic="sensors/sonar_left"/>
   <xacro:logitech_c920_camera_sim name="${namespace}/base_link/front_camera" topic_name="cameras/cam_front"/>
-  <xacro:logitech_c920_camera_sim name="${namespace}/base_link/bottom_camera" topic_name="cameras/cam_bottom"/>
+  <xacro:logitech_c920_camera_sim name="${namespace}/base_link/bottom_camera" topic_name="cameras/cam_bottom"
+    image_width="1920" image_height="1080" hfov="1.2724"
+    distortion_k1="-0.330122" distortion_k2="0.135823" distortion_k3="0.0"
+    distortion_t1="0.001839" distortion_t2="0.000819"/>
   <xacro:logitech_c920_camera_sim name="${namespace}/base_link/torpedo_camera" topic_name="cameras/cam_torpedo"/>
   <xacro:bar30_sim name="${namespace}/base_link/external_pressure_sensor" update_rate="$(arg pressure_update_rate)" namespace="${namespace}"/>

Commit message: changes sim cameras to follow the parameters of the real ones

File: auv_sim/auv_sim_description/auv_common_sim_descriptions/urdf/sensors/logitech_c920_camera.urdf.xacro (robot description, xacro)
@@ -1,13 +1,15 @@
 <?xml version="1.0"?>
 <robot xmlns:xacro="http://ros.org/wiki/xacro" name="logitech_c920_camera">
-  <xacro:macro name="logitech_c920_camera_sim" params="name topic_name">
+  <xacro:macro name="logitech_c920_camera_sim" params="name topic_name
+    image_width image_height hfov
+    distortion_k1 distortion_k2 distortion_k3 distortion_t1 distortion_t2">
     <gazebo reference="${name}_link">
       <sensor type="camera" name="${name}_sensor">
         <update_rate>30.0</update_rate>
         <camera name="head">
-          <horizontal_fov>1.229</horizontal_fov>
+          <horizontal_fov>${hfov}</horizontal_fov>
           <image>
-            <width>640</width>
-            <height>480</height>
+            <width>${image_width}</width>
+            <height>${image_height}</height>
             <format>B8G8R8</format>
           </image>
@@ -16,4 +18,12 @@
             <far>300</far>
           </clip>
+          <distortion>
+            <k1>${distortion_k1}</k1>
+            <k2>${distortion_k2}</k2>
+            <k3>${distortion_k3}</k3>
+            <p1>${distortion_t1}</p1>
+            <p2>${distortion_t2}</p2>
+            <center>0.5 0.5</center>
+          </distortion>
           <noise>
             <type>gaussian</type>
@@ -32,9 +42,9 @@
           <frameName>${name}_optical_link</frameName>
           <hackBaseline>0.07</hackBaseline>
-          <distortionK1>0.0</distortionK1>
-          <distortionK2>0.0</distortionK2>
-          <distortionK3>0.0</distortionK3>
-          <distortionT1>0.0</distortionT1>
-          <distortionT2>0.0</distortionT2>
+          <distortionK1>${distortion_k1}</distortionK1>
+          <distortionK2>${distortion_k2}</distortionK2>
+          <distortionK3>${distortion_k3}</distortionK3>
+          <distortionT1>${distortion_t1}</distortionT1>
+          <distortionT2>${distortion_t2}</distortionT2>
         </plugin>
       </sensor>

File: auv_sim/auv_sim_description/taluy_mini_sim_description/urdf/sensors.urdf.xacro (robot description, xacro)
@@ -5,5 +5,23 @@
   <xacro:arg name="pressure_update_rate" default="20"/>
   <xacro:include filename="$(find auv_common_sim_descriptions)/urdf/sensors.urdf.xacro"/>
-  <xacro:logitech_c920_camera_sim name="${namespace}/base_link/front_camera" topic_name="cameras/cam_front"/>
+  <!-- Share camera calibration with hardware. Plumb-bob order: [k1, k2, p1, p2, k3]. -->
+  <xacro:property name="cam_cfg" value="${xacro.load_yaml('$(find auv_bringup)/config/cameras_taluy_mini.yaml')}"/>
+  <xacro:property name="front_cfg" value="${cam_cfg['cam_front']}"/>
+  <xacro:property name="front_w" value="${front_cfg['image_width']}"/>
+  <xacro:property name="front_h" value="${front_cfg['image_height']}"/>
+  <xacro:property name="front_fx" value="${front_cfg['camera_matrix']['data'][0]}"/>
+  <xacro:property name="front_d" value="${front_cfg['distortion_coefficients']['data']}"/>
+  <xacro:logitech_c920_camera_sim
+    name="${namespace}/base_link/front_camera"
+    topic_name="cameras/cam_front"
+    image_width="${front_w}"
+    image_height="${front_h}"
+    hfov="${2 * atan2(front_w, 2 * front_fx)}"
+    distortion_k1="${front_d[0]}"
+    distortion_k2="${front_d[1]}"
+    distortion_k3="${front_d[4]}"
+    distortion_t1="${front_d[2]}"
+    distortion_t2="${front_d[3]}"
+  />
   <xacro:bar30_sim name="${namespace}/base_link/external_pressure_sensor" update_rate="$(arg pressure_update_rate)" namespace="${namespace}"/>
   <xacro:xsens_mti_g710_sim name="${namespace}/base_link/imu" namespace="${namespace}" static_reference_frame="${inertial_reference_frame}" update_rate="$(arg imu_update_rate)"/>

File: auv_sim/auv_sim_description/taluy_sim_description/urdf/sensors.urdf.xacro (robot description, xacro)
@@ -9,7 +9,57 @@
   <xacro:sonar_sim name="${namespace}/base_link/sonar_right" topic="sensors/sonar_right"/>
   <xacro:sonar_sim name="${namespace}/base_link/sonar_left" topic="sensors/sonar_left"/>
-  <xacro:logitech_c920_camera_sim name="${namespace}/base_link/front_camera" topic_name="cameras/cam_front"/>
-  <xacro:logitech_c920_camera_sim name="${namespace}/base_link/bottom_camera" topic_name="cameras/cam_bottom"/>
-  <xacro:logitech_c920_camera_sim name="${namespace}/base_link/torpedo_camera" topic_name="cameras/cam_torpedo"/>
+  <!-- Share camera calibration with hardware. Plumb-bob order: [k1, k2, p1, p2, k3]. -->
+  <xacro:property name="cam_cfg" value="${xacro.load_yaml('$(find auv_bringup)/config/cameras_taluy.yaml')}"/>
+  <xacro:property name="front_cfg" value="${cam_cfg['cam_front']}"/>
+  <xacro:property name="front_w" value="${front_cfg['image_width']}"/>
+  <xacro:property name="front_h" value="${front_cfg['image_height']}"/>
+  <xacro:property name="front_fx" value="${front_cfg['camera_matrix']['data'][0]}"/>
+  <xacro:property name="front_d" value="${front_cfg['distortion_coefficients']['data']}"/>
+  <xacro:property name="bottom_cfg" value="${cam_cfg['cam_bottom']}"/>
+  <xacro:property name="bottom_w" value="${bottom_cfg['image_width']}"/>
+  <xacro:property name="bottom_h" value="${bottom_cfg['image_height']}"/>
+  <xacro:property name="bottom_fx" value="${bottom_cfg['camera_matrix']['data'][0]}"/>
+  <xacro:property name="bottom_d" value="${bottom_cfg['distortion_coefficients']['data']}"/>
+  <xacro:property name="torpedo_cfg" value="${cam_cfg['cam_torpedo']}"/>
+  <xacro:property name="torpedo_w" value="${torpedo_cfg['image_width']}"/>
+  <xacro:property name="torpedo_h" value="${torpedo_cfg['image_height']}"/>
+  <xacro:property name="torpedo_fx" value="${torpedo_cfg['camera_matrix']['data'][0]}"/>
+  <xacro:property name="torpedo_d" value="${torpedo_cfg['distortion_coefficients']['data']}"/>
+  <xacro:logitech_c920_camera_sim
+    name="${namespace}/base_link/front_camera"
+    topic_name="cameras/cam_front"
+    image_width="${front_w}"
+    image_height="${front_h}"
+    hfov="${2 * atan2(front_w, 2 * front_fx)}"
+    distortion_k1="${front_d[0]}"
+    distortion_k2="${front_d[1]}"
+    distortion_k3="${front_d[4]}"
+    distortion_t1="${front_d[2]}"
+    distortion_t2="${front_d[3]}"
+  />
+  <xacro:logitech_c920_camera_sim
+    name="${namespace}/base_link/bottom_camera"
+    topic_name="cameras/cam_bottom"
+    image_width="${bottom_w}"
+    image_height="${bottom_h}"
+    hfov="${2 * atan2(bottom_w, 2 * bottom_fx)}"
+    distortion_k1="${bottom_d[0]}"
+    distortion_k2="${bottom_d[1]}"
+    distortion_k3="${bottom_d[4]}"
+    distortion_t1="${bottom_d[2]}"
+    distortion_t2="${bottom_d[3]}"
+  />
+  <xacro:logitech_c920_camera_sim
+    name="${namespace}/base_link/torpedo_camera"
+    topic_name="cameras/cam_torpedo"
+    image_width="${torpedo_w}"
+    image_height="${torpedo_h}"
+    hfov="${2 * atan2(torpedo_w, 2 * torpedo_fx)}"
+    distortion_k1="${torpedo_d[0]}"
+    distortion_k2="${torpedo_d[1]}"
+    distortion_k3="${torpedo_d[4]}"
+    distortion_t1="${torpedo_d[2]}"
+    distortion_t2="${torpedo_d[3]}"
+  />
   <xacro:bar30_sim name="${namespace}/base_link/external_pressure_sensor" update_rate="$(arg pressure_update_rate)" namespace="${namespace}"/>
   <xacro:xsens_mti_g710_sim name="${namespace}/base_link/imu" namespace="${namespace}" static_reference_frame="${inertial_reference_frame}" update_rate="$(arg imu_update_rate)"/>

Commit message: cleanup xacro files

File: auv_sim/auv_sim_description/auv_common_sim_descriptions/urdf/sensors/logitech_c920_camera.urdf.xacro (robot description, xacro)
@@ -1,15 +1,14 @@
 <?xml version="1.0"?>
 <robot xmlns:xacro="http://ros.org/wiki/xacro" name="logitech_c920_camera">
-  <xacro:macro name="logitech_c920_camera_sim" params="name topic_name
-    image_width image_height hfov
-    distortion_k1 distortion_k2 distortion_k3 distortion_t1 distortion_t2">
+  <xacro:macro name="logitech_c920_camera_sim" params="name topic_name calibration_params">
+    <xacro:property name="distortion" value="${calibration_params['distortion_coefficients']['data']}"/>
     <gazebo reference="${name}_link">
       <sensor type="camera" name="${name}_sensor">
         <update_rate>30.0</update_rate>
         <camera name="head">
-          <horizontal_fov>${hfov}</horizontal_fov>
+          <horizontal_fov>${2 * atan2(calibration_params['image_width'], 2 * calibration_params['camera_matrix']['data'][0])}</horizontal_fov>
           <image>
-            <width>${image_width}</width>
-            <height>${image_height}</height>
+            <width>${calibration_params['image_width']}</width>
+            <height>${calibration_params['image_height']}</height>
             <format>B8G8R8</format>
           </image>
@@ -19,9 +18,9 @@
           </clip>
           <distortion>
-            <k1>${distortion_k1}</k1>
-            <k2>${distortion_k2}</k2>
-            <k3>${distortion_k3}</k3>
-            <p1>${distortion_t1}</p1>
-            <p2>${distortion_t2}</p2>
+            <k1>${distortion[0]}</k1>
+            <k2>${distortion[1]}</k2>
+            <k3>${distortion[4]}</k3>
+            <p1>${distortion[2]}</p1>
+            <p2>${distortion[3]}</p2>
             <center>0.5 0.5</center>
           </distortion>
@@ -42,9 +41,9 @@
           <frameName>${name}_optical_link</frameName>
           <hackBaseline>0.07</hackBaseline>
-          <distortionK1>${distortion_k1}</distortionK1>
-          <distortionK2>${distortion_k2}</distortionK2>
-          <distortionK3>${distortion_k3}</distortionK3>
-          <distortionT1>${distortion_t1}</distortionT1>
-          <distortionT2>${distortion_t2}</distortionT2>
+          <distortionK1>${distortion[0]}</distortionK1>
+          <distortionK2>${distortion[1]}</distortionK2>
+          <distortionK3>${distortion[4]}</distortionK3>
+          <distortionT1>${distortion[2]}</distortionT1>
+          <distortionT2>${distortion[3]}</distortionT2>
         </plugin>
       </sensor>

File: auv_sim/auv_sim_description/taluy_mini_sim_description/urdf/sensors.urdf.xacro (robot description, xacro)
@@ -5,23 +5,6 @@
   <xacro:arg name="pressure_update_rate" default="20"/>
   <xacro:include filename="$(find auv_common_sim_descriptions)/urdf/sensors.urdf.xacro"/>
-  <!-- Share camera calibration with hardware. Plumb-bob order: [k1, k2, p1, p2, k3]. -->
-  <xacro:property name="cam_cfg" value="${xacro.load_yaml('$(find auv_bringup)/config/cameras_taluy_mini.yaml')}"/>
-  <xacro:property name="front_cfg" value="${cam_cfg['cam_front']}"/>
-  <xacro:property name="front_w" value="${front_cfg['image_width']}"/>
-  <xacro:property name="front_h" value="${front_cfg['image_height']}"/>
-  <xacro:property name="front_fx" value="${front_cfg['camera_matrix']['data'][0]}"/>
-  <xacro:property name="front_d" value="${front_cfg['distortion_coefficients']['data']}"/>
-  <xacro:logitech_c920_camera_sim
-    name="${namespace}/base_link/front_camera"
-    topic_name="cameras/cam_front"
-    image_width="${front_w}"
-    image_height="${front_h}"
-    hfov="${2 * atan2(front_w, 2 * front_fx)}"
-    distortion_k1="${front_d[0]}"
-    distortion_k2="${front_d[1]}"
-    distortion_k3="${front_d[4]}"
-    distortion_t1="${front_d[2]}"
-    distortion_t2="${front_d[3]}"
-  />
+  <xacro:property name="camera_calibrations" value="${xacro.load_yaml('$(find auv_bringup)/config/cameras_taluy_mini.yaml')}"/>
+  <xacro:logitech_c920_camera_sim name="${namespace}/base_link/front_camera" topic_name="cameras/cam_front" calibration_params="${camera_calibrations['cam_front']}"/>
   <xacro:bar30_sim name="${namespace}/base_link/external_pressure_sensor" update_rate="$(arg pressure_update_rate)" namespace="${namespace}"/>
   <xacro:xsens_mti_g710_sim name="${namespace}/base_link/imu" namespace="${namespace}" static_reference_frame="${inertial_reference_frame}" update_rate="$(arg imu_update_rate)"/>

File: auv_sim/auv_sim_description/taluy_sim_description/urdf/sensors.urdf.xacro (robot description, xacro)
@@ -9,57 +9,8 @@
   <xacro:sonar_sim name="${namespace}/base_link/sonar_right" topic="sensors/sonar_right"/>
   <xacro:sonar_sim name="${namespace}/base_link/sonar_left" topic="sensors/sonar_left"/>
-  <!-- Share camera calibration with hardware. Plumb-bob order: [k1, k2, p1, p2, k3]. -->
-  <xacro:property name="cam_cfg" value="${xacro.load_yaml('$(find auv_bringup)/config/cameras_taluy.yaml')}"/>
-  <xacro:property name="front_cfg" value="${cam_cfg['cam_front']}"/>
-  <xacro:property name="front_w" value="${front_cfg['image_width']}"/>
-  <xacro:property name="front_h" value="${front_cfg['image_height']}"/>
-  <xacro:property name="front_fx" value="${front_cfg['camera_matrix']['data'][0]}"/>
-  <xacro:property name="front_d" value="${front_cfg['distortion_coefficients']['data']}"/>
-  <xacro:property name="bottom_cfg" value="${cam_cfg['cam_bottom']}"/>
-  <xacro:property name="bottom_w" value="${bottom_cfg['image_width']}"/>
-  <xacro:property name="bottom_h" value="${bottom_cfg['image_height']}"/>
-  <xacro:property name="bottom_fx" value="${bottom_cfg['camera_matrix']['data'][0]}"/>
-  <xacro:property name="bottom_d" value="${bottom_cfg['distortion_coefficients']['data']}"/>
-  <xacro:property name="torpedo_cfg" value="${cam_cfg['cam_torpedo']}"/>
-  <xacro:property name="torpedo_w" value="${torpedo_cfg['image_width']}"/>
-  <xacro:property name="torpedo_h" value="${torpedo_cfg['image_height']}"/>
-  <xacro:property name="torpedo_fx" value="${torpedo_cfg['camera_matrix']['data'][0]}"/>
-  <xacro:property name="torpedo_d" value="${torpedo_cfg['distortion_coefficients']['data']}"/>
-  <xacro:logitech_c920_camera_sim
-    name="${namespace}/base_link/front_camera"
-    topic_name="cameras/cam_front"
-    image_width="${front_w}"
-    image_height="${front_h}"
-    hfov="${2 * atan2(front_w, 2 * front_fx)}"
-    distortion_k1="${front_d[0]}"
-    distortion_k2="${front_d[1]}"
-    distortion_k3="${front_d[4]}"
-    distortion_t1="${front_d[2]}"
-    distortion_t2="${front_d[3]}"
-  />
-  <xacro:logitech_c920_camera_sim
-    name="${namespace}/base_link/bottom_camera"
-    topic_name="cameras/cam_bottom"
-    image_width="${bottom_w}"
-    image_height="${bottom_h}"
-    hfov="${2 * atan2(bottom_w, 2 * bottom_fx)}"
-    distortion_k1="${bottom_d[0]}"
-    distortion_k2="${bottom_d[1]}"
-    distortion_k3="${bottom_d[4]}"
-    distortion_t1="${bottom_d[2]}"
-    distortion_t2="${bottom_d[3]}"
-  />
-  <xacro:logitech_c920_camera_sim
-    name="${namespace}/base_link/torpedo_camera"
-    topic_name="cameras/cam_torpedo"
-    image_width="${torpedo_w}"
-    image_height="${torpedo_h}"
-    hfov="${2 * atan2(torpedo_w, 2 * torpedo_fx)}"
-    distortion_k1="${torpedo_d[0]}"
-    distortion_k2="${torpedo_d[1]}"
-    distortion_k3="${torpedo_d[4]}"
-    distortion_t1="${torpedo_d[2]}"
-    distortion_t2="${torpedo_d[3]}"
-  />
+  <xacro:property name="camera_calibrations" value="${xacro.load_yaml('$(find auv_bringup)/config/cameras_taluy.yaml')}"/>
+  <xacro:logitech_c920_camera_sim name="${namespace}/base_link/front_camera" topic_name="cameras/cam_front" calibration_params="${camera_calibrations['cam_front']}"/>
+  <xacro:logitech_c920_camera_sim name="${namespace}/base_link/bottom_camera" topic_name="cameras/cam_bottom" calibration_params="${camera_calibrations['cam_bottom']}"/>
+  <xacro:logitech_c920_camera_sim name="${namespace}/base_link/torpedo_camera" topic_name="cameras/cam_torpedo" calibration_params="${camera_calibrations['cam_torpedo']}"/>
   <xacro:bar30_sim name="${namespace}/base_link/external_pressure_sensor" update_rate="$(arg pressure_update_rate)" namespace="${namespace}"/>
   <xacro:xsens_mti_g710_sim name="${namespace}/base_link/imu" namespace="${namespace}" static_reference_frame="${inertial_reference_frame}" update_rate="$(arg imu_update_rate)"/>
