Commit message: init

File: auv_sim/auv_sim_description/auv_common_sim_descriptions/urdf/sensors/logitech_c920_camera.urdf.xacro (robot description, xacro)
@@ -1,8 +1,8 @@
 <?xml version="1.0"?>
 <robot xmlns:xacro="http://ros.org/wiki/xacro" name="logitech_c920_camera">
-  <xacro:macro name="logitech_c920_camera_sim" params="name topic_name">
+  <xacro:macro name="logitech_c920_camera_sim" params="name topic_name update_rate:=10.0">
     <gazebo reference="${name}_link">
       <sensor type="camera" name="${name}_sensor">
-        <update_rate>30.0</update_rate>
+        <update_rate>${update_rate}</update_rate>
         <camera name="head">
           <horizontal_fov>1.229</horizontal_fov>
@@ -27,5 +27,5 @@
         <plugin name="camera_controller" filename="libgazebo_ros_camera.so">
           <alwaysOn>true</alwaysOn>
-          <updateRate>0.0</updateRate>
+          <updateRate>${update_rate}</updateRate>
           <cameraName>${topic_name}</cameraName>
           <imageTopicName>image_raw</imageTopicName>

File: auv_sim/auv_sim_description/taluy_sim_description/urdf/sensors.urdf.xacro (robot description, xacro)
@@ -4,4 +4,6 @@
   <xacro:arg name="dvl_update_rate" default="20"/>
   <xacro:arg name="pressure_update_rate" default="20"/>
+  <xacro:arg name="camera_update_rate" default="10.0"/>
+  <xacro:arg name="pointcloud_filter" default="true"/>
   <xacro:include filename="$(find auv_common_sim_descriptions)/urdf/sensors.urdf.xacro"/>
   <xacro:sonar_sim name="${namespace}/base_link/sonar_front" topic="sensors/sonar_front"/>
@@ -9,10 +11,12 @@
   <xacro:sonar_sim name="${namespace}/base_link/sonar_right" topic="sensors/sonar_right"/>
   <xacro:sonar_sim name="${namespace}/base_link/sonar_left" topic="sensors/sonar_left"/>
-  <xacro:logitech_c920_camera_sim name="${namespace}/base_link/front_camera" topic_name="cameras/cam_front"/>
-  <xacro:logitech_c920_camera_sim name="${namespace}/base_link/bottom_camera" topic_name="cameras/cam_bottom"/>
-  <xacro:logitech_c920_camera_sim name="${namespace}/base_link/torpedo_camera" topic_name="cameras/cam_torpedo"/>
+  <xacro:logitech_c920_camera_sim name="${namespace}/base_link/front_camera" topic_name="cameras/cam_front" update_rate="$(arg camera_update_rate)"/>
+  <xacro:logitech_c920_camera_sim name="${namespace}/base_link/bottom_camera" topic_name="cameras/cam_bottom" update_rate="$(arg camera_update_rate)"/>
+  <xacro:logitech_c920_camera_sim name="${namespace}/base_link/torpedo_camera" topic_name="cameras/cam_torpedo" update_rate="$(arg camera_update_rate)"/>
   <xacro:bar30_sim name="${namespace}/base_link/external_pressure_sensor" update_rate="$(arg pressure_update_rate)" namespace="${namespace}"/>
   <xacro:xsens_mti_g710_sim name="${namespace}/base_link/imu" namespace="${namespace}" static_reference_frame="${inertial_reference_frame}" update_rate="$(arg imu_update_rate)"/>
   <xacro:wayfinder_dvl_sim name="${namespace}/base_link/dvl" namespace="${namespace}" static_reference_frame="${inertial_reference_frame}" update_rate="$(arg dvl_update_rate)"/>
-  <xacro:realsense_d435_sim name="${namespace}/camera"/>
+  <xacro:if value="$(arg pointcloud_filter)">
+    <xacro:realsense_d435_sim name="${namespace}/camera"/>
+  </xacro:if>
 </robot>
