Commit message: depth anything correction sim brigde logic okkey

File: auv_sim/auv_sim_description/auv_common_sim_descriptions/urdf/sensors/realsense_d435.urdf.xacro (robot description, xacro)
@@ -1,6 +1,7 @@
 <?xml version="1.0"?>
 <robot xmlns:xacro="http://www.ros.org/wiki/xacro">
-  <xacro:macro name="realsense_d435_sim" params="name">
-    <gazebo reference="${name}">
+  <xacro:macro name="realsense_d435_sim"
+               params="name reference_name:='${name}' frame_name:='${name}_depth_optical_frame' depth_image_topic:='depth/image_raw' depth_camera_info_topic:='depth/camera_info'">
+    <gazebo reference="${reference_name}">
       <sensor type="depth" name="${name}_depth_sensor">
         <update_rate>30.0</update_rate>
@@ -23,8 +24,8 @@
           <imageTopicName>color/image_raw</imageTopicName>
           <cameraInfoTopicName>color/camera_info</cameraInfoTopicName>
-          <depthImageTopicName>depth/image_raw</depthImageTopicName>
-          <depthImageCameraInfoTopicName>depth/camera_info</depthImageCameraInfoTopicName>
+          <depthImageTopicName>${depth_image_topic}</depthImageTopicName>
+          <depthImageCameraInfoTopicName>${depth_camera_info_topic}</depthImageCameraInfoTopicName>
           <pointCloudTopicName>/points_filtered</pointCloudTopicName>
-          <frameName>${name}_depth_optical_frame</frameName>
+          <frameName>${frame_name}</frameName>
           <pointCloudCutoff>0.1</pointCloudCutoff>
           <pointCloudCutoffMax>10.0</pointCloudCutoffMax>

File: auv_sim/auv_sim_description/taluy_sim_description/urdf/sensors.urdf.xacro (robot description, xacro)
@@ -18,5 +18,8 @@
   <xacro:wayfinder_dvl_sim name="${namespace}/base_link/dvl" namespace="${namespace}" static_reference_frame="${inertial_reference_frame}" update_rate="$(arg dvl_update_rate)"/>
   <xacro:if value="$(arg pointcloud_filter)">
-    <xacro:realsense_d435_sim name="${namespace}/camera"/>
+    <xacro:realsense_d435_sim
+      name="${namespace}/camera"
+      reference_name="${namespace}/base_link/torpedo_camera_link"
+      frame_name="${namespace}/base_link/torpedo_camera_optical_link"/>
   </xacro:if>
 </robot>

Commit message: pre commit

File: auv_sim/auv_sim_description/auv_common_sim_descriptions/urdf/sensors/realsense_d435.urdf.xacro (robot description, xacro)
@@ -1,6 +1,8 @@
 <?xml version="1.0"?>
 <robot xmlns:xacro="http://www.ros.org/wiki/xacro">
-  <xacro:macro name="realsense_d435_sim"
-               params="name reference_name:='${name}' frame_name:='${name}_depth_optical_frame' depth_image_topic:='depth/image_raw' depth_camera_info_topic:='depth/camera_info'">
+  <xacro:macro
+    name="realsense_d435_sim"
+    params="name reference_name:='${name}' frame_name:='${name}_depth_optical_frame' depth_image_topic:='depth/image_raw' depth_camera_info_topic:='depth/camera_info'"
+  >
     <gazebo reference="${reference_name}">
       <sensor type="depth" name="${name}_depth_sensor">

File: auv_sim/auv_sim_description/taluy_sim_description/urdf/sensors.urdf.xacro (robot description, xacro)
@@ -18,8 +18,5 @@
   <xacro:wayfinder_dvl_sim name="${namespace}/base_link/dvl" namespace="${namespace}" static_reference_frame="${inertial_reference_frame}" update_rate="$(arg dvl_update_rate)"/>
   <xacro:if value="$(arg pointcloud_filter)">
-    <xacro:realsense_d435_sim
-      name="${namespace}/camera"
-      reference_name="${namespace}/base_link/torpedo_camera_link"
-      frame_name="${namespace}/base_link/torpedo_camera_optical_link"/>
+    <xacro:realsense_d435_sim name="${namespace}/camera" reference_name="${namespace}/base_link/torpedo_camera_link" frame_name="${namespace}/base_link/torpedo_camera_optical_link"/>
   </xacro:if>
 </robot>
