Commit message: update torpedos-to be continued

File: auv_description/auv_common_descriptions/urdf/actuators/torpedo.urdf.xacro (robot description, xacro)
@@ -7,16 +7,16 @@
         <origin xyz="0 0 0" rpy="0 0 0"/>
         <geometry>
-          <cylinder length="0.2" radius="0.0175"/>
+          <mesh filename="package://auv_common_descriptions/meshes/torpedo/torpedo.dae" scale="0.001 0.001 0.001"/>
         </geometry>
       </visual>
-      <collision name="${name}_collision">
+      <collision name="${name}_upper_collision">
         <origin xyz="0 0 0" rpy="0 0 0"/>
         <geometry>
-          <cylinder length="0.2" radius="0.0175"/>
+          <mesh filename="package://auv_common_descriptions/meshes/torpedo/torpedo.dae" scale="0.001 0.001 0.001"/>
         </geometry>
       </collision>
       <inertial>
-        <mass value="0.00001"/>
-        <inertia ixx="0.000001" ixy="0.0" ixz="0.0" iyy="0.000001" iyz="0.0" izz="0.000001"/>
+        <mass value="0.001"/> <!-- Adjusted mass for more realistic simulation -->
+        <inertia ixx="0.001" ixy="0.0" ixz="0.0" iyy="0.001" iyz="0.0" izz="0.001"/> <!-- Adjusted inertia -->
       </inertial>
     </link>
@@ -25,16 +25,16 @@
         <origin xyz="0 0 0" rpy="0 0 0"/>
         <geometry>
-          <cylinder length="0.2" radius="0.0175"/>
+          <mesh filename="package://auv_common_descriptions/meshes/torpedo/torpedo.dae" scale="0.001 0.001 0.001"/>
         </geometry>
       </visual>
-      <collision name="${name}_collision">
+      <collision name="${name}_lower_collision">
         <origin xyz="0 0 0" rpy="0 0 0"/>
         <geometry>
-          <cylinder length="0.2" radius="0.0175"/>
+          <mesh filename="package://auv_common_descriptions/meshes/torpedo/torpedo.dae" scale="0.001 0.001 0.001"/>
         </geometry>
       </collision>
       <inertial>
-        <mass value="0.000001"/>
-        <inertia ixx="0.000001" ixy="0.0" ixz="0.0" iyy="0.000001" iyz="0.0" izz="0.000001"/>
+        <mass value="0.001"/> <!-- Adjusted mass for more realistic simulation -->
+        <inertia ixx="0.001" ixy="0.0" ixz="0.0" iyy="0.001" iyz="0.0" izz="0.001"/> <!-- Adjusted inertia -->
       </inertial>
     </link>
@@ -43,17 +43,16 @@
       <child link="${name}_link"/>
       <origin xyz="${position}" rpy="${orientation}"/>
-      <axis rpy="0 0 0" xyz="0 0 1"/>
     </joint>
     <joint name="${name}_upper_joint" type="fixed">
-      <axis rpy="0 0 0" xyz="0 0 1"/>
+      <axis rpy="0 0 0" xyz="0 0 0"/>
       <parent link="${name}_link"/>
       <child link="${name}_upper_link"/>
-      <origin xyz="0.1 0 -0.0175" rpy="0 ${math.pi/2} 0"/>
+      <origin xyz="0 0 0" rpy="0 0 0"/>
     </joint>
     <joint name="${name}_lower_joint" type="fixed">
-      <axis rpy="0 0 0" xyz="0 0 1"/>
+      <axis rpy="0 0 0" xyz="0 0 0"/>
       <parent link="${name}_link"/>
       <child link="${name}_lower_link"/>
-      <origin xyz="0.1 0 -0.0525" rpy="0 ${math.pi/2} 0"/>
+      <origin xyz="0 0 0" rpy="0 0 0"/>
     </joint>
   </xacro:macro>

File: auv_description/taluy_description/urdf/auv_base.urdf.xacro (robot description, xacro)
@@ -52,6 +52,5 @@
     <xacro:logitech_c920_camera name="${namespace}/base_link/front_camera" parent="${namespace}/base_link" position="0.35 0 0" orientation="0 0 0"/>
     <xacro:logitech_c920_camera name="${namespace}/base_link/bottom_camera" parent="${namespace}/base_link" position="0 0 -0.07" orientation="0 ${math.pi/2} ${math.pi/2}"/>
-    <xacro:torpedo name="${namespace}/base_link/left_torpedo" parent="${namespace}/base_link" position="0.2 0.1 -0.11" orientation="0 0 0"/>
-    <xacro:torpedo name="${namespace}/base_link/right_torpedo" parent="${namespace}/base_link" position="0.2 -0.1 -0.11" orientation="0 0 0"/>
+    <xacro:torpedo name="${namespace}/base_link/torpedo" parent="${namespace}/base_link" position="0.27 -0.12 -0.07" orientation="0 0 0"/>
     <xacro:sonar name="${namespace}/base_link/sonar_front" parent="${namespace}/base_link" position="0.38 0.09 0.09" orientation="0 0 0"/>
     <xacro:sonar name="${namespace}/base_link/sonar_back" parent="${namespace}/base_link" position="-0.42 -0.09 0.09" orientation="0 0 ${math.pi}"/>

Commit message: pre_commit

File: auv_description/auv_common_descriptions/urdf/actuators/torpedo.urdf.xacro (robot description, xacro)
@@ -17,6 +17,8 @@
       </collision>
       <inertial>
-        <mass value="0.001"/> <!-- Adjusted mass for more realistic simulation -->
-        <inertia ixx="0.001" ixy="0.0" ixz="0.0" iyy="0.001" iyz="0.0" izz="0.001"/> <!-- Adjusted inertia -->
+        <mass value="0.001"/>
+        <!-- Adjusted mass for more realistic simulation -->
+        <inertia ixx="0.001" ixy="0.0" ixz="0.0" iyy="0.001" iyz="0.0" izz="0.001"/>
+        <!-- Adjusted inertia -->
       </inertial>
     </link>
@@ -35,6 +37,8 @@
       </collision>
       <inertial>
-        <mass value="0.001"/> <!-- Adjusted mass for more realistic simulation -->
-        <inertia ixx="0.001" ixy="0.0" ixz="0.0" iyy="0.001" iyz="0.0" izz="0.001"/> <!-- Adjusted inertia -->
+        <mass value="0.001"/>
+        <!-- Adjusted mass for more realistic simulation -->
+        <inertia ixx="0.001" ixy="0.0" ixz="0.0" iyy="0.001" iyz="0.0" izz="0.001"/>
+        <!-- Adjusted inertia -->
       </inertial>
     </link>
