Commit message: change t200 orientations

File: auv_description/auv_common_descriptions/urdf/actuators/t200.urdf.xacro (robot description, xacro)
@@ -4,5 +4,5 @@
     <link name="${name}_link">
       <visual>
-        <origin xyz="0 0 0" rpy="0 -${pi/2} ${-pi/2}" />
+        <origin xyz="0 0 0" rpy="0 ${pi/2} ${-pi/2}" />
         <geometry>
           <mesh filename="package://auv_common_descriptions/meshes/t200/shell.dae"
@@ -11,5 +11,5 @@
       </visual>
       <collision name="${name}_collision">
-        <origin xyz="0 0 0" rpy="0 -${pi/2} ${-pi/2}" />
+        <origin xyz="0 0 0" rpy="0 ${pi/2} ${-pi/2}" />
         <geometry>
           <mesh filename="package://auv_common_descriptions/meshes/t200/shell.dae"

File: auv_description/taluy_description/urdf/auv_base.urdf.xacro (robot description, xacro)
@@ -26,12 +26,12 @@
       </collision>
     </link>
-    <xacro:t200_thruster name="thruster_0" parent="base_link" position="0.14250 0.20070 -0.00525" orientation="0 0 ${-pi/2}"/>
-    <xacro:t200_thruster name="thruster_1" parent="base_link" position="0.14250 -0.20070 -0.00525" orientation="0 0 ${pi/2}"/>
-    <xacro:t200_thruster name="thruster_2" parent="base_link" position="-0.14250 0.20070 -0.00525" orientation="0 0 ${-pi/2}"/>
-    <xacro:t200_thruster name="thruster_3" parent="base_link" position="-0.14250 -0.20070 -0.00525" orientation="0 0 ${pi/2}"/>
-    <xacro:t200_thruster name="thruster_4" parent="base_link" position="0.352398 0.216638 -0.030881" orientation="${pi/2} 0 ${pi/4}"/>
-    <xacro:t200_thruster name="thruster_5" parent="base_link" position="0.352398 -0.216638 -0.030881" orientation="${-pi/2} 0 ${-pi/4}"/>
-    <xacro:t200_thruster name="thruster_6" parent="base_link" position="-0.352398 0.216638 -0.030881" orientation="${pi/2} 0 ${7*pi/4}"/>
-    <xacro:t200_thruster name="thruster_7" parent="base_link" position="-0.352398 -0.216638 -0.030881" orientation="${-pi/2} 0 ${-7*pi/4}"/>
+    <xacro:t200_thruster name="thruster_0" parent="base_link" position="0.14250 0.20070 -0.00525" orientation="${pi} 0 ${-pi/2}"/>
+    <xacro:t200_thruster name="thruster_1" parent="base_link" position="0.14250 -0.20070 -0.00525" orientation="${pi} 0 ${pi/2}"/>
+    <xacro:t200_thruster name="thruster_2" parent="base_link" position="-0.14250 0.20070 -0.00525" orientation="${pi} 0 ${-pi/2}"/>
+    <xacro:t200_thruster name="thruster_3" parent="base_link" position="-0.14250 -0.20070 -0.00525" orientation="${pi} 0 ${pi/2}"/>
+    <xacro:t200_thruster name="thruster_4" parent="base_link" position="0.352398 0.216638 -0.030881" orientation="${-pi/2} 0 ${-7*pi/4}"/>
+    <xacro:t200_thruster name="thruster_5" parent="base_link" position="0.352398 -0.216638 -0.030881" orientation="${pi/2} 0 ${7*pi/4}"/>
+    <xacro:t200_thruster name="thruster_6" parent="base_link" position="-0.352398 0.216638 -0.030881" orientation="${-pi/2} 0 ${-pi/4}"/>
+    <xacro:t200_thruster name="thruster_7" parent="base_link" position="-0.352398 -0.216638 -0.030881" orientation="${pi/2} 0 ${pi/4}"/>
   </xacro:macro>
 </robot>

Commit message: move gazebo tags in `t200.urdf.xacro` to it's auv_sim macro

File: auv_description/auv_common_descriptions/urdf/actuators/t200.urdf.xacro (robot description, xacro)
@@ -52,10 +52,4 @@
       <dynamics friction="0.05" damping="0.05"/>
     </joint>
-    <gazebo reference="${name}_propeller_link">
-      <material>Gazebo/Orange</material>
-    </gazebo>
-    <gazebo reference="${name}_link">
-      <material>Gazebo/Orange</material>
-    </gazebo>
   </xacro:macro>
 </robot>

Commit message: move gazebo tags in `t200.urdf.xacro` to it's auv_sim macro

File: auv_description/auv_common_descriptions/urdf/actuators/t200.urdf.xacro (robot description, xacro)
@@ -56,10 +56,4 @@
       <dynamics friction="0.05" damping="0.05" />
     </joint>
-    <gazebo reference="${name}_propeller_link">
-      <material>Gazebo/Orange</material>
-    </gazebo>
-    <gazebo reference="${name}_link">
-      <material>Gazebo/Orange</material>
-    </gazebo>
   </xacro:macro>
 </robot>

File: auv_sim/auv_sim_description/urdf/gazebo_plugins.urdf.xacro (robot description, xacro)
@@ -83,5 +83,9 @@
     </gazebo>
     <gazebo reference="${name}_propeller_link">
+      <material>Gazebo/Orange</material>
       <selfCollide>false</selfCollide>
+    </gazebo>
+    <gazebo reference="${name}_link">
+      <material>Gazebo/Orange</material>
     </gazebo>
   </xacro:macro>

Commit message: reduce dummy masses

File: auv_description/auv_common_descriptions/urdf/actuators/t200.urdf.xacro (robot description, xacro)
@@ -16,6 +16,6 @@
       </collision>
       <inertial>
-        <mass value="0.5"/>
-        <inertia ixx="0.008545" ixy="0.0" ixz="0.0" iyy="0.008545" iyz="0.0" izz="0.0144"/>
+        <mass value="0.001" />
+        <inertia ixx="0.0000001" ixy="0.0" ixz="0.0" iyy="0.0000001" iyz="0.0" izz="0.0000001" />
       </inertial>
     </link>
@@ -34,6 +34,6 @@
       </collision>
       <inertial>
-        <mass value="0.5"/>
-        <inertia ixx="0.008545" ixy="0.0" ixz="0.0" iyy="0.008545" iyz="0.0" izz="0.0144"/>
+        <mass value="0.001" />
+        <inertia ixx="0.0000001" ixy="0.0" ixz="0.0" iyy="0.0000001" iyz="0.0" izz="0.0000001" />
       </inertial>
     </link>
@@ -45,10 +45,13 @@
     </joint>
     <joint name="${name}_propeller_joint" type="continuous">
-      <axis rpy="0 0 0" xyz="0 0 1"/>
-      <parent link="${name}_link"/>
-      <child link="${name}_propeller_link"/>
-      <origin xyz="0 0 0" rpy="0 0 0"/>
-      <limit effort="100" velocity="100"/>
-      <dynamics friction="0.05" damping="0.05"/>
+      <axis rpy="0 0 0" xyz="0 0 1" />
+      <parent link="${name}_link" />
+      <child link="${name}_propeller_link" />
+      <origin xyz="0 0 0" rpy="0 0 0" />
+      <!-- TODO: This breaks the Gazebo Sim -->
+      <!-- <dynamics friction="0.05" damping="0.05" /> -->
+      <!-- TODO: This does not break, but the 100 velocity limit must be evaluated, why limit
+      anyway? -->
+      <!-- <limit effort="100" velocity="100" /> -->
     </joint>
   </xacro:macro>

File: auv_description/auv_common_descriptions/urdf/actuators/torpedo.urdf.xacro (robot description, xacro)
@@ -17,6 +17,6 @@
       </collision>
       <inertial>
-        <mass value="0.5"/>
-        <inertia ixx="0.008545" ixy="0.0" ixz="0.0" iyy="0.008545" iyz="0.0" izz="0.0144"/>
+        <mass value="0.00001" />
+        <inertia ixx="0.000001" ixy="0.0" ixz="0.0" iyy="0.000001" iyz="0.0" izz="0.000001" />
       </inertial>
     </link>
@@ -35,6 +35,6 @@
       </collision>
       <inertial>
-        <mass value="0.5"/>
-        <inertia ixx="0.008545" ixy="0.0" ixz="0.0" iyy="0.008545" iyz="0.0" izz="0.0144"/>
+        <mass value="0.000001" />
+        <inertia ixx="0.000001" ixy="0.0" ixz="0.0" iyy="0.000001" iyz="0.0" izz="0.000001" />
       </inertial>
     </link>

File: auv_description/auv_common_descriptions/urdf/sensors/bar30.urdf.xacro (robot description, xacro)
@@ -16,6 +16,6 @@
       </collision>
       <inertial>
-        <mass value="0.5"/>
-        <inertia ixx="0.008545" ixy="0.0" ixz="0.0" iyy="0.008545" iyz="0.0" izz="0.0144"/>
+        <mass value="0.00001" />
+        <inertia ixx="0.000001" ixy="0.0" ixz="0.0" iyy="0.000001" iyz="0.0" izz="0.000001" />
       </inertial>
     </link>

File: auv_description/auv_common_descriptions/urdf/sensors/h2c_hydrophone.urdf.xacro (robot description, xacro)
@@ -16,6 +16,6 @@
       </collision>
       <inertial>
-        <mass value="0.5"/>
-        <inertia ixx="0.008545" ixy="0.0" ixz="0.0" iyy="0.008545" iyz="0.0" izz="0.0144"/>
+        <mass value="0.0001" />
+        <inertia ixx="0.0000001" ixy="0.0" ixz="0.0" iyy="0.0000001" iyz="0.0" izz="0.0000001" />
       </inertial>
     </link>

File: auv_description/auv_common_descriptions/urdf/sensors/ping360.urdf.xacro (robot description, xacro)
@@ -16,6 +16,6 @@
       </collision>
       <inertial>
-        <mass value="0.5"/>
-        <inertia ixx="0.008545" ixy="0.0" ixz="0.0" iyy="0.008545" iyz="0.0" izz="0.0144"/>
+        <mass value="0.5" />
+        <inertia ixx="0.000001" ixy="0.0" ixz="0.0" iyy="0.000001" iyz="0.0" izz="0.000001" />
       </inertial>
     </link>

File: auv_description/auv_common_descriptions/urdf/sensors/xsens_mti_g710.urdf.xacro (robot description, xacro)
@@ -16,6 +16,6 @@
       </collision>
       <inertial>
-        <mass value="0.5"/>
-        <inertia ixx="0.008545" ixy="0.0" ixz="0.0" iyy="0.008545" iyz="0.0" izz="0.0144"/>
+        <mass value="0.0001" />
+        <inertia ixx="0.000001" ixy="0.0" ixz="0.0" iyy="0.000001" iyz="0.0" izz="0.000001" />
       </inertial>
     </link>

Commit message: reduce dummy masses

File: auv_description/auv_common_descriptions/urdf/actuators/t200.urdf.xacro (robot description, xacro)
@@ -18,6 +18,6 @@
       </collision>
       <inertial>
-        <mass value="0.5" />
-        <inertia ixx="0.008545" ixy="0.0" ixz="0.0" iyy="0.008545" iyz="0.0" izz="0.0144" />
+        <mass value="0.001" />
+        <inertia ixx="0.0000001" ixy="0.0" ixz="0.0" iyy="0.0000001" iyz="0.0" izz="0.0000001" />
       </inertial>
     </link>
@@ -38,6 +38,6 @@
       </collision>
       <inertial>
-        <mass value="0.5" />
-        <inertia ixx="0.008545" ixy="0.0" ixz="0.0" iyy="0.008545" iyz="0.0" izz="0.0144" />
+        <mass value="0.001" />
+        <inertia ixx="0.0000001" ixy="0.0" ixz="0.0" iyy="0.0000001" iyz="0.0" izz="0.0000001" />
       </inertial>
     </link>
@@ -53,6 +53,9 @@
       <child link="${name}_propeller_link" />
       <origin xyz="0 0 0" rpy="0 0 0" />
-      <limit effort="100" velocity="100" />
-      <dynamics friction="0.05" damping="0.05" />
+      <!-- TODO: This breaks the Gazebo Sim -->
+      <!-- <dynamics friction="0.05" damping="0.05" /> -->
+      <!-- TODO: This does not break, but the 100 velocity limit must be evaluated, why limit
+      anyway? -->
+      <!-- <limit effort="100" velocity="100" /> -->
     </joint>
   </xacro:macro>

File: auv_description/auv_common_descriptions/urdf/actuators/torpedo.urdf.xacro (robot description, xacro)
@@ -17,6 +17,6 @@
       </collision>
       <inertial>
-        <mass value="0.5" />
-        <inertia ixx="0.008545" ixy="0.0" ixz="0.0" iyy="0.008545" iyz="0.0" izz="0.0144" />
+        <mass value="0.00001" />
+        <inertia ixx="0.000001" ixy="0.0" ixz="0.0" iyy="0.000001" iyz="0.0" izz="0.000001" />
       </inertial>
     </link>
@@ -35,6 +35,6 @@
       </collision>
       <inertial>
-        <mass value="0.5" />
-        <inertia ixx="0.008545" ixy="0.0" ixz="0.0" iyy="0.008545" iyz="0.0" izz="0.0144" />
+        <mass value="0.000001" />
+        <inertia ixx="0.000001" ixy="0.0" ixz="0.0" iyy="0.000001" iyz="0.0" izz="0.000001" />
       </inertial>
     </link>

File: auv_description/auv_common_descriptions/urdf/sensors/bar30.urdf.xacro (robot description, xacro)
@@ -20,6 +20,6 @@
       </collision>
       <inertial>
-        <mass value="0.5" />
-        <inertia ixx="0.008545" ixy="0.0" ixz="0.0" iyy="0.008545" iyz="0.0" izz="0.0144" />
+        <mass value="0.00001" />
+        <inertia ixx="0.000001" ixy="0.0" ixz="0.0" iyy="0.000001" iyz="0.0" izz="0.000001" />
       </inertial>
     </link>

File: auv_description/auv_common_descriptions/urdf/sensors/h2c_hydrophone.urdf.xacro (robot description, xacro)
@@ -16,6 +16,6 @@
       </collision>
       <inertial>
-        <mass value="0.5" />
-        <inertia ixx="0.008545" ixy="0.0" ixz="0.0" iyy="0.008545" iyz="0.0" izz="0.0144" />
+        <mass value="0.0001" />
+        <inertia ixx="0.0000001" ixy="0.0" ixz="0.0" iyy="0.0000001" iyz="0.0" izz="0.0000001" />
       </inertial>
     </link>

File: auv_description/auv_common_descriptions/urdf/sensors/ping360.urdf.xacro (robot description, xacro)
@@ -21,5 +21,5 @@
       <inertial>
         <mass value="0.5" />
-        <inertia ixx="0.008545" ixy="0.0" ixz="0.0" iyy="0.008545" iyz="0.0" izz="0.0144" />
+        <inertia ixx="0.000001" ixy="0.0" ixz="0.0" iyy="0.000001" iyz="0.0" izz="0.000001" />
       </inertial>
     </link>

File: auv_description/auv_common_descriptions/urdf/sensors/xsens_mti_g710.urdf.xacro (robot description, xacro)
@@ -20,6 +20,6 @@
       </collision>
       <inertial>
-        <mass value="0.5" />
-        <inertia ixx="0.008545" ixy="0.0" ixz="0.0" iyy="0.008545" iyz="0.0" izz="0.0144" />
+        <mass value="0.0001" />
+        <inertia ixx="0.000001" ixy="0.0" ixz="0.0" iyy="0.000001" iyz="0.0" izz="0.000001" />
       </inertial>
     </link>
