Commit message: run pre-commit

File: auv_description/auv_common_descriptions/urdf/actuators/t200.urdf.xacro (robot description, xacro)
@@ -16,6 +16,6 @@
       </collision>
       <inertial>
-        <mass value="0.001" />
-        <inertia ixx="0.0000001" ixy="0.0" ixz="0.0" iyy="0.0000001" iyz="0.0" izz="0.0000001" />
+        <mass value="0.001"/>
+        <inertia ixx="0.0000001" ixy="0.0" ixz="0.0" iyy="0.0000001" iyz="0.0" izz="0.0000001"/>
       </inertial>
     </link>
@@ -34,6 +34,6 @@
       </collision>
       <inertial>
-        <mass value="0.001" />
-        <inertia ixx="0.0000001" ixy="0.0" ixz="0.0" iyy="0.0000001" iyz="0.0" izz="0.0000001" />
+        <mass value="0.001"/>
+        <inertia ixx="0.0000001" ixy="0.0" ixz="0.0" iyy="0.0000001" iyz="0.0" izz="0.0000001"/>
       </inertial>
     </link>
@@ -45,8 +45,8 @@
     </joint>
     <joint name="${name}_propeller_joint" type="continuous">
-      <axis rpy="0 0 0" xyz="0 0 1" />
-      <parent link="${name}_link" />
-      <child link="${name}_propeller_link" />
-      <origin xyz="0 0 0" rpy="0 0 0" />
+      <axis rpy="0 0 0" xyz="0 0 1"/>
+      <parent link="${name}_link"/>
+      <child link="${name}_propeller_link"/>
+      <origin xyz="0 0 0" rpy="0 0 0"/>
       <!-- TODO: This breaks the Gazebo Sim -->
       <!-- <dynamics friction="0.05" damping="0.05" /> -->

File: auv_description/auv_common_descriptions/urdf/actuators/torpedo.urdf.xacro (robot description, xacro)
@@ -17,6 +17,6 @@
       </collision>
       <inertial>
-        <mass value="0.00001" />
-        <inertia ixx="0.000001" ixy="0.0" ixz="0.0" iyy="0.000001" iyz="0.0" izz="0.000001" />
+        <mass value="0.00001"/>
+        <inertia ixx="0.000001" ixy="0.0" ixz="0.0" iyy="0.000001" iyz="0.0" izz="0.000001"/>
       </inertial>
     </link>
@@ -35,6 +35,6 @@
       </collision>
       <inertial>
-        <mass value="0.000001" />
-        <inertia ixx="0.000001" ixy="0.0" ixz="0.0" iyy="0.000001" iyz="0.0" izz="0.000001" />
+        <mass value="0.000001"/>
+        <inertia ixx="0.000001" ixy="0.0" ixz="0.0" iyy="0.000001" iyz="0.0" izz="0.000001"/>
       </inertial>
     </link>

File: auv_description/auv_common_descriptions/urdf/sensors/bar30.urdf.xacro (robot description, xacro)
@@ -16,14 +16,14 @@
       </collision>
       <inertial>
-        <mass value="0.00001" />
-        <inertia ixx="0.000001" ixy="0.0" ixz="0.0" iyy="0.000001" iyz="0.0" izz="0.000001" />
+        <mass value="0.00001"/>
+        <inertia ixx="0.000001" ixy="0.0" ixz="0.0" iyy="0.000001" iyz="0.0" izz="0.000001"/>
       </inertial>
     </link>
-    <link name="${name}_link" />
+    <link name="${name}_link"/>
     <joint name="${name}_joint" type="fixed">
-      <parent link="${parent}" />
-      <child link="${name}_chasis_link" />
-      <origin xyz="${position}" rpy="${orientation}" />
-      <axis rpy="0 0 0" xyz="0 0 1" />
+      <parent link="${parent}"/>
+      <child link="${name}_chasis_link"/>
+      <origin xyz="${position}" rpy="${orientation}"/>
+      <axis rpy="0 0 0" xyz="0 0 1"/>
     </joint>
     <joint name="${name}_sensor_joint" type="fixed">

File: auv_description/auv_common_descriptions/urdf/sensors/h2c_hydrophone.urdf.xacro (robot description, xacro)
@@ -16,6 +16,6 @@
       </collision>
       <inertial>
-        <mass value="0.0001" />
-        <inertia ixx="0.0000001" ixy="0.0" ixz="0.0" iyy="0.0000001" iyz="0.0" izz="0.0000001" />
+        <mass value="0.0001"/>
+        <inertia ixx="0.0000001" ixy="0.0" ixz="0.0" iyy="0.0000001" iyz="0.0" izz="0.0000001"/>
       </inertial>
     </link>

File: auv_description/auv_common_descriptions/urdf/sensors/ping360.urdf.xacro (robot description, xacro)
@@ -16,6 +16,6 @@
       </collision>
       <inertial>
-        <mass value="0.5" />
-        <inertia ixx="0.000001" ixy="0.0" ixz="0.0" iyy="0.000001" iyz="0.0" izz="0.000001" />
+        <mass value="0.5"/>
+        <inertia ixx="0.000001" ixy="0.0" ixz="0.0" iyy="0.000001" iyz="0.0" izz="0.000001"/>
       </inertial>
     </link>

File: auv_description/auv_common_descriptions/urdf/sensors/xsens_mti_g710.urdf.xacro (robot description, xacro)
@@ -16,13 +16,13 @@
       </collision>
       <inertial>
-        <mass value="0.0001" />
-        <inertia ixx="0.000001" ixy="0.0" ixz="0.0" iyy="0.000001" iyz="0.0" izz="0.000001" />
+        <mass value="0.0001"/>
+        <inertia ixx="0.000001" ixy="0.0" ixz="0.0" iyy="0.000001" iyz="0.0" izz="0.000001"/>
       </inertial>
     </link>
     <joint name="${name}_joint" type="fixed">
-      <parent link="${parent}" />
-      <child link="${name}_link" />
-      <origin xyz="${position}" rpy="${orientation}" />
-      <axis rpy="0 0 0" xyz="0 0 1" />
+      <parent link="${parent}"/>
+      <child link="${name}_link"/>
+      <origin xyz="${position}" rpy="${orientation}"/>
+      <axis rpy="0 0 0" xyz="0 0 1"/>
     </joint>
   </xacro:macro>

File: auv_description/taluy_description/urdf/auv_base.urdf.xacro (robot description, xacro)
@@ -1,18 +1,16 @@
 <?xml version="1.0"?>
-<robot name="taluy" xmlns:xacro="http://www.ros.org/wiki/xacro">
+<robot xmlns:xacro="http://www.ros.org/wiki/xacro" name="taluy">
   <!-- create xacro property -->
-  <xacro:property name="namespace" value="taluy" />
+  <xacro:property name="namespace" value="taluy"/>
   <xacro:macro name="taluy_base">
-    <xacro:include filename="$(find auv_common_descriptions)/urdf/actuators.urdf.xacro" />
-    <xacro:include
-      filename="$(find auv_common_descriptions)/urdf/sensors.urdf.xacro" />
-    <xacro:include
-      filename="$(find auv_common_descriptions)/urdf/materials.urdf.xacro" />
-    <xacro:arg name="angled_thruster_z_offset" default="-0.01" />
+    <xacro:include filename="$(find auv_common_descriptions)/urdf/actuators.urdf.xacro"/>
+    <xacro:include filename="$(find auv_common_descriptions)/urdf/sensors.urdf.xacro"/>
+    <xacro:include filename="$(find auv_common_descriptions)/urdf/materials.urdf.xacro"/>
+    <xacro:arg name="angled_thruster_z_offset" default="-0.01"/>
     <link name="${namespace}/base_link">
       <inertial>
-        <origin xyz="0 0 0" rpy="0 0 0" />
-        <mass value="25.37" />
-        <inertia ixx="0.1" iyy="0.1" izz="0.1" ixy="0.01" iyz="0.01" ixz="0.1" />
+        <origin xyz="0 0 0" rpy="0 0 0"/>
+        <mass value="25.37"/>
+        <inertia ixx="0.1" iyy="0.1" izz="0.1" ixy="0.01" iyz="0.01" ixz="0.1"/>
       </inertial>
       <visual>
@@ -36,77 +34,28 @@
       <child link="${namespace}/base_link" />
     </joint> -->
-    <xacro:t200_thruster name="${namespace}/thruster_0" parent="${namespace}/base_link"
-      position="0.14250 0.20070 -0.00525"
-      orientation="${pi} 0 ${-pi/2}" />
-    <xacro:t200_thruster name="${namespace}/thruster_1" parent="${namespace}/base_link"
-      position="0.14250 -0.20070 -0.00525"
-      orientation="${pi} 0 ${pi/2}" />
-    <xacro:t200_thruster name="${namespace}/thruster_2" parent="${namespace}/base_link"
-      position="-0.14250 0.20070 -0.00525"
-      orientation="${pi} 0 ${-pi/2}" />
-    <xacro:t200_thruster name="${namespace}/thruster_3" parent="${namespace}/base_link"
-      position="-0.14250 -0.20070 -0.00525"
-      orientation="${pi} 0 ${pi/2}" />
-    <xacro:t200_thruster name="${namespace}/thruster_4" parent="${namespace}/base_link"
-      position="0.352398 0.216638 $(arg angled_thruster_z_offset)"
-      orientation="${-pi/2} 0 ${-7*pi/4}" />
-    <xacro:t200_thruster name="${namespace}/thruster_5" parent="${namespace}/base_link"
-      position="0.352398 -0.216638 $(arg angled_thruster_z_offset)"
-      orientation="${pi/2} 0 ${7*pi/4}" />
-    <xacro:t200_thruster name="${namespace}/thruster_6" parent="${namespace}/base_link"
-      position="-0.352398 0.216638 $(arg angled_thruster_z_offset)"
-      orientation="${-pi/2} 0 ${-pi/4}" />
-    <xacro:t200_thruster name="${namespace}/thruster_7" parent="${namespace}/base_link"
-      position="-0.352398 -0.216638 $(arg angled_thruster_z_offset)" orientation="${pi/2} 0 ${pi/4}" />
-    <xacro:wayfinder_dvl
-      name="${namespace}/base_link/dvl" parent="${namespace}/base_link" position="0.2 0 -0.11"
-      orientation="0 0 0" />
-    <xacro:xsens_mti_g710 name="${namespace}/base_link/imu" parent="${namespace}/base_link"
-      position="-0.199 0 -0.0108"
-      orientation="0 0 ${math.pi}" />
-    <xacro:h2c_hydrophone name="${namespace}/base_link/hydrophone_0"
-      parent="${namespace}/base_link"
-      position="0.325 0.205 -0.15"
-      orientation="0 0 0" />
-    <xacro:h2c_hydrophone name="${namespace}/base_link/hydrophone_1" parent="${namespace}/base_link"
-      position="0.325 -0.205 -0.15"
-      orientation="0 0 0" />
-    <xacro:h2c_hydrophone name="${namespace}/base_link/hydrophone_2" parent="${namespace}/base_link"
-      position="-0.325 0.205 -0.15"
-      orientation="0 0 0" />
-    <xacro:h2c_hydrophone name="${namespace}/base_link/hydrophone_3" parent="${namespace}/base_link"
-      position="-0.325 -0.205 -0.15"
-      orientation="0 0 0" />
-    <xacro:ping360 name="${namespace}/base_link/ping360" parent="${namespace}/base_link"
-      position="0.2 0 0.134"
-      orientation="0 0 0" />
-    <xacro:bar30 name="${namespace}/base_link/external_pressure_sensor"
-      parent="${namespace}/base_link"
-      position="0 0 0.07"
-      orientation="0 0 0" />
-    <xacro:logitech_c920_camera name="${namespace}/base_link/front_camera"
-      parent="${namespace}/base_link" position="0.35 0 0"
-      orientation="0 0 0" />
-    <xacro:logitech_c920_camera name="${namespace}/base_link/bottom_camera"
-      parent="${namespace}/base_link" position="0 0 -0.07"
-      orientation="0 ${math.pi/2} ${math.pi/2}" />
-    <xacro:torpedo name="${namespace}/base_link/left_torpedo"
-      parent="${namespace}/base_link" position="0.2 0.1 -0.11"
-      orientation="0 0 0" />
-    <xacro:torpedo name="${namespace}/base_link/right_torpedo"
-      parent="${namespace}/base_link" position="0.2 -0.1 -0.11"
-      orientation="0 0 0" />
-    <xacro:sonar name="${namespace}/base_link/sonar_front" parent="${namespace}/base_link"
-      position="0.38 0.09 0.09"
-      orientation="0 0 0" />
-    <xacro:sonar name="${namespace}/base_link/sonar_back" parent="${namespace}/base_link"
-      position="-0.42 -0.09 0.09"
-      orientation="0 0 ${math.pi}" />
-    <xacro:sonar name="${namespace}/base_link/sonar_right" parent="${namespace}/base_link"
-      position="0.02 -0.21 -0.14"
-      orientation="0 0 ${-math.pi/2}" />
-    <xacro:sonar name="${namespace}/base_link/sonar_left" parent="${namespace}/base_link"
-      position="0.02 0.21 -0.14"
-      orientation="0 0 ${math.pi/2}" />
+    <xacro:t200_thruster name="${namespace}/thruster_0" parent="${namespace}/base_link" position="0.14250 0.20070 -0.00525" orientation="${pi} 0 ${-pi/2}"/>
+    <xacro:t200_thruster name="${namespace}/thruster_1" parent="${namespace}/base_link" position="0.14250 -0.20070 -0.00525" orientation="${pi} 0 ${pi/2}"/>
+    <xacro:t200_thruster name="${namespace}/thruster_2" parent="${namespace}/base_link" position="-0.14250 0.20070 -0.00525" orientation="${pi} 0 ${-pi/2}"/>
+    <xacro:t200_thruster name="${namespace}/thruster_3" parent="${namespace}/base_link" position="-0.14250 -0.20070 -0.00525" orientation="${pi} 0 ${pi/2}"/>
+    <xacro:t200_thruster name="${namespace}/thruster_4" parent="${namespace}/base_link" position="0.352398 0.216638 $(arg angled_thruster_z_offset)" orientation="${-pi/2} 0 ${-7*pi/4}"/>
+    <xacro:t200_thruster name="${namespace}/thruster_5" parent="${namespace}/base_link" position="0.352398 -0.216638 $(arg angled_thruster_z_offset)" orientation="${pi/2} 0 ${7*pi/4}"/>
+    <xacro:t200_thruster name="${namespace}/thruster_6" parent="${namespace}/base_link" position="-0.352398 0.216638 $(arg angled_thruster_z_offset)" orientation="${-pi/2} 0 ${-pi/4}"/>
+    <xacro:t200_thruster name="${namespace}/thruster_7" parent="${namespace}/base_link" position="-0.352398 -0.216638 $(arg angled_thruster_z_offset)" orientation="${pi/2} 0 ${pi/4}"/>
+    <xacro:wayfinder_dvl name="${namespace}/base_link/dvl" parent="${namespace}/base_link" position="0.2 0 -0.11" orientation="0 0 0"/>
+    <xacro:xsens_mti_g710 name="${namespace}/base_link/imu" parent="${namespace}/base_link" position="-0.199 0 -0.0108" orientation="0 0 ${math.pi}"/>
+    <xacro:h2c_hydrophone name="${namespace}/base_link/hydrophone_0" parent="${namespace}/base_link" position="0.325 0.205 -0.15" orientation="0 0 0"/>
+    <xacro:h2c_hydrophone name="${namespace}/base_link/hydrophone_1" parent="${namespace}/base_link" position="0.325 -0.205 -0.15" orientation="0 0 0"/>
+    <xacro:h2c_hydrophone name="${namespace}/base_link/hydrophone_2" parent="${namespace}/base_link" position="-0.325 0.205 -0.15" orientation="0 0 0"/>
+    <xacro:h2c_hydrophone name="${namespace}/base_link/hydrophone_3" parent="${namespace}/base_link" position="-0.325 -0.205 -0.15" orientation="0 0 0"/>
+    <xacro:ping360 name="${namespace}/base_link/ping360" parent="${namespace}/base_link" position="0.2 0 0.134" orientation="0 0 0"/>
+    <xacro:bar30 name="${namespace}/base_link/external_pressure_sensor" parent="${namespace}/base_link" position="0 0 0.07" orientation="0 0 0"/>
+    <xacro:logitech_c920_camera name="${namespace}/base_link/front_camera" parent="${namespace}/base_link" position="0.35 0 0" orientation="0 0 0"/>
+    <xacro:logitech_c920_camera name="${namespace}/base_link/bottom_camera" parent="${namespace}/base_link" position="0 0 -0.07" orientation="0 ${math.pi/2} ${math.pi/2}"/>
+    <xacro:torpedo name="${namespace}/base_link/left_torpedo" parent="${namespace}/base_link" position="0.2 0.1 -0.11" orientation="0 0 0"/>
+    <xacro:torpedo name="${namespace}/base_link/right_torpedo" parent="${namespace}/base_link" position="0.2 -0.1 -0.11" orientation="0 0 0"/>
+    <xacro:sonar name="${namespace}/base_link/sonar_front" parent="${namespace}/base_link" position="0.38 0.09 0.09" orientation="0 0 0"/>
+    <xacro:sonar name="${namespace}/base_link/sonar_back" parent="${namespace}/base_link" position="-0.42 -0.09 0.09" orientation="0 0 ${math.pi}"/>
+    <xacro:sonar name="${namespace}/base_link/sonar_right" parent="${namespace}/base_link" position="0.02 -0.21 -0.14" orientation="0 0 ${-math.pi/2}"/>
+    <xacro:sonar name="${namespace}/base_link/sonar_left" parent="${namespace}/base_link" position="0.02 0.21 -0.14" orientation="0 0 ${math.pi/2}"/>
     <!-- <link name="base_footprint">
       <inertial>

File: auv_sim/auv_sim_description/auv_common_sim_descriptions/urdf/actuators.urdf.xacro (robot description, xacro)
@@ -1,4 +1,4 @@
 <?xml version="1.0"?>
 <robot xmlns:xacro="http://www.ros.org/wiki/xacro">
-  <xacro:include filename="$(find auv_common_sim_descriptions)/urdf/actuators/t200.urdf.xacro" />
+  <xacro:include filename="$(find auv_common_sim_descriptions)/urdf/actuators/t200.urdf.xacro"/>
 </robot>

File: auv_sim/auv_sim_description/auv_common_sim_descriptions/urdf/actuators/t200.urdf.xacro (robot description, xacro)
@@ -1,4 +1,4 @@
 <?xml version="1.0"?>
-<robot name="t200_thruster" xmlns:xacro="http://ros.org/wiki/xacro">
+<robot xmlns:xacro="http://ros.org/wiki/xacro" name="t200_thruster">
   <xacro:macro name="t200_thruster_sim" params="name thruster_id">
     <gazebo>

File: auv_sim/auv_sim_description/auv_common_sim_descriptions/urdf/sensors.urdf.xacro (robot description, xacro)
@@ -1,13 +1,8 @@
 <?xml version="1.0"?>
 <robot xmlns:xacro="http://www.ros.org/wiki/xacro">
-  <xacro:include
-    filename="$(find auv_common_sim_descriptions)/urdf/sensors/xsens_mti_g710.urdf.xacro" />
-  <xacro:include
-    filename="$(find auv_common_sim_descriptions)/urdf/sensors/bar30.urdf.xacro" />
-  <xacro:include
-    filename="$(find auv_common_sim_descriptions)/urdf/sensors/logitech_c920_camera.urdf.xacro" />
-  <xacro:include
-    filename="$(find auv_common_sim_descriptions)/urdf/sensors/sonar.urdf.xacro" />
-  <xacro:include
-    filename="$(find auv_common_sim_descriptions)/urdf/sensors/wayfinder_dvl.urdf.xacro" />
+  <xacro:include filename="$(find auv_common_sim_descriptions)/urdf/sensors/xsens_mti_g710.urdf.xacro"/>
+  <xacro:include filename="$(find auv_common_sim_descriptions)/urdf/sensors/bar30.urdf.xacro"/>
+  <xacro:include filename="$(find auv_common_sim_descriptions)/urdf/sensors/logitech_c920_camera.urdf.xacro"/>
+  <xacro:include filename="$(find auv_common_sim_descriptions)/urdf/sensors/sonar.urdf.xacro"/>
+  <xacro:include filename="$(find auv_common_sim_descriptions)/urdf/sensors/wayfinder_dvl.urdf.xacro"/>
 </robot>

File: auv_sim/auv_sim_description/auv_common_sim_descriptions/urdf/sensors/bar30.urdf.xacro (robot description, xacro)
@@ -1,28 +1,27 @@
 <?xml version="1.0"?>
-<robot name="bar30" xmlns:xacro="http://www.ros.org/wiki/xacro">
+<robot xmlns:xacro="http://www.ros.org/wiki/xacro" name="bar30">
   <xacro:macro name="bar30_sim" params="name">
     <link name="${name}_sim_link">
       <inertial>
-        <mass value="0.001" />
-        <origin xyz="0 0 0" rpy="0 0 0" />
-        <inertia ixx="0.0000001" ixy="0" ixz="0" iyy="0.0000001" iyz="0" izz="0.0000001" />
+        <mass value="0.001"/>
+        <origin xyz="0 0 0" rpy="0 0 0"/>
+        <inertia ixx="0.0000001" ixy="0" ixz="0" iyy="0.0000001" iyz="0" izz="0.0000001"/>
       </inertial>
       <collision>
         <geometry>
-          <cylinder length="${0.000001}" radius="${0.000001}" />
+          <cylinder length="${0.000001}" radius="${0.000001}"/>
         </geometry>
-        <origin xyz="0 0 0" rpy="0 ${0.5*pi} 0" />
+        <origin xyz="0 0 0" rpy="0 ${0.5*pi} 0"/>
       </collision>
     </link>
     <joint name="${name}_sim_joint" type="revolute">
-      <parent link="${name}_chasis_link" />
-      <child link="${name}_sim_link" />
-      <origin xyz="0 0 0" rpy="0 0 0" />
-      <axis rpy="0 0 0" xyz="0 0 1" />
-      <limit lower="0.0" upper="0.0" effort="0.0" velocity="0.0" />
+      <parent link="${name}_chasis_link"/>
+      <child link="${name}_sim_link"/>
+      <origin xyz="0 0 0" rpy="0 0 0"/>
+      <axis rpy="0 0 0" xyz="0 0 1"/>
+      <limit lower="0.0" upper="0.0" effort="0.0" velocity="0.0"/>
     </joint>
     <gazebo>
-      <plugin filename="libuuv_gazebo_ros_subsea_pressure_plugin.so"
-        name="${name}_pressure_plugin">
+      <plugin filename="libuuv_gazebo_ros_subsea_pressure_plugin.so" name="${name}_pressure_plugin">
         <robot_namespace>taluy</robot_namespace>
         <link_name>${name}_sim_link</link_name>

File: auv_sim/auv_sim_description/auv_common_sim_descriptions/urdf/sensors/logitech_c920_camera.urdf.xacro (robot description, xacro)
@@ -1,4 +1,4 @@
 <?xml version="1.0"?>
-<robot name="logitech_c920_camera" xmlns:xacro="http://ros.org/wiki/xacro">
+<robot xmlns:xacro="http://ros.org/wiki/xacro" name="logitech_c920_camera">
   <xacro:macro name="logitech_c920_camera_sim" params="name topic_name">
     <gazebo reference="${name}_link">

File: auv_sim/auv_sim_description/auv_common_sim_descriptions/urdf/sensors/sonar.urdf.xacro (robot description, xacro)
@@ -1,4 +1,4 @@
 <?xml version="1.0"?>
-<robot name="sonar" xmlns:xacro="http://ros.org/wiki/xacro">
+<robot xmlns:xacro="http://ros.org/wiki/xacro" name="sonar">
   <xacro:macro name="sonar_sim" params="name topic">
     <gazebo reference="${name}_link">
