Commit message: run pre-commit

File: auv_sim/auv_sim_description/auv_common_sim_descriptions/urdf/sensors/wayfinder_dvl.urdf.xacro (robot description, xacro)
@@ -1,24 +1,25 @@
 <?xml version="1.0"?>
-<robot name="wayfinder_dvl" xmlns:xacro="http://ros.org/wiki/xacro">
+<robot xmlns:xacro="http://ros.org/wiki/xacro" name="wayfinder_dvl">
   <xacro:macro name="dvl_single_sonar" params="namespace name index update_rate">
     <link name="${namespace}/dvl_sonar${index}_link">
       <inertial>
-        <mass value="0.001" />  <!-- [kg] -->
-        <origin xyz="0 0 0" rpy="0 0 0" />
-        <inertia ixx="0.000000017" ixy="0" ixz="0" iyy="0.000000017" iyz="0" izz="0.000000017" />
+        <mass value="0.001"/>
+        <!-- [kg] -->
+        <origin xyz="0 0 0" rpy="0 0 0"/>
+        <inertia ixx="0.000000017" ixy="0" ixz="0" iyy="0.000000017" iyz="0" izz="0.000000017"/>
       </inertial>
       <collision>
         <geometry>
-          <cylinder length="${0.000001}" radius="${0.000001}" />
+          <cylinder length="${0.000001}" radius="${0.000001}"/>
         </geometry>
-        <origin xyz="0 0 0" rpy="0 ${0.5*pi} 0" />
+        <origin xyz="0 0 0" rpy="0 ${0.5*pi} 0"/>
       </collision>
     </link>
     <joint name="${namespace}/dvl_sonar${index}_joint" type="revolute">
-      <origin xyz="0 0 -0.07" rpy="0 ${math.pi/2} 0" />
-      <parent link="${name}_mount_link" />
-      <child link="${namespace}/dvl_sonar${index}_link" />
-      <limit upper="0" lower="0" effort="0" velocity="0" />
-      <axis xyz="1 0 0" />
+      <origin xyz="0 0 -0.07" rpy="0 ${math.pi/2} 0"/>
+      <parent link="${name}_mount_link"/>
+      <child link="${namespace}/dvl_sonar${index}_link"/>
+      <limit upper="0" lower="0" effort="0" velocity="0"/>
+      <axis xyz="1 0 0"/>
     </joint>
     <gazebo reference="${namespace}/dvl_sonar${index}_link">
@@ -66,49 +67,32 @@
     </gazebo>
   </xacro:macro>
-  <xacro:macro name="wayfinder_dvl_sim"
-    params="name namespace static_reference_frame update_rate">
+  <xacro:macro name="wayfinder_dvl_sim" params="name namespace static_reference_frame update_rate">
     <link name="${name}_sim_link">
       <inertial>
-        <mass value="0.001" />
-        <origin xyz="0 0 0" rpy="0 0 0" />
-        <inertia ixx="0.0000001" ixy="0" ixz="0" iyy="0.0000001" iyz="0" izz="0.0000001" />
+        <mass value="0.001"/>
+        <origin xyz="0 0 0" rpy="0 0 0"/>
+        <inertia ixx="0.0000001" ixy="0" ixz="0" iyy="0.0000001" iyz="0" izz="0.0000001"/>
       </inertial>
       <collision>
         <geometry>
-          <cylinder length="${0.000001}" radius="${0.000001}" />
+          <cylinder length="${0.000001}" radius="${0.000001}"/>
         </geometry>
-        <origin xyz="0 0 0" rpy="0 ${0.5*pi} 0" />
+        <origin xyz="0 0 0" rpy="0 ${0.5*pi} 0"/>
       </collision>
     </link>
     <joint name="${name}_sim_joint" type="revolute">
-      <parent link="${name}_mount_link" />
-      <child link="${name}_sim_link" />
-      <origin xyz="0 0 0" rpy="0 0 0" />
-      <axis rpy="0 0 0" xyz="0 0 1" />
-      <limit lower="0.0" upper="0.0" effort="0.0" velocity="0.0" />
+      <parent link="${name}_mount_link"/>
+      <child link="${name}_sim_link"/>
+      <origin xyz="0 0 0" rpy="0 0 0"/>
+      <axis rpy="0 0 0" xyz="0 0 1"/>
+      <limit lower="0.0" upper="0.0" effort="0.0" velocity="0.0"/>
     </joint>
-    <xacro:dvl_single_sonar
-      namespace="${namespace}"
-      name="${name}"
-      index="0"
-      update_rate="${update_rate}">
+    <xacro:dvl_single_sonar namespace="${namespace}" name="${name}" index="0" update_rate="${update_rate}">
     </xacro:dvl_single_sonar>
-    <xacro:dvl_single_sonar
-      namespace="${namespace}"
-      name="${name}"
-      index="1"
-      update_rate="${update_rate}">
+    <xacro:dvl_single_sonar namespace="${namespace}" name="${name}" index="1" update_rate="${update_rate}">
     </xacro:dvl_single_sonar>
-    <xacro:dvl_single_sonar
-      namespace="${namespace}"
-      name="${name}"
-      index="2"
-      update_rate="${update_rate}">
+    <xacro:dvl_single_sonar namespace="${namespace}" name="${name}" index="2" update_rate="${update_rate}">
     </xacro:dvl_single_sonar>
-    <xacro:dvl_single_sonar
-      namespace="${namespace}"
-      name="${name}"
-      index="3"
-      update_rate="${update_rate}">
+    <xacro:dvl_single_sonar namespace="${namespace}" name="${name}" index="3" update_rate="${update_rate}">
     </xacro:dvl_single_sonar>
     <gazebo>

File: auv_sim/auv_sim_description/auv_common_sim_descriptions/urdf/sensors/xsens_mti_g710.urdf.xacro (robot description, xacro)
@@ -1,28 +1,27 @@
 <?xml version="1.0"?>
-<robot name="xsens_mti_g710" xmlns:xacro="http://www.ros.org/wiki/xacro">
+<robot xmlns:xacro="http://www.ros.org/wiki/xacro" name="xsens_mti_g710">
   <xacro:macro name="xsens_mti_g710_sim" params="name namespace static_reference_frame">
     <link name="${name}_sim_link">
       <inertial>
-        <mass value="0.001" />
-        <origin xyz="0 0 0" rpy="0 0 0" />
-        <inertia ixx="0.0000001" ixy="0" ixz="0" iyy="0.0000001" iyz="0" izz="0.0000001" />
+        <mass value="0.001"/>
+        <origin xyz="0 0 0" rpy="0 0 0"/>
+        <inertia ixx="0.0000001" ixy="0" ixz="0" iyy="0.0000001" iyz="0" izz="0.0000001"/>
       </inertial>
       <collision>
         <geometry>
-          <cylinder length="${0.000001}" radius="${0.000001}" />
+          <cylinder length="${0.000001}" radius="${0.000001}"/>
         </geometry>
-        <origin xyz="0 0 0" rpy="0 ${0.5*pi} 0" />
+        <origin xyz="0 0 0" rpy="0 ${0.5*pi} 0"/>
       </collision>
     </link>
     <joint name="${name}_sim_joint" type="revolute">
-      <parent link="${name}_link" />
-      <child link="${name}_sim_link" />
-      <origin xyz="0 0 0" rpy="${math.pi} ${math.pi} 0" />
-      <axis rpy="0 0 0" xyz="0 0 1" />
-      <limit lower="0.0" upper="0.0" effort="0.0" velocity="0.0" />
+      <parent link="${name}_link"/>
+      <child link="${name}_sim_link"/>
+      <origin xyz="0 0 0" rpy="${math.pi} ${math.pi} 0"/>
+      <axis rpy="0 0 0" xyz="0 0 1"/>
+      <limit lower="0.0" upper="0.0" effort="0.0" velocity="0.0"/>
     </joint>
     <gazebo>
-      <plugin filename="libuuv_gazebo_ros_imu_plugin.so"
-        name="${name}_imu_plugin">
+      <plugin filename="libuuv_gazebo_ros_imu_plugin.so" name="${name}_imu_plugin">
         <robot_namespace>${namespace}</robot_namespace>
         <link_name>${name}_sim_link</link_name>

File: auv_sim/auv_sim_description/taluy_sim_description/urdf/actuators.urdf.xacro (robot description, xacro)
@@ -1,12 +1,12 @@
 <?xml version="1.0"?>
 <robot xmlns:xacro="http://www.ros.org/wiki/xacro">
-  <xacro:include filename="$(find auv_common_sim_descriptions)/urdf/actuators.urdf.xacro" />
-  <xacro:t200_thruster_sim name="${namespace}/thruster_0" thruster_id="0" />
-  <xacro:t200_thruster_sim name="${namespace}/thruster_1" thruster_id="1" />
-  <xacro:t200_thruster_sim name="${namespace}/thruster_2" thruster_id="2" />
-  <xacro:t200_thruster_sim name="${namespace}/thruster_3" thruster_id="3" />
-  <xacro:t200_thruster_sim name="${namespace}/thruster_4" thruster_id="4" />
-  <xacro:t200_thruster_sim name="${namespace}/thruster_5" thruster_id="5" />
-  <xacro:t200_thruster_sim name="${namespace}/thruster_6" thruster_id="6" />
-  <xacro:t200_thruster_sim name="${namespace}/thruster_7" thruster_id="7" />
+  <xacro:include filename="$(find auv_common_sim_descriptions)/urdf/actuators.urdf.xacro"/>
+  <xacro:t200_thruster_sim name="${namespace}/thruster_0" thruster_id="0"/>
+  <xacro:t200_thruster_sim name="${namespace}/thruster_1" thruster_id="1"/>
+  <xacro:t200_thruster_sim name="${namespace}/thruster_2" thruster_id="2"/>
+  <xacro:t200_thruster_sim name="${namespace}/thruster_3" thruster_id="3"/>
+  <xacro:t200_thruster_sim name="${namespace}/thruster_4" thruster_id="4"/>
+  <xacro:t200_thruster_sim name="${namespace}/thruster_5" thruster_id="5"/>
+  <xacro:t200_thruster_sim name="${namespace}/thruster_6" thruster_id="6"/>
+  <xacro:t200_thruster_sim name="${namespace}/thruster_7" thruster_id="7"/>
 </robot>

File: auv_sim/auv_sim_description/taluy_sim_description/urdf/base.urdf.xacro (robot description, xacro)
@@ -2,9 +2,9 @@
 <robot xmlns:xacro="http://www.ros.org/wiki/xacro">
   <xacro:macro name="auv_sim_base" params="namespace *gazebo inertial_reference_frame">
-    <xacro:insert_block name="gazebo" />
-    <xacro:include filename="$(find taluy_description)/urdf/auv_base.urdf.xacro" />
-    <xacro:taluy_base />
-    <xacro:include filename="$(find taluy_sim_description)/urdf/actuators.urdf.xacro" />
-    <xacro:include filename="$(find taluy_sim_description)/urdf/sensors.urdf.xacro" />
+    <xacro:insert_block name="gazebo"/>
+    <xacro:include filename="$(find taluy_description)/urdf/auv_base.urdf.xacro"/>
+    <xacro:taluy_base/>
+    <xacro:include filename="$(find taluy_sim_description)/urdf/actuators.urdf.xacro"/>
+    <xacro:include filename="$(find taluy_sim_description)/urdf/sensors.urdf.xacro"/>
   </xacro:macro>
 </robot>

File: auv_sim/auv_sim_description/taluy_sim_description/urdf/dynamics.urdf.xacro (robot description, xacro)
@@ -18,7 +18,7 @@
     assume NWU (otherwise cob is below cog?).
     -->
-  <xacro:property name="cob" value="0.0 0.0 0.2" />
+  <xacro:property name="cob" value="0.0 0.0 0.2"/>
   <!-- Volume, see p.31 in Berg2012, normally 0.009165088 -->
-  <xacro:property name="volume" value="0.027" />
+  <xacro:property name="volume" value="0.027"/>
   <xacro:macro name="auv_hydro_model" params="namespace">
     <link name="${namespace}/base_link">

File: auv_sim/auv_sim_description/taluy_sim_description/urdf/sensors.urdf.xacro (robot description, xacro)
@@ -1,17 +1,13 @@
 <?xml version="1.0"?>
 <robot xmlns:xacro="http://www.ros.org/wiki/xacro">
-  <xacro:include filename="$(find auv_common_sim_descriptions)/urdf/sensors.urdf.xacro" />
-  <xacro:bar30_sim name="${namespace}/base_link/external_pressure_sensor" />
-  <xacro:sonar_sim name="${namespace}/base_link/sonar_front" topic="sensors/sonar_front" />
-  <xacro:sonar_sim name="${namespace}/base_link/sonar_back" topic="sensors/sonar_back" />
-  <xacro:sonar_sim name="${namespace}/base_link/sonar_right" topic="sensors/sonar_right" />
-  <xacro:sonar_sim name="${namespace}/base_link/sonar_left" topic="sensors/sonar_left" />
-  <xacro:logitech_c920_camera_sim name="${namespace}/base_link/front_camera"
-    topic_name="cameras/cam_front" />
-  <xacro:logitech_c920_camera_sim name="${namespace}/base_link/bottom_camera"
-    topic_name="cameras/cam_bottom" />
-  <xacro:xsens_mti_g710_sim name="${namespace}/base_link/imu" namespace="${namespace}"
-    static_reference_frame="${inertial_reference_frame}" />
-  <xacro:wayfinder_dvl_sim name="${namespace}/base_link/dvl" namespace="${namespace}"
-    static_reference_frame="${inertial_reference_frame}" update_rate="10" />
+  <xacro:include filename="$(find auv_common_sim_descriptions)/urdf/sensors.urdf.xacro"/>
+  <xacro:bar30_sim name="${namespace}/base_link/external_pressure_sensor"/>
+  <xacro:sonar_sim name="${namespace}/base_link/sonar_front" topic="sensors/sonar_front"/>
+  <xacro:sonar_sim name="${namespace}/base_link/sonar_back" topic="sensors/sonar_back"/>
+  <xacro:sonar_sim name="${namespace}/base_link/sonar_right" topic="sensors/sonar_right"/>
+  <xacro:sonar_sim name="${namespace}/base_link/sonar_left" topic="sensors/sonar_left"/>
+  <xacro:logitech_c920_camera_sim name="${namespace}/base_link/front_camera" topic_name="cameras/cam_front"/>
+  <xacro:logitech_c920_camera_sim name="${namespace}/base_link/bottom_camera" topic_name="cameras/cam_bottom"/>
+  <xacro:xsens_mti_g710_sim name="${namespace}/base_link/imu" namespace="${namespace}" static_reference_frame="${inertial_reference_frame}"/>
+  <xacro:wayfinder_dvl_sim name="${namespace}/base_link/dvl" namespace="${namespace}" static_reference_frame="${inertial_reference_frame}" update_rate="10"/>
 </robot>

File: auv_sim/auv_sim_description/taluy_sim_description/urdf/taluy_sim.urdf.xacro (robot description, xacro)
@@ -1,13 +1,11 @@
 <?xml version="1.0"?>
-<robot name="taluy" xmlns:xacro="http://www.ros.org/wiki/xacro">
-  <xacro:arg name="debug" default="0" />
-  <xacro:arg name="namespace" default="taluy" />
-  <xacro:arg name="control_rate" default="20" />
-  <xacro:arg name="inertial_reference_frame" default="world" />
-  <xacro:include filename="$(find taluy_sim_description)/urdf/base.urdf.xacro" />
-  <xacro:include filename="$(find taluy_sim_description)/urdf/dynamics.urdf.xacro" />
-  <xacro:auv_sim_base
-    namespace="$(arg namespace)"
-    inertial_reference_frame="$(arg inertial_reference_frame)">
+<robot xmlns:xacro="http://www.ros.org/wiki/xacro" name="taluy">
+  <xacro:arg name="debug" default="0"/>
+  <xacro:arg name="namespace" default="taluy"/>
+  <xacro:arg name="control_rate" default="20"/>
+  <xacro:arg name="inertial_reference_frame" default="world"/>
+  <xacro:include filename="$(find taluy_sim_description)/urdf/base.urdf.xacro"/>
+  <xacro:include filename="$(find taluy_sim_description)/urdf/dynamics.urdf.xacro"/>
+  <xacro:auv_sim_base namespace="$(arg namespace)" inertial_reference_frame="$(arg inertial_reference_frame)">
     <gazebo>
       <plugin name="uuv_plugin" filename="libuuv_underwater_object_ros_plugin.so">
@@ -15,25 +13,15 @@
         <flow_velocity_topic>hydrodynamics/current_velocity</flow_velocity_topic>
         <debug>$(arg debug)</debug>
-        <xacro:auv_hydro_model namespace="$(arg namespace)" />
+        <xacro:auv_hydro_model namespace="$(arg namespace)"/>
       </plugin>
     </gazebo>
   </xacro:auv_sim_base>
   <!-- joint state publisher -->
-  <xacro:include filename="$(find uuv_gazebo_ros_plugins)/urdf/misc.xacro" />
-  <xacro:include filename="$(find uuv_sensor_ros_plugins)/urdf/pose_3d_snippets.xacro" />
-  <xacro:default_joint_state_publisher namespace="$(arg namespace)"
-    update_rate="$(arg control_rate)" />
+  <xacro:include filename="$(find uuv_gazebo_ros_plugins)/urdf/misc.xacro"/>
+  <xacro:include filename="$(find uuv_sensor_ros_plugins)/urdf/pose_3d_snippets.xacro"/>
+  <xacro:default_joint_state_publisher namespace="$(arg namespace)" update_rate="$(arg control_rate)"/>
   <!-- ground truth odometry -->
-  <xacro:pose_3d_macro
-    namespace="$(arg namespace)"
-    parent_link="$(arg namespace)/base_link"
-    topic="odometry_gt"
-    update_rate="$(arg control_rate)"
-    noise_sigma="0.0"
-    noise_amplitude="0.0"
-    suffix="default"
-    reference_frame="odom"
-    publish_ned_odom="false">
-    <origin xyz="0 0 0" rpy="0 0 0" />
+  <xacro:pose_3d_macro namespace="$(arg namespace)" parent_link="$(arg namespace)/base_link" topic="odometry_gt" update_rate="$(arg control_rate)" noise_sigma="0.0" noise_amplitude="0.0" suffix="default" reference_frame="odom" publish_ned_odom="false">
+    <origin xyz="0 0 0" rpy="0 0 0"/>
   </xacro:pose_3d_macro>
 </robot>
