Commit message: Add UUV Simulation (#94)
* create package structure for auv_sim

* Added descriptions, spawn.launch and start_gazebo.launch files

* Delete urdf's in auv_sim_description

* Change default namespace to taluy

* Use auv_description instead of auv_sim_description

* start control nodes at gazebo launch

* restructure `auv_sim_description`

- remove unnecessary folder

* use taluy_sim.urdf.xacro as main simulation macro

- we will use this to include gazebo plugins

* create camera, imu and thruster gazebo plugins

- plugin settings need to be edited

* add gazebo plugin for bottom camera

* add `topic_name` parameter to gazebo camera plugin

- use `topic_name` to match the original camera topic names
- also update plugin specs with logitech c920 specs

* rename `thrusterID` to `thruster_id`

it is urdf/xacro convention to use snake_case

* move gazebo tags in `t200.urdf.xacro` to it's auv_sim macro

* use the uuv_simulator plugin for imu

- Replace the libgazebo_ros imu plugin with libuuv_gazebo_ros imu plugin. This is how it was in the legacy repo, so I thought this should be better.
- Changed the joint type of the IMU link from `fixed` to `revolute` (with movement limits) to resolve an issue where libuuv_gazebo_ros plugins couldn't detect fixed links in Gazebo.
- Noted that Gazebo doesn't recognize links with fixed joints as standalone links, which seems to cause this issue.

* create bar30 gazebo plugin

- use libuuv_gazebo_ros_subsea_pressure_plugin
- Changed the joint type of the bar30 link from `fixed` to `revolute` (with movement limits) to resolve an issue where libuuv_gazebo_ros plugins couldn't detect fixed links in Gazebo.
- Noted that Gazebo doesn't recognize links with fixed joints as standalone links, which seems to cause this issue.

* create sonar gazebo plugin

- implemented from legacy repo (ituauv-uuv-descriptions)

* added base bridge nodes (not ready yet)

* modify package.xml files

* create base_link hydrodynamics plugin

- the values in base_link_ned are robot spesific and belongs to turquoise, we need to change them with taluy's values

* Add Singapore pool world and model

* create package structure for auv_sim

* Added descriptions, spawn.launch and start_gazebo.launch files

* Delete urdf's in auv_sim_description

* Use auv_description instead of auv_sim_description

* start control nodes at gazebo launch

* restructure `auv_sim_description`

- remove unnecessary folder

* use taluy_sim.urdf.xacro as main simulation macro

- we will use this to include gazebo plugins

* create camera, imu and thruster gazebo plugins

- plugin settings need to be edited

* add gazebo plugin for bottom camera

* add `topic_name` parameter to gazebo camera plugin

- use `topic_name` to match the original camera topic names
- also update plugin specs with logitech c920 specs

* rename `thrusterID` to `thruster_id`

it is urdf/xacro convention to use snake_case

* move gazebo tags in `t200.urdf.xacro` to it's auv_sim macro

* use the uuv_simulator plugin for imu

- Replace the libgazebo_ros imu plugin with libuuv_gazebo_ros imu plugin. This is how it was in the legacy repo, so I thought this should be better.
- Changed the joint type of the IMU link from `fixed` to `revolute` (with movement limits) to resolve an issue where libuuv_gazebo_ros plugins couldn't detect fixed links in Gazebo.
- Noted that Gazebo doesn't recognize links with fixed joints as standalone links, which seems to cause this issue.

* create bar30 gazebo plugin

- use libuuv_gazebo_ros_subsea_pressure_plugin
- Changed the joint type of the bar30 link from `fixed` to `revolute` (with movement limits) to resolve an issue where libuuv_gazebo_ros plugins couldn't detect fixed links in Gazebo.
- Noted that Gazebo doesn't recognize links with fixed joints as standalone links, which seems to cause this issue.

* create sonar gazebo plugin

- implemented from legacy repo (ituauv-uuv-descriptions)

* added base bridge nodes (not ready yet)

* modify package.xml files

* create base_link hydrodynamics plugin

- the values in base_link_ned are robot spesific and belongs to turquoise, we need to change them with taluy's values

* update

* reduce dummy masses

* remove base link ned pub

* update rviz

* update

* add sim deps

* update

* create auv_common_sim and taluy_sim

* remove the `_sim` suffix, call plugins in base

* move worlds and config to 'auv_sim_description'

* update

* fix typo

* improve simulation_mock_node and fix thruster issue (#83)

* add navigation launch file

* add dvl velocity implementation to auv_sim (#86)

* create dvl plugin and bridge

* remove dvl plugin

- velocity and altitude values we get from uuv_simulator plugin is not consistent with the ground truth

* use odometry_gt in dvl bridge

- rotate the velocity from the ground truth by 135 degrees to compensate for the rotation at `dvl_odometry_node`

* add altimeter

- use ray sensor and range plugin from gazebo to mock an altimeter
- invalidate the dvl data and set dvl/isValid to false when altitude < 0.3

* add noise to dvl data

- use the pre-calculated dvl covariances from `auv_localization`

* set gt reference frame to odom

* use reference instead of copy

* create kMinDvlAltitude constant

* use ros timer instead of `rate.sleep()`

* use dvl frame for dvl_altimeter

- rename altimeter to dvl_altimeter to make it easier to understand altimeter is used to mock the dvl in simulation

* revert arg default

* remove legacy variable

- remove the duplicate dvl_rate variable and remove the usage of ros::Rate since now we use ROS timer to do its job

* add uuv_simulator dvl plugin

- use it both for the altitude and the velocity, works as intended

* create another link for sim dvl

* remove position and orientation params

* remove unused parameters in dvl macro

* enhancements to simulation launch files (#85)

* add model.config files (#88)

Co-authored-by: frk781 <mimarlarf@gmail.com>

Squashed commit of the following:

commit 2b6ced176456bdcd87a606976f173f5f8813151a
Author: frk781 <mimarlarf@gmail.com>
Date:   Sat Dec 7 19:11:35 2024 +0300

    added model.config files

* Add props to the pool world (#100)

* Add texture models (gate and torpedo)

* Change prop locations

* fix IMU, Sonar and Bar30 in simulation (#96)

* revert IMU joint type from `revolute` to `fixed`

- add rotation to fix imu plugin values

* fix sonar plugin topic name

- removed namespace at the start of the topic name since it was causing issues
- also change update rate and range according to sensor specifications

* revert Bar30 joint type from `revolute` to `fixed`

* add imu offset to simulation

* fix drift ros param

* rename topics

- renamed it in the code and remapped it to same place.
- this is just to make it more understandable

---------

Co-authored-by: Ozan Hakan Tunca <t.ozanhakan@gmail.com>

* run pre-commit

* update package isolation

* add update rate across files

* add option to run gazebo headless with use_gui (#116)

* create a seperate control config for simulation (#110)

* create a seperate control config for simulation

* remove remapping from sim bridge

* use config_file param to load rosparams

* add pid params for sim

* add additional light

* fix starting pos

* remove unnecessary light, fix buoy pose

---------

Co-authored-by: Ozan Hakan Tunca <t.ozanhakan@gmail.com>
Co-authored-by: meydanoglu <eminmeydanoglu@gmail.com>
Co-authored-by: Sencer Yazici <senceryazici@gmail.com>
Co-authored-by: Ozan Hakan Tunca <155637446+ozanhakantunca@users.noreply.github.com>

File: auv_description/auv_common_descriptions/urdf/actuators/t200.urdf.xacro (robot description, xacro)
@@ -16,6 +16,6 @@
       </collision>
       <inertial>
-        <mass value="0.5"/>
-        <inertia ixx="0.008545" ixy="0.0" ixz="0.0" iyy="0.008545" iyz="0.0" izz="0.0144"/>
+        <mass value="0.001"/>
+        <inertia ixx="0.0000001" ixy="0.0" ixz="0.0" iyy="0.0000001" iyz="0.0" izz="0.0000001"/>
       </inertial>
     </link>
@@ -34,6 +34,6 @@
       </collision>
       <inertial>
-        <mass value="0.5"/>
-        <inertia ixx="0.008545" ixy="0.0" ixz="0.0" iyy="0.008545" iyz="0.0" izz="0.0144"/>
+        <mass value="0.001"/>
+        <inertia ixx="0.0000001" ixy="0.0" ixz="0.0" iyy="0.0000001" iyz="0.0" izz="0.0000001"/>
       </inertial>
     </link>
@@ -49,13 +49,10 @@
       <child link="${name}_propeller_link"/>
       <origin xyz="0 0 0" rpy="0 0 0"/>
-      <limit effort="100" velocity="100"/>
-      <dynamics friction="0.05" damping="0.05"/>
+      <!-- TODO: This breaks the Gazebo Sim -->
+      <!-- <dynamics friction="0.05" damping="0.05" /> -->
+      <!-- TODO: This does not break, but the 100 velocity limit must be evaluated, why limit
+      anyway? -->
+      <!-- <limit effort="100" velocity="100" /> -->
     </joint>
-    <gazebo reference="${name}_propeller_link">
-      <material>Gazebo/Orange</material>
-    </gazebo>
-    <gazebo reference="${name}_link">
-      <material>Gazebo/Orange</material>
-    </gazebo>
   </xacro:macro>
 </robot>

File: auv_description/auv_common_descriptions/urdf/actuators/torpedo.urdf.xacro (robot description, xacro)
@@ -17,6 +17,6 @@
       </collision>
       <inertial>
-        <mass value="0.5"/>
-        <inertia ixx="0.008545" ixy="0.0" ixz="0.0" iyy="0.008545" iyz="0.0" izz="0.0144"/>
+        <mass value="0.00001"/>
+        <inertia ixx="0.000001" ixy="0.0" ixz="0.0" iyy="0.000001" iyz="0.0" izz="0.000001"/>
       </inertial>
     </link>
@@ -35,6 +35,6 @@
       </collision>
       <inertial>
-        <mass value="0.5"/>
-        <inertia ixx="0.008545" ixy="0.0" ixz="0.0" iyy="0.008545" iyz="0.0" izz="0.0144"/>
+        <mass value="0.000001"/>
+        <inertia ixx="0.000001" ixy="0.0" ixz="0.0" iyy="0.000001" iyz="0.0" izz="0.000001"/>
       </inertial>
     </link>

File: auv_description/auv_common_descriptions/urdf/sensors/bar30.urdf.xacro (robot description, xacro)
@@ -16,6 +16,6 @@
       </collision>
       <inertial>
-        <mass value="0.5"/>
-        <inertia ixx="0.008545" ixy="0.0" ixz="0.0" iyy="0.008545" iyz="0.0" izz="0.0144"/>
+        <mass value="0.00001"/>
+        <inertia ixx="0.000001" ixy="0.0" ixz="0.0" iyy="0.000001" iyz="0.0" izz="0.000001"/>
       </inertial>
     </link>

File: auv_description/auv_common_descriptions/urdf/sensors/h2c_hydrophone.urdf.xacro (robot description, xacro)
@@ -16,6 +16,6 @@
       </collision>
       <inertial>
-        <mass value="0.5"/>
-        <inertia ixx="0.008545" ixy="0.0" ixz="0.0" iyy="0.008545" iyz="0.0" izz="0.0144"/>
+        <mass value="0.0001"/>
+        <inertia ixx="0.0000001" ixy="0.0" ixz="0.0" iyy="0.0000001" iyz="0.0" izz="0.0000001"/>
       </inertial>
     </link>

File: auv_description/auv_common_descriptions/urdf/sensors/ping360.urdf.xacro (robot description, xacro)
@@ -17,5 +17,5 @@
       <inertial>
         <mass value="0.5"/>
-        <inertia ixx="0.008545" ixy="0.0" ixz="0.0" iyy="0.008545" iyz="0.0" izz="0.0144"/>
+        <inertia ixx="0.000001" ixy="0.0" ixz="0.0" iyy="0.000001" iyz="0.0" izz="0.000001"/>
       </inertial>
     </link>

File: auv_description/auv_common_descriptions/urdf/sensors/xsens_mti_g710.urdf.xacro (robot description, xacro)
@@ -16,6 +16,6 @@
       </collision>
       <inertial>
-        <mass value="0.5"/>
-        <inertia ixx="0.008545" ixy="0.0" ixz="0.0" iyy="0.008545" iyz="0.0" izz="0.0144"/>
+        <mass value="0.0001"/>
+        <inertia ixx="0.000001" ixy="0.0" ixz="0.0" iyy="0.000001" iyz="0.0" izz="0.000001"/>
       </inertial>
     </link>

File: auv_description/taluy_description/urdf/auv_base.urdf.xacro (robot description, xacro)
@@ -1,4 +1,6 @@
 <?xml version="1.0"?>
 <robot xmlns:xacro="http://www.ros.org/wiki/xacro" name="taluy">
+  <!-- create xacro property -->
+  <xacro:property name="namespace" value="taluy"/>
   <xacro:macro name="taluy_base">
     <xacro:include filename="$(find auv_common_descriptions)/urdf/actuators.urdf.xacro"/>
@@ -6,8 +8,8 @@
     <xacro:include filename="$(find auv_common_descriptions)/urdf/materials.urdf.xacro"/>
     <xacro:arg name="angled_thruster_z_offset" default="-0.01"/>
-    <link name="base_link">
+    <link name="${namespace}/base_link">
       <inertial>
         <origin xyz="0 0 0" rpy="0 0 0"/>
-        <mass value="25.0"/>
+        <mass value="25.37"/>
         <inertia ixx="0.1" iyy="0.1" izz="0.1" ixy="0.01" iyz="0.01" ixz="0.1"/>
       </inertial>
@@ -26,34 +28,34 @@
       </collision>
     </link>
-    <link name="base_link_ned"/>
+    <!-- <link name="${namespace}/base_link_ned" />
     <joint name="base_link_joint" type="fixed">
-      <origin xyz="0 0 0" rpy="${math.pi} 0 0"/>
-      <parent link="base_link_ned"/>
-      <child link="base_link"/>
-    </joint>
-    <xacro:t200_thruster name="thruster_0" parent="base_link" position="0.14250 0.20070 -0.00525" orientation="${pi} 0 ${-pi/2}"/>
-    <xacro:t200_thruster name="thruster_1" parent="base_link" position="0.14250 -0.20070 -0.00525" orientation="${pi} 0 ${pi/2}"/>
-    <xacro:t200_thruster name="thruster_2" parent="base_link" position="-0.14250 0.20070 -0.00525" orientation="${pi} 0 ${-pi/2}"/>
-    <xacro:t200_thruster name="thruster_3" parent="base_link" position="-0.14250 -0.20070 -0.00525" orientation="${pi} 0 ${pi/2}"/>
-    <xacro:t200_thruster name="thruster_4" parent="base_link" position="0.352398 0.216638 $(arg angled_thruster_z_offset)" orientation="${-pi/2} 0 ${-7*pi/4}"/>
-    <xacro:t200_thruster name="thruster_5" parent="base_link" position="0.352398 -0.216638 $(arg angled_thruster_z_offset)" orientation="${pi/2} 0 ${7*pi/4}"/>
-    <xacro:t200_thruster name="thruster_6" parent="base_link" position="-0.352398 0.216638 $(arg angled_thruster_z_offset)" orientation="${-pi/2} 0 ${-pi/4}"/>
-    <xacro:t200_thruster name="thruster_7" parent="base_link" position="-0.352398 -0.216638 $(arg angled_thruster_z_offset)" orientation="${pi/2} 0 ${pi/4}"/>
-    <xacro:wayfinder_dvl name="base_link/dvl" parent="base_link" position="0.2 0 -0.11" orientation="0 0 0"/>
-    <xacro:xsens_mti_g710 name="base_link/imu" parent="base_link" position="-0.199 0 -0.0108" orientation="0 0 ${math.pi}"/>
-    <xacro:h2c_hydrophone name="base_link/hydrophone_0" parent="base_link" position="0.325 0.205 -0.15" orientation="0 0 0"/>
-    <xacro:h2c_hydrophone name="base_link/hydrophone_1" parent="base_link" position="0.325 -0.205 -0.15" orientation="0 0 0"/>
-    <xacro:h2c_hydrophone name="base_link/hydrophone_2" parent="base_link" position="-0.325 0.205 -0.15" orientation="0 0 0"/>
-    <xacro:h2c_hydrophone name="base_link/hydrophone_3" parent="base_link" position="-0.325 -0.205 -0.15" orientation="0 0 0"/>
-    <xacro:ping360 name="base_link/ping360" parent="base_link" position="0.2 0 0.134" orientation="0 0 0"/>
-    <xacro:bar30 name="base_link/external_pressure_sensor" parent="base_link" position="0 0 0.07" orientation="0 0 0"/>
-    <xacro:logitech_c920_camera name="base_link/front_camera" parent="base_link" position="0.35 0 0" orientation="0 0 0"/>
-    <xacro:logitech_c920_camera name="base_link/bottom_camera" parent="base_link" position="0 0 -0.07" orientation="0 ${math.pi/2} ${math.pi/2}"/>
-    <xacro:torpedo name="base_link/left_torpedo" parent="base_link" position="0.2 0.1 -0.11" orientation="0 0 0"/>
-    <xacro:torpedo name="base_link/right_torpedo" parent="base_link" position="0.2 -0.1 -0.11" orientation="0 0 0"/>
-    <xacro:sonar name="base_link/sonar_front" parent="base_link" position="0.38 0.09 0.09" orientation="0 0 0"/>
-    <xacro:sonar name="base_link/sonar_back" parent="base_link" position="-0.42 -0.09 0.09" orientation="0 0 ${math.pi}"/>
-    <xacro:sonar name="base_link/sonar_right" parent="base_link" position="0.02 -0.21 -0.14" orientation="0 0 ${-math.pi/2}"/>
-    <xacro:sonar name="base_link/sonar_left" parent="base_link" position="0.02 0.21 -0.14" orientation="0 0 ${math.pi/2}"/>
+      <origin xyz="0 0 0" rpy="${math.pi} 0 0" />
+      <parent link="${namespace}/base_link_ned" />
+      <child link="${namespace}/base_link" />
+    </joint> -->
+    <xacro:t200_thruster name="${namespace}/thruster_0" parent="${namespace}/base_link" position="0.14250 0.20070 -0.00525" orientation="${pi} 0 ${-pi/2}"/>
+    <xacro:t200_thruster name="${namespace}/thruster_1" parent="${namespace}/base_link" position="0.14250 -0.20070 -0.00525" orientation="${pi} 0 ${pi/2}"/>
+    <xacro:t200_thruster name="${namespace}/thruster_2" parent="${namespace}/base_link" position="-0.14250 0.20070 -0.00525" orientation="${pi} 0 ${-pi/2}"/>
+    <xacro:t200_thruster name="${namespace}/thruster_3" parent="${namespace}/base_link" position="-0.14250 -0.20070 -0.00525" orientation="${pi} 0 ${pi/2}"/>
+    <xacro:t200_thruster name="${namespace}/thruster_4" parent="${namespace}/base_link" position="0.352398 0.216638 $(arg angled_thruster_z_offset)" orientation="${-pi/2} 0 ${-7*pi/4}"/>
+    <xacro:t200_thruster name="${namespace}/thruster_5" parent="${namespace}/base_link" position="0.352398 -0.216638 $(arg angled_thruster_z_offset)" orientation="${pi/2} 0 ${7*pi/4}"/>
+    <xacro:t200_thruster name="${namespace}/thruster_6" parent="${namespace}/base_link" position="-0.352398 0.216638 $(arg angled_thruster_z_offset)" orientation="${-pi/2} 0 ${-pi/4}"/>
+    <xacro:t200_thruster name="${namespace}/thruster_7" parent="${namespace}/base_link" position="-0.352398 -0.216638 $(arg angled_thruster_z_offset)" orientation="${pi/2} 0 ${pi/4}"/>
+    <xacro:wayfinder_dvl name="${namespace}/base_link/dvl" parent="${namespace}/base_link" position="0.2 0 -0.11" orientation="0 0 0"/>
+    <xacro:xsens_mti_g710 name="${namespace}/base_link/imu" parent="${namespace}/base_link" position="-0.199 0 -0.0108" orientation="0 0 ${math.pi}"/>
+    <xacro:h2c_hydrophone name="${namespace}/base_link/hydrophone_0" parent="${namespace}/base_link" position="0.325 0.205 -0.15" orientation="0 0 0"/>
+    <xacro:h2c_hydrophone name="${namespace}/base_link/hydrophone_1" parent="${namespace}/base_link" position="0.325 -0.205 -0.15" orientation="0 0 0"/>
+    <xacro:h2c_hydrophone name="${namespace}/base_link/hydrophone_2" parent="${namespace}/base_link" position="-0.325 0.205 -0.15" orientation="0 0 0"/>
+    <xacro:h2c_hydrophone name="${namespace}/base_link/hydrophone_3" parent="${namespace}/base_link" position="-0.325 -0.205 -0.15" orientation="0 0 0"/>
+    <xacro:ping360 name="${namespace}/base_link/ping360" parent="${namespace}/base_link" position="0.2 0 0.134" orientation="0 0 0"/>
+    <xacro:bar30 name="${namespace}/base_link/external_pressure_sensor" parent="${namespace}/base_link" position="0 0 0.07" orientation="0 0 0"/>
+    <xacro:logitech_c920_camera name="${namespace}/base_link/front_camera" parent="${namespace}/base_link" position="0.35 0 0" orientation="0 0 0"/>
+    <xacro:logitech_c920_camera name="${namespace}/base_link/bottom_camera" parent="${namespace}/base_link" position="0 0 -0.07" orientation="0 ${math.pi/2} ${math.pi/2}"/>
+    <xacro:torpedo name="${namespace}/base_link/left_torpedo" parent="${namespace}/base_link" position="0.2 0.1 -0.11" orientation="0 0 0"/>
+    <xacro:torpedo name="${namespace}/base_link/right_torpedo" parent="${namespace}/base_link" position="0.2 -0.1 -0.11" orientation="0 0 0"/>
+    <xacro:sonar name="${namespace}/base_link/sonar_front" parent="${namespace}/base_link" position="0.38 0.09 0.09" orientation="0 0 0"/>
+    <xacro:sonar name="${namespace}/base_link/sonar_back" parent="${namespace}/base_link" position="-0.42 -0.09 0.09" orientation="0 0 ${math.pi}"/>
+    <xacro:sonar name="${namespace}/base_link/sonar_right" parent="${namespace}/base_link" position="0.02 -0.21 -0.14" orientation="0 0 ${-math.pi/2}"/>
+    <xacro:sonar name="${namespace}/base_link/sonar_left" parent="${namespace}/base_link" position="0.02 0.21 -0.14" orientation="0 0 ${math.pi/2}"/>
     <!-- <link name="base_footprint">
       <inertial>
