Commit message: replace models with boxes, disable shadows(not stable??)

File: auv_description/auv_common_descriptions/urdf/actuators/t200.urdf.xacro (robot description, xacro)
@@ -6,5 +6,5 @@
         <origin xyz="0 0 0" rpy="0 ${pi/2} ${-pi/2}"/>
         <geometry>
-          <mesh filename="package://auv_common_descriptions/meshes/t200/shell.dae" scale="1 1 1"/>
+            <box size="0.1 0.1 0.1"/>
         </geometry>
       </visual>
@@ -12,5 +12,5 @@
         <origin xyz="0 0 0" rpy="0 ${pi/2} ${-pi/2}"/>
         <geometry>
-          <mesh filename="package://auv_common_descriptions/meshes/t200/shell.dae" scale="1 1 1"/>
+            <box size="0.1 0.1 0.1"/>
         </geometry>
       </collision>
@@ -24,5 +24,5 @@
         <origin xyz="0 0 0" rpy="0 ${pi/2} 0"/>
         <geometry>
-          <mesh filename="package://auv_common_descriptions/meshes/t200/propeller.dae" scale="1.0 1.0 1.0"/>
+            <box size="0.1 0.1 0.1"/>
         </geometry>
       </visual>
@@ -30,5 +30,5 @@
         <origin xyz="0 0 0" rpy="0 ${pi/2} 0"/>
         <geometry>
-          <mesh filename="package://auv_common_descriptions/meshes/t200/propeller.dae" scale="1 1 1"/>
+            <box size="0.1 0.1 0.1"/>
         </geometry>
       </collision>

File: auv_description/auv_common_descriptions/urdf/actuators/torpedo_bottom.urdf.xacro (robot description, xacro)
@@ -6,5 +6,5 @@
         <origin xyz="0 0 0" rpy="0 0 0"/>
         <geometry>
-          <mesh filename="package://auv_common_descriptions/meshes/torpedo/torpedo_bottom.dae" scale="0.001 0.001 0.001"/>
+            <box size="0.1 0.1 0.1"/>
         </geometry>
       </visual>
@@ -12,5 +12,5 @@
         <origin xyz="0 0 0" rpy="0 0 0"/>
         <geometry>
-          <mesh filename="package://auv_common_descriptions/meshes/torpedo/torpedo_bottom.dae" scale="0.001 0.001 0.001"/>
+            <box size="0.1 0.1 0.1"/>
         </geometry>
       </collision>

File: auv_description/auv_common_descriptions/urdf/actuators/torpedo_upper.urdf.xacro (robot description, xacro)
@@ -6,5 +6,5 @@
         <origin xyz="0 0 0" rpy="0 0 0"/>
         <geometry>
-          <mesh filename="package://auv_common_descriptions/meshes/torpedo/torpedo_upper.dae" scale="0.001 0.001 0.001"/>
+            <box size="0.1 0.1 0.1"/>
         </geometry>
       </visual>
@@ -12,5 +12,5 @@
         <origin xyz="0 0 0" rpy="0 0 0"/>
         <geometry>
-          <mesh filename="package://auv_common_descriptions/meshes/torpedo/torpedo_upper.dae" scale="0.001 0.001 0.001"/>
+            <box size="0.1 0.1 0.1"/>
         </geometry>
       </collision>

File: auv_description/auv_common_descriptions/urdf/sensors/bar30.urdf.xacro (robot description, xacro)
@@ -6,5 +6,5 @@
         <origin xyz="0 0 0" rpy="0 0 ${math.pi}"/>
         <geometry>
-          <mesh filename="package://auv_common_descriptions/meshes/bar30/bar30.dae" scale="0.001 0.001 0.001"/>
+            <box size="0.1 0.1 0.1"/>
         </geometry>
       </visual>
@@ -12,5 +12,5 @@
         <origin xyz="0 0 0" rpy="0 0 ${math.pi}"/>
         <geometry>
-          <mesh filename="package://auv_common_descriptions/meshes/bar30/bar30.dae" scale="0.001 0.001 0.001"/>
+            <box size="0.1 0.1 0.1"/>
         </geometry>
       </collision>

File: auv_description/auv_common_descriptions/urdf/sensors/ping360.urdf.xacro (robot description, xacro)
@@ -6,5 +6,5 @@
         <origin xyz="0 0 0" rpy="0 0 ${math.pi}"/>
         <geometry>
-          <mesh filename="package://auv_common_descriptions/meshes/ping360/ping360.dae" scale="0.001 0.001 0.001"/>
+            <box size="0.1 0.1 0.1"/>
         </geometry>
       </visual>
@@ -12,5 +12,5 @@
         <origin xyz="0 0 0" rpy="0 0 ${math.pi}"/>
         <geometry>
-          <mesh filename="package://auv_common_descriptions/meshes/ping360/ping360.dae" scale="0.001 0.001 0.001"/>
+            <box size="0.1 0.1 0.1"/>
         </geometry>
       </collision>

File: auv_description/auv_common_descriptions/urdf/sensors/sonar.urdf.xacro (robot description, xacro)
@@ -6,5 +6,5 @@
         <origin xyz="0 0 0" rpy="0 0 0"/>
         <geometry>
-          <mesh filename="package://auv_common_descriptions/meshes/sonar/sonar.dae" scale="0.001 0.001 0.001"/>
+            <box size="0.1 0.1 0.1"/>
         </geometry>
       </visual>
@@ -12,5 +12,5 @@
         <origin xyz="0 0 0" rpy="0 0 0"/>
         <geometry>
-          <mesh filename="package://auv_common_descriptions/meshes/sonar/sonar.dae" scale="0.001 0.001 0.001"/>
+            <box size="0.1 0.1 0.1"/>
         </geometry>
       </collision>

File: auv_description/auv_common_descriptions/urdf/sensors/wayfinder_dvl.urdf.xacro (robot description, xacro)
@@ -6,5 +6,5 @@
         <origin xyz="0 0 0" rpy="${math.pi} 0 0"/>
         <geometry>
-          <mesh filename="package://auv_common_descriptions/meshes/wayfinder_dvl/dvl.dae" scale="0.001 0.001 0.001"/>
+            <box size="0.1 0.1 0.1"/>
           <material name="black"/>
         </geometry>
@@ -13,5 +13,5 @@
         <origin xyz="0 0 0" rpy="${math.pi} 0 0"/>
         <geometry>
-          <mesh filename="package://auv_common_descriptions/meshes/wayfinder_dvl/dvl.dae" scale="0.001 0.001 0.001"/>
+            <box size="0.1 0.1 0.1"/>
           <material name="black"/>
         </geometry>

File: auv_description/auv_common_descriptions/urdf/sensors/xsens_mti_g710.urdf.xacro (robot description, xacro)
@@ -6,5 +6,5 @@
         <origin xyz="0 0 0" rpy="0 0 ${math.pi}"/>
         <geometry>
-          <mesh filename="package://auv_common_descriptions/meshes/xsens_mti_g710/xsens_mti_g710.dae" scale="0.001 0.001 0.001"/>
+            <box size="0.1 0.1 0.1"/>
         </geometry>
       </visual>
@@ -12,5 +12,5 @@
         <origin xyz="0 0 0" rpy="0 0 ${math.pi}"/>
         <geometry>
-          <mesh filename="package://auv_common_descriptions/meshes/xsens_mti_g710/xsens_mti_g710.dae" scale="0.001 0.001 0.001"/>
+            <box size="0.1 0.1 0.1"/>
         </geometry>
       </collision>

File: auv_description/taluy_description/urdf/auv_base.urdf.xacro (robot description, xacro)
@@ -17,5 +17,6 @@
         <origin xyz="0.0 0.0 0.0" rpy="0 0 0"/>
         <geometry>
-          <mesh filename="package://taluy_description/meshes/body/body.stl" scale="1 1 1"/>
+            <box size="0.1 0.1 0.1"/>
+            <!-- <mesh filename="package://taluy_description/meshes/body/body.stl" scale="1 1 1"/> -->
         </geometry>
         <material name="black"/>
