Commit message: delete everything

File: auv_description/auv_common_descriptions/urdf/actuators/ball_dropper.urdf.xacro (robot description, xacro)
@@ -1,3 +1,3 @@
-<?xml version="1.0"?>
+<?xml version='1.0' encoding='UTF-8'?>
 <robot xmlns:xacro="http://ros.org/wiki/xacro" name="ball_dropper">
   <xacro:macro name="ball_dropper" params="name parent position:='0 0 0' orientation:='0 0 0'">
@@ -6,5 +6,5 @@
         <origin xyz="0 0 0" rpy="0 0 0"/>
         <geometry>
-          <mesh filename="package://auv_common_descriptions/meshes/ball_dropper/ball_dropper.dae" scale="0.001 0.001 0.001"/>
+          <box size="0.1 0.1 0.1"/>
         </geometry>
       </visual>
@@ -12,5 +12,5 @@
         <origin xyz="0 0 0" rpy="0 0 0"/>
         <geometry>
-          <mesh filename="package://auv_common_descriptions/meshes/ball_dropper/ball_dropper.dae" scale="0.001 0.001 0.001"/>
+          <box size="0.1 0.1 0.1"/>
         </geometry>
       </collision>

File: auv_description/auv_common_descriptions/urdf/actuators/torpedo_upper.urdf.xacro (robot description, xacro)
@@ -1,3 +1,3 @@
-<?xml version="1.0"?>
+<?xml version='1.0' encoding='UTF-8'?>
 <robot xmlns:xacro="http://ros.org/wiki/xacro" name="torpedo_upper">
   <xacro:macro name="torpedo_upper" params="name parent position:='0 0 0' orientation:='0 0 0'">
@@ -6,5 +6,5 @@
         <origin xyz="0 0 0" rpy="0 0 0"/>
         <geometry>
-          <mesh filename="package://auv_common_descriptions/meshes/torpedo/torpedo_upper.dae" scale="0.001 0.001 0.001"/>
+          <box size="0.1 0.1 0.1"/>
         </geometry>
       </visual>
@@ -12,5 +12,5 @@
         <origin xyz="0 0 0" rpy="0 0 0"/>
         <geometry>
-          <mesh filename="package://auv_common_descriptions/meshes/torpedo/torpedo_upper.dae" scale="0.001 0.001 0.001"/>
+          <box size="0.1 0.1 0.1"/>
         </geometry>
       </collision>

File: auv_description/auv_common_descriptions/urdf/sensors/ping360.urdf.xacro (robot description, xacro)
@@ -1,3 +1,3 @@
-<?xml version="1.0"?>
+<?xml version='1.0' encoding='UTF-8'?>
 <robot xmlns:xacro="http://ros.org/wiki/xacro" name="ping360">
   <xacro:macro name="ping360" params="name parent position:='0 0 0' orientation:='0 0 0'">
@@ -6,5 +6,5 @@
         <origin xyz="0 0 0" rpy="0 0 ${math.pi}"/>
         <geometry>
-          <mesh filename="package://auv_common_descriptions/meshes/ping360/ping360.dae" scale="0.001 0.001 0.001"/>
+          <box size="0.1 0.1 0.1"/>
         </geometry>
       </visual>
@@ -12,5 +12,5 @@
         <origin xyz="0 0 0" rpy="0 0 ${math.pi}"/>
         <geometry>
-          <mesh filename="package://auv_common_descriptions/meshes/ping360/ping360.dae" scale="0.001 0.001 0.001"/>
+          <box size="0.1 0.1 0.1"/>
         </geometry>
       </collision>

File: auv_description/auv_common_descriptions/urdf/sensors/sonar.urdf.xacro (robot description, xacro)
@@ -1,3 +1,3 @@
-<?xml version="1.0"?>
+<?xml version='1.0' encoding='UTF-8'?>
 <robot xmlns:xacro="http://ros.org/wiki/xacro" name="sonar">
   <xacro:macro name="sonar" params="name parent position:='0 0 0' orientation:='0 0 0'">
@@ -6,5 +6,5 @@
         <origin xyz="0 0 0" rpy="0 0 0"/>
         <geometry>
-          <mesh filename="package://auv_common_descriptions/meshes/sonar/sonar.dae" scale="0.001 0.001 0.001"/>
+          <box size="0.1 0.1 0.1"/>
         </geometry>
       </visual>
@@ -12,5 +12,5 @@
         <origin xyz="0 0 0" rpy="0 0 0"/>
         <geometry>
-          <mesh filename="package://auv_common_descriptions/meshes/sonar/sonar.dae" scale="0.001 0.001 0.001"/>
+          <box size="0.1 0.1 0.1"/>
         </geometry>
       </collision>

Commit message: delete all sensor/actuator collisions/visuals and replace taluy base model with a box with (a bit) respect the actual measurements

File: auv_description/auv_common_descriptions/urdf/actuators/ball_dropper.urdf.xacro (robot description, xacro)
@@ -3,16 +3,4 @@
   <xacro:macro name="ball_dropper" params="name parent position:='0 0 0' orientation:='0 0 0'">
     <link name="${name}_link">
-      <visual>
-        <origin xyz="0 0 0" rpy="0 0 0"/>
-        <geometry>
-          <mesh filename="package://auv_common_descriptions/meshes/ball_dropper/ball_dropper.dae" scale="0.001 0.001 0.001"/>
-        </geometry>
-      </visual>
-      <collision name="${name}_collision">
-        <origin xyz="0 0 0" rpy="0 0 0"/>
-        <geometry>
-          <mesh filename="package://auv_common_descriptions/meshes/ball_dropper/ball_dropper.dae" scale="0.001 0.001 0.001"/>
-        </geometry>
-      </collision>
       <inertial>
         <mass value="0.001"/>

File: auv_description/auv_common_descriptions/urdf/actuators/t200.urdf.xacro (robot description, xacro)
@@ -3,16 +3,4 @@
   <xacro:macro name="t200_thruster" params="name parent position:='0 0 0' orientation:='0 0 0'">
     <link name="${name}_link">
-      <visual>
-        <origin xyz="0 0 0" rpy="0 ${pi/2} ${-pi/2}"/>
-        <geometry>
-            <box size="0.1 0.1 0.1"/>
-        </geometry>
-      </visual>
-      <collision name="${name}_collision">
-        <origin xyz="0 0 0" rpy="0 ${pi/2} ${-pi/2}"/>
-        <geometry>
-            <box size="0.1 0.1 0.1"/>
-        </geometry>
-      </collision>
       <inertial>
         <mass value="0.001"/>
@@ -21,16 +9,4 @@
     </link>
     <link name="${name}_propeller_link">
-      <visual>
-        <origin xyz="0 0 0" rpy="0 ${pi/2} 0"/>
-        <geometry>
-            <box size="0.1 0.1 0.1"/>
-        </geometry>
-      </visual>
-      <collision name="${name}_propeller_collision">
-        <origin xyz="0 0 0" rpy="0 ${pi/2} 0"/>
-        <geometry>
-            <box size="0.1 0.1 0.1"/>
-        </geometry>
-      </collision>
       <inertial>
         <mass value="0.001"/>

File: auv_description/auv_common_descriptions/urdf/actuators/torpedo_bottom.urdf.xacro (robot description, xacro)
@@ -3,16 +3,4 @@
   <xacro:macro name="torpedo_bottom" params="name parent position:='0 0 0' orientation:='0 0 0'">
     <link name="${name}_link">
-      <visual>
-        <origin xyz="0 0 0" rpy="0 0 0"/>
-        <geometry>
-            <box size="0.1 0.1 0.1"/>
-        </geometry>
-      </visual>
-      <collision name="${name}_collision">
-        <origin xyz="0 0 0" rpy="0 0 0"/>
-        <geometry>
-            <box size="0.1 0.1 0.1"/>
-        </geometry>
-      </collision>
       <inertial>
         <mass value="0.001"/>

File: auv_description/auv_common_descriptions/urdf/actuators/torpedo_upper.urdf.xacro (robot description, xacro)
@@ -3,16 +3,4 @@
   <xacro:macro name="torpedo_upper" params="name parent position:='0 0 0' orientation:='0 0 0'">
     <link name="${name}_link">
-      <visual>
-        <origin xyz="0 0 0" rpy="0 0 0"/>
-        <geometry>
-            <box size="0.1 0.1 0.1"/>
-        </geometry>
-      </visual>
-      <collision name="${name}_collision">
-        <origin xyz="0 0 0" rpy="0 0 0"/>
-        <geometry>
-            <box size="0.1 0.1 0.1"/>
-        </geometry>
-      </collision>
       <inertial>
         <mass value="0.001"/>

File: auv_description/auv_common_descriptions/urdf/sensors/bar30.urdf.xacro (robot description, xacro)
@@ -3,16 +3,4 @@
   <xacro:macro name="bar30" params="name parent position:='0 0 0' orientation:='0 0 0'">
     <link name="${name}_chasis_link">
-      <visual>
-        <origin xyz="0 0 0" rpy="0 0 ${math.pi}"/>
-        <geometry>
-            <box size="0.1 0.1 0.1"/>
-        </geometry>
-      </visual>
-      <collision name="${name}_collision">
-        <origin xyz="0 0 0" rpy="0 0 ${math.pi}"/>
-        <geometry>
-            <box size="0.1 0.1 0.1"/>
-        </geometry>
-      </collision>
       <inertial>
         <mass value="0.00001"/>

File: auv_description/auv_common_descriptions/urdf/sensors/h2c_hydrophone.urdf.xacro (robot description, xacro)
@@ -3,16 +3,4 @@
   <xacro:macro name="h2c_hydrophone" params="name parent position:='0 0 0' orientation:='0 0 0'">
     <link name="${name}_link">
-      <visual>
-        <origin xyz="0 0 0" rpy="0 0 0"/>
-        <geometry>
-          <cylinder length="0.05695" radius="0.0125"/>
-        </geometry>
-      </visual>
-      <collision name="${name}_collision">
-        <origin xyz="0 0 0" rpy="0 0 0"/>
-        <geometry>
-          <cylinder length="0.05695" radius="0.02489"/>
-        </geometry>
-      </collision>
       <inertial>
         <mass value="0.0001"/>

File: auv_description/auv_common_descriptions/urdf/sensors/logitech_c920_camera.urdf.xacro (robot description, xacro)
@@ -3,22 +3,4 @@
   <xacro:macro name="logitech_c920_camera" params="name parent position:='0 0 0' orientation:='0 0 0'">
     <link name="${name}_link">
-      <visual>
-        <origin xyz="0 0 0" rpy="0 0 ${math.pi}"/>
-        <geometry>
-          <box size="0.02 0.094 0.0433"/>
-          <!-- <mesh
-            filename="package://auv_common_descriptions/meshes/bar30/bar30.dae"
-            scale="0.001 0.001 0.001" /> -->
-        </geometry>
-      </visual>
-      <collision name="${name}_collision">
-        <origin xyz="0 0 0" rpy="0 0 ${math.pi}"/>
-        <geometry>
-          <box size="0.02 0.094 0.0433"/>
-          <!-- <mesh
-            filename="package://auv_common_descriptions/meshes/bar30/bar30.dae"
-            scale="0.001 0.001 0.001" /> -->
-        </geometry>
-      </collision>
       <inertial>
         <mass value="0.162"/>

File: auv_description/auv_common_descriptions/urdf/sensors/ping360.urdf.xacro (robot description, xacro)
@@ -3,16 +3,4 @@
   <xacro:macro name="ping360" params="name parent position:='0 0 0' orientation:='0 0 0'">
     <link name="${name}_mount_link">
-      <visual>
-        <origin xyz="0 0 0" rpy="0 0 ${math.pi}"/>
-        <geometry>
-            <box size="0.1 0.1 0.1"/>
-        </geometry>
-      </visual>
-      <collision name="${name}_collision">
-        <origin xyz="0 0 0" rpy="0 0 ${math.pi}"/>
-        <geometry>
-            <box size="0.1 0.1 0.1"/>
-        </geometry>
-      </collision>
       <inertial>
         <mass value="0.5"/>

File: auv_description/auv_common_descriptions/urdf/sensors/sonar.urdf.xacro (robot description, xacro)
@@ -3,16 +3,4 @@
   <xacro:macro name="sonar" params="name parent position:='0 0 0' orientation:='0 0 0'">
     <link name="${name}_link">
-      <visual>
-        <origin xyz="0 0 0" rpy="0 0 0"/>
-        <geometry>
-            <box size="0.1 0.1 0.1"/>
-        </geometry>
-      </visual>
-      <collision name="${name}_collision">
-        <origin xyz="0 0 0" rpy="0 0 0"/>
-        <geometry>
-            <box size="0.1 0.1 0.1"/>
-        </geometry>
-      </collision>
       <inertial>
         <mass value="0.15"/>

File: auv_description/auv_common_descriptions/urdf/sensors/wayfinder_dvl.urdf.xacro (robot description, xacro)
@@ -3,18 +3,4 @@
   <xacro:macro name="wayfinder_dvl" params="name parent position:='0 0 0' orientation:='0 0 0'">
     <link name="${name}_mount_link">
-      <visual>
-        <origin xyz="0 0 0" rpy="${math.pi} 0 0"/>
-        <geometry>
-            <box size="0.1 0.1 0.1"/>
-          <material name="black"/>
-        </geometry>
-      </visual>
-      <collision name="${name}_collision">
-        <origin xyz="0 0 0" rpy="${math.pi} 0 0"/>
-        <geometry>
-            <box size="0.1 0.1 0.1"/>
-          <material name="black"/>
-        </geometry>
-      </collision>
     </link>
     <link name="${name}_cog">

File: auv_description/auv_common_descriptions/urdf/sensors/xsens_mti_g710.urdf.xacro (robot description, xacro)
@@ -3,16 +3,4 @@
   <xacro:macro name="xsens_mti_g710" params="name parent position:='0 0 0' orientation:='0 0 0'">
     <link name="${name}_link">
-      <visual>
-        <origin xyz="0 0 0" rpy="0 0 ${math.pi}"/>
-        <geometry>
-            <box size="0.1 0.1 0.1"/>
-        </geometry>
-      </visual>
-      <collision name="${name}_collision">
-        <origin xyz="0 0 0" rpy="0 0 ${math.pi}"/>
-        <geometry>
-            <box size="0.1 0.1 0.1"/>
-        </geometry>
-      </collision>
       <inertial>
         <mass value="0.0001"/>

File: auv_description/taluy_description/urdf/auv_base.urdf.xacro (robot description, xacro)
@@ -17,6 +17,5 @@
         <origin xyz="0.0 0.0 0.0" rpy="0 0 0"/>
         <geometry>
-            <box size="0.1 0.1 0.1"/>
-            <!-- <mesh filename="package://taluy_description/meshes/body/body.stl" scale="1 1 1"/> -->
+            <box size="1.5 0.8 0.3"/>
         </geometry>
         <material name="black"/>
@@ -25,5 +24,5 @@
         <origin xyz="0.0 0.0 0.0" rpy="0 0 0"/>
         <geometry>
-          <mesh filename="package://taluy_description/meshes/body/body.stl" scale="1 1 1"/>
+            <box size="1.5 0.8 0.3"/>
         </geometry>
       </collision>

File: auv_sim/auv_sim_description/auv_common_sim_descriptions/urdf/sensors/bar30.urdf.xacro (robot description, xacro)
@@ -8,10 +8,4 @@
         <inertia ixx="0.0000001" ixy="0" ixz="0" iyy="0.0000001" iyz="0" izz="0.0000001"/>
       </inertial>
-      <collision>
-        <geometry>
-          <cylinder length="${0.000001}" radius="${0.000001}"/>
-        </geometry>
-        <origin xyz="0 0 0" rpy="0 ${0.5*pi} 0"/>
-      </collision>
     </link>
     <joint name="${name}_sim_joint" type="revolute">

File: auv_sim/auv_sim_description/auv_common_sim_descriptions/urdf/sensors/wayfinder_dvl.urdf.xacro (robot description, xacro)
@@ -9,10 +9,4 @@
         <inertia ixx="0.000000017" ixy="0" ixz="0" iyy="0.000000017" iyz="0" izz="0.000000017"/>
       </inertial>
-      <collision>
-        <geometry>
-          <cylinder length="${0.000001}" radius="${0.000001}"/>
-        </geometry>
-        <origin xyz="0 0 0" rpy="0 ${0.5*pi} 0"/>
-      </collision>
     </link>
     <joint name="${namespace}/dvl_sonar${index}_joint" type="revolute">
@@ -74,10 +68,4 @@
         <inertia ixx="0.0000001" ixy="0" ixz="0" iyy="0.0000001" iyz="0" izz="0.0000001"/>
       </inertial>
-      <collision>
-        <geometry>
-          <cylinder length="${0.000001}" radius="${0.000001}"/>
-        </geometry>
-        <origin xyz="0 0 0" rpy="0 ${0.5*pi} 0"/>
-      </collision>
     </link>
     <joint name="${name}_sim_joint" type="revolute">

File: auv_sim/auv_sim_description/auv_common_sim_descriptions/urdf/sensors/xsens_mti_g710.urdf.xacro (robot description, xacro)
@@ -8,10 +8,4 @@
         <inertia ixx="0.0000001" ixy="0" ixz="0" iyy="0.0000001" iyz="0" izz="0.0000001"/>
       </inertial>
-      <collision>
-        <geometry>
-          <cylinder length="${0.000001}" radius="${0.000001}"/>
-        </geometry>
-        <origin xyz="0 0 0" rpy="0 ${0.5*pi} 0"/>
-      </collision>
     </link>
     <joint name="${name}_sim_joint" type="revolute">
