Commit message: Improve gazebo performance (#482)
* replace models with boxes, disable shadows(not stable??)

* delete all sensor/actuator collisions/visuals and replace taluy base model with a box with (a bit) respect the actual measurements

* fix space

* format

* add use_models as an argument

* enable taluy model

* one more attempt for shadow disabling (gazebo ;)) + change physics time factors

File: auv_description/auv_common_descriptions/urdf/actuators/ball_dropper.urdf.xacro (robot description, xacro)
@@ -1,22 +1,25 @@
 <?xml version="1.0"?>
 <robot xmlns:xacro="http://ros.org/wiki/xacro" name="ball_dropper">
-  <xacro:macro name="ball_dropper" params="name parent position:='0 0 0' orientation:='0 0 0'">
+  <xacro:macro name="ball_dropper" params="name parent position:='0 0 0' orientation:='0 0 0' use_models:='false'">
     <link name="${name}_link">
-      <visual>
-        <origin xyz="0 0 0" rpy="0 0 0"/>
-        <geometry>
-          <mesh filename="package://auv_common_descriptions/meshes/ball_dropper/ball_dropper.dae" scale="0.001 0.001 0.001"/>
-        </geometry>
-      </visual>
-      <collision name="${name}_collision">
-        <origin xyz="0 0 0" rpy="0 0 0"/>
-        <geometry>
-          <mesh filename="package://auv_common_descriptions/meshes/ball_dropper/ball_dropper.dae" scale="0.001 0.001 0.001"/>
-        </geometry>
-      </collision>
       <inertial>
         <mass value="0.001"/>
         <inertia ixx="0.001" ixy="0.0" ixz="0.0" iyy="0.001" iyz="0.0" izz="0.001"/>
       </inertial>
+      <xacro:if value="${use_models}">
+        <visual>
+          <origin xyz="0 0 0" rpy="0 0 0"/>
+          <geometry>
+            <mesh filename="package://auv_common_descriptions/meshes/ball_dropper/ball_dropper.dae" scale="0.001 0.001 0.001"/>
+          </geometry>
+          <material name="black"/>
+        </visual>
+        <collision>
+          <origin xyz="0 0 0" rpy="0 0 0"/>
+          <geometry>
+            <mesh filename="package://auv_common_descriptions/meshes/ball_dropper/ball_dropper.dae" scale="0.001 0.001 0.001"/>
+          </geometry>
+        </collision>
+      </xacro:if>
     </link>
     <joint name="${name}_joint" type="fixed">

File: auv_description/auv_common_descriptions/urdf/actuators/t200.urdf.xacro (robot description, xacro)
@@ -1,36 +1,40 @@
 <?xml version="1.0"?>
 <robot xmlns:xacro="http://ros.org/wiki/xacro" name="t200_thruster">
-  <xacro:macro name="t200_thruster" params="name parent position:='0 0 0' orientation:='0 0 0'">
+  <xacro:macro name="t200_thruster" params="name parent position:='0 0 0' orientation:='0 0 0' use_models:='false'">
     <link name="${name}_link">
-      <visual>
-        <origin xyz="0 0 0" rpy="0 ${pi/2} ${-pi/2}"/>
-        <geometry>
-          <mesh filename="package://auv_common_descriptions/meshes/t200/shell.dae" scale="1 1 1"/>
-        </geometry>
-      </visual>
-      <collision name="${name}_collision">
-        <origin xyz="0 0 0" rpy="0 ${pi/2} ${-pi/2}"/>
-        <geometry>
-          <mesh filename="package://auv_common_descriptions/meshes/t200/shell.dae" scale="1 1 1"/>
-        </geometry>
-      </collision>
       <inertial>
         <mass value="0.001"/>
         <inertia ixx="0.0000001" ixy="0.0" ixz="0.0" iyy="0.0000001" iyz="0.0" izz="0.0000001"/>
       </inertial>
+      <xacro:if value="${use_models}">
+        <visual>
+          <origin xyz="0 0 0" rpy="0 ${pi/2} ${-pi/2}"/>
+          <geometry>
+            <mesh filename="package://auv_common_descriptions/meshes/t200/shell.dae" scale="1 1 1"/>
+          </geometry>
+        </visual>
+        <collision name="${name}_collision">
+          <origin xyz="0 0 0" rpy="0 ${pi/2} ${-pi/2}"/>
+          <geometry>
+            <mesh filename="package://auv_common_descriptions/meshes/t200/shell.dae" scale="1 1 1"/>
+          </geometry>
+        </collision>
+      </xacro:if>
     </link>
     <link name="${name}_propeller_link">
-      <visual>
-        <origin xyz="0 0 0" rpy="0 ${pi/2} 0"/>
-        <geometry>
-          <mesh filename="package://auv_common_descriptions/meshes/t200/propeller.dae" scale="1.0 1.0 1.0"/>
-        </geometry>
-      </visual>
-      <collision name="${name}_propeller_collision">
-        <origin xyz="0 0 0" rpy="0 ${pi/2} 0"/>
-        <geometry>
-          <mesh filename="package://auv_common_descriptions/meshes/t200/propeller.dae" scale="1 1 1"/>
-        </geometry>
-      </collision>
+      <xacro:if value="${use_models}">
+        <visual>
+          <origin xyz="0 0 0" rpy="0 ${pi/2} 0"/>
+          <geometry>
+            <mesh filename="package://auv_common_descriptions/meshes/t200/propeller.dae" scale="1.0 1.0 1.0"/>
+          </geometry>
+        </visual>
+        <collision name="${name}_propeller_collision">
+          <origin xyz="0 0 0" rpy="0 ${pi/2} 0"/>
+          <geometry>
+            <mesh filename="package://auv_common_descriptions/meshes/t200/propeller.dae" scale="1 1 1"/>
+          </geometry>
+        </collision>
+      </xacro:if>
       <inertial>
         <mass value="0.001"/>

File: auv_description/auv_common_descriptions/urdf/actuators/torpedo_bottom.urdf.xacro (robot description, xacro)
@@ -1,22 +1,24 @@
 <?xml version="1.0"?>
 <robot xmlns:xacro="http://ros.org/wiki/xacro" name="torpedo_bottom">
-  <xacro:macro name="torpedo_bottom" params="name parent position:='0 0 0' orientation:='0 0 0'">
+  <xacro:macro name="torpedo_bottom" params="name parent position:='0 0 0' orientation:='0 0 0' use_models:='false'">
     <link name="${name}_link">
-      <visual>
-        <origin xyz="0 0 0" rpy="0 0 0"/>
-        <geometry>
-          <mesh filename="package://auv_common_descriptions/meshes/torpedo/torpedo_bottom.dae" scale="0.001 0.001 0.001"/>
-        </geometry>
-      </visual>
-      <collision name="${name}_collision">
-        <origin xyz="0 0 0" rpy="0 0 0"/>
-        <geometry>
-          <mesh filename="package://auv_common_descriptions/meshes/torpedo/torpedo_bottom.dae" scale="0.001 0.001 0.001"/>
-        </geometry>
-      </collision>
       <inertial>
         <mass value="0.001"/>
         <inertia ixx="0.001" ixy="0.0" ixz="0.0" iyy="0.001" iyz="0.0" izz="0.001"/>
       </inertial>
+      <xacro:if value="${use_models}">
+        <visual>
+          <origin xyz="0 0 0" rpy="0 0 0"/>
+          <geometry>
+            <mesh filename="package://auv_common_descriptions/meshes/torpedo/torpedo_bottom.dae" scale="0.001 0.001 0.001"/>
+          </geometry>
+        </visual>
+        <collision name="${name}_collision">
+          <origin xyz="0 0 0" rpy="0 0 0"/>
+          <geometry>
+            <mesh filename="package://auv_common_descriptions/meshes/torpedo/torpedo_bottom.dae" scale="0.001 0.001 0.001"/>
+          </geometry>
+        </collision>
+      </xacro:if>
     </link>
     <joint name="${name}_joint" type="fixed">

File: auv_description/auv_common_descriptions/urdf/actuators/torpedo_upper.urdf.xacro (robot description, xacro)
@@ -1,22 +1,24 @@
 <?xml version="1.0"?>
 <robot xmlns:xacro="http://ros.org/wiki/xacro" name="torpedo_upper">
-  <xacro:macro name="torpedo_upper" params="name parent position:='0 0 0' orientation:='0 0 0'">
+  <xacro:macro name="torpedo_upper" params="name parent position:='0 0 0' orientation:='0 0 0' use_models:='false'">
     <link name="${name}_link">
-      <visual>
-        <origin xyz="0 0 0" rpy="0 0 0"/>
-        <geometry>
-          <mesh filename="package://auv_common_descriptions/meshes/torpedo/torpedo_upper.dae" scale="0.001 0.001 0.001"/>
-        </geometry>
-      </visual>
-      <collision name="${name}_collision">
-        <origin xyz="0 0 0" rpy="0 0 0"/>
-        <geometry>
-          <mesh filename="package://auv_common_descriptions/meshes/torpedo/torpedo_upper.dae" scale="0.001 0.001 0.001"/>
-        </geometry>
-      </collision>
       <inertial>
         <mass value="0.001"/>
         <inertia ixx="0.001" ixy="0.0" ixz="0.0" iyy="0.001" iyz="0.0" izz="0.001"/>
       </inertial>
+      <xacro:if value="${use_models}">
+        <visual>
+          <origin xyz="0 0 0" rpy="0 0 0"/>
+          <geometry>
+            <mesh filename="package://auv_common_descriptions/meshes/torpedo/torpedo_upper.dae" scale="0.001 0.001 0.001"/>
+          </geometry>
+        </visual>
+        <collision name="${name}_collision">
+          <origin xyz="0 0 0" rpy="0 0 0"/>
+          <geometry>
+            <mesh filename="package://auv_common_descriptions/meshes/torpedo/torpedo_upper.dae" scale="0.001 0.001 0.001"/>
+          </geometry>
+        </collision>
+      </xacro:if>
     </link>
     <joint name="${name}_joint" type="fixed">

File: auv_description/auv_common_descriptions/urdf/sensors/bar30.urdf.xacro (robot description, xacro)
@@ -1,22 +1,24 @@
 <?xml version="1.0"?>
 <robot xmlns:xacro="http://ros.org/wiki/xacro" name="bar30">
-  <xacro:macro name="bar30" params="name parent position:='0 0 0' orientation:='0 0 0'">
+  <xacro:macro name="bar30" params="name parent position:='0 0 0' orientation:='0 0 0' use_models:='false'">
     <link name="${name}_chasis_link">
-      <visual>
-        <origin xyz="0 0 0" rpy="0 0 ${math.pi}"/>
-        <geometry>
-          <mesh filename="package://auv_common_descriptions/meshes/bar30/bar30.dae" scale="0.001 0.001 0.001"/>
-        </geometry>
-      </visual>
-      <collision name="${name}_collision">
-        <origin xyz="0 0 0" rpy="0 0 ${math.pi}"/>
-        <geometry>
-          <mesh filename="package://auv_common_descriptions/meshes/bar30/bar30.dae" scale="0.001 0.001 0.001"/>
-        </geometry>
-      </collision>
       <inertial>
         <mass value="0.00001"/>
         <inertia ixx="0.000001" ixy="0.0" ixz="0.0" iyy="0.000001" iyz="0.0" izz="0.000001"/>
       </inertial>
+      <xacro:if value="${use_models}">
+        <visual>
+          <origin xyz="0 0 0" rpy="0 0 ${math.pi}"/>
+          <geometry>
+            <mesh filename="package://auv_common_descriptions/meshes/bar30/bar30.dae" scale="0.001 0.001 0.001"/>
+          </geometry>
+        </visual>
+        <collision name="${name}_collision">
+          <origin xyz="0 0 0" rpy="0 0 ${math.pi}"/>
+          <geometry>
+            <mesh filename="package://auv_common_descriptions/meshes/bar30/bar30.dae" scale="0.001 0.001 0.001"/>
+          </geometry>
+        </collision>
+      </xacro:if>
     </link>
     <link name="${name}_link"/>

File: auv_description/auv_common_descriptions/urdf/sensors/h2c_hydrophone.urdf.xacro (robot description, xacro)
@@ -1,18 +1,20 @@
 <?xml version="1.0"?>
 <robot xmlns:xacro="http://ros.org/wiki/xacro" name="h2c_hydrophone">
-  <xacro:macro name="h2c_hydrophone" params="name parent position:='0 0 0' orientation:='0 0 0'">
+  <xacro:macro name="h2c_hydrophone" params="name parent position:='0 0 0' orientation:='0 0 0' use_models:='false'">
     <link name="${name}_link">
-      <visual>
-        <origin xyz="0 0 0" rpy="0 0 0"/>
-        <geometry>
-          <cylinder length="0.05695" radius="0.0125"/>
-        </geometry>
-      </visual>
-      <collision name="${name}_collision">
-        <origin xyz="0 0 0" rpy="0 0 0"/>
-        <geometry>
-          <cylinder length="0.05695" radius="0.02489"/>
-        </geometry>
-      </collision>
+      <xacro:if value="${use_models}">
+        <visual>
+          <origin xyz="0 0 0" rpy="0 0 0"/>
+          <geometry>
+            <cylinder length="0.05695" radius="0.0125"/>
+          </geometry>
+        </visual>
+        <collision name="${name}_collision">
+          <origin xyz="0 0 0" rpy="0 0 0"/>
+          <geometry>
+            <cylinder length="0.05695" radius="0.02489"/>
+          </geometry>
+        </collision>
+      </xacro:if>
       <inertial>
         <mass value="0.0001"/>

File: auv_description/auv_common_descriptions/urdf/sensors/logitech_c920_camera.urdf.xacro (robot description, xacro)
@@ -1,24 +1,26 @@
 <?xml version="1.0"?>
 <robot xmlns:xacro="http://ros.org/wiki/xacro" name="logitech_c920_camera">
-  <xacro:macro name="logitech_c920_camera" params="name parent position:='0 0 0' orientation:='0 0 0'">
+  <xacro:macro name="logitech_c920_camera" params="name parent position:='0 0 0' orientation:='0 0 0' use_models:='false'">
     <link name="${name}_link">
-      <visual>
-        <origin xyz="0 0 0" rpy="0 0 ${math.pi}"/>
-        <geometry>
-          <box size="0.02 0.094 0.0433"/>
-          <!-- <mesh
+      <xacro:if value="${use_models}">
+        <visual>
+          <origin xyz="0 0 0" rpy="0 0 ${math.pi}"/>
+          <geometry>
+            <box size="0.02 0.094 0.0433"/>
+            <!-- <mesh
             filename="package://auv_common_descriptions/meshes/bar30/bar30.dae"
             scale="0.001 0.001 0.001" /> -->
-        </geometry>
-      </visual>
-      <collision name="${name}_collision">
-        <origin xyz="0 0 0" rpy="0 0 ${math.pi}"/>
-        <geometry>
-          <box size="0.02 0.094 0.0433"/>
-          <!-- <mesh
+          </geometry>
+        </visual>
+        <collision name="${name}_collision">
+          <origin xyz="0 0 0" rpy="0 0 ${math.pi}"/>
+          <geometry>
+            <box size="0.02 0.094 0.0433"/>
+            <!-- <mesh
             filename="package://auv_common_descriptions/meshes/bar30/bar30.dae"
             scale="0.001 0.001 0.001" /> -->
-        </geometry>
-      </collision>
+          </geometry>
+        </collision>
+      </xacro:if>
       <inertial>
         <mass value="0.162"/>

File: auv_description/auv_common_descriptions/urdf/sensors/ping360.urdf.xacro (robot description, xacro)
@@ -1,22 +1,24 @@
 <?xml version="1.0"?>
 <robot xmlns:xacro="http://ros.org/wiki/xacro" name="ping360">
-  <xacro:macro name="ping360" params="name parent position:='0 0 0' orientation:='0 0 0'">
+  <xacro:macro name="ping360" params="name parent position:='0 0 0' orientation:='0 0 0' use_models:='false'">
     <link name="${name}_mount_link">
-      <visual>
-        <origin xyz="0 0 0" rpy="0 0 ${math.pi}"/>
-        <geometry>
-          <mesh filename="package://auv_common_descriptions/meshes/ping360/ping360.dae" scale="0.001 0.001 0.001"/>
-        </geometry>
-      </visual>
-      <collision name="${name}_collision">
-        <origin xyz="0 0 0" rpy="0 0 ${math.pi}"/>
-        <geometry>
-          <mesh filename="package://auv_common_descriptions/meshes/ping360/ping360.dae" scale="0.001 0.001 0.001"/>
-        </geometry>
-      </collision>
       <inertial>
         <mass value="0.5"/>
         <inertia ixx="0.000001" ixy="0.0" ixz="0.0" iyy="0.000001" iyz="0.0" izz="0.000001"/>
       </inertial>
+      <xacro:if value="${use_models}">
+        <visual>
+          <origin xyz="0 0 0" rpy="0 0 ${math.pi}"/>
+          <geometry>
+            <mesh filename="package://auv_common_descriptions/meshes/ping360/ping360.dae" scale="0.001 0.001 0.001"/>
+          </geometry>
+        </visual>
+        <collision name="${name}_collision">
+          <origin xyz="0 0 0" rpy="0 0 ${math.pi}"/>
+          <geometry>
+            <mesh filename="package://auv_common_descriptions/meshes/ping360/ping360.dae" scale="0.001 0.001 0.001"/>
+          </geometry>
+        </collision>
+      </xacro:if>
     </link>
     <link name="${name}_link"/>

File: auv_description/auv_common_descriptions/urdf/sensors/sonar.urdf.xacro (robot description, xacro)
@@ -1,22 +1,24 @@
 <?xml version="1.0"?>
 <robot xmlns:xacro="http://ros.org/wiki/xacro" name="sonar">
-  <xacro:macro name="sonar" params="name parent position:='0 0 0' orientation:='0 0 0'">
+  <xacro:macro name="sonar" params="name parent position:='0 0 0' orientation:='0 0 0' use_models:='false'">
     <link name="${name}_link">
-      <visual>
-        <origin xyz="0 0 0" rpy="0 0 0"/>
-        <geometry>
-          <mesh filename="package://auv_common_descriptions/meshes/sonar/sonar.dae" scale="0.001 0.001 0.001"/>
-        </geometry>
-      </visual>
-      <collision name="${name}_collision">
-        <origin xyz="0 0 0" rpy="0 0 0"/>
-        <geometry>
-          <mesh filename="package://auv_common_descriptions/meshes/sonar/sonar.dae" scale="0.001 0.001 0.001"/>
-        </geometry>
-      </collision>
       <inertial>
         <mass value="0.15"/>
         <inertia ixx="0.001" ixy="0.0" ixz="0.0" iyy="0.001" iyz="0.0" izz="0.001"/>
       </inertial>
+      <xacro:if value="${use_models}">
+        <visual>
+          <origin xyz="0 0 0" rpy="0 0 0"/>
+          <geometry>
+            <mesh filename="package://auv_common_descriptions/meshes/sonar/sonar.dae" scale="0.001 0.001 0.001"/>
+          </geometry>
+        </visual>
+        <collision name="${name}_collision">
+          <origin xyz="0 0 0" rpy="0 0 0"/>
+          <geometry>
+            <mesh filename="package://auv_common_descriptions/meshes/sonar/sonar.dae" scale="0.001 0.001 0.001"/>
+          </geometry>
+        </collision>
+      </xacro:if>
     </link>
     <joint name="${name}_joint" type="fixed">

File: auv_description/auv_common_descriptions/urdf/sensors/wayfinder_dvl.urdf.xacro (robot description, xacro)
@@ -1,20 +1,22 @@
 <?xml version="1.0"?>
 <robot xmlns:xacro="http://ros.org/wiki/xacro" name="wayfinder_dvl">
-  <xacro:macro name="wayfinder_dvl" params="name parent position:='0 0 0' orientation:='0 0 0'">
+  <xacro:macro name="wayfinder_dvl" params="name parent position:='0 0 0' orientation:='0 0 0' use_models:='false'">
     <link name="${name}_mount_link">
-      <visual>
-        <origin xyz="0 0 0" rpy="${math.pi} 0 0"/>
-        <geometry>
-          <mesh filename="package://auv_common_descriptions/meshes/wayfinder_dvl/dvl.dae" scale="0.001 0.001 0.001"/>
-          <material name="black"/>
-        </geometry>
-      </visual>
-      <collision name="${name}_collision">
-        <origin xyz="0 0 0" rpy="${math.pi} 0 0"/>
-        <geometry>
-          <mesh filename="package://auv_common_descriptions/meshes/wayfinder_dvl/dvl.dae" scale="0.001 0.001 0.001"/>
-          <material name="black"/>
-        </geometry>
-      </collision>
+      <xacro:if value="${use_models}">
+        <visual>
+          <origin xyz="0 0 0" rpy="${math.pi} 0 0"/>
+          <geometry>
+            <mesh filename="package://auv_common_descriptions/meshes/wayfinder_dvl/dvl.dae" scale="0.001 0.001 0.001"/>
+            <material name="black"/>
+          </geometry>
+        </visual>
+        <collision name="${name}_collision">
+          <origin xyz="0 0 0" rpy="${math.pi} 0 0"/>
+          <geometry>
+            <mesh filename="package://auv_common_descriptions/meshes/wayfinder_dvl/dvl.dae" scale="0.001 0.001 0.001"/>
+            <material name="black"/>
+          </geometry>
+        </collision>
+      </xacro:if>
     </link>
     <link name="${name}_cog">

File: auv_description/auv_common_descriptions/urdf/sensors/xsens_mti_g710.urdf.xacro (robot description, xacro)
@@ -1,22 +1,24 @@
 <?xml version="1.0"?>
 <robot xmlns:xacro="http://ros.org/wiki/xacro" name="xsens_mti_g710">
-  <xacro:macro name="xsens_mti_g710" params="name parent position:='0 0 0' orientation:='0 0 0'">
+  <xacro:macro name="xsens_mti_g710" params="name parent position:='0 0 0' orientation:='0 0 0' use_models:='false'">
     <link name="${name}_link">
-      <visual>
-        <origin xyz="0 0 0" rpy="0 0 ${math.pi}"/>
-        <geometry>
-          <mesh filename="package://auv_common_descriptions/meshes/xsens_mti_g710/xsens_mti_g710.dae" scale="0.001 0.001 0.001"/>
-        </geometry>
-      </visual>
-      <collision name="${name}_collision">
-        <origin xyz="0 0 0" rpy="0 0 ${math.pi}"/>
-        <geometry>
-          <mesh filename="package://auv_common_descriptions/meshes/xsens_mti_g710/xsens_mti_g710.dae" scale="0.001 0.001 0.001"/>
-        </geometry>
-      </collision>
       <inertial>
         <mass value="0.0001"/>
         <inertia ixx="0.000001" ixy="0.0" ixz="0.0" iyy="0.000001" iyz="0.0" izz="0.000001"/>
       </inertial>
+      <xacro:if value="${use_models}">
+        <visual>
+          <origin xyz="0 0 0" rpy="0 0 ${math.pi}"/>
+          <geometry>
+            <mesh filename="package://auv_common_descriptions/meshes/xsens_mti_g710/xsens_mti_g710.dae" scale="0.001 0.001 0.001"/>
+          </geometry>
+        </visual>
+        <collision name="${name}_collision">
+          <origin xyz="0 0 0" rpy="0 0 ${math.pi}"/>
+          <geometry>
+            <mesh filename="package://auv_common_descriptions/meshes/xsens_mti_g710/xsens_mti_g710.dae" scale="0.001 0.001 0.001"/>
+          </geometry>
+        </collision>
+      </xacro:if>
     </link>
     <joint name="${name}_joint" type="fixed">
