Commit message: Improve gazebo performance (#482)
* replace models with boxes, disable shadows(not stable??)

* delete all sensor/actuator collisions/visuals and replace taluy base model with a box with (a bit) respect the actual measurements

* fix space

* format

* add use_models as an argument

* enable taluy model

* one more attempt for shadow disabling (gazebo ;)) + change physics time factors

File: auv_description/taluy_description/urdf/auv_base.urdf.xacro (robot description, xacro)
@@ -3,9 +3,10 @@
   <!-- create xacro property -->
   <xacro:property name="namespace" value="taluy"/>
-  <xacro:macro name="taluy_base">
+  <xacro:macro name="taluy_base" params="use_models">
     <xacro:include filename="$(find auv_common_descriptions)/urdf/actuators.urdf.xacro"/>
     <xacro:include filename="$(find auv_common_descriptions)/urdf/sensors.urdf.xacro"/>
     <xacro:include filename="$(find auv_common_descriptions)/urdf/materials.urdf.xacro"/>
     <xacro:arg name="angled_thruster_z_offset" default="-0.01"/>
+    <xacro:arg name="use_models" default="${use_models}"/>
     <link name="${namespace}/base_link">
       <inertial>
@@ -28,51 +29,63 @@
       </collision>
     </link>
-    <!-- <link name="${namespace}/base_link_ned" />
-    <joint name="base_link_joint" type="fixed">
-      <origin xyz="0 0 0" rpy="${math.pi} 0 0" />
-      <parent link="${namespace}/base_link_ned" />
-      <child link="${namespace}/base_link" />
-    </joint> -->
-    <xacro:t200_thruster name="${namespace}/thruster_0" parent="${namespace}/base_link" position="0.15895 0.20070 -0.00525" orientation="${pi} 0 ${-pi/2}"/>
-    <xacro:t200_thruster name="${namespace}/thruster_1" parent="${namespace}/base_link" position="0.15895 -0.20070 -0.00525" orientation="${pi} 0 ${pi/2}"/>
-    <xacro:t200_thruster name="${namespace}/thruster_2" parent="${namespace}/base_link" position="-0.15895 0.20070 -0.00525" orientation="${pi} 0 ${-pi/2}"/>
-    <xacro:t200_thruster name="${namespace}/thruster_3" parent="${namespace}/base_link" position="-0.15895 -0.20070 -0.00525" orientation="${pi} 0 ${pi/2}"/>
-    <xacro:t200_thruster name="${namespace}/thruster_4" parent="${namespace}/base_link" position="0.352398 0.216638 $(arg angled_thruster_z_offset)" orientation="${-pi/2} 0 ${-7*pi/4}"/>
-    <xacro:t200_thruster name="${namespace}/thruster_5" parent="${namespace}/base_link" position="0.352398 -0.216638 $(arg angled_thruster_z_offset)" orientation="${pi/2} 0 ${7*pi/4}"/>
-    <xacro:t200_thruster name="${namespace}/thruster_6" parent="${namespace}/base_link" position="-0.352398 0.216638 $(arg angled_thruster_z_offset)" orientation="${-pi/2} 0 ${-pi/4}"/>
-    <xacro:t200_thruster name="${namespace}/thruster_7" parent="${namespace}/base_link" position="-0.352398 -0.216638 $(arg angled_thruster_z_offset)" orientation="${pi/2} 0 ${pi/4}"/>
-    <xacro:wayfinder_dvl name="${namespace}/base_link/dvl" parent="${namespace}/base_link" position="0.2 0 -0.11" orientation="0 0 0"/>
-    <xacro:xsens_mti_g710 name="${namespace}/base_link/imu" parent="${namespace}/base_link" position="-0.162 0 -0.0108" orientation="0 0 ${math.pi}"/>
-    <xacro:xsens_mti_g710 name="${namespace}/base_link/imu_expansion" parent="${namespace}/base_link" position="-0.282 -0.1 -0.0108" orientation="0 0 ${math.pi}"/>
-    <xacro:h2c_hydrophone name="${namespace}/base_link/hydrophone_0" parent="${namespace}/base_link" position="0.315 0.1675 0.1715" orientation="0 0 0"/>
-    <xacro:h2c_hydrophone name="${namespace}/base_link/hydrophone_1" parent="${namespace}/base_link" position="0.315 -0.1675 0.1715" orientation="0 0 0"/>
-    <xacro:h2c_hydrophone name="${namespace}/base_link/hydrophone_2" parent="${namespace}/base_link" position="-0.315 0.1675 0.1715" orientation="0 0 0"/>
-    <xacro:h2c_hydrophone name="${namespace}/base_link/hydrophone_3" parent="${namespace}/base_link" position="-0.315 -0.1675 0.1715" orientation="0 0 0"/>
-    <xacro:ping360 name="${namespace}/base_link/ping360" parent="${namespace}/base_link" position="0.2 0 0.134" orientation="0 0 0"/>
-    <xacro:bar30 name="${namespace}/base_link/external_pressure_sensor" parent="${namespace}/base_link" position="0 0 0.079" orientation="0 0 0"/>
-    <xacro:logitech_c920_camera name="${namespace}/base_link/front_camera" parent="${namespace}/base_link" position="0.40125 0 0" orientation="0 0 0"/>
-    <xacro:logitech_c920_camera name="${namespace}/base_link/bottom_camera" parent="${namespace}/base_link" position="0 0 -0.07" orientation="0 ${math.pi/2} ${-math.pi/2}"/>
-    <xacro:torpedo_upper name="${namespace}/base_link/torpedo_upper" parent="${namespace}/base_link" position="0.4057 -0.1038 -0.049" orientation="0 0 0"/>
-    <xacro:torpedo_bottom name="${namespace}/base_link/torpedo_bottom" parent="${namespace}/base_link" position="0.4057 -0.1038 -0.084" orientation="0 0 0"/>
-    <xacro:sonar name="${namespace}/base_link/sonar_front" parent="${namespace}/base_link" position="0.38 0.09 0.09" orientation="0 0 0"/>
-    <xacro:sonar name="${namespace}/base_link/sonar_back" parent="${namespace}/base_link" position="-0.42 -0.09 0.09" orientation="0 0 ${math.pi}"/>
-    <xacro:sonar name="${namespace}/base_link/sonar_right" parent="${namespace}/base_link" position="0.02 -0.21 -0.14" orientation="0 0 ${-math.pi/2}"/>
-    <xacro:sonar name="${namespace}/base_link/sonar_left" parent="${namespace}/base_link" position="0.02 0.21 -0.14" orientation="0 0 ${math.pi/2}"/>
-    <!-- 0.0931 -->
-    <xacro:ball_dropper name="${namespace}/base_link/ball_dropper" parent="${namespace}/base_link" position="0.1004 0.0745 -0.1953" orientation="0 0 0"/>
-    <xacro:realsense_d435 name="${namespace}/camera" parent="${namespace}/base_link" position="-0.35 0 0" orientation="0 0 ${math.pi}"/>
-    <!-- <link name="base_footprint">
-      <inertial>
-        <origin xyz="0 0 0" rpy="0 0 0" />
-        <mass value="15.0" />
-        <inertia ixx="39.351246" iyy="103.261717" izz="127.702526" ixy="-5e-06" iyz="6e-06"
-          ixz="4.403436" />
-      </inertial>
-    </link>
-    <joint name="base_link_joint" type="fixed">
-      <origin xyz="0 0 ${-base_z_offsett + 0.06 - draft}" rpy="0 0 0" />
-      <parent link="base_footprint" />
-      <child link="base_link" />
-    </joint> -->
+    <!-- Thrusters -->
+    <xacro:t200_thruster name="${namespace}/thruster_0" parent="${namespace}/base_link" position="0.15895 0.20070 -0.00525" orientation="${pi} 0 ${-pi/2}" use_models="$(arg use_models)"/>
+    <xacro:t200_thruster name="${namespace}/thruster_1" parent="${namespace}/base_link" position="0.15895 -0.20070 -0.00525" orientation="${pi} 0 ${pi/2}" use_models="$(arg use_models)"/>
+    <xacro:t200_thruster name="${namespace}/thruster_2" parent="${namespace}/base_link" position="-0.15895 0.20070 -0.00525" orientation="${pi} 0 ${-pi/2}" use_models="$(arg use_models)"/>
+    <xacro:t200_thruster name="${namespace}/thruster_3" parent="${namespace}/base_link" position="-0.15895 -0.20070 -0.00525" orientation="${pi} 0 ${pi/2}" use_models="$(arg use_models)"/>
+    <xacro:t200_thruster
+      name="${namespace}/thruster_4"
+      parent="${namespace}/base_link"
+      position="0.352398 0.216638 $(arg angled_thruster_z_offset)"
+      orientation="${-pi/2} 0 ${-7*pi/4}"
+      use_models="$(arg use_models)"
+    />
+    <xacro:t200_thruster
+      name="${namespace}/thruster_5"
+      parent="${namespace}/base_link"
+      position="0.352398 -0.216638 $(arg angled_thruster_z_offset)"
+      orientation="${pi/2} 0 ${7*pi/4}"
+      use_models="$(arg use_models)"
+    />
+    <xacro:t200_thruster
+      name="${namespace}/thruster_6"
+      parent="${namespace}/base_link"
+      position="-0.352398 0.216638 $(arg angled_thruster_z_offset)"
+      orientation="${-pi/2} 0 ${-pi/4}"
+      use_models="$(arg use_models)"
+    />
+    <xacro:t200_thruster
+      name="${namespace}/thruster_7"
+      parent="${namespace}/base_link"
+      position="-0.352398 -0.216638 $(arg angled_thruster_z_offset)"
+      orientation="${pi/2} 0 ${pi/4}"
+      use_models="$(arg use_models)"
+    />
+    <!-- Sensors -->
+    <xacro:wayfinder_dvl name="${namespace}/base_link/dvl" parent="${namespace}/base_link" position="0.2 0 -0.11" orientation="0 0 0" use_models="$(arg use_models)"/>
+    <xacro:xsens_mti_g710 name="${namespace}/base_link/imu" parent="${namespace}/base_link" position="-0.162 0 -0.0108" orientation="0 0 ${math.pi}" use_models="$(arg use_models)"/>
+    <xacro:xsens_mti_g710 name="${namespace}/base_link/imu_expansion" parent="${namespace}/base_link" position="-0.282 -0.1 -0.0108" orientation="0 0 ${math.pi}" use_models="$(arg use_models)"/>
+    <xacro:h2c_hydrophone name="${namespace}/base_link/hydrophone_0" parent="${namespace}/base_link" position="0.315 0.1675 0.1715" orientation="0 0 0" use_models="$(arg use_models)"/>
+    <xacro:h2c_hydrophone name="${namespace}/base_link/hydrophone_1" parent="${namespace}/base_link" position="0.315 -0.1675 0.1715" orientation="0 0 0" use_models="$(arg use_models)"/>
+    <xacro:h2c_hydrophone name="${namespace}/base_link/hydrophone_2" parent="${namespace}/base_link" position="-0.315 0.1675 0.1715" orientation="0 0 0" use_models="$(arg use_models)"/>
+    <xacro:h2c_hydrophone name="${namespace}/base_link/hydrophone_3" parent="${namespace}/base_link" position="-0.315 -0.1675 0.1715" orientation="0 0 0" use_models="$(arg use_models)"/>
+    <xacro:ping360 name="${namespace}/base_link/ping360" parent="${namespace}/base_link" position="0.2 0 0.134" orientation="0 0 0" use_models="$(arg use_models)"/>
+    <xacro:bar30 name="${namespace}/base_link/external_pressure_sensor" parent="${namespace}/base_link" position="0 0 0.079" orientation="0 0 0" use_models="$(arg use_models)"/>
+    <xacro:logitech_c920_camera name="${namespace}/base_link/front_camera" parent="${namespace}/base_link" position="0.40125 0 0" orientation="0 0 0" use_models="$(arg use_models)"/>
+    <xacro:logitech_c920_camera
+      name="${namespace}/base_link/bottom_camera"
+      parent="${namespace}/base_link"
+      position="0 0 -0.07"
+      orientation="0 ${math.pi/2} ${-math.pi/2}"
+      use_models="$(arg use_models)"
+    />
+    <xacro:torpedo_upper name="${namespace}/base_link/torpedo_upper" parent="${namespace}/base_link" position="0.4057 -0.1038 -0.049" orientation="0 0 0" use_models="$(arg use_models)"/>
+    <xacro:torpedo_bottom name="${namespace}/base_link/torpedo_bottom" parent="${namespace}/base_link" position="0.4057 -0.1038 -0.084" orientation="0 0 0" use_models="$(arg use_models)"/>
+    <xacro:sonar name="${namespace}/base_link/sonar_front" parent="${namespace}/base_link" position="0.38 0.09 0.09" orientation="0 0 0" use_models="$(arg use_models)"/>
+    <xacro:sonar name="${namespace}/base_link/sonar_back" parent="${namespace}/base_link" position="-0.42 -0.09 0.09" orientation="0 0 ${math.pi}" use_models="$(arg use_models)"/>
+    <xacro:sonar name="${namespace}/base_link/sonar_right" parent="${namespace}/base_link" position="0.02 -0.21 -0.14" orientation="0 0 ${-math.pi/2}" use_models="$(arg use_models)"/>
+    <xacro:sonar name="${namespace}/base_link/sonar_left" parent="${namespace}/base_link" position="0.02 0.21 -0.14" orientation="0 0 ${math.pi/2}" use_models="$(arg use_models)"/>
+    <xacro:ball_dropper name="${namespace}/base_link/ball_dropper" parent="${namespace}/base_link" position="0.1004 0.0745 -0.1953" orientation="0 0 0" use_models="$(arg use_models)"/>
+    <xacro:realsense_d435 name="${namespace}/camera" parent="${namespace}/base_link" position="-0.35 0 0" orientation="0 0 ${math.pi}" use_models="$(arg use_models)"/>
   </xacro:macro>
 </robot>
