Commit message: simulation environment changes

File: auv_description/auv_common_descriptions/urdf/actuators/docking_puck.urdf.xacro (robot description, xacro)
@@ -4,6 +4,6 @@
     <link name="${name}_link">
       <inertial>
-        <mass value="0.5"/>
-        <inertia ixx="0.001" ixy="0.0" ixz="0.0" iyy="0.001" iyz="0.0" izz="0.001"/>
+        <mass value="0.001"/>
+        <inertia ixx="0.000001" ixy="0.0" ixz="0.0" iyy="0.000001" iyz="0.0" izz="0.000001"/>
       </inertial>
       <visual>
@@ -30,4 +30,8 @@
       <axis rpy="0 0 0" xyz="0 0 1"/>
     </joint>
+    <gazebo reference="${name}_link">
+      <min_depth>0.005</min_depth>
+      <max_vel>0.1</max_vel>
+    </gazebo>
   </xacro:macro>
 </robot>

Commit message: Rebased and cleaned up, changed the aruco node to be config based

File: auv_description/auv_common_descriptions/urdf/actuators/docking_puck.urdf.xacro (robot description, xacro)
@@ -8,6 +8,6 @@
       </inertial>
       <visual>
-        <!-- Rotate mesh so flat surface faces down (Y axis in mesh becomes -Z in robot frame) -->
-        <origin xyz="0 0 0" rpy="${pi/2} 0 0"/>
+        <!-- Rotate mesh so cylinder axis aligns with link Z, then shift up so the bottom face sits at link z=0 -->
+        <origin xyz="0 0 0.0368" rpy="${pi/2} 0 0"/>
         <geometry>
           <mesh filename="package://auv_common_descriptions/meshes/docking_puck/docking_puck.stl" scale="0.001 0.001 0.001"/>
@@ -18,5 +18,5 @@
       </visual>
       <collision>
-        <origin xyz="0 0 0" rpy="${pi/2} 0 0"/>
+        <origin xyz="0 0 0.0368" rpy="${pi/2} 0 0"/>
         <geometry>
           <mesh filename="package://auv_common_descriptions/meshes/docking_puck/docking_puck.stl" scale="0.001 0.001 0.001"/>

File: auv_sim/auv_sim_description/auv_common_sim_descriptions/urdf/sensors/logitech_c920_camera.urdf.xacro (robot description, xacro)
@@ -1,16 +1,13 @@
 <?xml version="1.0"?>
 <robot xmlns:xacro="http://ros.org/wiki/xacro" name="logitech_c920_camera">
-  <xacro:macro name="logitech_c920_camera_sim" params="name topic_name
-    image_width:=640 image_height:=480 hfov:=1.229
-    distortion_k1:=0.0 distortion_k2:=0.0 distortion_k3:=0.0
-    distortion_t1:=0.0 distortion_t2:=0.0">
+  <xacro:macro name="logitech_c920_camera_sim" params="name topic_name">
     <gazebo reference="${name}_link">
       <sensor type="camera" name="${name}_sensor">
         <update_rate>30.0</update_rate>
         <camera name="head">
-          <horizontal_fov>${hfov}</horizontal_fov>
+          <horizontal_fov>1.229</horizontal_fov>
           <image>
-            <width>${image_width}</width>
-            <height>${image_height}</height>
+            <width>640</width>
+            <height>480</height>
             <format>B8G8R8</format>
           </image>
@@ -27,12 +24,4 @@
             <stddev>0.007</stddev>
           </noise>
-          <distortion>
-            <k1>${distortion_k1}</k1>
-            <k2>${distortion_k2}</k2>
-            <k3>${distortion_k3}</k3>
-            <p1>${distortion_t1}</p1>
-            <p2>${distortion_t2}</p2>
-            <center>0.5 0.5</center>
-          </distortion>
         </camera>
         <plugin name="camera_controller" filename="libgazebo_ros_camera.so">
@@ -43,9 +32,9 @@
           <frameName>${name}_optical_link</frameName>
           <hackBaseline>0.07</hackBaseline>
-          <distortionK1>${distortion_k1}</distortionK1>
-          <distortionK2>${distortion_k2}</distortionK2>
-          <distortionK3>${distortion_k3}</distortionK3>
-          <distortionT1>${distortion_t1}</distortionT1>
-          <distortionT2>${distortion_t2}</distortionT2>
+          <distortionK1>0.0</distortionK1>
+          <distortionK2>0.0</distortionK2>
+          <distortionK3>0.0</distortionK3>
+          <distortionT1>0.0</distortionT1>
+          <distortionT2>0.0</distortionT2>
         </plugin>
       </sensor>

File: auv_sim/auv_sim_description/taluy_sim_description/urdf/sensors.urdf.xacro (robot description, xacro)
@@ -10,8 +10,5 @@
   <xacro:sonar_sim name="${namespace}/base_link/sonar_left" topic="sensors/sonar_left"/>
   <xacro:logitech_c920_camera_sim name="${namespace}/base_link/front_camera" topic_name="cameras/cam_front"/>
-  <xacro:logitech_c920_camera_sim name="${namespace}/base_link/bottom_camera" topic_name="cameras/cam_bottom"
-    image_width="1920" image_height="1080" hfov="1.2724"
-    distortion_k1="-0.330122" distortion_k2="0.135823" distortion_k3="0.0"
-    distortion_t1="0.001839" distortion_t2="0.000819"/>
+  <xacro:logitech_c920_camera_sim name="${namespace}/base_link/bottom_camera" topic_name="cameras/cam_bottom"/>
   <xacro:logitech_c920_camera_sim name="${namespace}/base_link/torpedo_camera" topic_name="cameras/cam_torpedo"/>
   <xacro:bar30_sim name="${namespace}/base_link/external_pressure_sensor" update_rate="$(arg pressure_update_rate)" namespace="${namespace}"/>

Commit message: added pre-touch frame, lighhtened aruco detection load

File: auv_description/auv_common_descriptions/urdf/actuators/docking_puck.urdf.xacro (robot description, xacro)
@@ -7,14 +7,4 @@
         <inertia ixx="0.000001" ixy="0.0" ixz="0.0" iyy="0.000001" iyz="0.0" izz="0.000001"/>
       </inertial>
-      <visual>
-        <!-- Rotate mesh so cylinder axis aligns with link Z, then shift up so the bottom face sits at link z=0 -->
-        <origin xyz="0 0 0.0368" rpy="${pi/2} 0 0"/>
-        <geometry>
-          <mesh filename="package://auv_common_descriptions/meshes/docking_puck/docking_puck.stl" scale="0.001 0.001 0.001"/>
-        </geometry>
-        <material name="grey">
-          <color rgba="0.5 0.5 0.5 1.0"/>
-        </material>
-      </visual>
       <collision>
         <origin xyz="0 0 0.0368" rpy="${pi/2} 0 0"/>

Commit message: docking test mode, works in sim

File: auv_description/auv_common_descriptions/urdf/actuators/docking_puck.urdf.xacro (robot description, xacro)
@@ -3,14 +3,5 @@
   <xacro:macro name="docking_puck" params="name parent position:='0 0 0' orientation:='0 0 0' use_models:='false'">
     <link name="${name}_link">
-      <inertial>
-        <mass value="0.001"/>
-        <inertia ixx="0.000001" ixy="0.0" ixz="0.0" iyy="0.000001" iyz="0.0" izz="0.000001"/>
-      </inertial>
-      <collision>
-        <origin xyz="0 0 0.0368" rpy="${pi/2} 0 0"/>
-        <geometry>
-          <mesh filename="package://auv_common_descriptions/meshes/docking_puck/docking_puck.stl" scale="0.001 0.001 0.001"/>
-        </geometry>
-      </collision>
+      <!-- Collision/inertial disabled: puck is invisible and non-colliding, kept only as a frame on the AUV base -->
     </link>
     <joint name="${name}_joint" type="fixed">
@@ -20,8 +11,4 @@
       <axis rpy="0 0 0" xyz="0 0 1"/>
     </joint>
-    <gazebo reference="${name}_link">
-      <min_depth>0.005</min_depth>
-      <max_vel>0.1</max_vel>
-    </gazebo>
   </xacro:macro>
 </robot>
