Commit message: fix sonar urdf

File: auv_description/auv_common_descriptions/urdf/sensors.urdf.xacro (robot description, xacro)
@@ -6,3 +6,4 @@
 	<xacro:include filename="$(find auv_common_descriptions)/urdf/sensors/bar30.urdf.xacro" />
 	<xacro:include filename="$(find auv_common_descriptions)/urdf/sensors/logitech_c920_camera.urdf.xacro" />
+	<xacro:include filename="$(find auv_common_descriptions)/urdf/sensors/sonar.urdf.xacro" />
 </robot>

File: auv_description/auv_common_descriptions/urdf/sensors/sonar.urdf.xacro (robot description, xacro)
@@ -4,9 +4,9 @@
     <link name="${name}_link">
       <visual>
-        <origin xyz="0 0 0" rpy="0 0 0" />
+        <origin xyz="0 0 0" rpy="0 ${-math.pi/2} 0" />
         <geometry>
           <mesh
             filename="package://auv_common_descriptions/meshes/sonar/sonar.dae"
-            scale="1 1 1" />
+            scale="0.001 0.001 0.001" />
         </geometry>
       </visual>
@@ -16,5 +16,5 @@
           <mesh
             filename="package://auv_common_descriptions/meshes/sonar/sonar.dae"
-            scale="1 1 1" />
+            scale="0.001 0.001 0.001" />
         </geometry>
       </collision>

File: auv_description/taluy_description/urdf/auv_base.urdf.xacro (robot description, xacro)
@@ -90,14 +90,14 @@
     <xacro:sonar name="base_link/sonar_front" parent="base_link"
       position="0.38 0.09 0.09"
-      orientation="0 0 0" />
+      orientation="0 ${math.pi/2} 0" />
     <xacro:sonar name="base_link/sonar_back" parent="base_link"
       position="-0.42 -0.09 0.09"
-      orientation="0 0 ${math.pi}" />
+      orientation="0 ${math.pi/2} ${math.pi}" />
     <xacro:sonar name="base_link/sonar_left" parent="base_link"
       position="0.02 -0.21 -0.14"
-      orientation="0 0 ${-math.pi/2}" />
+      orientation="0 ${math.pi/2} ${-math.pi/2}" />
     <xacro:sonar name="base_link/sonar_right" parent="base_link"
       position="0.02 0.21 -0.14"
-      orientation="0 0 ${math.pi/2}" />
+      orientation="0 ${math.pi/2} ${math.pi/2}" />
     <!-- <link name="base_footprint">
       <inertial>

Commit message: init

File: auv_description/auv_common_descriptions/urdf/sensors.urdf.xacro (robot description, xacro)
@@ -8,3 +8,4 @@
   <xacro:include filename="$(find auv_common_descriptions)/urdf/sensors/logitech_c920_camera.urdf.xacro"/>
   <xacro:include filename="$(find auv_common_descriptions)/urdf/sensors/sonar.urdf.xacro"/>
+  <xacro:include filename="$(find auv_common_descriptions)/urdf/sensors/depth_camera.urdf.xacro"/>
 </robot>

File: auv_description/taluy_description/urdf/auv_base.urdf.xacro (robot description, xacro)
@@ -52,4 +52,7 @@
     <xacro:logitech_c920_camera name="${namespace}/base_link/front_camera" parent="${namespace}/base_link" position="0.35 0 0" orientation="0 0 0"/>
     <xacro:logitech_c920_camera name="${namespace}/base_link/bottom_camera" parent="${namespace}/base_link" position="0 0 -0.07" orientation="0 ${math.pi/2} ${math.pi/2}"/>
+    <xacro:depth_camera name="${namespace}/base_link/depth_camera" parent="${namespace}/base_link">
+      <origin xyz="0.35 0 0" rpy="0 0 0"/>
+    </xacro:depth_camera>
     <xacro:torpedo name="${namespace}/base_link/left_torpedo" parent="${namespace}/base_link" position="0.2 0.1 -0.11" orientation="0 0 0"/>
     <xacro:torpedo name="${namespace}/base_link/right_torpedo" parent="${namespace}/base_link" position="0.2 -0.1 -0.11" orientation="0 0 0"/>

Commit message: init

File: auv_description/auv_common_descriptions/urdf/sensors.urdf.xacro (robot description, xacro)
@@ -8,4 +8,3 @@
   <xacro:include filename="$(find auv_common_descriptions)/urdf/sensors/logitech_c920_camera.urdf.xacro"/>
   <xacro:include filename="$(find auv_common_descriptions)/urdf/sensors/sonar.urdf.xacro"/>
-  <xacro:include filename="$(find auv_common_descriptions)/urdf/sensors/depth_camera.urdf.xacro"/>
 </robot>

File: auv_description/taluy_description/urdf/auv_base.urdf.xacro (robot description, xacro)
@@ -52,7 +52,4 @@
     <xacro:logitech_c920_camera name="${namespace}/base_link/front_camera" parent="${namespace}/base_link" position="0.35 0 0" orientation="0 0 0"/>
     <xacro:logitech_c920_camera name="${namespace}/base_link/bottom_camera" parent="${namespace}/base_link" position="0 0 -0.07" orientation="0 ${math.pi/2} ${math.pi/2}"/>
-    <xacro:depth_camera name="${namespace}/base_link/depth_camera" parent="${namespace}/base_link">
-      <origin xyz="0.35 0 0" rpy="0 0 0"/>
-    </xacro:depth_camera>
     <xacro:torpedo name="${namespace}/base_link/left_torpedo" parent="${namespace}/base_link" position="0.2 0.1 -0.11" orientation="0 0 0"/>
     <xacro:torpedo name="${namespace}/base_link/right_torpedo" parent="${namespace}/base_link" position="0.2 -0.1 -0.11" orientation="0 0 0"/>
