Commit message: add torpedo and camera

File: auv_description/auv_common_descriptions/urdf/actuators.urdf.xacro (robot description, xacro)
@@ -1,3 +1,4 @@
 <robot xmlns:xacro="http://www.ros.org/wiki/xacro">
 	<xacro:include filename="$(find auv_common_descriptions)/urdf/actuators/t200.urdf.xacro" />
+	<xacro:include filename="$(find auv_common_descriptions)/urdf/actuators/torpedo.urdf.xacro" />
 </robot>

File: auv_description/auv_common_descriptions/urdf/sensors.urdf.xacro (robot description, xacro)
@@ -5,3 +5,4 @@
 	<xacro:include filename="$(find auv_common_descriptions)/urdf/sensors/ping360.urdf.xacro" />
 	<xacro:include filename="$(find auv_common_descriptions)/urdf/sensors/bar30.urdf.xacro" />
+	<xacro:include filename="$(find auv_common_descriptions)/urdf/sensors/logitech_c920_camera.urdf.xacro" />
 </robot>

File: auv_description/auv_common_descriptions/urdf/sensors/wayfinder_dvl.urdf.xacro (robot description, xacro)
@@ -19,7 +19,12 @@
         </geometry>
       </collision>
+    </link>
+    <link name="${name}_cog">
       <inertial>
-        <mass value="0.5" />
-        <inertia ixx="0.008545" ixy="0.0" ixz="0.0" iyy="0.008545" iyz="0.0" izz="0.0144" />
+        <!-- 0.313 in water -->
+        <mass value="0.947" />
+        <!-- volume: 100mm x 100mm x 70mm -->
+        <!-- 0.0007 m^3-->
+        <inertia ixx="0.001176" ixy="0.0" ixz="0.0" iyy="0.001176" iyz="0.0" izz="0.001578" />
       </inertial>
     </link>
@@ -36,5 +41,11 @@
       <parent link="${name}_mount_link" />
       <child link="${name}_sensor_surface_link" />
-      <origin xyz="0 0 -0.07" rpy="${math.pi} 0 0" />
+      <origin xyz="0 0 -0.07" rpy="0 0 0" />
+    </joint>
+    <joint name="${name}_cog_joint" type="fixed">
+      <axis rpy="0 0 0" xyz="0 0 1" />
+      <parent link="${name}_mount_link" />
+      <child link="${name}_cog" />
+      <origin xyz="0 0 -0.035" rpy="0 0 0" />
     </joint>
     <joint name="${name}_sensor_joint" type="fixed">
@@ -42,5 +53,5 @@
       <parent link="${name}_sensor_surface_link" />
       <child link="${name}_link" />
-      <origin xyz="0 0 0" rpy="0 0 ${math.pi/4}" />
+      <origin xyz="0 0 0" rpy="0 0 ${-3*math.pi/4}" />
     </joint>
     <!-- <gazebo reference="${name}_propeller_link">

File: auv_description/taluy_description/urdf/auv_base.urdf.xacro (robot description, xacro)
@@ -3,6 +3,8 @@
   <xacro:macro name="taluy_base">
     <xacro:include filename="$(find auv_common_descriptions)/urdf/actuators.urdf.xacro" />
-    <xacro:include filename="$(find auv_common_descriptions)/urdf/sensors.urdf.xacro" />
-    <xacro:include filename="$(find auv_common_descriptions)/urdf/materials.urdf.xacro" />
+    <xacro:include
+      filename="$(find auv_common_descriptions)/urdf/sensors.urdf.xacro" />
+    <xacro:include
+      filename="$(find auv_common_descriptions)/urdf/materials.urdf.xacro" />
     <link name="base_link">
       <inertial>
@@ -27,34 +29,75 @@
       </collision>
     </link>
-    <xacro:t200_thruster name="thruster_0" parent="base_link" position="0.14250 0.20070 -0.00525"
+    <link name="base_link_ned"/>
+    <joint name="base_link_joint" type="fixed">
+      <origin xyz="0 0 0" rpy="${math.pi} 0 0" />
+      <parent link="base_link_ned" />
+      <child link="base_link" />
+    </joint>
+    <xacro:t200_thruster
+      name="base_link/thruster_0" parent="base_link"
+      position="0.14250 0.20070 -0.00525"
       orientation="0 0 ${-pi/2}" />
-    <xacro:t200_thruster name="thruster_1" parent="base_link" position="0.14250 -0.20070 -0.00525"
+    <xacro:t200_thruster name="base_link/thruster_1"
+      parent="base_link"
+      position="0.14250 -0.20070 -0.00525"
       orientation="0 0 ${pi/2}" />
-    <xacro:t200_thruster name="thruster_2" parent="base_link" position="-0.14250 0.20070 -0.00525"
+    <xacro:t200_thruster name="base_link/thruster_2"
+      parent="base_link"
+      position="-0.14250 0.20070 -0.00525"
       orientation="0 0 ${-pi/2}" />
-    <xacro:t200_thruster name="thruster_3" parent="base_link" position="-0.14250 -0.20070 -0.00525"
+    <xacro:t200_thruster name="base_link/thruster_3"
+      parent="base_link"
+      position="-0.14250 -0.20070 -0.00525"
       orientation="0 0 ${pi/2}" />
-    <xacro:t200_thruster name="thruster_4" parent="base_link" position="0.352398 0.216638 -0.030881"
+    <xacro:t200_thruster name="base_link/thruster_4"
+      parent="base_link"
+      position="0.352398 0.216638 -0.030881"
       orientation="${pi/2} 0 ${pi/4}" />
-    <xacro:t200_thruster name="thruster_5" parent="base_link"
+    <xacro:t200_thruster name="base_link/thruster_5"
+      parent="base_link"
       position="0.352398 -0.216638 -0.030881" orientation="${-pi/2} 0 ${-pi/4}" />
-    <xacro:t200_thruster name="thruster_6" parent="base_link"
+    <xacro:t200_thruster
+      name="base_link/thruster_6" parent="base_link"
       position="-0.352398 0.216638 -0.030881" orientation="${pi/2} 0 ${3*pi/4}" />
-    <xacro:t200_thruster name="thruster_7" parent="base_link"
+    <xacro:t200_thruster
+      name="base_link/thruster_7" parent="base_link"
       position="-0.352398 -0.216638 -0.030881" orientation="${-pi/2} 0 ${-3*pi/4}" />
-    <xacro:wayfinder_dvl name="dvl" parent="base_link" position="0.2 0 -0.11" orientation="0 0 0" />
-    <xacro:xsens_mti_g710 name="imu" parent="base_link" position="-0.199 0 -0.0108"
+    <xacro:wayfinder_dvl
+      name="base_link/dvl" parent="base_link" position="0.2 0 -0.11"
+      orientation="0 0 0" />
+    <xacro:xsens_mti_g710 name="base_link/imu" parent="base_link"
+      position="-0.199 0 -0.0108"
       orientation="0 0 ${math.pi}" />
-    <xacro:h2c_hydrophone name="hydrophone_0" parent="base_link" position="0.325 0.205 -0.15"
+    <xacro:h2c_hydrophone name="base_link/hydrophone_0"
+      parent="base_link"
+      position="0.325 0.205 -0.15"
       orientation="0 0 0" />
-    <xacro:h2c_hydrophone name="hydrophone_1" parent="base_link" position="0.325 -0.205 -0.15"
+    <xacro:h2c_hydrophone name="base_link/hydrophone_1" parent="base_link"
+      position="0.325 -0.205 -0.15"
       orientation="0 0 0" />
-    <xacro:h2c_hydrophone name="hydrophone_2" parent="base_link" position="-0.325 0.205 -0.15"
+    <xacro:h2c_hydrophone name="base_link/hydrophone_2" parent="base_link"
+      position="-0.325 0.205 -0.15"
       orientation="0 0 0" />
-    <xacro:h2c_hydrophone name="hydrophone_3" parent="base_link" position="-0.325 -0.205 -0.15"
+    <xacro:h2c_hydrophone name="base_link/hydrophone_3" parent="base_link"
+      position="-0.325 -0.205 -0.15"
       orientation="0 0 0" />
-    <xacro:ping360 name="ping360" parent="base_link" position="0.2 0 0.134"
+    <xacro:ping360 name="base_link/ping360" parent="base_link"
+      position="0.2 0 0.134"
       orientation="0 0 0" />
-    <xacro:bar30 name="bar30" parent="base_link" position="0 0 0.07"
+    <xacro:bar30 name="base_link/bar30" parent="base_link"
+      position="0 0 0.07"
+      orientation="0 0 0" />
+    <xacro:logitech_c920_camera name="base_link/front_camera"
+      parent="base_link" position="0.35 0 0"
+      orientation="0 0 0" />
+    <xacro:logitech_c920_camera name="base_link/bottom_camera"
+      parent="base_link" position="0 0 -0.07"
+      orientation="0 ${math.pi/2} ${math.pi/2}" />
+    <xacro:torpedo name="base_link/left_torpedo"
+      parent="base_link" position="0.2 0.1 -0.11"
+      orientation="0 0 0" />
+    <xacro:torpedo name="base_link/right_torpedo"
+      parent="base_link" position="0.2 -0.1 -0.11"
       orientation="0 0 0" />
     <!-- <link name="base_footprint">

Commit message: add torpedo & marker

File: auv_description/auv_common_descriptions/urdf/actuators.urdf.xacro (robot description, xacro)
@@ -2,3 +2,4 @@
 	<xacro:include filename="$(find auv_common_descriptions)/urdf/actuators/t200.urdf.xacro" />
 	<xacro:include filename="$(find auv_common_descriptions)/urdf/actuators/torpedo.urdf.xacro" />
+	<xacro:include filename="$(find auv_common_descriptions)/urdf/actuators/marker.urdf.xacro" />
 </robot>

File: auv_description/auv_common_descriptions/urdf/actuators/torpedo.urdf.xacro (robot description, xacro)
@@ -2,10 +2,10 @@
 <robot name="torpedo" xmlns:xacro="http://ros.org/wiki/xacro">
   <xacro:macro name="torpedo" params="name parent position:='0 0 0' orientation:='0 0 0'">
-    <link name="${name}_link" />
-    <link name="${name}_upper_link">
+    <link name="${name}_link">
       <visual>
-        <origin xyz="0 0 0" rpy="0 0 0" />
+        <origin xyz="0 0 0" rpy="0 0 -0.05" />
         <geometry>
-          <cylinder length="0.2" radius="0.0175" />
+          <mesh filename="package://auv_common_descriptions/meshes/torpedo/torpedo.dae"
+            scale="0.001 0.001 0.001" />
         </geometry>
       </visual>
@@ -13,5 +13,6 @@
         <origin xyz="0 0 0" rpy="0 0 0" />
         <geometry>
-          <cylinder length="0.2" radius="0.0175" />
+          <mesh filename="package://auv_common_descriptions/meshes/torpedo/torpedo.dae"
+            scale="0.001 0.001 0.001" />
         </geometry>
       </collision>
@@ -21,22 +22,6 @@
       </inertial>
     </link>
-    <link name="${name}_lower_link">
-      <visual>
-        <origin xyz="0 0 0" rpy="0 0 0" />
-        <geometry>
-          <cylinder length="0.2" radius="0.0175" />
-        </geometry>
-      </visual>
-      <collision name="${name}_collision">
-        <origin xyz="0 0 0" rpy="0 0 0" />
-        <geometry>
-          <cylinder length="0.2" radius="0.0175" />
-        </geometry>
-      </collision>
-      <inertial>
-        <mass value="0.5" />
-        <inertia ixx="0.008545" ixy="0.0" ixz="0.0" iyy="0.008545" iyz="0.0" izz="0.0144" />
-      </inertial>
-    </link>
+    <link name="${name}_top_torpedo_link" />
+    <link name="${name}_bottom_torpedo_link" />
     <joint name="${name}_chasis_joint" type="fixed">
       <parent link="${parent}" />
@@ -45,15 +30,13 @@
       <axis rpy="0 0 0" xyz="0 0 1" />
     </joint>
-    <joint name="${name}_upper_joint" type="fixed">
-      <axis rpy="0 0 0" xyz="0 0 1" />
+    <joint name="${name}_top_torpedo_joint" type="fixed">
       <parent link="${name}_link" />
-      <child link="${name}_upper_link" />
-      <origin xyz="0.1 0 -0.0175" rpy="0 ${math.pi/2} 0" />
+      <child link="${name}_top_torpedo_link" />
+      <origin xyz="0 0 0" rpy="0 ${math.pi/2} 0" />
     </joint>
-    <joint name="${name}_lower_joint" type="fixed">
-      <axis rpy="0 0 0" xyz="0 0 1" />
+    <joint name="${name}_bottom_torpedo_joint" type="fixed">
       <parent link="${name}_link" />
-      <child link="${name}_lower_link" />
-      <origin xyz="0.1 0 -0.0525" rpy="0 ${math.pi/2} 0" />
+      <child link="${name}_bottom_torpedo_link" />
+      <origin xyz="0 0 -0.035" rpy="0 ${math.pi/2} 0" />
     </joint>
   </xacro:macro>

File: auv_description/taluy_description/urdf/auv_base.urdf.xacro (robot description, xacro)
@@ -29,5 +29,5 @@
       </collision>
     </link>
-    <link name="base_link_ned"/>
+    <link name="base_link_ned" />
     <joint name="base_link_joint" type="fixed">
       <origin xyz="0 0 0" rpy="${math.pi} 0 0" />
@@ -95,9 +95,9 @@
       parent="base_link" position="0 0 -0.07"
       orientation="0 ${math.pi/2} ${math.pi/2}" />
-    <xacro:torpedo name="base_link/left_torpedo"
-      parent="base_link" position="0.2 0.1 -0.11"
+    <xacro:torpedo name="base_link/torpedo"
+      parent="base_link" position="0.39 0.121 -0.056"
       orientation="0 0 0" />
-    <xacro:torpedo name="base_link/right_torpedo"
-      parent="base_link" position="0.2 -0.1 -0.11"
+    <xacro:marker name="base_link/marker"
+      parent="base_link" position="0.093 -0.075 -0.188"
       orientation="0 0 0" />
     <!-- <link name="base_footprint">

Commit message: Add TF tree (#29)
* add frame transformations

* add torpedo and camera

* update

* add torpedo & marker

File: auv_description/auv_common_descriptions/urdf/actuators.urdf.xacro (robot description, xacro)
@@ -1,3 +1,5 @@
 <robot xmlns:xacro="http://www.ros.org/wiki/xacro">
 	<xacro:include filename="$(find auv_common_descriptions)/urdf/actuators/t200.urdf.xacro" />
+	<xacro:include filename="$(find auv_common_descriptions)/urdf/actuators/torpedo.urdf.xacro" />
+	<xacro:include filename="$(find auv_common_descriptions)/urdf/actuators/marker.urdf.xacro" />
 </robot>

File: auv_description/taluy_description/urdf/auv_base.urdf.xacro (robot description, xacro)
@@ -3,5 +3,8 @@
   <xacro:macro name="taluy_base">
     <xacro:include filename="$(find auv_common_descriptions)/urdf/actuators.urdf.xacro" />
-    <xacro:include filename="$(find auv_common_descriptions)/urdf/materials.urdf.xacro" />
+    <xacro:include
+      filename="$(find auv_common_descriptions)/urdf/sensors.urdf.xacro" />
+    <xacro:include
+      filename="$(find auv_common_descriptions)/urdf/materials.urdf.xacro" />
     <link name="base_link">
       <inertial>
@@ -26,12 +29,76 @@
       </collision>
     </link>
-    <xacro:t200_thruster name="thruster_0" parent="base_link" position="0.14250 0.20070 -0.00525" orientation="0 0 ${-pi/2}"/>
-    <xacro:t200_thruster name="thruster_1" parent="base_link" position="0.14250 -0.20070 -0.00525" orientation="0 0 ${pi/2}"/>
-    <xacro:t200_thruster name="thruster_2" parent="base_link" position="-0.14250 0.20070 -0.00525" orientation="0 0 ${-pi/2}"/>
-    <xacro:t200_thruster name="thruster_3" parent="base_link" position="-0.14250 -0.20070 -0.00525" orientation="0 0 ${pi/2}"/>
-    <xacro:t200_thruster name="thruster_4" parent="base_link" position="0.352398 0.216638 -0.030881" orientation="${pi/2} 0 ${pi/4}"/>
-    <xacro:t200_thruster name="thruster_5" parent="base_link" position="0.352398 -0.216638 -0.030881" orientation="${-pi/2} 0 ${-pi/4}"/>
-    <xacro:t200_thruster name="thruster_6" parent="base_link" position="-0.352398 0.216638 -0.030881" orientation="${pi/2} 0 ${3*pi/4}"/>
-    <xacro:t200_thruster name="thruster_7" parent="base_link" position="-0.352398 -0.216638 -0.030881" orientation="${-pi/2} 0 ${-3*pi/4}"/>
+    <link name="base_link_ned" />
+    <joint name="base_link_joint" type="fixed">
+      <origin xyz="0 0 0" rpy="${math.pi} 0 0" />
+      <parent link="base_link_ned" />
+      <child link="base_link" />
+    </joint>
+    <xacro:t200_thruster
+      name="base_link/thruster_0" parent="base_link"
+      position="0.14250 0.20070 -0.00525"
+      orientation="0 0 ${-pi/2}" />
+    <xacro:t200_thruster name="base_link/thruster_1"
+      parent="base_link"
+      position="0.14250 -0.20070 -0.00525"
+      orientation="0 0 ${pi/2}" />
+    <xacro:t200_thruster name="base_link/thruster_2"
+      parent="base_link"
+      position="-0.14250 0.20070 -0.00525"
+      orientation="0 0 ${-pi/2}" />
+    <xacro:t200_thruster name="base_link/thruster_3"
+      parent="base_link"
+      position="-0.14250 -0.20070 -0.00525"
+      orientation="0 0 ${pi/2}" />
+    <xacro:t200_thruster name="base_link/thruster_4"
+      parent="base_link"
+      position="0.352398 0.216638 -0.030881"
+      orientation="${pi/2} 0 ${pi/4}" />
+    <xacro:t200_thruster name="base_link/thruster_5"
+      parent="base_link"
+      position="0.352398 -0.216638 -0.030881" orientation="${-pi/2} 0 ${-pi/4}" />
+    <xacro:t200_thruster
+      name="base_link/thruster_6" parent="base_link"
+      position="-0.352398 0.216638 -0.030881" orientation="${pi/2} 0 ${3*pi/4}" />
+    <xacro:t200_thruster
+      name="base_link/thruster_7" parent="base_link"
+      position="-0.352398 -0.216638 -0.030881" orientation="${-pi/2} 0 ${-3*pi/4}" />
+    <xacro:wayfinder_dvl
+      name="base_link/dvl" parent="base_link" position="0.2 0 -0.11"
+      orientation="0 0 0" />
+    <xacro:xsens_mti_g710 name="base_link/imu" parent="base_link"
+      position="-0.199 0 -0.0108"
+      orientation="0 0 ${math.pi}" />
+    <xacro:h2c_hydrophone name="base_link/hydrophone_0"
+      parent="base_link"
+      position="0.325 0.205 -0.15"
+      orientation="0 0 0" />
+    <xacro:h2c_hydrophone name="base_link/hydrophone_1" parent="base_link"
+      position="0.325 -0.205 -0.15"
+      orientation="0 0 0" />
+    <xacro:h2c_hydrophone name="base_link/hydrophone_2" parent="base_link"
+      position="-0.325 0.205 -0.15"
+      orientation="0 0 0" />
+    <xacro:h2c_hydrophone name="base_link/hydrophone_3" parent="base_link"
+      position="-0.325 -0.205 -0.15"
+      orientation="0 0 0" />
+    <xacro:ping360 name="base_link/ping360" parent="base_link"
+      position="0.2 0 0.134"
+      orientation="0 0 0" />
+    <xacro:bar30 name="base_link/bar30" parent="base_link"
+      position="0 0 0.07"
+      orientation="0 0 0" />
+    <xacro:logitech_c920_camera name="base_link/front_camera"
+      parent="base_link" position="0.35 0 0"
+      orientation="0 0 0" />
+    <xacro:logitech_c920_camera name="base_link/bottom_camera"
+      parent="base_link" position="0 0 -0.07"
+      orientation="0 ${math.pi/2} ${math.pi/2}" />
+    <xacro:torpedo name="base_link/torpedo"
+      parent="base_link" position="0.39 0.121 -0.056"
+      orientation="0 0 0" />
+    <xacro:marker name="base_link/marker"
+      parent="base_link" position="0.093 -0.075 -0.188"
+      orientation="0 0 0" />
     <!-- <link name="base_footprint">
       <inertial>
