Commit message: format xml

File: auv_description/auv_common_descriptions/urdf/actuators.urdf.xacro (robot description, xacro)
@@ -1,4 +1,5 @@
+<?xml version="1.0"?>
 <robot xmlns:xacro="http://www.ros.org/wiki/xacro">
-	<xacro:include filename="$(find auv_common_descriptions)/urdf/actuators/t200.urdf.xacro" />
-	<xacro:include filename="$(find auv_common_descriptions)/urdf/actuators/torpedo.urdf.xacro" />
+  <xacro:include filename="$(find auv_common_descriptions)/urdf/actuators/t200.urdf.xacro"/>
+  <xacro:include filename="$(find auv_common_descriptions)/urdf/actuators/torpedo.urdf.xacro"/>
 </robot>

File: auv_description/auv_common_descriptions/urdf/actuators/t200.urdf.xacro (robot description, xacro)
@@ -1,58 +1,54 @@
 <?xml version="1.0"?>
-<robot name="t200_thruster" xmlns:xacro="http://ros.org/wiki/xacro">
+<robot xmlns:xacro="http://ros.org/wiki/xacro" name="t200_thruster">
   <xacro:macro name="t200_thruster" params="name parent position:='0 0 0' orientation:='0 0 0'">
     <link name="${name}_link">
       <visual>
-        <origin xyz="0 0 0" rpy="0 ${pi/2} ${-pi/2}" />
+        <origin xyz="0 0 0" rpy="0 ${pi/2} ${-pi/2}"/>
         <geometry>
-          <mesh filename="package://auv_common_descriptions/meshes/t200/shell.dae"
-            scale="1 1 1" />
+          <mesh filename="package://auv_common_descriptions/meshes/t200/shell.dae" scale="1 1 1"/>
         </geometry>
       </visual>
       <collision name="${name}_collision">
-        <origin xyz="0 0 0" rpy="0 ${pi/2} ${-pi/2}" />
+        <origin xyz="0 0 0" rpy="0 ${pi/2} ${-pi/2}"/>
         <geometry>
-          <mesh filename="package://auv_common_descriptions/meshes/t200/shell.dae"
-            scale="1 1 1" />
+          <mesh filename="package://auv_common_descriptions/meshes/t200/shell.dae" scale="1 1 1"/>
         </geometry>
       </collision>
       <inertial>
-        <mass value="0.5" />
-        <inertia ixx="0.008545" ixy="0.0" ixz="0.0" iyy="0.008545" iyz="0.0" izz="0.0144" />
+        <mass value="0.5"/>
+        <inertia ixx="0.008545" ixy="0.0" ixz="0.0" iyy="0.008545" iyz="0.0" izz="0.0144"/>
       </inertial>
     </link>
     <link name="${name}_propeller_link">
       <visual>
-        <origin xyz="0 0 0" rpy="0 ${pi/2} 0" />
+        <origin xyz="0 0 0" rpy="0 ${pi/2} 0"/>
         <geometry>
-          <mesh filename="package://auv_common_descriptions/meshes/t200/propeller.dae"
-            scale="1.0 1.0 1.0" />
+          <mesh filename="package://auv_common_descriptions/meshes/t200/propeller.dae" scale="1.0 1.0 1.0"/>
         </geometry>
       </visual>
       <collision name="${name}_propeller_collision">
-        <origin xyz="0 0 0" rpy="0 ${pi/2} 0" />
+        <origin xyz="0 0 0" rpy="0 ${pi/2} 0"/>
         <geometry>
-          <mesh filename="package://auv_common_descriptions/meshes/t200/propeller.dae"
-            scale="1 1 1" />
+          <mesh filename="package://auv_common_descriptions/meshes/t200/propeller.dae" scale="1 1 1"/>
         </geometry>
       </collision>
       <inertial>
-        <mass value="0.5" />
-        <inertia ixx="0.008545" ixy="0.0" ixz="0.0" iyy="0.008545" iyz="0.0" izz="0.0144" />
+        <mass value="0.5"/>
+        <inertia ixx="0.008545" ixy="0.0" ixz="0.0" iyy="0.008545" iyz="0.0" izz="0.0144"/>
       </inertial>
     </link>
     <joint name="${name}_chasis_joint" type="fixed">
-      <parent link="${parent}" />
-      <child link="${name}_link" />
-      <origin xyz="${position}" rpy="${orientation}" />
-      <axis rpy="0 0 0" xyz="0 0 1" />
+      <parent link="${parent}"/>
+      <child link="${name}_link"/>
+      <origin xyz="${position}" rpy="${orientation}"/>
+      <axis rpy="0 0 0" xyz="0 0 1"/>
     </joint>
     <joint name="${name}_propeller_joint" type="continuous">
-      <axis rpy="0 0 0" xyz="0 0 1" />
-      <parent link="${name}_link" />
-      <child link="${name}_propeller_link" />
-      <origin xyz="0 0 0" rpy="0 0 0" />
-      <limit effort="100" velocity="100" />
-      <dynamics friction="0.05" damping="0.05" />
+      <axis rpy="0 0 0" xyz="0 0 1"/>
+      <parent link="${name}_link"/>
+      <child link="${name}_propeller_link"/>
+      <origin xyz="0 0 0" rpy="0 0 0"/>
+      <limit effort="100" velocity="100"/>
+      <dynamics friction="0.05" damping="0.05"/>
     </joint>
     <gazebo reference="${name}_propeller_link">

File: auv_description/auv_common_descriptions/urdf/actuators/torpedo.urdf.xacro (robot description, xacro)
@@ -1,59 +1,59 @@
 <?xml version="1.0"?>
-<robot name="torpedo" xmlns:xacro="http://ros.org/wiki/xacro">
+<robot xmlns:xacro="http://ros.org/wiki/xacro" name="torpedo">
   <xacro:macro name="torpedo" params="name parent position:='0 0 0' orientation:='0 0 0'">
-    <link name="${name}_link" />
+    <link name="${name}_link"/>
     <link name="${name}_upper_link">
       <visual>
-        <origin xyz="0 0 0" rpy="0 0 0" />
+        <origin xyz="0 0 0" rpy="0 0 0"/>
         <geometry>
-          <cylinder length="0.2" radius="0.0175" />
+          <cylinder length="0.2" radius="0.0175"/>
         </geometry>
       </visual>
       <collision name="${name}_collision">
-        <origin xyz="0 0 0" rpy="0 0 0" />
+        <origin xyz="0 0 0" rpy="0 0 0"/>
         <geometry>
-          <cylinder length="0.2" radius="0.0175" />
+          <cylinder length="0.2" radius="0.0175"/>
         </geometry>
       </collision>
       <inertial>
-        <mass value="0.5" />
-        <inertia ixx="0.008545" ixy="0.0" ixz="0.0" iyy="0.008545" iyz="0.0" izz="0.0144" />
+        <mass value="0.5"/>
+        <inertia ixx="0.008545" ixy="0.0" ixz="0.0" iyy="0.008545" iyz="0.0" izz="0.0144"/>
       </inertial>
     </link>
     <link name="${name}_lower_link">
       <visual>
-        <origin xyz="0 0 0" rpy="0 0 0" />
+        <origin xyz="0 0 0" rpy="0 0 0"/>
         <geometry>
-          <cylinder length="0.2" radius="0.0175" />
+          <cylinder length="0.2" radius="0.0175"/>
         </geometry>
       </visual>
       <collision name="${name}_collision">
-        <origin xyz="0 0 0" rpy="0 0 0" />
+        <origin xyz="0 0 0" rpy="0 0 0"/>
         <geometry>
-          <cylinder length="0.2" radius="0.0175" />
+          <cylinder length="0.2" radius="0.0175"/>
         </geometry>
       </collision>
       <inertial>
-        <mass value="0.5" />
-        <inertia ixx="0.008545" ixy="0.0" ixz="0.0" iyy="0.008545" iyz="0.0" izz="0.0144" />
+        <mass value="0.5"/>
+        <inertia ixx="0.008545" ixy="0.0" ixz="0.0" iyy="0.008545" iyz="0.0" izz="0.0144"/>
       </inertial>
     </link>
     <joint name="${name}_chasis_joint" type="fixed">
-      <parent link="${parent}" />
-      <child link="${name}_link" />
-      <origin xyz="${position}" rpy="${orientation}" />
-      <axis rpy="0 0 0" xyz="0 0 1" />
+      <parent link="${parent}"/>
+      <child link="${name}_link"/>
+      <origin xyz="${position}" rpy="${orientation}"/>
+      <axis rpy="0 0 0" xyz="0 0 1"/>
     </joint>
     <joint name="${name}_upper_joint" type="fixed">
-      <axis rpy="0 0 0" xyz="0 0 1" />
-      <parent link="${name}_link" />
-      <child link="${name}_upper_link" />
-      <origin xyz="0.1 0 -0.0175" rpy="0 ${math.pi/2} 0" />
+      <axis rpy="0 0 0" xyz="0 0 1"/>
+      <parent link="${name}_link"/>
+      <child link="${name}_upper_link"/>
+      <origin xyz="0.1 0 -0.0175" rpy="0 ${math.pi/2} 0"/>
     </joint>
     <joint name="${name}_lower_joint" type="fixed">
-      <axis rpy="0 0 0" xyz="0 0 1" />
-      <parent link="${name}_link" />
-      <child link="${name}_lower_link" />
-      <origin xyz="0.1 0 -0.0525" rpy="0 ${math.pi/2} 0" />
+      <axis rpy="0 0 0" xyz="0 0 1"/>
+      <parent link="${name}_link"/>
+      <child link="${name}_lower_link"/>
+      <origin xyz="0.1 0 -0.0525" rpy="0 ${math.pi/2} 0"/>
     </joint>
   </xacro:macro>

File: auv_description/auv_common_descriptions/urdf/materials.urdf.xacro (robot description, xacro)
@@ -2,17 +2,17 @@
 <robot>
   <material name="black">
-    <color rgba="0.0 0.0 0.0 1.0" />
+    <color rgba="0.0 0.0 0.0 1.0"/>
   </material>
   <material name="gray">
-    <color rgba="0.7 0.7 0.7 1.0" />
+    <color rgba="0.7 0.7 0.7 1.0"/>
   </material>
   <material name="dark_gray">
-    <color rgba="0.2 0.2 0.2 1.0" />
+    <color rgba="0.2 0.2 0.2 1.0"/>
   </material>
   <material name="white">
-    <color rgba="1.0 1.0 1.0 1.0" />
+    <color rgba="1.0 1.0 1.0 1.0"/>
   </material>
   <material name="yellow">
-    <color rgba="1.0 0.8 0.0 1.0" />
+    <color rgba="1.0 0.8 0.0 1.0"/>
   </material>
 </robot>

File: auv_description/auv_common_descriptions/urdf/sensors.urdf.xacro (robot description, xacro)
@@ -1,9 +1,10 @@
+<?xml version="1.0"?>
 <robot xmlns:xacro="http://www.ros.org/wiki/xacro">
-	<xacro:include filename="$(find auv_common_descriptions)/urdf/sensors/wayfinder_dvl.urdf.xacro" />
-	<xacro:include filename="$(find auv_common_descriptions)/urdf/sensors/xsens_mti_g710.urdf.xacro" />
-	<xacro:include filename="$(find auv_common_descriptions)/urdf/sensors/h2c_hydrophone.urdf.xacro" />
-	<xacro:include filename="$(find auv_common_descriptions)/urdf/sensors/ping360.urdf.xacro" />
-	<xacro:include filename="$(find auv_common_descriptions)/urdf/sensors/bar30.urdf.xacro" />
-	<xacro:include filename="$(find auv_common_descriptions)/urdf/sensors/logitech_c920_camera.urdf.xacro" />
-	<xacro:include filename="$(find auv_common_descriptions)/urdf/sensors/sonar.urdf.xacro" />
+  <xacro:include filename="$(find auv_common_descriptions)/urdf/sensors/wayfinder_dvl.urdf.xacro"/>
+  <xacro:include filename="$(find auv_common_descriptions)/urdf/sensors/xsens_mti_g710.urdf.xacro"/>
+  <xacro:include filename="$(find auv_common_descriptions)/urdf/sensors/h2c_hydrophone.urdf.xacro"/>
+  <xacro:include filename="$(find auv_common_descriptions)/urdf/sensors/ping360.urdf.xacro"/>
+  <xacro:include filename="$(find auv_common_descriptions)/urdf/sensors/bar30.urdf.xacro"/>
+  <xacro:include filename="$(find auv_common_descriptions)/urdf/sensors/logitech_c920_camera.urdf.xacro"/>
+  <xacro:include filename="$(find auv_common_descriptions)/urdf/sensors/sonar.urdf.xacro"/>
 </robot>

File: auv_description/auv_common_descriptions/urdf/sensors/bar30.urdf.xacro (robot description, xacro)
@@ -1,39 +1,35 @@
 <?xml version="1.0"?>
-<robot name="bar30" xmlns:xacro="http://ros.org/wiki/xacro">
+<robot xmlns:xacro="http://ros.org/wiki/xacro" name="bar30">
   <xacro:macro name="bar30" params="name parent position:='0 0 0' orientation:='0 0 0'">
     <link name="${name}_chasis_link">
       <visual>
-        <origin xyz="0 0 0" rpy="0 0 ${math.pi}" />
+        <origin xyz="0 0 0" rpy="0 0 ${math.pi}"/>
         <geometry>
-          <mesh
-            filename="package://auv_common_descriptions/meshes/bar30/bar30.dae"
-            scale="0.001 0.001 0.001" />
+          <mesh filename="package://auv_common_descriptions/meshes/bar30/bar30.dae" scale="0.001 0.001 0.001"/>
         </geometry>
       </visual>
       <collision name="${name}_collision">
-        <origin xyz="0 0 0" rpy="0 0 ${math.pi}" />
+        <origin xyz="0 0 0" rpy="0 0 ${math.pi}"/>
         <geometry>
-          <mesh
-            filename="package://auv_common_descriptions/meshes/bar30/bar30.dae"
-            scale="0.001 0.001 0.001" />
+          <mesh filename="package://auv_common_descriptions/meshes/bar30/bar30.dae" scale="0.001 0.001 0.001"/>
         </geometry>
       </collision>
       <inertial>
-        <mass value="0.5" />
-        <inertia ixx="0.008545" ixy="0.0" ixz="0.0" iyy="0.008545" iyz="0.0" izz="0.0144" />
+        <mass value="0.5"/>
+        <inertia ixx="0.008545" ixy="0.0" ixz="0.0" iyy="0.008545" iyz="0.0" izz="0.0144"/>
       </inertial>
     </link>
-    <link name="${name}_link" />
+    <link name="${name}_link"/>
     <joint name="${name}_joint" type="fixed">
-      <parent link="${parent}" />
-      <child link="${name}_chasis_link" />
-      <origin xyz="${position}" rpy="${orientation}" />
-      <axis rpy="0 0 0" xyz="0 0 1" />
+      <parent link="${parent}"/>
+      <child link="${name}_chasis_link"/>
+      <origin xyz="${position}" rpy="${orientation}"/>
+      <axis rpy="0 0 0" xyz="0 0 1"/>
     </joint>
     <joint name="${name}_sensor_joint" type="fixed">
-      <axis rpy="0 0 0" xyz="0 0 1" />
-      <parent link="${name}_chasis_link" />
-      <child link="${name}_link" />
-      <origin xyz="0 0 0.0075" rpy="0 0 0" />
+      <axis rpy="0 0 0" xyz="0 0 1"/>
+      <parent link="${name}_chasis_link"/>
+      <child link="${name}_link"/>
+      <origin xyz="0 0 0.0075" rpy="0 0 0"/>
     </joint>
   </xacro:macro>

File: auv_description/auv_common_descriptions/urdf/sensors/h2c_hydrophone.urdf.xacro (robot description, xacro)
@@ -1,28 +1,28 @@
 <?xml version="1.0"?>
-<robot name="h2c_hydrophone" xmlns:xacro="http://ros.org/wiki/xacro">
+<robot xmlns:xacro="http://ros.org/wiki/xacro" name="h2c_hydrophone">
   <xacro:macro name="h2c_hydrophone" params="name parent position:='0 0 0' orientation:='0 0 0'">
     <link name="${name}_link">
       <visual>
-        <origin xyz="0 0 0" rpy="0 0 0" />
+        <origin xyz="0 0 0" rpy="0 0 0"/>
         <geometry>
-          <cylinder length="0.05695" radius="0.0125" />
+          <cylinder length="0.05695" radius="0.0125"/>
         </geometry>
       </visual>
       <collision name="${name}_collision">
-        <origin xyz="0 0 0" rpy="0 0 0" />
+        <origin xyz="0 0 0" rpy="0 0 0"/>
         <geometry>
-          <cylinder length="0.05695" radius="0.02489" />
+          <cylinder length="0.05695" radius="0.02489"/>
         </geometry>
       </collision>
       <inertial>
-        <mass value="0.5" />
-        <inertia ixx="0.008545" ixy="0.0" ixz="0.0" iyy="0.008545" iyz="0.0" izz="0.0144" />
+        <mass value="0.5"/>
+        <inertia ixx="0.008545" ixy="0.0" ixz="0.0" iyy="0.008545" iyz="0.0" izz="0.0144"/>
       </inertial>
     </link>
     <joint name="${name}_joint" type="fixed">
-      <parent link="${parent}" />
-      <child link="${name}_link" />
-      <origin xyz="${position}" rpy="${orientation}" />
-      <axis rpy="0 0 0" xyz="0 0 1" />
+      <parent link="${parent}"/>
+      <child link="${name}_link"/>
+      <origin xyz="${position}" rpy="${orientation}"/>
+      <axis rpy="0 0 0" xyz="0 0 1"/>
     </joint>
   </xacro:macro>

File: auv_description/auv_common_descriptions/urdf/sensors/logitech_c920_camera.urdf.xacro (robot description, xacro)
@@ -1,11 +1,10 @@
 <?xml version="1.0"?>
-<robot name="logitech_c920_camera" xmlns:xacro="http://ros.org/wiki/xacro">
-  <xacro:macro name="logitech_c920_camera"
-    params="name parent position:='0 0 0' orientation:='0 0 0'">
+<robot xmlns:xacro="http://ros.org/wiki/xacro" name="logitech_c920_camera">
+  <xacro:macro name="logitech_c920_camera" params="name parent position:='0 0 0' orientation:='0 0 0'">
     <link name="${name}_link">
       <visual>
-        <origin xyz="0 0 0" rpy="0 0 ${math.pi}" />
+        <origin xyz="0 0 0" rpy="0 0 ${math.pi}"/>
         <geometry>
-          <box size="0.02 0.094 0.0433" />
+          <box size="0.02 0.094 0.0433"/>
           <!-- <mesh
             filename="package://auv_common_descriptions/meshes/bar30/bar30.dae"
@@ -14,7 +13,7 @@
       </visual>
       <collision name="${name}_collision">
-        <origin xyz="0 0 0" rpy="0 0 ${math.pi}" />
+        <origin xyz="0 0 0" rpy="0 0 ${math.pi}"/>
         <geometry>
-          <box size="0.02 0.094 0.0433" />
+          <box size="0.02 0.094 0.0433"/>
           <!-- <mesh
             filename="package://auv_common_descriptions/meshes/bar30/bar30.dae"
@@ -23,20 +22,20 @@
       </collision>
       <inertial>
-        <mass value="0.162" />
-        <inertia ixx="0.0001" ixy="0.0" ixz="0.0" iyy="0.0001" iyz="0.0" izz="0.0001" />
+        <mass value="0.162"/>
+        <inertia ixx="0.0001" ixy="0.0" ixz="0.0" iyy="0.0001" iyz="0.0" izz="0.0001"/>
       </inertial>
     </link>
-    <link name="${name}_optical_link" />
+    <link name="${name}_optical_link"/>
     <joint name="${name}_joint" type="fixed">
-      <parent link="${parent}" />
-      <child link="${name}_link" />
-      <origin xyz="${position}" rpy="${orientation}" />
-      <axis rpy="0 0 0" xyz="0 0 1" />
+      <parent link="${parent}"/>
+      <child link="${name}_link"/>
+      <origin xyz="${position}" rpy="${orientation}"/>
+      <axis rpy="0 0 0" xyz="0 0 1"/>
     </joint>
     <joint name="${name}_optical_joint" type="fixed">
-      <axis rpy="0 0 0" xyz="0 0 1" />
-      <parent link="${name}_link" />
-      <child link="${name}_optical_link" />
-      <origin xyz="0.01 0 0" rpy="${-math.pi/2} 0 ${-math.pi/2}" />
+      <axis rpy="0 0 0" xyz="0 0 1"/>
+      <parent link="${name}_link"/>
+      <child link="${name}_optical_link"/>
+      <origin xyz="0.01 0 0" rpy="${-math.pi/2} 0 ${-math.pi/2}"/>
     </joint>
   </xacro:macro>

File: auv_description/auv_common_descriptions/urdf/sensors/ping360.urdf.xacro (robot description, xacro)
@@ -1,39 +1,35 @@
 <?xml version="1.0"?>
-<robot name="ping360" xmlns:xacro="http://ros.org/wiki/xacro">
+<robot xmlns:xacro="http://ros.org/wiki/xacro" name="ping360">
   <xacro:macro name="ping360" params="name parent position:='0 0 0' orientation:='0 0 0'">
     <link name="${name}_mount_link">
       <visual>
-        <origin xyz="0 0 0" rpy="0 0 ${math.pi}" />
+        <origin xyz="0 0 0" rpy="0 0 ${math.pi}"/>
         <geometry>
-          <mesh
-            filename="package://auv_common_descriptions/meshes/ping360/ping360.dae"
-            scale="0.001 0.001 0.001" />
+          <mesh filename="package://auv_common_descriptions/meshes/ping360/ping360.dae" scale="0.001 0.001 0.001"/>
         </geometry>
       </visual>
       <collision name="${name}_collision">
-        <origin xyz="0 0 0" rpy="0 0 ${math.pi}" />
+        <origin xyz="0 0 0" rpy="0 0 ${math.pi}"/>
         <geometry>
-          <mesh
-            filename="package://auv_common_descriptions/meshes/ping360/ping360.dae"
-            scale="0.001 0.001 0.001" />
+          <mesh filename="package://auv_common_descriptions/meshes/ping360/ping360.dae" scale="0.001 0.001 0.001"/>
         </geometry>
       </collision>
       <inertial>
-        <mass value="0.5" />
-        <inertia ixx="0.008545" ixy="0.0" ixz="0.0" iyy="0.008545" iyz="0.0" izz="0.0144" />
+        <mass value="0.5"/>
+        <inertia ixx="0.008545" ixy="0.0" ixz="0.0" iyy="0.008545" iyz="0.0" izz="0.0144"/>
       </inertial>
     </link>
-    <link name="${name}_link" />
+    <link name="${name}_link"/>
     <joint name="${name}_joint" type="fixed">
-      <parent link="${parent}" />
-      <child link="${name}_mount_link" />
-      <origin xyz="${position}" rpy="${orientation}" />
-      <axis rpy="0 0 0" xyz="0 0 1" />
+      <parent link="${parent}"/>
+      <child link="${name}_mount_link"/>
+      <origin xyz="${position}" rpy="${orientation}"/>
+      <axis rpy="0 0 0" xyz="0 0 1"/>
     </joint>
     <joint name="${name}_scan_joint" type="fixed">
-      <axis rpy="0 0 0" xyz="0 0 1" />
-      <parent link="${name}_mount_link" />
-      <child link="${name}_link" />
-      <origin xyz="0 0 0.065" rpy="0 0 0" />
+      <axis rpy="0 0 0" xyz="0 0 1"/>
+      <parent link="${name}_mount_link"/>
+      <child link="${name}_link"/>
+      <origin xyz="0 0 0.065" rpy="0 0 0"/>
     </joint>
   </xacro:macro>

File: auv_description/auv_common_descriptions/urdf/sensors/sonar.urdf.xacro (robot description, xacro)
@@ -1,32 +1,28 @@
 <?xml version="1.0"?>
-<robot name="sonar" xmlns:xacro="http://ros.org/wiki/xacro">
+<robot xmlns:xacro="http://ros.org/wiki/xacro" name="sonar">
   <xacro:macro name="sonar" params="name parent position:='0 0 0' orientation:='0 0 0'">
     <link name="${name}_link">
       <visual>
-        <origin xyz="0 0 0" rpy="0 0 0" />
+        <origin xyz="0 0 0" rpy="0 0 0"/>
         <geometry>
-          <mesh
-            filename="package://auv_common_descriptions/meshes/sonar/sonar.dae"
-            scale="0.001 0.001 0.001" />
+          <mesh filename="package://auv_common_descriptions/meshes/sonar/sonar.dae" scale="0.001 0.001 0.001"/>
         </geometry>
       </visual>
       <collision name="${name}_collision">
-        <origin xyz="0 0 0" rpy="0 0 0" />
+        <origin xyz="0 0 0" rpy="0 0 0"/>
         <geometry>
-          <mesh
-            filename="package://auv_common_descriptions/meshes/sonar/sonar.dae"
-            scale="0.001 0.001 0.001" />
+          <mesh filename="package://auv_common_descriptions/meshes/sonar/sonar.dae" scale="0.001 0.001 0.001"/>
         </geometry>
       </collision>
       <inertial>
-        <mass value="0.15" />
-        <inertia ixx="0.001" ixy="0.0" ixz="0.0" iyy="0.001" iyz="0.0" izz="0.001" />
+        <mass value="0.15"/>
+        <inertia ixx="0.001" ixy="0.0" ixz="0.0" iyy="0.001" iyz="0.0" izz="0.001"/>
       </inertial>
     </link>
     <joint name="${name}_joint" type="fixed">
-      <parent link="${parent}" />
-      <child link="${name}_link" />
-      <origin xyz="${position}" rpy="${orientation}" />
-      <axis rpy="0 0 0" xyz="0 0 1" />
+      <parent link="${parent}"/>
+      <child link="${name}_link"/>
+      <origin xyz="${position}" rpy="${orientation}"/>
+      <axis rpy="0 0 0" xyz="0 0 1"/>
     </joint>
   </xacro:macro>
