Commit message: format xml

File: auv_description/auv_common_descriptions/urdf/sensors/wayfinder_dvl.urdf.xacro (robot description, xacro)
@@ -1,20 +1,18 @@
 <?xml version="1.0"?>
-<robot name="wayfinder_dvl" xmlns:xacro="http://ros.org/wiki/xacro">
+<robot xmlns:xacro="http://ros.org/wiki/xacro" name="wayfinder_dvl">
   <xacro:macro name="wayfinder_dvl" params="name parent position:='0 0 0' orientation:='0 0 0'">
     <link name="${name}_mount_link">
       <visual>
-        <origin xyz="0 0 0" rpy="${math.pi} 0 0" />
+        <origin xyz="0 0 0" rpy="${math.pi} 0 0"/>
         <geometry>
-          <mesh filename="package://auv_common_descriptions/meshes/wayfinder_dvl/dvl.dae"
-            scale="0.001 0.001 0.001" />
-          <material name="black" />
+          <mesh filename="package://auv_common_descriptions/meshes/wayfinder_dvl/dvl.dae" scale="0.001 0.001 0.001"/>
+          <material name="black"/>
         </geometry>
       </visual>
       <collision name="${name}_collision">
-        <origin xyz="0 0 0" rpy="${math.pi} 0 0" />
+        <origin xyz="0 0 0" rpy="${math.pi} 0 0"/>
         <geometry>
-          <mesh filename="package://auv_common_descriptions/meshes/wayfinder_dvl/dvl.dae"
-            scale="0.001 0.001 0.001" />
-          <material name="black" />
+          <mesh filename="package://auv_common_descriptions/meshes/wayfinder_dvl/dvl.dae" scale="0.001 0.001 0.001"/>
+          <material name="black"/>
         </geometry>
       </collision>
@@ -23,35 +21,35 @@
       <inertial>
         <!-- 0.313 in water -->
-        <mass value="0.947" />
+        <mass value="0.947"/>
         <!-- volume: 100mm x 100mm x 70mm -->
         <!-- 0.0007 m^3-->
-        <inertia ixx="0.001176" ixy="0.0" ixz="0.0" iyy="0.001176" iyz="0.0" izz="0.001578" />
+        <inertia ixx="0.001176" ixy="0.0" ixz="0.0" iyy="0.001176" iyz="0.0" izz="0.001578"/>
       </inertial>
     </link>
-    <link name="${name}_sensor_surface_link" />
-    <link name="${name}_link" />
+    <link name="${name}_sensor_surface_link"/>
+    <link name="${name}_link"/>
     <joint name="${name}_chasis_joint" type="fixed">
-      <parent link="${parent}" />
-      <child link="${name}_mount_link" />
-      <origin xyz="${position}" rpy="${orientation}" />
-      <axis rpy="0 0 0" xyz="0 0 1" />
+      <parent link="${parent}"/>
+      <child link="${name}_mount_link"/>
+      <origin xyz="${position}" rpy="${orientation}"/>
+      <axis rpy="0 0 0" xyz="0 0 1"/>
     </joint>
     <joint name="${name}_sensor_surface_joint" type="fixed">
-      <axis rpy="0 0 0" xyz="0 0 1" />
-      <parent link="${name}_mount_link" />
-      <child link="${name}_sensor_surface_link" />
-      <origin xyz="0 0 -0.07" rpy="0 0 0" />
+      <axis rpy="0 0 0" xyz="0 0 1"/>
+      <parent link="${name}_mount_link"/>
+      <child link="${name}_sensor_surface_link"/>
+      <origin xyz="0 0 -0.07" rpy="0 0 0"/>
     </joint>
     <joint name="${name}_cog_joint" type="fixed">
-      <axis rpy="0 0 0" xyz="0 0 1" />
-      <parent link="${name}_mount_link" />
-      <child link="${name}_cog" />
-      <origin xyz="0 0 -0.035" rpy="0 0 0" />
+      <axis rpy="0 0 0" xyz="0 0 1"/>
+      <parent link="${name}_mount_link"/>
+      <child link="${name}_cog"/>
+      <origin xyz="0 0 -0.035" rpy="0 0 0"/>
     </joint>
     <joint name="${name}_sensor_joint" type="fixed">
-      <axis rpy="0 0 0" xyz="0 0 1" />
-      <parent link="${name}_sensor_surface_link" />
-      <child link="${name}_link" />
-      <origin xyz="0 0 0" rpy="0 0 ${-3*math.pi/4}" />
+      <axis rpy="0 0 0" xyz="0 0 1"/>
+      <parent link="${name}_sensor_surface_link"/>
+      <child link="${name}_link"/>
+      <origin xyz="0 0 0" rpy="0 0 ${-3*math.pi/4}"/>
     </joint>
     <!-- <gazebo reference="${name}_propeller_link">

File: auv_description/auv_common_descriptions/urdf/sensors/xsens_mti_g710.urdf.xacro (robot description, xacro)
@@ -1,32 +1,28 @@
 <?xml version="1.0"?>
-<robot name="xsens_mti_g710" xmlns:xacro="http://ros.org/wiki/xacro">
+<robot xmlns:xacro="http://ros.org/wiki/xacro" name="xsens_mti_g710">
   <xacro:macro name="xsens_mti_g710" params="name parent position:='0 0 0' orientation:='0 0 0'">
     <link name="${name}_link">
       <visual>
-        <origin xyz="0 0 0" rpy="0 0 ${math.pi}" />
+        <origin xyz="0 0 0" rpy="0 0 ${math.pi}"/>
         <geometry>
-          <mesh
-            filename="package://auv_common_descriptions/meshes/xsens_mti_g710/xsens_mti_g710.dae"
-            scale="0.001 0.001 0.001" />
+          <mesh filename="package://auv_common_descriptions/meshes/xsens_mti_g710/xsens_mti_g710.dae" scale="0.001 0.001 0.001"/>
         </geometry>
       </visual>
       <collision name="${name}_collision">
-        <origin xyz="0 0 0" rpy="0 0 ${math.pi}" />
+        <origin xyz="0 0 0" rpy="0 0 ${math.pi}"/>
         <geometry>
-          <mesh
-            filename="package://auv_common_descriptions/meshes/xsens_mti_g710/xsens_mti_g710.dae"
-            scale="0.001 0.001 0.001" />
+          <mesh filename="package://auv_common_descriptions/meshes/xsens_mti_g710/xsens_mti_g710.dae" scale="0.001 0.001 0.001"/>
         </geometry>
       </collision>
       <inertial>
-        <mass value="0.5" />
-        <inertia ixx="0.008545" ixy="0.0" ixz="0.0" iyy="0.008545" iyz="0.0" izz="0.0144" />
+        <mass value="0.5"/>
+        <inertia ixx="0.008545" ixy="0.0" ixz="0.0" iyy="0.008545" iyz="0.0" izz="0.0144"/>
       </inertial>
     </link>
     <joint name="${name}_joint" type="fixed">
-      <parent link="${parent}" />
-      <child link="${name}_link" />
-      <origin xyz="${position}" rpy="${orientation}" />
-      <axis rpy="0 0 0" xyz="0 0 1" />
+      <parent link="${parent}"/>
+      <child link="${name}_link"/>
+      <origin xyz="${position}" rpy="${orientation}"/>
+      <axis rpy="0 0 0" xyz="0 0 1"/>
     </joint>
   </xacro:macro>

File: auv_description/taluy_description/urdf/auv.urdf.xacro (robot description, xacro)
@@ -1,5 +1,5 @@
 <?xml version="1.0"?>
-<robot name="taluy" xmlns:xacro="http://www.ros.org/wiki/xacro">
-  <xacro:include filename="$(find taluy_description)/urdf/auv_base.urdf.xacro" />
-  <xacro:taluy_base />
+<robot xmlns:xacro="http://www.ros.org/wiki/xacro" name="taluy">
+  <xacro:include filename="$(find taluy_description)/urdf/auv_base.urdf.xacro"/>
+  <xacro:taluy_base/>
 </robot>

File: auv_description/taluy_description/urdf/auv_base.urdf.xacro (robot description, xacro)
@@ -1,107 +1,59 @@
 <?xml version="1.0"?>
-<robot name="taluy" xmlns:xacro="http://www.ros.org/wiki/xacro">
+<robot xmlns:xacro="http://www.ros.org/wiki/xacro" name="taluy">
   <xacro:macro name="taluy_base">
-    <xacro:include filename="$(find auv_common_descriptions)/urdf/actuators.urdf.xacro" />
-    <xacro:include
-      filename="$(find auv_common_descriptions)/urdf/sensors.urdf.xacro" />
-    <xacro:include
-      filename="$(find auv_common_descriptions)/urdf/materials.urdf.xacro" />
-    <xacro:arg name="angled_thruster_z_offset" default="-0.01" />
+    <xacro:include filename="$(find auv_common_descriptions)/urdf/actuators.urdf.xacro"/>
+    <xacro:include filename="$(find auv_common_descriptions)/urdf/sensors.urdf.xacro"/>
+    <xacro:include filename="$(find auv_common_descriptions)/urdf/materials.urdf.xacro"/>
+    <xacro:arg name="angled_thruster_z_offset" default="-0.01"/>
     <link name="base_link">
       <inertial>
-        <origin xyz="0 0 0" rpy="0 0 0" />
-        <mass value="25.0" />
-        <inertia ixx="0.1" iyy="0.1" izz="0.1" ixy="0.01" iyz="0.01" ixz="0.1" />
+        <origin xyz="0 0 0" rpy="0 0 0"/>
+        <mass value="25.0"/>
+        <inertia ixx="0.1" iyy="0.1" izz="0.1" ixy="0.01" iyz="0.01" ixz="0.1"/>
       </inertial>
       <visual>
-        <origin xyz="0.0 0.0 0.0" rpy="0 0 0" />
+        <origin xyz="0.0 0.0 0.0" rpy="0 0 0"/>
         <geometry>
-          <mesh filename="package://taluy_description/meshes/body/body.stl"
-            scale="1 1 1" />
+          <mesh filename="package://taluy_description/meshes/body/body.stl" scale="1 1 1"/>
         </geometry>
-        <material name="black" />
+        <material name="black"/>
       </visual>
       <collision>
-        <origin xyz="0.0 0.0 0.0" rpy="0 0 0" />
+        <origin xyz="0.0 0.0 0.0" rpy="0 0 0"/>
         <geometry>
-          <mesh filename="package://taluy_description/meshes/body/body.stl"
-            scale="1 1 1" />
+          <mesh filename="package://taluy_description/meshes/body/body.stl" scale="1 1 1"/>
         </geometry>
       </collision>
     </link>
-    <link name="base_link_ned" />
+    <link name="base_link_ned"/>
     <joint name="base_link_joint" type="fixed">
-      <origin xyz="0 0 0" rpy="${math.pi} 0 0" />
-      <parent link="base_link_ned" />
-      <child link="base_link" />
+      <origin xyz="0 0 0" rpy="${math.pi} 0 0"/>
+      <parent link="base_link_ned"/>
+      <child link="base_link"/>
     </joint>
-    <xacro:t200_thruster name="thruster_0" parent="base_link" position="0.14250 0.20070 -0.00525"
-      orientation="${pi} 0 ${-pi/2}" />
-    <xacro:t200_thruster name="thruster_1" parent="base_link" position="0.14250 -0.20070 -0.00525"
-      orientation="${pi} 0 ${pi/2}" />
-    <xacro:t200_thruster name="thruster_2" parent="base_link" position="-0.14250 0.20070 -0.00525"
-      orientation="${pi} 0 ${-pi/2}" />
-    <xacro:t200_thruster name="thruster_3" parent="base_link" position="-0.14250 -0.20070 -0.00525"
-      orientation="${pi} 0 ${pi/2}" />
-    <xacro:t200_thruster name="thruster_4" parent="base_link"
-      position="0.352398 0.216638 $(arg angled_thruster_z_offset)"
-      orientation="${-pi/2} 0 ${-7*pi/4}" />
-    <xacro:t200_thruster name="thruster_5" parent="base_link"
-      position="0.352398 -0.216638 $(arg angled_thruster_z_offset)"
-      orientation="${pi/2} 0 ${7*pi/4}" />
-    <xacro:t200_thruster name="thruster_6" parent="base_link"
-      position="-0.352398 0.216638 $(arg angled_thruster_z_offset)"
-      orientation="${-pi/2} 0 ${-pi/4}" />
-    <xacro:t200_thruster name="thruster_7" parent="base_link"
-      position="-0.352398 -0.216638 $(arg angled_thruster_z_offset)" orientation="${pi/2} 0 ${pi/4}" />
-    <xacro:wayfinder_dvl
-      name="base_link/dvl" parent="base_link" position="0.2 0 -0.11"
-      orientation="0 0 0" />
-    <xacro:xsens_mti_g710 name="base_link/imu" parent="base_link"
-      position="-0.199 0 -0.0108"
-      orientation="0 0 ${math.pi}" />
-    <xacro:h2c_hydrophone name="base_link/hydrophone_0"
-      parent="base_link"
-      position="0.325 0.205 -0.15"
-      orientation="0 0 0" />
-    <xacro:h2c_hydrophone name="base_link/hydrophone_1" parent="base_link"
-      position="0.325 -0.205 -0.15"
-      orientation="0 0 0" />
-    <xacro:h2c_hydrophone name="base_link/hydrophone_2" parent="base_link"
-      position="-0.325 0.205 -0.15"
-      orientation="0 0 0" />
-    <xacro:h2c_hydrophone name="base_link/hydrophone_3" parent="base_link"
-      position="-0.325 -0.205 -0.15"
-      orientation="0 0 0" />
-    <xacro:ping360 name="base_link/ping360" parent="base_link"
-      position="0.2 0 0.134"
-      orientation="0 0 0" />
-    <xacro:bar30 name="base_link/external_pressure_sensor" parent="base_link"
-      position="0 0 0.07"
-      orientation="0 0 0" />
-    <xacro:logitech_c920_camera name="base_link/front_camera"
-      parent="base_link" position="0.35 0 0"
-      orientation="0 0 0" />
-    <xacro:logitech_c920_camera name="base_link/bottom_camera"
-      parent="base_link" position="0 0 -0.07"
-      orientation="0 ${math.pi/2} ${math.pi/2}" />
-    <xacro:torpedo name="base_link/left_torpedo"
-      parent="base_link" position="0.2 0.1 -0.11"
-      orientation="0 0 0" />
-    <xacro:torpedo name="base_link/right_torpedo"
-      parent="base_link" position="0.2 -0.1 -0.11"
-      orientation="0 0 0" />
-    <xacro:sonar name="base_link/sonar_front" parent="base_link"
-      position="0.38 0.09 0.09"
-      orientation="0 0 0" />
-    <xacro:sonar name="base_link/sonar_back" parent="base_link"
-      position="-0.42 -0.09 0.09"
-      orientation="0 0 ${math.pi}" />
-    <xacro:sonar name="base_link/sonar_right" parent="base_link"
-      position="0.02 -0.21 -0.14"
-      orientation="0 0 ${-math.pi/2}" />
-    <xacro:sonar name="base_link/sonar_left" parent="base_link"
-      position="0.02 0.21 -0.14"
-      orientation="0 0 ${math.pi/2}" />
+    <xacro:t200_thruster name="thruster_0" parent="base_link" position="0.14250 0.20070 -0.00525" orientation="${pi} 0 ${-pi/2}"/>
+    <xacro:t200_thruster name="thruster_1" parent="base_link" position="0.14250 -0.20070 -0.00525" orientation="${pi} 0 ${pi/2}"/>
+    <xacro:t200_thruster name="thruster_2" parent="base_link" position="-0.14250 0.20070 -0.00525" orientation="${pi} 0 ${-pi/2}"/>
+    <xacro:t200_thruster name="thruster_3" parent="base_link" position="-0.14250 -0.20070 -0.00525" orientation="${pi} 0 ${pi/2}"/>
+    <xacro:t200_thruster name="thruster_4" parent="base_link" position="0.352398 0.216638 $(arg angled_thruster_z_offset)" orientation="${-pi/2} 0 ${-7*pi/4}"/>
+    <xacro:t200_thruster name="thruster_5" parent="base_link" position="0.352398 -0.216638 $(arg angled_thruster_z_offset)" orientation="${pi/2} 0 ${7*pi/4}"/>
+    <xacro:t200_thruster name="thruster_6" parent="base_link" position="-0.352398 0.216638 $(arg angled_thruster_z_offset)" orientation="${-pi/2} 0 ${-pi/4}"/>
+    <xacro:t200_thruster name="thruster_7" parent="base_link" position="-0.352398 -0.216638 $(arg angled_thruster_z_offset)" orientation="${pi/2} 0 ${pi/4}"/>
+    <xacro:wayfinder_dvl name="base_link/dvl" parent="base_link" position="0.2 0 -0.11" orientation="0 0 0"/>
+    <xacro:xsens_mti_g710 name="base_link/imu" parent="base_link" position="-0.199 0 -0.0108" orientation="0 0 ${math.pi}"/>
+    <xacro:h2c_hydrophone name="base_link/hydrophone_0" parent="base_link" position="0.325 0.205 -0.15" orientation="0 0 0"/>
+    <xacro:h2c_hydrophone name="base_link/hydrophone_1" parent="base_link" position="0.325 -0.205 -0.15" orientation="0 0 0"/>
+    <xacro:h2c_hydrophone name="base_link/hydrophone_2" parent="base_link" position="-0.325 0.205 -0.15" orientation="0 0 0"/>
+    <xacro:h2c_hydrophone name="base_link/hydrophone_3" parent="base_link" position="-0.325 -0.205 -0.15" orientation="0 0 0"/>
+    <xacro:ping360 name="base_link/ping360" parent="base_link" position="0.2 0 0.134" orientation="0 0 0"/>
+    <xacro:bar30 name="base_link/external_pressure_sensor" parent="base_link" position="0 0 0.07" orientation="0 0 0"/>
+    <xacro:logitech_c920_camera name="base_link/front_camera" parent="base_link" position="0.35 0 0" orientation="0 0 0"/>
+    <xacro:logitech_c920_camera name="base_link/bottom_camera" parent="base_link" position="0 0 -0.07" orientation="0 ${math.pi/2} ${math.pi/2}"/>
+    <xacro:torpedo name="base_link/left_torpedo" parent="base_link" position="0.2 0.1 -0.11" orientation="0 0 0"/>
+    <xacro:torpedo name="base_link/right_torpedo" parent="base_link" position="0.2 -0.1 -0.11" orientation="0 0 0"/>
+    <xacro:sonar name="base_link/sonar_front" parent="base_link" position="0.38 0.09 0.09" orientation="0 0 0"/>
+    <xacro:sonar name="base_link/sonar_back" parent="base_link" position="-0.42 -0.09 0.09" orientation="0 0 ${math.pi}"/>
+    <xacro:sonar name="base_link/sonar_right" parent="base_link" position="0.02 -0.21 -0.14" orientation="0 0 ${-math.pi/2}"/>
+    <xacro:sonar name="base_link/sonar_left" parent="base_link" position="0.02 0.21 -0.14" orientation="0 0 ${math.pi/2}"/>
     <!-- <link name="base_footprint">
       <inertial>

Commit message: four finger

File: auv_description/auv_common_descriptions/urdf/actuators.urdf.xacro (robot description, xacro)
@@ -5,3 +5,4 @@
   <xacro:include filename="$(find auv_common_descriptions)/urdf/actuators/torpedo_bottom.urdf.xacro"/>
   <xacro:include filename="$(find auv_common_descriptions)/urdf/actuators/ball_dropper.urdf.xacro"/>
+  <xacro:include filename="$(find auv_common_descriptions)/urdf/actuators/gripper.urdf.xacro"/>
 </robot>

File: auv_description/taluy_description/urdf/auv_base.urdf.xacro (robot description, xacro)
@@ -62,17 +62,6 @@
     <xacro:ball_dropper name="${namespace}/base_link/ball_dropper" parent="${namespace}/base_link" position="0.1004 0.0745 -0.1953" orientation="0 0 0"/>
     <xacro:realsense_d435 name="${namespace}/camera" parent="${namespace}/base_link" position="-0.35 0 0" orientation="0 0 ${math.pi}"/>
-    <!-- <link name="base_footprint">
-      <inertial>
-        <origin xyz="0 0 0" rpy="0 0 0" />
-        <mass value="15.0" />
-        <inertia ixx="39.351246" iyy="103.261717" izz="127.702526" ixy="-5e-06" iyz="6e-06"
-          ixz="4.403436" />
-      </inertial>
-    </link>
-    <joint name="base_link_joint" type="fixed">
-      <origin xyz="0 0 ${-base_z_offsett + 0.06 - draft}" rpy="0 0 0" />
-      <parent link="base_footprint" />
-      <child link="base_link" />
-    </joint> -->
+    <!-- Gripper mounted underneath the robot, facing downwards -->
+    <xacro:gripper name="${namespace}/gripper" parent="${namespace}/base_link" position="0.15 0 -0.15" orientation="0 ${math.pi/2} 0" namespace="${namespace}"/>
   </xacro:macro>
 </robot>
