Commit message: ready for test

File: auv_sim/auv_sim_description/taluy_sim_description/urdf/dynamics.urdf.xacro (robot description, xacro)
@@ -18,5 +18,5 @@
     assume NWU (otherwise cob is below cog?).
     -->
-  <xacro:property name="cob" value="0.0 0.0 0.2"/>
+  <xacro:property name="cob" value="-0.02 0.0 0.2"/>
   <!-- Volume, see p.31 in Berg2012, normally 0.009165088 -->
   <xacro:property name="volume" value="0.027"/>

Commit message: civelekiz

File: auv_sim/auv_sim_description/taluy_sim_description/urdf/dynamics.urdf.xacro (robot description, xacro)
@@ -18,5 +18,5 @@
     assume NWU (otherwise cob is below cog?).
     -->
-  <xacro:property name="cob" value="-0.02 0.0 0.2"/>
+  <xacro:property name="cob" value="0.0 0.0 0.2"/>
   <!-- Volume, see p.31 in Berg2012, normally 0.009165088 -->
   <xacro:property name="volume" value="0.027"/>

Commit message: start.

File: auv_sim/auv_sim_description/taluy_sim_description/urdf/dynamics.urdf.xacro (robot description, xacro)
@@ -18,5 +18,5 @@
     assume NWU (otherwise cob is below cog?).
     -->
-  <xacro:property name="cob" value="0.0 0.0 0.2"/>
+  <xacro:property name="cob" value="0.0 0.0 0.02"/>
   <!-- Volume, see p.31 in Berg2012, normally 0.009165088 -->
   <xacro:property name="volume" value="0.027"/>
