Commit message: fix stl

File: auv_description/taluy_mini_description/urdf/auv_base.urdf.xacro (robot description, xacro)
@@ -14,14 +14,14 @@
       </inertial>
       <visual>
-        <origin xyz="0.0 0.0 0.0" rpy="0 0 0"/>
+        <origin xyz="0.2 0.0 0.0" rpy="0 0 ${math.pi/2}"/>
         <geometry>
-          <mesh filename="package://taluy_mini_description/meshes/body/body.stl" scale="1 1 1"/>
+          <mesh filename="package://taluy_mini_description/meshes/body/body.stl" scale="0.001 0.001 0.001"/>
         </geometry>
         <material name="black"/>
       </visual>
       <collision>
-        <origin xyz="0.0 0.0 0.0" rpy="0 0 0"/>
+        <origin xyz="0.2 0.0 0.0" rpy="0 0 ${math.pi/2}"/>
         <geometry>
-          <mesh filename="package://taluy_mini_description/meshes/body/body.stl" scale="1 1 1"/>
+          <mesh filename="package://taluy_mini_description/meshes/body/body.stl" scale="0.001 0.001 0.001"/>
         </geometry>
       </collision>
@@ -51,5 +51,5 @@
     <xacro:xsens_mti_g710 name="${namespace}/base_link/imu" parent="${namespace}/base_link" position="-0.162 0 -0.0108" orientation="0 0 ${math.pi}"/>
     <xacro:bar30 name="${namespace}/base_link/external_pressure_sensor" parent="${namespace}/base_link" position="0 0 0.07" orientation="0 0 0"/>
-    <xacro:logitech_c920_camera name="${namespace}/base_link/front_camera" parent="${namespace}/base_link" position="0.35 0 0" orientation="0 0 0"/>
+    <xacro:logitech_c920_camera name="${namespace}/base_link/front_camera" parent="${namespace}/base_link" position="0.08 0 0" orientation="0 0 0"/>
     <xacro:logitech_c920_camera name="${namespace}/base_link/bottom_camera" parent="${namespace}/base_link" position="0 0 -0.07" orientation="0 ${math.pi/2} ${-math.pi/2}"/>
   </xacro:macro>

Commit message: rviz

File: auv_description/taluy_mini_description/urdf/auv_base.urdf.xacro (robot description, xacro)
@@ -18,5 +18,5 @@
           <mesh filename="package://taluy_mini_description/meshes/body/body.stl" scale="0.001 0.001 0.001"/>
         </geometry>
-        <material name="black"/>
+        <material name="gray"/>
       </visual>
       <collision>

File: auv_sim/auv_sim_description/taluy_mini_sim_description/urdf/sensors.urdf.xacro (robot description, xacro)
@@ -7,5 +7,5 @@
   <xacro:logitech_c920_camera_sim name="${namespace}/base_link/front_camera" topic_name="cameras/cam_front"/>
   <xacro:logitech_c920_camera_sim name="${namespace}/base_link/bottom_camera" topic_name="cameras/cam_bottom"/>
-  <xacro:bar30_sim name="${namespace}/base_link/external_pressure_sensor" update_rate="$(arg pressure_update_rate)"/>
+  <xacro:bar30_sim name="${namespace}/base_link/external_pressure_sensor" namespace="${namespace}" update_rate="$(arg pressure_update_rate)"/>
   <xacro:xsens_mti_g710_sim name="${namespace}/base_link/imu" namespace="${namespace}" static_reference_frame="${inertial_reference_frame}" update_rate="$(arg imu_update_rate)"/>
 </robot>

Commit message: fixes

File: auv_description/taluy_mini_description/urdf/auv_base.urdf.xacro (robot description, xacro)
@@ -3,5 +3,5 @@
   <!-- create xacro property -->
   <xacro:property name="namespace" value="taluy_mini"/>
-  <xacro:macro name="taluy_mini_base">
+  <xacro:macro name="taluy_mini_base" params="use_models:=false">
     <xacro:include filename="$(find auv_common_descriptions)/urdf/actuators.urdf.xacro"/>
     <xacro:include filename="$(find auv_common_descriptions)/urdf/sensors.urdf.xacro"/>
@@ -54,4 +54,11 @@
     <xacro:logitech_c920_camera name="${namespace}/base_link/front_camera" parent="${namespace}/base_link" position="0.3 0 0" orientation="0.17 0 0"/>
     <xacro:logitech_c920_camera name="${namespace}/base_link/bottom_camera" parent="${namespace}/base_link" position="0 0 -0.07" orientation="0 ${math.pi/2} ${-math.pi/2}"/>
+    <xacro:wayfinder_dvl name="${namespace}/base_link/dvl" parent="${namespace}/base_link" position="0.2 0 -0.07" orientation="0 0 0"/>
+    <xacro:torpedo_camera name="${namespace}/base_link/torpedo_camera" parent="${namespace}/base_link" position="0.25 -0.09 -0.1" orientation="0 0 0"/>
+    <xacro:sonar name="${namespace}/base_link/sonar_front" parent="${namespace}/base_link" position="0.28 0 0.06" orientation="0 0 0"/>
+    <xacro:sonar name="${namespace}/base_link/sonar_back" parent="${namespace}/base_link" position="-0.28 0 0.06" orientation="0 0 ${math.pi}"/>
+    <xacro:sonar name="${namespace}/base_link/sonar_right" parent="${namespace}/base_link" position="0 -0.15 -0.07" orientation="0 0 ${-math.pi/2}"/>
+    <xacro:sonar name="${namespace}/base_link/sonar_left" parent="${namespace}/base_link" position="0 0.15 -0.07" orientation="0 0 ${math.pi/2}"/>
+    <xacro:realsense_d435 name="${namespace}/camera" parent="${namespace}/base_link" position="-0.25 0 0" orientation="0 0 ${math.pi}"/>
   </xacro:macro>
 </robot>

Commit message: imu

File: auv_description/taluy_mini_description/urdf/auv_base.urdf.xacro (robot description, xacro)
@@ -49,10 +49,10 @@
     <xacro:t200_thruster name="${namespace}/thruster_7" parent="${namespace}/base_link" position="-0.166012 -0.235802 -0.103472" orientation="0 ${pi/4} ${pi/4}"/>
     <!-- arka sag alt -->
-    <xacro:xsens_mti_g710 name="${namespace}/base_link/imu" parent="${namespace}/base_link" position="-0.162 0 -0.0108" orientation="${-math.pi / 2} 0 ${-math.pi / 2}"/>
+    <xacro:xsens_mti_g710 name="${namespace}/base_link/imu" parent="${namespace}/base_link" position="-0.162 0 -0.0108" orientation="0 0 ${math.pi}"/>
     <!-- <xacro:xsens_mti_g710 name="${namespace}/base_link/imu" parent="${namespace}/base_link" position="-0.162 0 -0.0108" orientation="0 0 0"/> -->
     <xacro:bar30 name="${namespace}/base_link/external_pressure_sensor" parent="${namespace}/base_link" position="0 0 0.07" orientation="0 0 0"/>
     <xacro:logitech_c920_camera name="${namespace}/base_link/front_camera" parent="${namespace}/base_link" position="0.3 0 0" orientation="0.17 0 0"/>
     <xacro:logitech_c920_camera name="${namespace}/base_link/bottom_camera" parent="${namespace}/base_link" position="0 0 -0.07" orientation="0 ${math.pi/2} ${-math.pi/2}"/>
-    <xacro:wayfinder_dvl name="${namespace}/base_link/dvl" parent="${namespace}/base_link" position="0.2 0 -0.07" orientation="0 0 0"/>
+    <xacro:wayfinder_dvl name="${namespace}/base_link/dvl" parent="${namespace}/base_link" position="0.0 0 -0.17" orientation="0 0 0"/>
     <xacro:torpedo_camera name="${namespace}/base_link/torpedo_camera" parent="${namespace}/base_link" position="0.25 -0.09 -0.1" orientation="0 0 0"/>
     <xacro:sonar name="${namespace}/base_link/sonar_front" parent="${namespace}/base_link" position="0.28 0 0.06" orientation="0 0 0"/>

File: auv_sim/auv_sim_description/taluy_mini_sim_description/urdf/dynamics.urdf.xacro (robot description, xacro)
@@ -13,6 +13,6 @@
 -->
 <robot xmlns:xacro="http://www.ros.org/wiki/xacro">
-  <xacro:property name="cob" value="0.0 0.0 0.15"/>
-  <xacro:property name="volume" value="0.015"/>
+  <xacro:property name="cob" value="0.0 0.0 0.2"/>
+  <xacro:property name="volume" value="0.027"/>
   <xacro:macro name="auv_hydro_model" params="namespace">
     <link name="${namespace}/base_link">
@@ -35,6 +35,6 @@
           0 0 0 0 0 0
         </added_mass>
-        <linear_damping>0 0 0 0 0 0</linear_damping>
-        <quadratic_damping>0 0 0 0 0 0</quadratic_damping>
+        <linear_damping>-30 -31 -89 -1.87 -1.87 -1.87</linear_damping>
+        <quadratic_damping>-77 -155 -136 -7.98 -7.98 -7.98</quadratic_damping>
       </hydrodynamic_model>
     </link>

Commit message: refactoring

File: auv_description/taluy_mini_description/urdf/auv_base.urdf.xacro (robot description, xacro)
@@ -1,5 +1,4 @@
 <?xml version="1.0"?>
 <robot xmlns:xacro="http://www.ros.org/wiki/xacro" name="taluy_mini">
-  <!-- create xacro property -->
   <xacro:property name="namespace" value="taluy_mini"/>
   <xacro:macro name="taluy_mini_base" params="use_models:=false">
@@ -27,10 +26,4 @@
       </collision>
     </link>
-    <!-- <link name="${namespace}/base_link_ned" />
-    <joint name="base_link_joint" type="fixed">
-      <origin xyz="0 0 0" rpy="${math.pi} 0 0" />
-      <parent link="${namespace}/base_link_ned" />
-      <child link="${namespace}/base_link" />
-    </joint> -->
     <xacro:t200_thruster name="${namespace}/thruster_0" parent="${namespace}/base_link" position="0.157582 0.234119 0.104193" orientation="0 ${-3*pi/4} ${pi/4}"/>
     <!-- on sol ust -->
@@ -50,15 +43,6 @@
     <!-- arka sag alt -->
     <xacro:xsens_mti_g710 name="${namespace}/base_link/imu" parent="${namespace}/base_link" position="-0.162 0 -0.0108" orientation="${math.pi} 0 ${math.pi/2}"/>
-    <!-- <xacro:xsens_mti_g710 name="${namespace}/base_link/imu" parent="${namespace}/base_link" position="-0.162 0 -0.0108" orientation="0 0 0"/> -->
     <xacro:bar30 name="${namespace}/base_link/external_pressure_sensor" parent="${namespace}/base_link" position="0 0 0.07" orientation="0 0 0"/>
-    <xacro:logitech_c920_camera name="${namespace}/base_link/front_camera" parent="${namespace}/base_link" position="0.3 0 0" orientation="0.0 0 0"/>
-    <xacro:logitech_c920_camera name="${namespace}/base_link/bottom_camera" parent="${namespace}/base_link" position="0 0 -0.07" orientation="0 ${math.pi/2} ${-math.pi/2}"/>
     <xacro:wayfinder_dvl name="${namespace}/base_link/dvl" parent="${namespace}/base_link" position="0.0 0 -0.17" orientation="0 0 0"/>
-    <xacro:torpedo_camera name="${namespace}/base_link/torpedo_camera" parent="${namespace}/base_link" position="0.25 -0.09 -0.1" orientation="0 0 0"/>
-    <xacro:sonar name="${namespace}/base_link/sonar_front" parent="${namespace}/base_link" position="0.28 0 0.06" orientation="0 0 0"/>
-    <xacro:sonar name="${namespace}/base_link/sonar_back" parent="${namespace}/base_link" position="-0.28 0 0.06" orientation="0 0 ${math.pi}"/>
-    <xacro:sonar name="${namespace}/base_link/sonar_right" parent="${namespace}/base_link" position="0 -0.15 -0.07" orientation="0 0 ${-math.pi/2}"/>
-    <xacro:sonar name="${namespace}/base_link/sonar_left" parent="${namespace}/base_link" position="0 0.15 -0.07" orientation="0 0 ${math.pi/2}"/>
-    <xacro:realsense_d435 name="${namespace}/camera" parent="${namespace}/base_link" position="-0.25 0 0" orientation="0 0 ${math.pi}"/>
   </xacro:macro>
 </robot>
