Commit message: need to fix close service

File: auv_description/taluy_description/urdf/parallel_gripper.xacro (robot description, xacro)
@@ -63,9 +63,11 @@
       <parent link="${namespace}/gripper_base"/>
       <child link="${namespace}/finger_left"/>
-      <origin rpy="0 0 0" xyz="0.0444267 0.0391376 0"/>
+      <!-- Y mesafesi artırıldı: 0.055 -> 0.065 (parmaklar arası mesafe daha da arttı) -->
+      <origin rpy="0 0 0" xyz="0.0444267 0.065 0"/>
       <axis xyz="0 0 1"/>
-      <dynamics damping="12" friction="1"/>
-      <!-- Lower max effort & speed so joint stalls on object instead of crushing it -->
-      <limit effort="15" lower="0.0" upper="0.35" velocity="0.1"/>
+      <!-- Dengeli ayar: Güçlü ama yumuşak (titreşim önleme) -->
+      <dynamics damping="30" friction="8"/>
+      <!-- Effort optimal: 100 -> 80 Nm (hala çok güçlü), velocity biraz daha yavaş -->
+      <limit effort="80" lower="-0.15" upper="0.25" velocity="0.02"/>
     </joint>
     <!-- Left Finger Tip -->
@@ -94,5 +96,6 @@
       <parent link="${namespace}/finger_left"/>
       <child link="${namespace}/finger_tip_left"/>
-      <origin rpy="3.14159265359 0 0" xyz="0.06431 0 0"/>
+      <!-- Ucu daha fazla içe doğru: Z ekseninde -0.15 rad (~-8.6°) rotasyon ekleyerek uç içe bakar -->
+      <origin rpy="3.14159265359 0 -0.15" xyz="0.06431 0 0"/>
     </joint>
     <!-- Right Finger -->
@@ -121,9 +124,11 @@
       <parent link="${namespace}/gripper_base"/>
       <child link="${namespace}/finger_right"/>
-      <origin rpy="3.14159265359 3.14159265359 3.14159265359" xyz="0.0444267 -0.0391376 0"/>
+      <!-- Y mesafesi artırıldı: -0.055 -> -0.065 (parmaklar arası mesafe daha da arttı) -->
+      <origin rpy="3.14159265359 3.14159265359 3.14159265359" xyz="0.0444267 -0.065 0"/>
       <axis xyz="0 0 -1"/>
-      <dynamics damping="12" friction="1"/>
-      <!-- Lower max effort & speed so joint stalls on object instead of crushing it -->
-      <limit effort="15" lower="0.0" upper="0.35" velocity="0.1"/>
+      <!-- Dengeli ayar: Güçlü ama yumuşak (titreşim önleme) -->
+      <dynamics damping="30" friction="8"/>
+      <!-- Effort optimal: 100 -> 80 Nm (hala çok güçlü), velocity biraz daha yavaş -->
+      <limit effort="80" lower="-0.15" upper="0.25" velocity="0.02"/>
     </joint>
     <!-- Right Finger Tip -->
@@ -152,90 +157,97 @@
       <parent link="${namespace}/finger_right"/>
       <child link="${namespace}/finger_tip_right"/>
-      <origin rpy="0 0 0" xyz="0.06431 0 0"/>
+      <!-- Ucu daha fazla içe doğru: Z ekseninde +0.15 rad (~+8.6°) rotasyon ekleyerek uç içe bakar -->
+      <origin rpy="0 0 0.15" xyz="0.06431 0 0"/>
     </joint>
     <!-- Contact parameters for gripper links: firm for grasping, prevent tunneling -->
+    <!-- Dengeli ayar: Yüksek sürtünme ama yumuşak temas (titreme önleme) -->
     <gazebo reference="${namespace}/finger_left">
       <self_collide>false</self_collide>
       <!-- gravity tag removed to re-enable gravity -->
-      <linearDamping>0.2</linearDamping>
-      <angularDamping>0.2</angularDamping>
-      <mu1>1.0</mu1>
-      <mu2>1.0</mu2>
-      <slip1>0.0</slip1>
-      <slip2>0.0</slip2>
-      <kp>80000</kp>
-      <kd>80</kd>
-      <max_contacts>10</max_contacts>
-      <max_vel>0.3</max_vel>
-      <min_depth>0.001</min_depth>
-      <contact_surface_layer>0.0002</contact_surface_layer>
+      <!-- Damping artırıldı: 0.3 -> 0.5 (titreşimi söndürür) -->
+      <linearDamping>0.5</linearDamping>
+      <angularDamping>0.5</angularDamping>
+      <!-- Sürtünme yüksek kalıyor -->
+      <mu1>8.0</mu1>
+      <mu2>8.0</mu2>
+      <slip1>0.0</slip1>
+      <slip2>0.0</slip2>
+      <!-- Contact stiffness hafif azaltıldı: 120k -> 100k (daha yumuşak temas) -->
+      <kp>100000</kp>
+      <!-- Contact damping artırıldı: 100 -> 150 (titreşim sönümleme) -->
+      <kd>150</kd>
+      <max_contacts>20</max_contacts>
+      <max_vel>0.2</max_vel>
+      <min_depth>0.0005</min_depth>
+      <contact_surface_layer>0.0001</contact_surface_layer>
     </gazebo>
     <gazebo reference="${namespace}/finger_right">
       <self_collide>false</self_collide>
-      <!-- gravity tag removed to re-enable gravity -->
-      <linearDamping>0.2</linearDamping>
-      <angularDamping>0.2</angularDamping>
-      <mu1>1.0</mu1>
-      <mu2>1.0</mu2>
-      <slip1>0.0</slip1>
-      <slip2>0.0</slip2>
-      <kp>80000</kp>
-      <kd>80</kd>
-      <max_contacts>10</max_contacts>
-      <max_vel>0.3</max_vel>
-      <min_depth>0.001</min_depth>
-      <contact_surface_layer>0.0002</contact_surface_layer>
+      <linearDamping>0.5</linearDamping>
+      <angularDamping>0.5</angularDamping>
+      <mu1>8.0</mu1>
+      <mu2>8.0</mu2>
+      <slip1>0.0</slip1>
+      <slip2>0.0</slip2>
+      <kp>100000</kp>
+      <kd>150</kd>
+      <max_contacts>20</max_contacts>
+      <max_vel>0.2</max_vel>
+      <min_depth>0.0005</min_depth>
+      <contact_surface_layer>0.0001</contact_surface_layer>
     </gazebo>
     <gazebo reference="${namespace}/finger_tip_left">
       <self_collide>false</self_collide>
-      <!-- gravity tag removed to re-enable gravity -->
-      <linearDamping>0.2</linearDamping>
-      <angularDamping>0.2</angularDamping>
-      <mu1>1.0</mu1>
-      <mu2>1.0</mu2>
-      <slip1>0.0</slip1>
-      <slip2>0.0</slip2>
-      <kp>80000</kp>
-      <kd>80</kd>
-      <max_contacts>10</max_contacts>
-      <max_vel>0.3</max_vel>
-      <min_depth>0.001</min_depth>
-      <contact_surface_layer>0.0002</contact_surface_layer>
+      <linearDamping>0.5</linearDamping>
+      <angularDamping>0.5</angularDamping>
+      <mu1>8.0</mu1>
+      <mu2>8.0</mu2>
+      <slip1>0.0</slip1>
+      <slip2>0.0</slip2>
+      <kp>100000</kp>
+      <kd>150</kd>
+      <max_contacts>20</max_contacts>
+      <max_vel>0.2</max_vel>
+      <min_depth>0.0005</min_depth>
+      <contact_surface_layer>0.0001</contact_surface_layer>
     </gazebo>
     <gazebo reference="${namespace}/finger_tip_right">
       <self_collide>false</self_collide>
-      <!-- gravity tag removed to re-enable gravity -->
-      <linearDamping>0.2</linearDamping>
-      <angularDamping>0.2</angularDamping>
-      <mu1>1.0</mu1>
-      <mu2>1.0</mu2>
-      <slip1>0.0</slip1>
-      <slip2>0.0</slip2>
-      <kp>80000</kp>
-      <kd>80</kd>
-      <max_contacts>10</max_contacts>
-      <max_vel>0.3</max_vel>
-      <min_depth>0.001</min_depth>
-      <contact_surface_layer>0.0002</contact_surface_layer>
+      <linearDamping>0.5</linearDamping>
+      <angularDamping>0.5</angularDamping>
+      <mu1>8.0</mu1>
+      <mu2>8.0</mu2>
+      <slip1>0.0</slip1>
+      <slip2>0.0</slip2>
+      <kp>100000</kp>
+      <kd>150</kd>
+      <max_contacts>20</max_contacts>
+      <max_vel>0.2</max_vel>
+      <min_depth>0.0005</min_depth>
+      <contact_surface_layer>0.0001</contact_surface_layer>
     </gazebo>
     <!-- Make joints soft but not mushy; single definition per joint -->
+    <!-- Joint sertliği artırıldı - daha güçlü tutma kabiliyeti -->
     <gazebo reference="${namespace}/finger_left_joint">
       <implicitSpringDamper>true</implicitSpringDamper>
-      <stop_kp>1500</stop_kp>
-      <stop_kd>15</stop_kd>
-      <cfm>0.001</cfm>
-      <erp>0.2</erp>
+      <!-- Stop stiffness artırıldı: 1500 -> 3000 (daha sert durma) -->
+      <stop_kp>3000</stop_kp>
+      <stop_kd>30</stop_kd>
+      <!-- CFM azaltıldı, ERP artırıldı: daha sert ve hızlı düzeltme -->
+      <cfm>0.0005</cfm>
+      <erp>0.3</erp>
       <spring_reference>0.0</spring_reference>
-      <spring_stiffness>5.0</spring_stiffness>
+      <!-- Spring stiffness artırıldı: 5.0 -> 15.0 (güçlü geri yay) -->
+      <spring_stiffness>15.0</spring_stiffness>
       <provideFeedback>true</provideFeedback>
     </gazebo>
     <gazebo reference="${namespace}/finger_right_joint">
       <implicitSpringDamper>true</implicitSpringDamper>
-      <stop_kp>1500</stop_kp>
-      <stop_kd>15</stop_kd>
-      <cfm>0.001</cfm>
-      <erp>0.2</erp>
+      <stop_kp>3000</stop_kp>
+      <stop_kd>30</stop_kd>
+      <cfm>0.0005</cfm>
+      <erp>0.3</erp>
       <spring_reference>0.0</spring_reference>
-      <spring_stiffness>5.0</spring_stiffness>
+      <spring_stiffness>15.0</spring_stiffness>
       <provideFeedback>true</provideFeedback>
     </gazebo>
@@ -267,8 +279,17 @@
           <gripper_link>${namespace}/finger_tip_right</gripper_link>
           <palm_link>${namespace}/gripper_base</palm_link>
-          <max_contacts>100</max_contacts>
-          <min_contact_count>2</min_contact_count>
-          <forces_angle_tolerance>25</forces_angle_tolerance>
-          <release_tolerance>0.002</release_tolerance>
+          <!-- Çok daha fazla contact izleme -->
+          <max_contacts>200</max_contacts>
+          <!-- Minimum 3 contact noktası gerekli (daha güvenli) -->
+          <min_contact_count>3</min_contact_count>
+          <!-- Kuvvet açı toleransı azaltıldı: 25 -> 20 (daha hassas) -->
+          <forces_angle_tolerance>20</forces_angle_tolerance>
+          <!-- Release tolerance azaltıldı: 0.002 -> 0.001 (daha sıkı tutma) -->
+          <release_tolerance>0.001</release_tolerance>
+          <!-- Attach ve detach kuvvet eşikleri eklendi -->
+          <grip_count_threshold>3</grip_count_threshold>
+          <max_grip_count>10</max_grip_count>
+          <release_count_threshold>2</release_count_threshold>
+          <disable_collisions_on_attach>false</disable_collisions_on_attach>
         </plugin>
       </gazebo>

Commit message: integrated the smach, turned off gripper collision, change valve names, added valve to sim keypoint node, deleted old file

File: auv_description/taluy_description/urdf/parallel_gripper.xacro (robot description, xacro)
@@ -53,10 +53,12 @@
         </geometry>
       </visual>
-      <collision>
+      <!-- Collision disabled: physical gripper is too large to fit at the
+           valve task workspace. Visual is kept for debugging. -->
+      <!-- <collision>
         <origin rpy="0 0 0" xyz="0.024426 0.0 0.0"/>
         <geometry>
           <box size="0.074326 0.117427 0.114298"/>
         </geometry>
-      </collision>
+      </collision> -->
     </link>
     <!-- Joint connecting the virtual mount link to gripper base -->
@@ -80,10 +82,11 @@
         </geometry>
       </visual>
-      <collision>
+      <!-- Collision disabled (gripper too large for valve workspace). -->
+      <!-- <collision>
         <origin rpy="0 0 0" xyz="0.032 0 0"/>
         <geometry>
           <box size="0.064 0.078 0.025"/>
         </geometry>
-      </collision>
+      </collision> -->
     </link>
     <!-- Left Finger Joint -->
@@ -113,10 +116,11 @@
         </geometry>
       </visual>
-      <collision>
+      <!-- Collision disabled (gripper too large for valve workspace). -->
+      <!-- <collision>
         <origin rpy="0 0 0" xyz="0.042 0 0"/>
         <geometry>
           <box size="0.084 0.048 0.024"/>
         </geometry>
-      </collision>
+      </collision> -->
     </link>
     <!-- Left Finger Tip Joint (fixed for stability) -->
@@ -141,10 +145,11 @@
         </geometry>
       </visual>
-      <collision>
+      <!-- Collision disabled (gripper too large for valve workspace). -->
+      <!-- <collision>
         <origin rpy="3.14159265359 0 0" xyz="0.032 0 0"/>
         <geometry>
           <box size="0.064 0.078 0.025"/>
         </geometry>
-      </collision>
+      </collision> -->
     </link>
     <!-- Right Finger Joint -->
@@ -174,10 +179,11 @@
         </geometry>
       </visual>
-      <collision>
+      <!-- Collision disabled (gripper too large for valve workspace). -->
+      <!-- <collision>
         <origin rpy="0 0 0" xyz="0.042 0 0"/>
         <geometry>
           <box size="0.084 0.048 0.024"/>
         </geometry>
-      </collision>
+      </collision> -->
     </link>
     <!-- Right Finger Tip Joint (fixed for stability) -->
