Commit message: update thruster orientations

File: auv_description/taluy_description/urdf/auv_base.urdf.xacro (robot description, xacro)
@@ -32,19 +32,6 @@
     <xacro:t200_thruster name="thruster_4" parent="base_link" position="0.352398 0.216638 -0.030881" orientation="${pi/2} 0 ${pi/4}"/>
     <xacro:t200_thruster name="thruster_5" parent="base_link" position="0.352398 -0.216638 -0.030881" orientation="${-pi/2} 0 ${-pi/4}"/>
-    <xacro:t200_thruster name="thruster_6" parent="base_link" position="-0.352398 0.216638 -0.030881" orientation="${pi/2} 0 ${3*pi/4}"/>
-    <xacro:t200_thruster name="thruster_7" parent="base_link" position="-0.352398 -0.216638 -0.030881" orientation="${-pi/2} 0 ${-3*pi/4}"/>
-    <!-- <link name="base_footprint">
-      <inertial>
-        <origin xyz="0 0 0" rpy="0 0 0" />
-        <mass value="15.0" />
-        <inertia ixx="39.351246" iyy="103.261717" izz="127.702526" ixy="-5e-06" iyz="6e-06"
-          ixz="4.403436" />
-      </inertial>
-    </link>
-    <joint name="base_link_joint" type="fixed">
-      <origin xyz="0 0 ${-base_z_offsett + 0.06 - draft}" rpy="0 0 0" />
-      <parent link="base_footprint" />
-      <child link="base_link" />
-    </joint> -->
+    <xacro:t200_thruster name="thruster_6" parent="base_link" position="-0.352398 0.216638 -0.030881" orientation="${pi/2} 0 ${7*pi/4}"/>
+    <xacro:t200_thruster name="thruster_7" parent="base_link" position="-0.352398 -0.216638 -0.030881" orientation="${-pi/2} 0 ${-7*pi/4}"/>
   </xacro:macro>
 </robot>

Commit message: add sonar xacro

File: auv_description/taluy_description/urdf/auv_base.urdf.xacro (robot description, xacro)
@@ -29,5 +29,5 @@
       </collision>
     </link>
-    <link name="base_link_ned"/>
+    <link name="base_link_ned" />
     <joint name="base_link_joint" type="fixed">
       <origin xyz="0 0 0" rpy="${math.pi} 0 0" />
@@ -35,12 +35,20 @@
       <child link="base_link" />
     </joint>
-    <xacro:t200_thruster name="thruster_0" parent="base_link" position="0.14250 0.20070 -0.00525" orientation="${pi} 0 ${-pi/2}"/>
-    <xacro:t200_thruster name="thruster_1" parent="base_link" position="0.14250 -0.20070 -0.00525" orientation="${pi} 0 ${pi/2}"/>
-    <xacro:t200_thruster name="thruster_2" parent="base_link" position="-0.14250 0.20070 -0.00525" orientation="${pi} 0 ${-pi/2}"/>
-    <xacro:t200_thruster name="thruster_3" parent="base_link" position="-0.14250 -0.20070 -0.00525" orientation="${pi} 0 ${pi/2}"/>
-    <xacro:t200_thruster name="thruster_4" parent="base_link" position="0.352398 0.216638 -0.030881" orientation="${-pi/2} 0 ${-7*pi/4}"/>
-    <xacro:t200_thruster name="thruster_5" parent="base_link" position="0.352398 -0.216638 -0.030881" orientation="${pi/2} 0 ${7*pi/4}"/>
-    <xacro:t200_thruster name="thruster_6" parent="base_link" position="-0.352398 0.216638 -0.030881" orientation="${-pi/2} 0 ${-pi/4}"/>
-    <xacro:t200_thruster name="thruster_7" parent="base_link" position="-0.352398 -0.216638 -0.030881" orientation="${pi/2} 0 ${pi/4}"/>
+    <xacro:t200_thruster name="thruster_0" parent="base_link" position="0.14250 0.20070 -0.00525"
+      orientation="${pi} 0 ${-pi/2}" />
+    <xacro:t200_thruster name="thruster_1" parent="base_link" position="0.14250 -0.20070 -0.00525"
+      orientation="${pi} 0 ${pi/2}" />
+    <xacro:t200_thruster name="thruster_2" parent="base_link" position="-0.14250 0.20070 -0.00525"
+      orientation="${pi} 0 ${-pi/2}" />
+    <xacro:t200_thruster name="thruster_3" parent="base_link" position="-0.14250 -0.20070 -0.00525"
+      orientation="${pi} 0 ${pi/2}" />
+    <xacro:t200_thruster name="thruster_4" parent="base_link" position="0.352398 0.216638 -0.030881"
+      orientation="${-pi/2} 0 ${-7*pi/4}" />
+    <xacro:t200_thruster name="thruster_5" parent="base_link"
+      position="0.352398 -0.216638 -0.030881" orientation="${pi/2} 0 ${7*pi/4}" />
+    <xacro:t200_thruster name="thruster_6" parent="base_link"
+      position="-0.352398 0.216638 -0.030881" orientation="${-pi/2} 0 ${-pi/4}" />
+    <xacro:t200_thruster name="thruster_7" parent="base_link"
+      position="-0.352398 -0.216638 -0.030881" orientation="${pi/2} 0 ${pi/4}" />
     <xacro:wayfinder_dvl
       name="base_link/dvl" parent="base_link" position="0.2 0 -0.11"
@@ -80,4 +88,16 @@
       parent="base_link" position="0.2 -0.1 -0.11"
       orientation="0 0 0" />
+    <xacro:sonar name="base_link/sonar_front" parent="base_link"
+      position="0.38 0.09 0.09"
+      orientation="0 0 0" />
+    <xacro:sonar name="base_link/sonar_back" parent="base_link"
+      position="-0.42 -0.09 0.09"
+      orientation="0 0 ${math.pi}" />
+    <xacro:sonar name="base_link/sonar_left" parent="base_link"
+      position="0.02 -0.21 -0.14"
+      orientation="0 0 ${-math.pi/2}" />
+    <xacro:sonar name="base_link/sonar_right" parent="base_link"
+      position="0.02 0.21 -0.14"
+      orientation="0 0 ${math.pi/2}" />
     <!-- <link name="base_footprint">
       <inertial>

Commit message: Sonar description (#41)
* add sonar xacro

* fix sonar urdf

* fix build error

---------

Co-authored-by: ituauvteam <auv@itu.edu.tr>

File: auv_description/taluy_description/urdf/auv_base.urdf.xacro (robot description, xacro)
@@ -29,5 +29,5 @@
       </collision>
     </link>
-    <link name="base_link_ned"/>
+    <link name="base_link_ned" />
     <joint name="base_link_joint" type="fixed">
       <origin xyz="0 0 0" rpy="${math.pi} 0 0" />
@@ -35,12 +35,20 @@
       <child link="base_link" />
     </joint>
-    <xacro:t200_thruster name="thruster_0" parent="base_link" position="0.14250 0.20070 -0.00525" orientation="${pi} 0 ${-pi/2}"/>
-    <xacro:t200_thruster name="thruster_1" parent="base_link" position="0.14250 -0.20070 -0.00525" orientation="${pi} 0 ${pi/2}"/>
-    <xacro:t200_thruster name="thruster_2" parent="base_link" position="-0.14250 0.20070 -0.00525" orientation="${pi} 0 ${-pi/2}"/>
-    <xacro:t200_thruster name="thruster_3" parent="base_link" position="-0.14250 -0.20070 -0.00525" orientation="${pi} 0 ${pi/2}"/>
-    <xacro:t200_thruster name="thruster_4" parent="base_link" position="0.352398 0.216638 -0.030881" orientation="${-pi/2} 0 ${-7*pi/4}"/>
-    <xacro:t200_thruster name="thruster_5" parent="base_link" position="0.352398 -0.216638 -0.030881" orientation="${pi/2} 0 ${7*pi/4}"/>
-    <xacro:t200_thruster name="thruster_6" parent="base_link" position="-0.352398 0.216638 -0.030881" orientation="${-pi/2} 0 ${-pi/4}"/>
-    <xacro:t200_thruster name="thruster_7" parent="base_link" position="-0.352398 -0.216638 -0.030881" orientation="${pi/2} 0 ${pi/4}"/>
+    <xacro:t200_thruster name="thruster_0" parent="base_link" position="0.14250 0.20070 -0.00525"
+      orientation="${pi} 0 ${-pi/2}" />
+    <xacro:t200_thruster name="thruster_1" parent="base_link" position="0.14250 -0.20070 -0.00525"
+      orientation="${pi} 0 ${pi/2}" />
+    <xacro:t200_thruster name="thruster_2" parent="base_link" position="-0.14250 0.20070 -0.00525"
+      orientation="${pi} 0 ${-pi/2}" />
+    <xacro:t200_thruster name="thruster_3" parent="base_link" position="-0.14250 -0.20070 -0.00525"
+      orientation="${pi} 0 ${pi/2}" />
+    <xacro:t200_thruster name="thruster_4" parent="base_link" position="0.352398 0.216638 -0.030881"
+      orientation="${-pi/2} 0 ${-7*pi/4}" />
+    <xacro:t200_thruster name="thruster_5" parent="base_link"
+      position="0.352398 -0.216638 -0.030881" orientation="${pi/2} 0 ${7*pi/4}" />
+    <xacro:t200_thruster name="thruster_6" parent="base_link"
+      position="-0.352398 0.216638 -0.030881" orientation="${-pi/2} 0 ${-pi/4}" />
+    <xacro:t200_thruster name="thruster_7" parent="base_link"
+      position="-0.352398 -0.216638 -0.030881" orientation="${pi/2} 0 ${pi/4}" />
     <xacro:wayfinder_dvl
       name="base_link/dvl" parent="base_link" position="0.2 0 -0.11"
@@ -80,4 +88,16 @@
       parent="base_link" position="0.2 -0.1 -0.11"
       orientation="0 0 0" />
+    <xacro:sonar name="base_link/sonar_front" parent="base_link"
+      position="0.38 0.09 0.09"
+      orientation="0 ${math.pi/2} 0" />
+    <xacro:sonar name="base_link/sonar_back" parent="base_link"
+      position="-0.42 -0.09 0.09"
+      orientation="0 ${math.pi/2} ${math.pi}" />
+    <xacro:sonar name="base_link/sonar_left" parent="base_link"
+      position="0.02 -0.21 -0.14"
+      orientation="0 ${math.pi/2} ${-math.pi/2}" />
+    <xacro:sonar name="base_link/sonar_right" parent="base_link"
+      position="0.02 0.21 -0.14"
+      orientation="0 ${math.pi/2} ${math.pi/2}" />
     <!-- <link name="base_footprint">
       <inertial>

Commit message: update

File: auv_description/taluy_description/urdf/auv_base.urdf.xacro (robot description, xacro)
@@ -1,14 +1,18 @@
 <?xml version="1.0"?>
-<robot xmlns:xacro="http://www.ros.org/wiki/xacro" name="taluy">
+<robot name="taluy" xmlns:xacro="http://www.ros.org/wiki/xacro">
+  <!-- create xacro property -->
+  <xacro:property name="namespace" value="taluy" />
   <xacro:macro name="taluy_base">
-    <xacro:include filename="$(find auv_common_descriptions)/urdf/actuators.urdf.xacro"/>
-    <xacro:include filename="$(find auv_common_descriptions)/urdf/sensors.urdf.xacro"/>
-    <xacro:include filename="$(find auv_common_descriptions)/urdf/materials.urdf.xacro"/>
-    <xacro:arg name="angled_thruster_z_offset" default="-0.01"/>
-    <link name="base_link">
+    <xacro:include filename="$(find auv_common_descriptions)/urdf/actuators.urdf.xacro" />
+    <xacro:include
+      filename="$(find auv_common_descriptions)/urdf/sensors.urdf.xacro" />
+    <xacro:include
+      filename="$(find auv_common_descriptions)/urdf/materials.urdf.xacro" />
+    <xacro:arg name="angled_thruster_z_offset" default="-0.01" />
+    <link name="${namespace}/base_link">
       <inertial>
-        <origin xyz="0 0 0" rpy="0 0 0"/>
-        <mass value="25.0"/>
-        <inertia ixx="0.1" iyy="0.1" izz="0.1" ixy="0.01" iyz="0.01" ixz="0.1"/>
+        <origin xyz="0 0 0" rpy="0 0 0" />
+        <mass value="27.0" />
+        <inertia ixx="0.1" iyy="0.1" izz="0.1" ixy="0.01" iyz="0.01" ixz="0.1" />
       </inertial>
       <visual>
@@ -26,34 +30,83 @@
       </collision>
     </link>
-    <link name="base_link_ned"/>
+    <link name="${namespace}/base_link_ned" />
     <joint name="base_link_joint" type="fixed">
-      <origin xyz="0 0 0" rpy="${math.pi} 0 0"/>
-      <parent link="base_link_ned"/>
-      <child link="base_link"/>
+      <origin xyz="0 0 0" rpy="${math.pi} 0 0" />
+      <parent link="${namespace}/base_link_ned" />
+      <child link="${namespace}/base_link" />
     </joint>
-    <xacro:t200_thruster name="thruster_0" parent="base_link" position="0.14250 0.20070 -0.00525" orientation="${pi} 0 ${-pi/2}"/>
-    <xacro:t200_thruster name="thruster_1" parent="base_link" position="0.14250 -0.20070 -0.00525" orientation="${pi} 0 ${pi/2}"/>
-    <xacro:t200_thruster name="thruster_2" parent="base_link" position="-0.14250 0.20070 -0.00525" orientation="${pi} 0 ${-pi/2}"/>
-    <xacro:t200_thruster name="thruster_3" parent="base_link" position="-0.14250 -0.20070 -0.00525" orientation="${pi} 0 ${pi/2}"/>
-    <xacro:t200_thruster name="thruster_4" parent="base_link" position="0.352398 0.216638 $(arg angled_thruster_z_offset)" orientation="${-pi/2} 0 ${-7*pi/4}"/>
-    <xacro:t200_thruster name="thruster_5" parent="base_link" position="0.352398 -0.216638 $(arg angled_thruster_z_offset)" orientation="${pi/2} 0 ${7*pi/4}"/>
-    <xacro:t200_thruster name="thruster_6" parent="base_link" position="-0.352398 0.216638 $(arg angled_thruster_z_offset)" orientation="${-pi/2} 0 ${-pi/4}"/>
-    <xacro:t200_thruster name="thruster_7" parent="base_link" position="-0.352398 -0.216638 $(arg angled_thruster_z_offset)" orientation="${pi/2} 0 ${pi/4}"/>
-    <xacro:wayfinder_dvl name="base_link/dvl" parent="base_link" position="0.2 0 -0.11" orientation="0 0 0"/>
-    <xacro:xsens_mti_g710 name="base_link/imu" parent="base_link" position="-0.199 0 -0.0108" orientation="0 0 ${math.pi}"/>
-    <xacro:h2c_hydrophone name="base_link/hydrophone_0" parent="base_link" position="0.325 0.205 -0.15" orientation="0 0 0"/>
-    <xacro:h2c_hydrophone name="base_link/hydrophone_1" parent="base_link" position="0.325 -0.205 -0.15" orientation="0 0 0"/>
-    <xacro:h2c_hydrophone name="base_link/hydrophone_2" parent="base_link" position="-0.325 0.205 -0.15" orientation="0 0 0"/>
-    <xacro:h2c_hydrophone name="base_link/hydrophone_3" parent="base_link" position="-0.325 -0.205 -0.15" orientation="0 0 0"/>
-    <xacro:ping360 name="base_link/ping360" parent="base_link" position="0.2 0 0.134" orientation="0 0 0"/>
-    <xacro:bar30 name="base_link/external_pressure_sensor" parent="base_link" position="0 0 0.07" orientation="0 0 0"/>
-    <xacro:logitech_c920_camera name="base_link/front_camera" parent="base_link" position="0.35 0 0" orientation="0 0 0"/>
-    <xacro:logitech_c920_camera name="base_link/bottom_camera" parent="base_link" position="0 0 -0.07" orientation="0 ${math.pi/2} ${math.pi/2}"/>
-    <xacro:torpedo name="base_link/left_torpedo" parent="base_link" position="0.2 0.1 -0.11" orientation="0 0 0"/>
-    <xacro:torpedo name="base_link/right_torpedo" parent="base_link" position="0.2 -0.1 -0.11" orientation="0 0 0"/>
-    <xacro:sonar name="base_link/sonar_front" parent="base_link" position="0.38 0.09 0.09" orientation="0 0 0"/>
-    <xacro:sonar name="base_link/sonar_back" parent="base_link" position="-0.42 -0.09 0.09" orientation="0 0 ${math.pi}"/>
-    <xacro:sonar name="base_link/sonar_right" parent="base_link" position="0.02 -0.21 -0.14" orientation="0 0 ${-math.pi/2}"/>
-    <xacro:sonar name="base_link/sonar_left" parent="base_link" position="0.02 0.21 -0.14" orientation="0 0 ${math.pi/2}"/>
+    <xacro:t200_thruster name="${namespace}/thruster_0" parent="${namespace}/base_link"
+      position="0.14250 0.20070 -0.00525"
+      orientation="${pi} 0 ${-pi/2}" />
+    <xacro:t200_thruster name="${namespace}/thruster_1" parent="${namespace}/base_link"
+      position="0.14250 -0.20070 -0.00525"
+      orientation="${pi} 0 ${pi/2}" />
+    <xacro:t200_thruster name="${namespace}/thruster_2" parent="${namespace}/base_link"
+      position="-0.14250 0.20070 -0.00525"
+      orientation="${pi} 0 ${-pi/2}" />
+    <xacro:t200_thruster name="${namespace}/thruster_3" parent="${namespace}/base_link"
+      position="-0.14250 -0.20070 -0.00525"
+      orientation="${pi} 0 ${pi/2}" />
+    <xacro:t200_thruster name="${namespace}/thruster_4" parent="${namespace}/base_link"
+      position="0.352398 0.216638 $(arg angled_thruster_z_offset)"
+      orientation="${-pi/2} 0 ${-7*pi/4}" />
+    <xacro:t200_thruster name="${namespace}/thruster_5" parent="${namespace}/base_link"
+      position="0.352398 -0.216638 $(arg angled_thruster_z_offset)"
+      orientation="${pi/2} 0 ${7*pi/4}" />
+    <xacro:t200_thruster name="${namespace}/thruster_6" parent="${namespace}/base_link"
+      position="-0.352398 0.216638 $(arg angled_thruster_z_offset)"
+      orientation="${-pi/2} 0 ${-pi/4}" />
+    <xacro:t200_thruster name="${namespace}/thruster_7" parent="${namespace}/base_link"
+      position="-0.352398 -0.216638 $(arg angled_thruster_z_offset)" orientation="${pi/2} 0 ${pi/4}" />
+    <xacro:wayfinder_dvl
+      name="${namespace}/base_link/dvl" parent="${namespace}/base_link" position="0.2 0 -0.11"
+      orientation="0 0 0" />
+    <xacro:xsens_mti_g710 name="${namespace}/base_link/imu" parent="${namespace}/base_link"
+      position="-0.199 0 -0.0108"
+      orientation="0 0 ${math.pi}" />
+    <xacro:h2c_hydrophone name="${namespace}/base_link/hydrophone_0"
+      parent="${namespace}/base_link"
+      position="0.325 0.205 -0.15"
+      orientation="0 0 0" />
+    <xacro:h2c_hydrophone name="${namespace}/base_link/hydrophone_1" parent="${namespace}/base_link"
+      position="0.325 -0.205 -0.15"
+      orientation="0 0 0" />
+    <xacro:h2c_hydrophone name="${namespace}/base_link/hydrophone_2" parent="${namespace}/base_link"
+      position="-0.325 0.205 -0.15"
+      orientation="0 0 0" />
+    <xacro:h2c_hydrophone name="${namespace}/base_link/hydrophone_3" parent="${namespace}/base_link"
+      position="-0.325 -0.205 -0.15"
+      orientation="0 0 0" />
+    <xacro:ping360 name="${namespace}/base_link/ping360" parent="${namespace}/base_link"
+      position="0.2 0 0.134"
+      orientation="0 0 0" />
+    <xacro:bar30 name="${namespace}/base_link/external_pressure_sensor"
+      parent="${namespace}/base_link"
+      position="0 0 0.07"
+      orientation="0 0 0" />
+    <xacro:logitech_c920_camera name="${namespace}/base_link/front_camera"
+      parent="${namespace}/base_link" position="0.35 0 0"
+      orientation="0 0 0" />
+    <xacro:logitech_c920_camera name="${namespace}/base_link/bottom_camera"
+      parent="${namespace}/base_link" position="0 0 -0.07"
+      orientation="0 ${math.pi/2} ${math.pi/2}" />
+    <xacro:torpedo name="${namespace}/base_link/left_torpedo"
+      parent="${namespace}/base_link" position="0.2 0.1 -0.11"
+      orientation="0 0 0" />
+    <xacro:torpedo name="${namespace}/base_link/right_torpedo"
+      parent="${namespace}/base_link" position="0.2 -0.1 -0.11"
+      orientation="0 0 0" />
+    <xacro:sonar name="${namespace}/base_link/sonar_front" parent="${namespace}/base_link"
+      position="0.38 0.09 0.09"
+      orientation="0 0 0" />
+    <xacro:sonar name="${namespace}/base_link/sonar_back" parent="${namespace}/base_link"
+      position="-0.42 -0.09 0.09"
+      orientation="0 0 ${math.pi}" />
+    <xacro:sonar name="${namespace}/base_link/sonar_right" parent="${namespace}/base_link"
+      position="0.02 -0.21 -0.14"
+      orientation="0 0 ${-math.pi/2}" />
+    <xacro:sonar name="${namespace}/base_link/sonar_left" parent="${namespace}/base_link"
+      position="0.02 0.21 -0.14"
+      orientation="0 0 ${math.pi/2}" />
     <!-- <link name="base_footprint">
       <inertial>
