Commit message: update

File: auv_description/taluy_description/urdf/auv_base.urdf.xacro (robot description, xacro)
@@ -1,4 +1,6 @@
 <?xml version="1.0"?>
 <robot name="taluy" xmlns:xacro="http://www.ros.org/wiki/xacro">
+  <!-- create xacro property -->
+  <xacro:property name="namespace" value="taluy" />
   <xacro:macro name="taluy_base">
     <xacro:include filename="$(find auv_common_descriptions)/urdf/actuators.urdf.xacro" />
@@ -8,8 +10,8 @@
       filename="$(find auv_common_descriptions)/urdf/materials.urdf.xacro" />
     <xacro:arg name="angled_thruster_z_offset" default="-0.01" />
-    <link name="base_link">
+    <link name="${namespace}/base_link">
       <inertial>
         <origin xyz="0 0 0" rpy="0 0 0" />
-        <mass value="25.0" />
+        <mass value="27.0" />
         <inertia ixx="0.1" iyy="0.1" izz="0.1" ixy="0.01" iyz="0.01" ixz="0.1" />
       </inertial>
@@ -30,76 +32,81 @@
       </collision>
     </link>
-    <link name="base_link_ned" />
+    <link name="${namespace}/base_link_ned" />
     <joint name="base_link_joint" type="fixed">
       <origin xyz="0 0 0" rpy="${math.pi} 0 0" />
-      <parent link="base_link_ned" />
-      <child link="base_link" />
+      <parent link="${namespace}/base_link_ned" />
+      <child link="${namespace}/base_link" />
     </joint>
-    <xacro:t200_thruster name="thruster_0" parent="base_link" position="0.14250 0.20070 -0.00525"
+    <xacro:t200_thruster name="${namespace}/thruster_0" parent="${namespace}/base_link"
+      position="0.14250 0.20070 -0.00525"
       orientation="${pi} 0 ${-pi/2}" />
-    <xacro:t200_thruster name="thruster_1" parent="base_link" position="0.14250 -0.20070 -0.00525"
+    <xacro:t200_thruster name="${namespace}/thruster_1" parent="${namespace}/base_link"
+      position="0.14250 -0.20070 -0.00525"
       orientation="${pi} 0 ${pi/2}" />
-    <xacro:t200_thruster name="thruster_2" parent="base_link" position="-0.14250 0.20070 -0.00525"
+    <xacro:t200_thruster name="${namespace}/thruster_2" parent="${namespace}/base_link"
+      position="-0.14250 0.20070 -0.00525"
       orientation="${pi} 0 ${-pi/2}" />
-    <xacro:t200_thruster name="thruster_3" parent="base_link" position="-0.14250 -0.20070 -0.00525"
+    <xacro:t200_thruster name="${namespace}/thruster_3" parent="${namespace}/base_link"
+      position="-0.14250 -0.20070 -0.00525"
       orientation="${pi} 0 ${pi/2}" />
-    <xacro:t200_thruster name="thruster_4" parent="base_link"
+    <xacro:t200_thruster name="${namespace}/thruster_4" parent="${namespace}/base_link"
       position="0.352398 0.216638 $(arg angled_thruster_z_offset)"
       orientation="${-pi/2} 0 ${-7*pi/4}" />
-    <xacro:t200_thruster name="thruster_5" parent="base_link"
+    <xacro:t200_thruster name="${namespace}/thruster_5" parent="${namespace}/base_link"
       position="0.352398 -0.216638 $(arg angled_thruster_z_offset)"
       orientation="${pi/2} 0 ${7*pi/4}" />
-    <xacro:t200_thruster name="thruster_6" parent="base_link"
+    <xacro:t200_thruster name="${namespace}/thruster_6" parent="${namespace}/base_link"
       position="-0.352398 0.216638 $(arg angled_thruster_z_offset)"
       orientation="${-pi/2} 0 ${-pi/4}" />
-    <xacro:t200_thruster name="thruster_7" parent="base_link"
+    <xacro:t200_thruster name="${namespace}/thruster_7" parent="${namespace}/base_link"
       position="-0.352398 -0.216638 $(arg angled_thruster_z_offset)" orientation="${pi/2} 0 ${pi/4}" />
     <xacro:wayfinder_dvl
-      name="base_link/dvl" parent="base_link" position="0.2 0 -0.11"
+      name="${namespace}/base_link/dvl" parent="${namespace}/base_link" position="0.2 0 -0.11"
       orientation="0 0 0" />
-    <xacro:xsens_mti_g710 name="base_link/imu" parent="base_link"
+    <xacro:xsens_mti_g710 name="${namespace}/base_link/imu" parent="${namespace}/base_link"
       position="-0.199 0 -0.0108"
       orientation="0 0 ${math.pi}" />
-    <xacro:h2c_hydrophone name="base_link/hydrophone_0"
-      parent="base_link"
+    <xacro:h2c_hydrophone name="${namespace}/base_link/hydrophone_0"
+      parent="${namespace}/base_link"
       position="0.325 0.205 -0.15"
       orientation="0 0 0" />
-    <xacro:h2c_hydrophone name="base_link/hydrophone_1" parent="base_link"
+    <xacro:h2c_hydrophone name="${namespace}/base_link/hydrophone_1" parent="${namespace}/base_link"
       position="0.325 -0.205 -0.15"
       orientation="0 0 0" />
-    <xacro:h2c_hydrophone name="base_link/hydrophone_2" parent="base_link"
+    <xacro:h2c_hydrophone name="${namespace}/base_link/hydrophone_2" parent="${namespace}/base_link"
       position="-0.325 0.205 -0.15"
       orientation="0 0 0" />
-    <xacro:h2c_hydrophone name="base_link/hydrophone_3" parent="base_link"
+    <xacro:h2c_hydrophone name="${namespace}/base_link/hydrophone_3" parent="${namespace}/base_link"
       position="-0.325 -0.205 -0.15"
       orientation="0 0 0" />
-    <xacro:ping360 name="base_link/ping360" parent="base_link"
+    <xacro:ping360 name="${namespace}/base_link/ping360" parent="${namespace}/base_link"
       position="0.2 0 0.134"
       orientation="0 0 0" />
-    <xacro:bar30 name="base_link/external_pressure_sensor" parent="base_link"
+    <xacro:bar30 name="${namespace}/base_link/external_pressure_sensor"
+      parent="${namespace}/base_link"
       position="0 0 0.07"
       orientation="0 0 0" />
-    <xacro:logitech_c920_camera name="base_link/front_camera"
-      parent="base_link" position="0.35 0 0"
+    <xacro:logitech_c920_camera name="${namespace}/base_link/front_camera"
+      parent="${namespace}/base_link" position="0.35 0 0"
       orientation="0 0 0" />
-    <xacro:logitech_c920_camera name="base_link/bottom_camera"
-      parent="base_link" position="0 0 -0.07"
+    <xacro:logitech_c920_camera name="${namespace}/base_link/bottom_camera"
+      parent="${namespace}/base_link" position="0 0 -0.07"
       orientation="0 ${math.pi/2} ${math.pi/2}" />
-    <xacro:torpedo name="base_link/left_torpedo"
-      parent="base_link" position="0.2 0.1 -0.11"
+    <xacro:torpedo name="${namespace}/base_link/left_torpedo"
+      parent="${namespace}/base_link" position="0.2 0.1 -0.11"
       orientation="0 0 0" />
-    <xacro:torpedo name="base_link/right_torpedo"
-      parent="base_link" position="0.2 -0.1 -0.11"
+    <xacro:torpedo name="${namespace}/base_link/right_torpedo"
+      parent="${namespace}/base_link" position="0.2 -0.1 -0.11"
       orientation="0 0 0" />
-    <xacro:sonar name="base_link/sonar_front" parent="base_link"
+    <xacro:sonar name="${namespace}/base_link/sonar_front" parent="${namespace}/base_link"
       position="0.38 0.09 0.09"
       orientation="0 0 0" />
-    <xacro:sonar name="base_link/sonar_back" parent="base_link"
+    <xacro:sonar name="${namespace}/base_link/sonar_back" parent="${namespace}/base_link"
       position="-0.42 -0.09 0.09"
       orientation="0 0 ${math.pi}" />
-    <xacro:sonar name="base_link/sonar_right" parent="base_link"
+    <xacro:sonar name="${namespace}/base_link/sonar_right" parent="${namespace}/base_link"
       position="0.02 -0.21 -0.14"
       orientation="0 0 ${-math.pi/2}" />
-    <xacro:sonar name="base_link/sonar_left" parent="base_link"
+    <xacro:sonar name="${namespace}/base_link/sonar_left" parent="${namespace}/base_link"
       position="0.02 0.21 -0.14"
       orientation="0 0 ${math.pi/2}" />

File: auv_sim/auv_sim_description/urdf/gazebo_plugins.urdf.xacro (robot description, xacro)
@@ -78,6 +78,22 @@
         </dynamics>
         <conversion>
-          <type>Basic</type>
-          <rotorConstant>0.00031</rotorConstant>
+          <type>
+            LinearInterp
+          </type>
+          <inputValues>
+            0 1009 1100 1110 1120 1130 1140 1150 1160 1170 1180 1190 1200 1210 1220 1230 1240 1250
+            1260 1270 1280 1290 1300 1310 1320 1330 1340 1350 1360 1370 1380 1390 1400 1410 1420
+            1430 1440 1450 1460 1470 1480 1490 1500 1510 1520 1530 1540 1550 1560 1570 1580 1590
+            1600 1610 1620 1630 1640 1650 1660 1670 1680 1690 1700 1710 1720 1730 1740 1750 1760
+            1770 1780 1790 1800 1810 1820 1830 1840 1850 1860 1870 1880 1890 1900 1901 1902
+          </inputValues>
+          <outputValues>
+            0 0 -17.34 -16.09 -15.47 -14.98 -14.13 -13.73 -12.97 -12.35 -11.86 -11.41 -10.83 -10.21
+            -9.72 -9.09 -8.38 -7.76 -7.40 -6.91 -6.55 -6.11 -5.71 -5.22 -4.64 -4.19 -3.92 -3.61
+            -3.21 -2.67 -2.27 -1.96 -1.65 -1.38 -1.03 -0.71 -0.49 -0.31 -0.13 -0.09 0.00 0.00 0.00
+            0.00 0.00 0.09 0.36 0.62 1.03 1.43 1.92 2.50 3.03 3.61 4.23 4.73 5.35 6.02 6.73 7.22
+            7.89 8.65 9.45 10.39 11.10 11.63 12.30 12.79 13.60 14.62 15.47 16.23 16.94 17.87 19.21
+            20.06 20.59 21.40 22.20 22.78 23.71 24.38 24.69 0 0
+          </outputValues>
         </conversion>
       </plugin>
@@ -156,42 +172,3 @@
     </gazebo>
   </xacro:macro>
-  <!-- base link hydrodynamics plugin -->
-  <xacro:macro name="base_link_sim">
-    <gazebo>
-      <plugin name="uuv_plugin" filename="libuuv_underwater_object_ros_plugin.so">
-        <fluid_density>1028.0</fluid_density>
-        <flow_velocity_topic>hydrodynamics/current_velocity</flow_velocity_topic>
-        <debug>$(arg debug)</debug>
-        <link name="base_link_ned">
-          <neutrally_buoyant>1</neutrally_buoyant>
-          <volume>0.024</volume>
-          <box>
-            <width>0.665</width>
-            <length>0.875</length>
-            <height>0.525</height>
-          </box>
-          <center_of_buoyancy>
-            0.013859156 0.000063641869 0.3332835841
-          </center_of_buoyancy>
-          <hydrodynamic_model>
-            <type>fossen</type>
-            <added_mass>
-              10.7727 0 0 0 0 0
-              0 10.7727 0 0 0 0
-              0 0 49.7679 0 0 0
-              0 0 0 1.0092 0 0
-              0 0 0 0 1.0092 0
-              0 0 0 0 0 0
-            </added_mass>
-            <linear_damping>
-              -19.5909 -19.5909 -50.5595 -13.3040 -13.2181 -1.1559
-            </linear_damping>
-            <quadratic_damping>
-              -5.1386 -5.1386 -26.1105 0 0 0
-            </quadratic_damping>
-          </hydrodynamic_model>
-        </link>
-      </plugin>
-    </gazebo>
-  </xacro:macro>
 </robot>

File: auv_sim/auv_sim_description/urdf/taluy_sim.urdf.xacro (robot description, xacro)
@@ -1,25 +1,23 @@
 <?xml version="1.0"?>
 <robot name="taluy" xmlns:xacro="http://www.ros.org/wiki/xacro">
-  <xacro:include filename="$(find taluy_description)/urdf/auv_base.urdf.xacro" />
-  <xacro:taluy_base />
-  <!-- Gazebo plugins -->
-  <xacro:include filename="$(find auv_sim_description)/urdf/gazebo_plugins.urdf.xacro" />
-  <xacro:base_link_sim />
-  <xacro:logitech_c920_camera_sim name="base_link/front_camera" topic_name="cameras/cam_front" />
-  <xacro:logitech_c920_camera_sim name="base_link/bottom_camera" topic_name="cameras/cam_bottom" />
-  <xacro:xsens_mti_g710_sim name="base_link/imu" />
-  <xacro:t200_thruster_sim name="thruster_0" thruster_id="0" />
-  <xacro:t200_thruster_sim name="thruster_1" thruster_id="1" />
-  <xacro:t200_thruster_sim name="thruster_2" thruster_id="2" />
-  <xacro:t200_thruster_sim name="thruster_3" thruster_id="3" />
-  <xacro:t200_thruster_sim name="thruster_4" thruster_id="4" />
-  <xacro:t200_thruster_sim name="thruster_5" thruster_id="5" />
-  <xacro:t200_thruster_sim name="thruster_6" thruster_id="6" />
-  <xacro:t200_thruster_sim name="thruster_7" thruster_id="7" />
-  <xacro:bar30_sim name="base_link/external_pressure_sensor" />
-  <xacro:sonar_sim name="base_link/sonar_front" />
-  <xacro:sonar_sim name="base_link/sonar_back" />
-  <xacro:sonar_sim name="base_link/sonar_right" />
-  <xacro:sonar_sim name="base_link/sonar_left" />
-  <!--  -->
+  <xacro:arg name="debug" default="0" />
+  <xacro:arg name="namespace" default="taluy" />
+  <xacro:arg name="inertial_reference_frame" default="world" />
+  <xacro:include filename="$(find auv_sim_description)/urdf/base.urdf.xacro" />
+  <xacro:include filename="$(find auv_sim_description)/urdf/dynamics.urdf.xacro" />
+  <xacro:auv_sim_base
+    namespace="$(arg namespace)"
+    inertial_reference_frame="$(arg inertial_reference_frame)">
+    <gazebo>
+      <plugin name="uuv_plugin" filename="libuuv_underwater_object_ros_plugin.so">
+        <fluid_density>1028.0</fluid_density>
+        <flow_velocity_topic>hydrodynamics/current_velocity</flow_velocity_topic>
+        <debug>$(arg debug)</debug>
+        <xacro:auv_hydro_model namespace="$(arg namespace)" />
+      </plugin>
+    </gazebo>
+  </xacro:auv_sim_base>
+  <!-- joint state publisher -->
+  <xacro:include filename="$(find uuv_gazebo_ros_plugins)/urdf/misc.xacro" />
+  <xacro:default_joint_state_publisher namespace="$(arg namespace)" update_rate="50" />
 </robot>

Commit message: remove base link ned pub

File: auv_description/taluy_description/urdf/auv_base.urdf.xacro (robot description, xacro)
@@ -13,5 +13,5 @@
       <inertial>
         <origin xyz="0 0 0" rpy="0 0 0" />
-        <mass value="27.0" />
+        <mass value="25.37" />
         <inertia ixx="0.1" iyy="0.1" izz="0.1" ixy="0.01" iyz="0.01" ixz="0.1" />
       </inertial>
@@ -30,10 +30,10 @@
       </collision>
     </link>
-    <link name="${namespace}/base_link_ned" />
+    <!-- <link name="${namespace}/base_link_ned" />
     <joint name="base_link_joint" type="fixed">
       <origin xyz="0 0 0" rpy="${math.pi} 0 0" />
       <parent link="${namespace}/base_link_ned" />
       <child link="${namespace}/base_link" />
-    </joint>
+    </joint> -->
     <xacro:t200_thruster name="${namespace}/thruster_0" parent="${namespace}/base_link"
       position="0.14250 0.20070 -0.00525"

Commit message: remove base link ned pub

File: auv_description/taluy_description/urdf/auv_base.urdf.xacro (robot description, xacro)
@@ -13,5 +13,5 @@
       <inertial>
         <origin xyz="0 0 0" rpy="0 0 0" />
-        <mass value="27.0" />
+        <mass value="25.37" />
         <inertia ixx="0.1" iyy="0.1" izz="0.1" ixy="0.01" iyz="0.01" ixz="0.1" />
       </inertial>
@@ -32,10 +32,10 @@
       </collision>
     </link>
-    <link name="${namespace}/base_link_ned" />
+    <!-- <link name="${namespace}/base_link_ned" />
     <joint name="base_link_joint" type="fixed">
       <origin xyz="0 0 0" rpy="${math.pi} 0 0" />
       <parent link="${namespace}/base_link_ned" />
       <child link="${namespace}/base_link" />
-    </joint>
+    </joint> -->
     <xacro:t200_thruster name="${namespace}/thruster_0" parent="${namespace}/base_link"
       position="0.14250 0.20070 -0.00525"

Commit message: good location

File: auv_description/taluy_description/urdf/auv_base.urdf.xacro (robot description, xacro)
@@ -64,5 +64,5 @@
     <xacro:realsense_d435 name="${namespace}/camera" parent="${namespace}/base_link" position="-0.35 0 0" orientation="0 0 ${math.pi}"/>
     <!-- Parallel Gripper -->
-    <xacro:parallel_gripper namespace="${namespace}" parent_link="${namespace}/base_link"/>
+    <xacro:parallel_gripper namespace="${namespace}" parent_link="${namespace}/base_link" mount_xyz="-0.1 0 -0.1" mount_rpy="0 ${math.pi/2} 0" mass_scale="0.001"/>
     <!-- <link name="base_footprint">
       <inertial>

File: auv_description/taluy_description/urdf/parallel_gripper.xacro (robot description, xacro)
@@ -10,11 +10,11 @@
   <!-- Parallel Gripper Macro -->
   <!-- Added parameter use_mimic_plugin (default: false) to avoid Gazebo errors when the plugin is not available yet. -->
-  <xacro:macro name="parallel_gripper" params="namespace parent_link use_mimic_plugin:=false">
+  <xacro:macro name="parallel_gripper" params="namespace parent_link use_mimic_plugin:=false mass_scale:=0.001 mount_xyz:='0 0 0' mount_rpy:='0 0 0'">
     <!-- Gripper Base Link -->
     <link name="${namespace}/gripper_base">
       <inertial>
         <origin rpy="0 0 0" xyz="0.024426 0.0 0.0"/>
-        <mass value="3.5"/>
-        <xacro:box_inertia mass="3.5" x="0.074326" y="0.117427" z="0.114298"/>
+        <mass value="${3.5*mass_scale}"/>
+        <xacro:box_inertia mass="${3.5*mass_scale}" x="0.074326" y="0.117427" z="0.114298"/>
       </inertial>
       <visual>
@@ -35,6 +35,6 @@
       <parent link="${parent_link}"/>
       <child link="${namespace}/gripper_base"/>
-      <!-- Adjusted mounting position - front and slightly down from base_link -->
-      <origin xyz="0.45 0 -0.05" rpy="0 0 0"/>
+      <!-- Mount pose provided by caller (auv_base) via mount_xyz/mount_rpy -->
+      <origin xyz="${mount_xyz}" rpy="${mount_rpy}"/>
     </joint>
     <!-- Left Finger -->
@@ -42,6 +42,6 @@
       <inertial>
         <origin rpy="0 0 0" xyz="0.025268 -0.001931 -0.000079"/>
-        <mass value="0.88"/>
-        <xacro:box_inertia mass="0.88" x="0.064" y="0.078" z="0.025"/>
+        <mass value="${0.88*mass_scale}"/>
+        <xacro:box_inertia mass="${0.88*mass_scale}" x="0.064" y="0.078" z="0.025"/>
       </inertial>
       <visual>
@@ -72,6 +72,6 @@
       <inertial>
         <origin rpy="0 0 0" xyz="0.027744 0.017278 0.0"/>
-        <mass value="1.13"/>
-        <xacro:box_inertia mass="1.13" x="0.084" y="0.048" z="0.024"/>
+        <mass value="${1.13*mass_scale}"/>
+        <xacro:box_inertia mass="${1.13*mass_scale}" x="0.084" y="0.048" z="0.024"/>
       </inertial>
       <visual>
@@ -101,6 +101,6 @@
       <inertial>
         <origin rpy="0 0 0" xyz="0.025268 -0.001931 -0.000079"/>
-        <mass value="0.88"/>
-        <xacro:box_inertia mass="0.88" x="0.064" y="0.078" z="0.025"/>
+        <mass value="${0.88*mass_scale}"/>
+        <xacro:box_inertia mass="${0.88*mass_scale}" x="0.064" y="0.078" z="0.025"/>
       </inertial>
       <visual>
@@ -131,6 +131,6 @@
       <inertial>
         <origin rpy="0 0 0" xyz="0.027744 0.017278 0.0"/>
-        <mass value="1.13"/>
-        <xacro:box_inertia mass="1.13" x="0.084" y="0.048" z="0.024"/>
+        <mass value="${1.13*mass_scale}"/>
+        <xacro:box_inertia mass="${1.13*mass_scale}" x="0.084" y="0.048" z="0.024"/>
       </inertial>
       <visual>

Commit message: initial smach working commit

File: auv_description/taluy_description/urdf/auv_base.urdf.xacro (robot description, xacro)
@@ -65,4 +65,17 @@
     <!-- Parallel Gripper -->
     <xacro:parallel_gripper namespace="${namespace}" parent_link="${namespace}/base_link" mount_xyz="-0.1 0 -0.1" mount_rpy="0 ${math.pi/2} 0" mass_scale="0.001"/>
+    <!-- Gripper Link (fixed frame) -->
+    <link name="${namespace}/gripper_link">
+      <inertial>
+        <origin xyz="0 0 0" rpy="0 0 0"/>
+        <mass value="0.001"/>
+        <inertia ixx="0.000001" ixy="0.0" ixz="0.0" iyy="0.000001" iyz="0.0" izz="0.000001"/>
+      </inertial>
+    </link>
+    <joint name="gripper_link_joint" type="fixed">
+      <origin xyz="-0.1 0 -0.1" rpy="0 0 0"/>
+      <parent link="${namespace}/base_link"/>
+      <child link="${namespace}/gripper_link"/>
+    </joint>
     <!-- <link name="base_footprint">
       <inertial>

Commit message: files moved

File: auv_description/taluy_description/urdf/auv_base.urdf.xacro (robot description, xacro)
@@ -7,5 +7,4 @@
     <xacro:include filename="$(find auv_common_descriptions)/urdf/sensors.urdf.xacro"/>
     <xacro:include filename="$(find auv_common_descriptions)/urdf/materials.urdf.xacro"/>
-    <xacro:include filename="$(find taluy_description)/urdf/parallel_gripper.xacro"/>
     <xacro:arg name="angled_thruster_z_offset" default="-0.01"/>
     <link name="${namespace}/base_link">
@@ -63,6 +62,4 @@
     <xacro:ball_dropper name="${namespace}/base_link/ball_dropper" parent="${namespace}/base_link" position="0.1004 0.0745 -0.1953" orientation="0 0 0"/>
     <xacro:realsense_d435 name="${namespace}/camera" parent="${namespace}/base_link" position="-0.35 0 0" orientation="0 0 ${math.pi}"/>
-    <!-- Parallel Gripper -->
-    <xacro:parallel_gripper namespace="${namespace}" parent_link="${namespace}/base_link" mount_xyz="-0.1 0 -0.1" mount_rpy="0 ${math.pi/2} 0" mass_scale="0.001"/>
     <!-- <link name="base_footprint">
       <inertial>

File: auv_sim/auv_sim_description/taluy_sim_description/urdf/base.urdf.xacro (robot description, xacro)
@@ -7,4 +7,7 @@
     <xacro:include filename="$(find taluy_sim_description)/urdf/actuators.urdf.xacro"/>
     <xacro:include filename="$(find taluy_sim_description)/urdf/sensors.urdf.xacro"/>
+    <xacro:include filename="$(find taluy_sim_description)/urdf/parallel_gripper.xacro"/>
+    <!-- Parallel Gripper -->
+    <xacro:parallel_gripper namespace="${namespace}" parent_link="${namespace}/base_link" mount_xyz="-0.1 0 -0.1" mount_rpy="0 ${math.pi/2} 0" mass_scale="0.001"/>
   </xacro:macro>
 </robot>

File: auv_sim/auv_sim_description/taluy_sim_description/urdf/parallel_gripper.xacro (robot description, xacro)
@@ -21,5 +21,5 @@
         <origin rpy="0 0 0" xyz="0 0 0"/>
         <geometry>
-          <mesh filename="package://taluy_description/meshes/parallel_gripper/visual/BaseGripper.dae"/>
+          <mesh filename="package://auv_common_sim_descriptions/meshes/parallel_gripper/visual/BaseGripper.dae"/>
         </geometry>
       </visual>
@@ -49,5 +49,5 @@
         <origin rpy="0 0 0" xyz="0 0 0"/>
         <geometry>
-          <mesh filename="package://taluy_description/meshes/parallel_gripper/visual/Finger.dae"/>
+          <mesh filename="package://auv_common_sim_descriptions/meshes/parallel_gripper/visual/Finger.dae"/>
         </geometry>
       </visual>
@@ -82,5 +82,5 @@
         <origin rpy="0 0 0" xyz="0 0 0"/>
         <geometry>
-          <mesh filename="package://taluy_description/meshes/parallel_gripper/visual/FingerTip.dae"/>
+          <mesh filename="package://auv_common_sim_descriptions/meshes/parallel_gripper/visual/FingerTip.dae"/>
         </geometry>
       </visual>
@@ -110,5 +110,5 @@
         <origin rpy="3.14159265359 0 0" xyz="0 0 0"/>
         <geometry>
-          <mesh filename="package://taluy_description/meshes/parallel_gripper/visual/Finger.dae"/>
+          <mesh filename="package://auv_common_sim_descriptions/meshes/parallel_gripper/visual/Finger.dae"/>
         </geometry>
       </visual>
@@ -143,5 +143,5 @@
         <origin rpy="0 0 0" xyz="0 0 0"/>
         <geometry>
-          <mesh filename="package://taluy_description/meshes/parallel_gripper/visual/FingerTip.dae"/>
+          <mesh filename="package://auv_common_sim_descriptions/meshes/parallel_gripper/visual/FingerTip.dae"/>
         </geometry>
       </visual>

Commit message: fix space

File: auv_description/taluy_description/urdf/auv_base.urdf.xacro (robot description, xacro)
@@ -17,5 +17,5 @@
         <origin xyz="0.0 0.0 0.0" rpy="0 0 0"/>
         <geometry>
-            <box size="1.5 0.8 0.3"/>
+          <box size="1.5 0.8 0.3"/>
         </geometry>
         <material name="black"/>
@@ -24,5 +24,5 @@
         <origin xyz="0.0 0.0 0.0" rpy="0 0 0"/>
         <geometry>
-            <box size="1.5 0.8 0.3"/>
+          <box size="1.5 0.8 0.3"/>
         </geometry>
       </collision>
