Commit message: enable taluy model

File: auv_description/taluy_description/urdf/auv_base.urdf.xacro (robot description, xacro)
@@ -15,34 +15,17 @@
         <inertia ixx="0.1" iyy="0.1" izz="0.1" ixy="0.01" iyz="0.01" ixz="0.1"/>
       </inertial>
-      <xacro:if value="$(arg use_models)">
-        <visual>
-          <origin xyz="0.0 0.0 0.0" rpy="0 0 0"/>
-          <geometry>
-            <mesh filename="package://taluy_description/meshes/body/body.stl" scale="1 1 1"/>
-          </geometry>
-          <material name="black"/>
-        </visual>
-        <collision>
-          <origin xyz="0.0 0.0 0.0" rpy="0 0 0"/>
-          <geometry>
-            <mesh filename="package://taluy_description/meshes/body/body.stl" scale="1 1 1"/>
-          </geometry>
-        </collision>
-      </xacro:if>
-      <xacro:unless value="$(arg use_models)">
-        <visual>
-          <origin xyz="0.0 0.0 0.0" rpy="0 0 0"/>
-          <geometry>
-            <box size="1.5 0.8 0.3"/>
-          </geometry>
-          <material name="black"/>
-        </visual>
-        <collision>
-          <origin xyz="0.0 0.0 0.0" rpy="0 0 0"/>
-          <geometry>
-            <box size="1.5 0.8 0.3"/>
-          </geometry>
-        </collision>
-      </xacro:unless>
+      <visual>
+        <origin xyz="0.0 0.0 0.0" rpy="0 0 0"/>
+        <geometry>
+          <mesh filename="package://taluy_description/meshes/body/body.stl" scale="1 1 1"/>
+        </geometry>
+        <material name="black"/>
+      </visual>
+      <collision>
+        <origin xyz="0.0 0.0 0.0" rpy="0 0 0"/>
+        <geometry>
+          <mesh filename="package://taluy_description/meshes/body/body.stl" scale="1 1 1"/>
+        </geometry>
+      </collision>
     </link>
     <!-- Thrusters -->

Commit message: urdf fix

File: auv_description/taluy_description/urdf/auv_base.urdf.xacro (robot description, xacro)
@@ -64,5 +64,5 @@
     />
     <!-- Parallel Gripper -->
-    <xacro:parallel_gripper namespace="${namespace}" parent_link="${namespace}/base_link" mount_xyz="-0.1 0 -0.1" mount_rpy="0 ${math.pi/2} 0" mass_scale="0.001"/>
+    <xacro:parallel_gripper namespace="${namespace}" parent_link="${namespace}/base_link" mount_xyz="0 0.1929 -0.0347" mount_rpy="0 ${math.pi/2} ${math.pi/2}" mass_scale="0.001"/>
     <!-- Gripper Link (fixed frame) -->
     <link name="${namespace}/gripper_link">
@@ -74,5 +74,5 @@
     </link>
     <joint name="gripper_link_joint" type="fixed">
-      <origin xyz="-0.1 0 -0.1" rpy="0 0 0"/>
+      <origin xyz="0 0.1929 -0.0347" rpy="0 0 ${math.pi/2}"/>
       <parent link="${namespace}/base_link"/>
       <child link="${namespace}/gripper_link"/>

Commit message: feb8changes

File: auv_description/taluy_description/urdf/auv_base.urdf.xacro (robot description, xacro)
@@ -74,5 +74,5 @@
     </link>
     <joint name="gripper_link_joint" type="fixed">
-      <origin xyz="0 0.1929 -0.0347" rpy="0 0 ${math.pi/2}"/>
+      <origin xyz="0 0.1929 -0.0347" rpy="0 0 0"/>
       <parent link="${namespace}/base_link"/>
       <child link="${namespace}/gripper_link"/>

Commit message: 19FEB

File: auv_description/taluy_description/urdf/auv_base.urdf.xacro (robot description, xacro)
@@ -74,5 +74,5 @@
     </link>
     <joint name="gripper_link_joint" type="fixed">
-      <origin xyz="0 0.1929 -0.0347" rpy="0 0 0"/>
+      <origin xyz="-0.09791 0.205121 -0.40520" rpy="0 0 0"/>
       <parent link="${namespace}/base_link"/>
       <child link="${namespace}/gripper_link"/>

Commit message: cn

File: auv_description/taluy_description/urdf/auv_base.urdf.xacro (robot description, xacro)
@@ -74,5 +74,5 @@
     </link>
     <joint name="gripper_link_joint" type="fixed">
-      <origin xyz="-0.09791 0.205121 -0.40520" rpy="0 0 0"/>
+      <origin xyz="-0.128 0.0 -0.4285" rpy="0 0 0"/>
       <parent link="${namespace}/base_link"/>
       <child link="${namespace}/gripper_link"/>

Commit message: simulation damping

File: auv_description/taluy_description/urdf/auv_base.urdf.xacro (robot description, xacro)
@@ -12,5 +12,5 @@
       <inertial>
         <origin xyz="0 0 0" rpy="0 0 0"/>
-        <mass value="25.37"/>
+        <mass value="29"/>
         <inertia ixx="0.1" iyy="0.1" izz="0.1" ixy="0.01" iyz="0.01" ixz="0.1"/>
       </inertial>

Commit message: fix gripper in sim

File: auv_description/taluy_description/urdf/auv_base.urdf.xacro (robot description, xacro)
@@ -63,6 +63,4 @@
       use_models="$(arg use_models)"
     />
-    <!-- Parallel Gripper -->
-    <xacro:parallel_gripper namespace="${namespace}" parent_link="${namespace}/base_link" mount_xyz="0 0.1929 -0.0347" mount_rpy="0 ${math.pi/2} ${math.pi/2}" mass_scale="0.001"/>
     <!-- Gripper Link (fixed frame) -->
     <link name="${namespace}/gripper_link">
@@ -78,4 +76,19 @@
       <child link="${namespace}/gripper_link"/>
     </joint>
+    <!-- Gripper Mount Link (offset from tip) -->
+    <link name="${namespace}/gripper_mount_link">
+      <inertial>
+        <origin xyz="0 0 0" rpy="0 0 0"/>
+        <mass value="0.001"/>
+        <inertia ixx="0.000001" ixy="0.0" ixz="0.0" iyy="0.000001" iyz="0.0" izz="0.000001"/>
+      </inertial>
+    </link>
+    <joint name="gripper_mount_joint" type="fixed">
+      <origin xyz="0 0 0.193" rpy="0 0 0"/>
+      <parent link="${namespace}/gripper_link"/>
+      <child link="${namespace}/gripper_mount_link"/>
+    </joint>
+    <!-- Parallel Gripper -->
+    <xacro:parallel_gripper namespace="${namespace}" parent_link="${namespace}/gripper_mount_link" mount_xyz="0 0 0" mount_rpy="0 ${math.pi/2} 0" mass_scale="0.001"/>
     <!-- <link name="base_footprint">
       <inertial>

Commit message: refactor gripper import

File: auv_description/taluy_description/urdf/auv_base.urdf.xacro (robot description, xacro)
@@ -63,32 +63,6 @@
       use_models="$(arg use_models)"
     />
-    <!-- Gripper Link (fixed frame) -->
-    <link name="${namespace}/gripper_link">
-      <inertial>
-        <origin xyz="0 0 0" rpy="0 0 0"/>
-        <mass value="0.001"/>
-        <inertia ixx="0.000001" ixy="0.0" ixz="0.0" iyy="0.000001" iyz="0.0" izz="0.000001"/>
-      </inertial>
-    </link>
-    <joint name="gripper_link_joint" type="fixed">
-      <origin xyz="-0.128 0.0 -0.4285" rpy="0 0 0"/>
-      <parent link="${namespace}/base_link"/>
-      <child link="${namespace}/gripper_link"/>
-    </joint>
-    <!-- Gripper Mount Link (offset from tip) -->
-    <link name="${namespace}/gripper_mount_link">
-      <inertial>
-        <origin xyz="0 0 0" rpy="0 0 0"/>
-        <mass value="0.001"/>
-        <inertia ixx="0.000001" ixy="0.0" ixz="0.0" iyy="0.000001" iyz="0.0" izz="0.000001"/>
-      </inertial>
-    </link>
-    <joint name="gripper_mount_joint" type="fixed">
-      <origin xyz="0 0 0.193" rpy="0 0 0"/>
-      <parent link="${namespace}/gripper_link"/>
-      <child link="${namespace}/gripper_mount_link"/>
-    </joint>
     <!-- Parallel Gripper -->
-    <xacro:parallel_gripper namespace="${namespace}" parent_link="${namespace}/gripper_mount_link" mount_xyz="0 0 0" mount_rpy="0 ${math.pi/2} 0" mass_scale="0.001"/>
+    <xacro:parallel_gripper namespace="${namespace}" parent_link="${namespace}/base_link" mount_xyz="-0.128 0.0 -0.4285" mount_rpy="0 0 0" mass_scale="0.001"/>
     <!-- <link name="base_footprint">
       <inertial>

File: auv_description/taluy_description/urdf/parallel_gripper.xacro (robot description, xacro)
@@ -11,4 +11,33 @@
   <!-- Added parameter use_mimic_plugin (default: false) to avoid Gazebo errors when the plugin is not available yet. -->
   <xacro:macro name="parallel_gripper" params="namespace parent_link use_mimic_plugin:=false use_grasp_fix:=true mass_scale:=0.001 mount_xyz:='0 0 0' mount_rpy:='0 0 0'">
+<!-- Custom connection mapping to attach from base to the tip backward to gripper base -->
+    <!-- Virtual link representing the tip (where the gripper actually touches what it holds) -->
+    <link name="${namespace}/gripper_link">
+      <inertial>
+        <origin xyz="0 0 0" rpy="0 0 0"/>
+        <mass value="0.001"/>
+        <inertia ixx="0.000001" ixy="0.0" ixz="0.0" iyy="0.000001" iyz="0.0" izz="0.000001"/>
+      </inertial>
+    </link>
+    <!-- Joint connecting parent (e.g. base_link) to gripper_link -->
+    <joint name="${namespace}/gripper_link_joint" type="fixed">
+      <origin xyz="${mount_xyz}" rpy="${mount_rpy}"/>
+      <parent link="${parent_link}"/>
+      <child link="${namespace}/gripper_link"/>
+    </joint>
+    <!-- Gripper Mount Link (offset from tip up to the base of the gripper) -->
+    <link name="${namespace}/gripper_mount_link">
+      <inertial>
+        <origin xyz="0 0 0" rpy="0 0 0"/>
+        <mass value="0.001"/>
+        <inertia ixx="0.000001" ixy="0.0" ixz="0.0" iyy="0.000001" iyz="0.0" izz="0.000001"/>
+      </inertial>
+    </link>
+    <!-- The offset from tip backwards to the base -->
+    <joint name="${namespace}/gripper_mount_joint" type="fixed">
+      <origin xyz="0 0 0.193" rpy="0 0 0"/>
+      <parent link="${namespace}/gripper_link"/>
+      <child link="${namespace}/gripper_mount_link"/>
+    </joint>
     <!-- Gripper Base Link -->
     <link name="${namespace}/gripper_base">
@@ -31,10 +60,9 @@
       </collision>
     </link>
-    <!-- Joint connecting parent to gripper base -->
-    <joint name="${namespace}/gripper_mount_joint" type="fixed">
-      <parent link="${parent_link}"/>
+    <!-- Joint connecting the virtual mount link to gripper base -->
+    <joint name="${namespace}/gripper_base_joint" type="fixed">
+      <parent link="${namespace}/gripper_mount_link"/>
       <child link="${namespace}/gripper_base"/>
-      <!-- Mount pose provided by caller (auv_base) via mount_xyz/mount_rpy -->
-      <origin xyz="${mount_xyz}" rpy="${mount_rpy}"/>
+      <origin xyz="0 0 0" rpy="0 ${math.pi/2} 0"/>
     </joint>
     <!-- Left Finger -->

Commit message: cog for allocation

File: auv_description/taluy_description/urdf/auv_base.urdf.xacro (robot description, xacro)
@@ -29,4 +29,11 @@
       </collision>
     </link>
+    <!-- Center of Gravity -->
+    <link name="${namespace}/center_of_gravity"/>
+    <joint name="${namespace}/base_link_to_cog" type="fixed">
+      <parent link="${namespace}/base_link"/>
+      <child link="${namespace}/center_of_gravity"/>
+      <origin xyz="0 0 -0.05" rpy="0 0 0"/>
+    </joint>
     <!-- Thrusters -->
     <xacro:t200_thruster name="${namespace}/thruster_0" parent="${namespace}/base_link" position="0.16040 0.20070 -0.012879" orientation="${pi} 0 ${-pi/2}" use_models="$(arg use_models)"/>

Commit message: cog for allocation

File: auv_description/taluy_description/urdf/auv_base.urdf.xacro (robot description, xacro)
@@ -29,4 +29,11 @@
       </collision>
     </link>
+    <!-- Center of Gravity -->
+    <link name="${namespace}/center_of_gravity"/>
+    <joint name="${namespace}/base_link_to_cog" type="fixed">
+      <parent link="${namespace}/base_link"/>
+      <child link="${namespace}/center_of_gravity"/>
+      <origin xyz="0 0 -0.05" rpy="0 0 0"/>
+    </joint>
     <!-- Thrusters -->
     <xacro:t200_thruster name="${namespace}/thruster_0" parent="${namespace}/base_link" position="0.16040 0.20070 -0.012879" orientation="${pi} 0 ${-pi/2}" use_models="$(arg use_models)"/>

File: auv_sim/auv_sim_description/taluy_sim_description/urdf/dynamics.urdf.xacro (robot description, xacro)
@@ -18,5 +18,5 @@
     assume NWU (otherwise cob is below cog?).
     -->
-  <xacro:property name="cob" value="0.0 0.0 0.2"/>
+  <xacro:property name="cob" value="0.0 0.0 0.05"/>
   <!-- Volume, see p.31 in Berg2012, normally 0.009165088 -->
   <xacro:property name="volume" value="0.027"/>
@@ -31,4 +31,5 @@
       </box>
       <center_of_buoyancy>${cob}</center_of_buoyancy>
+      <center_of_gravity>0 0 -0.05</center_of_gravity>
       <hydrodynamic_model>
         <type>fossen</type>

Commit message: 30mart

File: auv_description/taluy_description/urdf/auv_base.urdf.xacro (robot description, xacro)
@@ -12,6 +12,6 @@
       <inertial>
         <origin xyz="0 0 0" rpy="0 0 0"/>
-        <mass value="29"/>
-        <inertia ixx="0.1" iyy="0.1" izz="0.1" ixy="0.01" iyz="0.01" ixz="0.1"/>
+        <mass value="29.8419"/>
+        <inertia ixx="0.9430" iyy="2.12" izz="2.18" ixy="0.0" iyz="0.0" ixz="0.0"/>
       </inertial>
       <visual>

File: auv_sim/auv_sim_description/taluy_sim_description/urdf/dynamics.urdf.xacro (robot description, xacro)
@@ -41,6 +41,6 @@
           0 0 0 0 0 0
         </added_mass>
-        <linear_damping>-45.8 -42.37 -89.2 -1.87 -1.87 -5.646</linear_damping>
-        <quadratic_damping>-141.9 -221.7 -136.16 -7.98 -7.98 -2.608</quadratic_damping>
+        <linear_damping>-62.8822 -106.733 -89.2 -1.87 -1.87 -4.04997</linear_damping>
+        <quadratic_damping>-116.822 -82.556 -136.16 -7.98 -7.98 -2.41789</quadratic_damping>
       </hydrodynamic_model>
     </link>

Commit message: sim succeded ?

File: auv_description/taluy_description/urdf/auv_base.urdf.xacro (robot description, xacro)
@@ -12,5 +12,5 @@
       <inertial>
         <origin xyz="0 0 0" rpy="0 0 0"/>
-        <mass value="25.37"/>
+        <mass value="29.8419"/>
         <inertia ixx="0.1" iyy="0.1" izz="0.1" ixy="0.01" iyz="0.01" ixz="0.1"/>
       </inertial>

Commit message: added pitch error to align frame, changed cog in sim, integrated trajectory publisher from another branch, smach is still unintegrated

File: auv_description/taluy_description/urdf/auv_base.urdf.xacro (robot description, xacro)
@@ -12,5 +12,5 @@
     <link name="${namespace}/base_link">
       <inertial>
-        <origin xyz="0 0 0" rpy="0 0 0"/>
+        <origin xyz="0 0 0.16" rpy="0 0 0"/>
         <mass value="25.37"/>
         <inertia ixx="0.1" iyy="0.1" izz="0.1" ixy="0.01" iyz="0.01" ixz="0.1"/>

File: auv_description/taluy_mini_description/urdf/auv_base.urdf.xacro (robot description, xacro)
@@ -9,5 +9,5 @@
     <link name="${namespace}/base_link">
       <inertial>
-        <origin xyz="0 0 0" rpy="0 0 0"/>
+        <origin xyz="0 0 0.18" rpy="0 0 0"/>
         <mass value="15.0"/>
         <inertia ixx="0.1" iyy="0.1" izz="0.1" ixy="0.01" iyz="0.01" ixz="0.1"/>

Commit message: cleaned up, also changed how the smach works

File: auv_description/taluy_description/urdf/auv_base.urdf.xacro (robot description, xacro)
@@ -89,4 +89,10 @@
     <xacro:bar30 name="${namespace}/base_link/external_pressure_sensor" parent="${namespace}/base_link" position="0 0 0.079" orientation="0 0 0" use_models="$(arg use_models)"/>
     <xacro:logitech_c920_camera name="${namespace}/base_link/front_camera" parent="${namespace}/base_link" position="0.40125 0 0" orientation="0 0 0" use_models="$(arg use_models)"/>
+    <link name="${namespace}/base_link/valve_gripper_front_link"/>
+    <joint name="${namespace}/base_link/valve_gripper_front_joint" type="fixed">
+      <parent link="${namespace}/base_link/front_camera_link"/>
+      <child link="${namespace}/base_link/valve_gripper_front_link"/>
+      <origin xyz="0.30 0 0" rpy="0 0 0"/>
+    </joint>
     <xacro:logitech_c920_camera
       name="${namespace}/base_link/bottom_camera"

Commit message: Dynamic Model (#683)
Co-authored-by: meydanoglu <eminmeydanoglu@gmail.com>
Co-authored-by: Talha Karasu <talha@karasu.me>

File: auv_description/taluy_description/urdf/auv_base.urdf.xacro (robot description, xacro)
@@ -13,5 +13,5 @@
       <inertial>
         <origin xyz="0 0 0" rpy="0 0 0"/>
-        <mass value="25.37"/>
+        <mass value="29.8419"/>
         <inertia ixx="0.1" iyy="0.1" izz="0.1" ixy="0.01" iyz="0.01" ixz="0.1"/>
       </inertial>

Commit message: wip

File: auv_description/taluy_description/urdf/auv_base.urdf.xacro (robot description, xacro)
@@ -102,4 +102,14 @@
       use_models="$(arg use_models)"
     />
+    <!-- Bottom valve gripper: PLACEHOLDER position — 30cm below the bottom
+         camera. Mounted via base_link so the rpy is unambiguous: pitch
+         -π/2 rotates +X to point along -Z_base (straight down when
+         the AUV is level). -->
+    <link name="${namespace}/base_link/valve_gripper_bottom_link"/>
+    <joint name="${namespace}/base_link/valve_gripper_bottom_joint" type="fixed">
+      <parent link="${namespace}/base_link"/>
+      <child link="${namespace}/base_link/valve_gripper_bottom_link"/>
+      <origin xyz="0 0 -0.37" rpy="0 ${-math.pi/2} 0"/>
+    </joint>
     <xacro:torpedo_camera
       name="${namespace}/base_link/torpedo_camera"

Commit message: still wip but finally works in sim

File: auv_description/taluy_description/urdf/auv_base.urdf.xacro (robot description, xacro)
@@ -102,13 +102,12 @@
       use_models="$(arg use_models)"
     />
-    <!-- Bottom valve gripper: PLACEHOLDER position — 30cm below the bottom
-         camera. Mounted via base_link so the rpy is unambiguous: pitch
-         -π/2 rotates +X to point along -Z_base (straight down when
-         the AUV is level). -->
+    <!-- Bottom valve gripper: PLACEHOLDER position — 37cm below base_link.
+         Identity orientation (same as base_link) — the trajectory publisher
+         handles the full 3D look-at orientation for the target frames. -->
     <link name="${namespace}/base_link/valve_gripper_bottom_link"/>
     <joint name="${namespace}/base_link/valve_gripper_bottom_joint" type="fixed">
       <parent link="${namespace}/base_link"/>
       <child link="${namespace}/base_link/valve_gripper_bottom_link"/>
-      <origin xyz="0 0 -0.37" rpy="0 ${-math.pi/2} 0"/>
+      <origin xyz="0 0 -0.37" rpy="0 0 0"/>
     </joint>
     <xacro:torpedo_camera

Commit message: changed gripper position

File: auv_description/taluy_description/urdf/auv_base.urdf.xacro (robot description, xacro)
@@ -91,7 +91,7 @@
     <link name="${namespace}/base_link/valve_gripper_front_link"/>
     <joint name="${namespace}/base_link/valve_gripper_front_joint" type="fixed">
-      <parent link="${namespace}/base_link/front_camera_link"/>
+      <parent link="${namespace}/base_link"/>
       <child link="${namespace}/base_link/valve_gripper_front_link"/>
-      <origin xyz="0.30 0 0" rpy="0 0 0"/>
+      <origin xyz="0.626109 -0.06965 -0.075051" rpy="0 0 0"/>
     </joint>
     <xacro:logitech_c920_camera

Commit message: working dynamic model an also viisual servoing

File: auv_description/taluy_description/urdf/auv_base.urdf.xacro (robot description, xacro)
@@ -91,7 +91,7 @@
     <link name="${namespace}/base_link/valve_gripper_front_link"/>
     <joint name="${namespace}/base_link/valve_gripper_front_joint" type="fixed">
-      <parent link="${namespace}/base_link/front_camera_link"/>
+      <parent link="${namespace}/base_link"/>
       <child link="${namespace}/base_link/valve_gripper_front_link"/>
-      <origin xyz="0.30 0 0" rpy="0 0 0"/>
+      <origin xyz="0.626 -0.04 -0.075" rpy="0 0 0"/>
     </joint>
     <xacro:logitech_c920_camera

Commit message: tracking changes

File: auv_description/taluy_description/urdf/auv_base.urdf.xacro (robot description, xacro)
@@ -93,5 +93,5 @@
       <parent link="${namespace}/base_link"/>
       <child link="${namespace}/base_link/valve_gripper_front_link"/>
-      <origin xyz="0.626 -0.04 -0.075" rpy="0 0 0"/>
+      <origin xyz="0.626109 -0.06965 -0.075051" rpy="0 0 0"/>
     </joint>
     <xacro:logitech_c920_camera

Commit message: change urdf

File: auv_description/taluy_description/urdf/auv_base.urdf.xacro (robot description, xacro)
@@ -102,5 +102,5 @@
       use_models="$(arg use_models)"
     />
-    <!-- Bottom valve gripper: PLACEHOLDER position — 37cm below base_link.
+    <!-- Bottom valve gripper: position from CAD sketch point (Y taken as 0).
          Identity orientation (same as base_link) — the trajectory publisher
          handles the full 3D look-at orientation for the target frames. -->
@@ -109,5 +109,5 @@
       <parent link="${namespace}/base_link"/>
       <child link="${namespace}/base_link/valve_gripper_bottom_link"/>
-      <origin xyz="0 0 -0.37" rpy="0 0 0"/>
+      <origin xyz="-0.145 0 -0.369736" rpy="0 0 0"/>
     </joint>
     <xacro:torpedo_camera

Commit message: new bottom gripper urdf

File: auv_description/taluy_description/urdf/auv_base.urdf.xacro (robot description, xacro)
@@ -109,5 +109,5 @@
       <parent link="${namespace}/base_link"/>
       <child link="${namespace}/base_link/valve_gripper_bottom_link"/>
-      <origin xyz="-0.145 0 -0.369736" rpy="0 0 0"/>
+      <origin xyz="-0.1385 0 -0.368736" rpy="0 0 0"/>
     </joint>
     <xacro:torpedo_camera

Commit message: Revert "Merge remote-tracking branch 'origin/baykara-slalom-torpedocam' into furkan/main"
This reverts commit 30cde790c58806990b38b523a89a90f84d5eacba, reversing
changes made to e00cee0c054e3f5d92092aedb322ce8fa89c4f2f.

File: auv_description/taluy_description/urdf/auv_base.urdf.xacro (robot description, xacro)
@@ -30,11 +30,4 @@
       </collision>
     </link>
-    <!-- child frame: base_link_180 - same position, rotated 180° around Z -->
-    <link name="${namespace}/base_link_180"/>
-    <joint name="${namespace}/base_link_to_base_link_180" type="fixed">
-      <parent link="${namespace}/base_link"/>
-      <child link="${namespace}/base_link_180"/>
-      <origin xyz="0 0 0" rpy="0 0 ${math.pi}"/>
-    </joint>
     <!-- Thrusters -->
     <xacro:t200_thruster name="${namespace}/thruster_0" parent="${namespace}/base_link" position="0.16040 0.20070 -0.012879" orientation="${pi} 0 ${-pi/2}" use_models="$(arg use_models)"/>

File: auv_description/taluy_mini_description/urdf/auv_base.urdf.xacro (robot description, xacro)
@@ -27,11 +27,4 @@
       </collision>
     </link>
-    <!-- child frame: base_link_180 - same position, rotated 180° around Z -->
-    <link name="${namespace}/base_link_180"/>
-    <joint name="${namespace}/base_link_to_base_link_180" type="fixed">
-      <parent link="${namespace}/base_link"/>
-      <child link="${namespace}/base_link_180"/>
-      <origin xyz="0 0 0" rpy="0 0 ${math.pi}"/>
-    </joint>
     <xacro:t200_thruster
       name="${namespace}/thruster_0"
