Commit message: nazar degmez ins

File: auv_description/taluy_description/urdf/auv_base.urdf.xacro (robot description, xacro)
@@ -64,5 +64,5 @@
     />
     <!-- Parallel Gripper -->
-    <xacro:parallel_gripper namespace="${namespace}" parent_link="${namespace}/base_link" mount_xyz="-0.102 0.0 -0.425" mount_rpy="0 0 0" mass_scale="0.001"/>
+    <xacro:parallel_gripper namespace="${namespace}" parent_link="${namespace}/base_link" mount_xyz="-0.107 0.0 -0.425" mount_rpy="0 0 0" mass_scale="0.001"/>
     <!-- <link name="base_footprint">
       <inertial>

File: auv_description/taluy_description/urdf/parallel_gripper.xacro (robot description, xacro)
@@ -25,4 +25,28 @@
       <parent link="${parent_link}"/>
       <child link="${namespace}/gripper_link"/>
+    </joint>
+    <link name="${namespace}/gripper_link_p2"/>
+    <link name="${namespace}/gripper_link_p4"/>
+    <link name="${namespace}/gripper_link_n2"/>
+    <link name="${namespace}/gripper_link_n4"/>
+    <joint name="${namespace}/gripper_front_joint" type="fixed">
+      <origin xyz="0.02 0 0" rpy="0 0 0"/>
+      <parent link="${namespace}/gripper_link"/>
+      <child link="${namespace}/gripper_link_p2"/>
+    </joint>
+    <joint name="${namespace}/gripper_rear_joint" type="fixed">
+      <origin xyz="0.04 0 0" rpy="0 0 0"/>
+      <parent link="${namespace}/gripper_link"/>
+      <child link="${namespace}/gripper_link_p4"/>
+    </joint>
+    <joint name="${namespace}/gripper_front_joint_2" type="fixed">
+      <origin xyz="-0.02 0 0" rpy="0 0 0"/>
+      <parent link="${namespace}/gripper_link"/>
+      <child link="${namespace}/gripper_link_n2"/>
+    </joint>
+    <joint name="${namespace}/gripper_rear_joint_2" type="fixed">
+      <origin xyz="-0.04 0 0" rpy="0 0 0"/>
+      <parent link="${namespace}/gripper_link"/>
+      <child link="${namespace}/gripper_link_n4"/>
     </joint>
     <!-- Gripper Mount Link (offset from tip up to the base of the gripper) -->
